File: DCCStepperDrive/DCCStepperDrive.kicad_pcb (KiCad board)
At the start: 2 copper layers, 100 x 100 mm, 34 parts, among them J1 12v, J2 CBUS, J3 5V select, J4 DCC, J5 Grove 2mm, J6 GROVE-CONNECTOR-DIP_4P-2.0_, J7 Sensor, J8 Motor, J9 Mode Select, Q1 DMG2305UX-7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

Commit message: 19:27 Arrakis.local
Parts:
- J6: value GROVE-CONNECTOR-DIP_4P-2.0_ -> I2C
Connections:
- A1 pad 8: +12V -> /12V
- C1 pad 1: Net-(D1-Pad1) -> /12V
- C4 pad 1: +5V -> /5V
- D1 pad 1: Net-(D1-Pad1) -> /12V
- D1 pad 2: +12V -> Net-(D1-Pad2)
- J1 pad 2: +12V -> Net-(D1-Pad2)
- J2 pad 1: +12V -> Net-(D1-Pad2)
- J3 pad 1: +5V -> /5V
- J5 pad 1: GND -> /SCL
- J5 pad 2: /3V3 -> /SDA
- J5 pad 3: /SDA -> /3V3
- J5 pad 4: /SCL -> GND
- J6 pad 1: Net-(J6-Pad1) -> /SCL
- J6 pad 2: Net-(J6-Pad2) -> /SDA
- J6 pad 3: /SDA -> /3V3
- J6 pad 4: /SCL -> GND
- J9 pad 10: +5V -> /+5V
- J9 pad 6: +5V -> /+5V
- J9 pad 8: +5V -> /+5V
- Q1 pad 3: +5V -> /5V
- U2 pad 2: +5V -> /5V
- U2 pad 3: Net-(D1-Pad1) -> /12V
Routing:
- net +5V: track 98.7 -> 0.00 mm, vias 1 -> 0
- net +12V: track 93.0 -> 0.00 mm
- net /12V: track 0.00 -> 81.2 mm
- net Net-(D1-Pad2): track 0.00 -> 58.6 mm
- net /5V: track 0.00 -> 46.4 mm
- net Net-(J7-Pad3): track 103.0 -> 80.2 mm, vias 0 -> 1
- net Net-(D1-Pad1): track 22.4 -> 0.00 mm
- net Net-(J6-Pad2): track 12.9 -> 0.00 mm
- net Net-(J6-Pad1): track 11.6 -> 0.00 mm
- net Net-(A1-Pad16): track 80.7 -> 72.0 mm
- net /DccIn: track 74.0 -> 65.5 mm
- net /3V3: track 136.2 -> 144.6 mm
- net /VBUS: track 89.7 -> 95.7 mm
- net GND: track 295.2 -> 301.1 mm, vias 1 -> 0
- net /+5V: track 0.00 -> 5.08 mm
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
Commit message: 21:55 Arrakis.local
Parts:
- D1: value 1N4004 -> 1N5819
- J1, J4: footprint TerminalBlock_Phoenix:TerminalBlock_Phoenix_PT-1,5-2-5.0-H_1x02_P5.00mm_Horizontal -> TerminalBlock_Phoenix:TerminalBlock_Phoenix_PT-1,5-2-3.5-H_1x02_P3.50mm_Horizontal
- U4: footprint MCU_RaspberryPi_and_Boards:RPi_Pico_SMD_TH -> MCU_RaspberryPi_and_Boards:RP2040Pico
- turned SW1 to 180 degrees
Routing:
- net GND: track 301.1 -> 319.3 mm
- net Net-(SW1-Pad2): track 51.5 -> 43.3 mm
- net /VBUS: track 95.7 -> 103.5 mm
- net /5V: track 46.4 -> 48.5 mm
- net Net-(D1-Pad2): track 58.6 -> 60.3 mm
- net /5Vopt: track 25.6 -> 24.0 mm
- net /12V: track 81.2 -> 82.6 mm
- net /VSYS: track 68.3 -> 69.7 mm
- net Net-(J7-Pad3): track 80.2 -> 81.5 mm
- net /SCL: track 79.8 -> 78.6 mm
- net Net-(C2-Pad1): track 61.5 -> 62.4 mm
- net Net-(J7-Pad2): track 50.6 -> 50.0 mm
