File: DCCStepperDrive/DCCStepperDrive.kicad_pcb (KiCad board)
At the start: 2 copper layers, 100 x 100 mm, 35 parts, among them J1 12v, J2 CBUS, J3 5V select, J4 DCC, J5 Grove 2mm, J6 I2C, J7 Sensor, J8 Motor, J9 Mode Select, Q1 DMG2305UX-7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

Commit message: 18:34 Arrakis.local
Other:
- board text added: "DCC Stepper Drive v3.0"
- board text removed: "DCC Stepper Drive v2.0"
Changed lines of the file:
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@@
   (gr_arc (start 103 150) (mid 100.87868 149.12132) (end 100 147) (layer "Edge.Cuts") (width 0.1))
   (gr_arc (start 197 50) (mid 199.12132 50.87868) (end 200 53) (layer "Edge.Cuts") (width 0.2))
-  (gr_text "DCC Stepper Drive v2.0\n" (at 150 53) (layer "F.SilkS")
+  (gr_text "DCC Stepper Drive v3.0\n" (at 150 53) (layer "F.SilkS")
     (effects (font (size 2 2) (thickness 0.15)))
   )
