File: PicoXpressSmdK/PicoXpressSmdK.kicad_pcb (KiCad board)
At the start: 2 copper layers, 100 x 80 mm, 22 parts, among them J1 6P6C, J2 Screw_Terminal_01x09, J3 I2C, J4 Screw_Terminal_01x03, J5 I2C, J6 Screw_Terminal_01x09, Q1 DMG2305UX-7, SW1 SW_Push, U1 AMS1117-5.0, U2 MCP23008-xSO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

Commit message: 12:08 Arrakis.local
Parts:
- moved J3 4.00 mm to (157.0, 120.0)
Routing:
- net /GND: track 0.00 -> 267.3 mm
- net /3V3: track 0.00 -> 135.5 mm, vias 0 -> 2
- net /RUN: track 0.00 -> 124.9 mm
- net /5V: track 0.00 -> 96.2 mm
- net /SCL: track 0.00 -> 83.5 mm
- net /SDA: track 0.00 -> 83.5 mm
- net /GP0: track 0.00 -> 73.0 mm
- net /GP1: track 0.00 -> 67.5 mm
- net /RTS: track 0.00 -> 66.3 mm
- net /VBUS: track 0.00 -> 40.0 mm
- net /VIN: track 0.00 -> 37.8 mm
- net Net-(J6-Pad8): track 0.00 -> 37.3 mm
- net Net-(J6-Pad5): track 0.00 -> 35.2 mm
- net Net-(J1-Pad3): track 0.00 -> 32.8 mm
- net Net-(J6-Pad7): track 0.00 -> 31.6 mm
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
Commit message: 13:19 Arrakis.local
Parts:
- added J6: Screw_Terminal_01x05, Connector_PinHeader_2.54mm:PinHeader_1x05_P2.54mm_Vertical, F.Cu at (135.0, 119.0)
- moved C2 36.2 mm to (147.6, 74.0)
- moved C1 34.8 mm to (103.6, 88.0)
- moved D1 6.92 mm to (116.1, 79.0)
- moved U4 5.00 mm to (137.0, 87.0)
- moved U1 4.24 mm to (137.0, 76.0)
- renumbered J6 to J7
Connections:
- J3 pad 1: /GND -> /SCL
- J3 pad 2: /3V3 -> /SDA
- J3 pad 3: /SDA -> /3V3
- J3 pad 4: /SCL -> /GND
- J5 pad 1: /GND -> /SCL
- J5 pad 2: /3V3 -> /SDA
- J5 pad 3: /SDA -> /3V3
- J5 pad 4: /SCL -> /GND
Routing:
- net /GND: track 267.3 -> 319.6 mm
- net Net-(J1-Pad3): track 32.8 -> 46.1 mm
- net /3V3: track 135.5 -> 147.0 mm, vias 2 -> 0
- net /SDA: track 83.5 -> 91.9 mm
- net /RUN: track 124.9 -> 118.0 mm
- net /SCL: track 83.5 -> 90.2 mm
- net /5Vopt: track 21.2 -> 16.5 mm
- net /VIN: track 37.8 -> 34.3 mm
- net Net-(J1-Pad4): track 31.5 -> 28.6 mm
- net /12V: track 11.3 -> 13.8 mm
- net Net-(J7-Pad6): track 29.4 -> 31.5 mm
- net Net-(J7-Pad5): track 35.2 -> 37.3 mm
- net /VBUS: track 40.0 -> 39.1 mm
- net /GP0: track 73.0 -> 73.5 mm
- net /5V: vias 0 -> 1
Other:
- board text added: "3v3"
- board text added: "Gnd"
- board text added: "SCL"
- board text added: "SDA"

Commit message: 19:27 Arrakis.local
Parts:
- added H1: 0, MountingHole:MountingHole_3.2mm_M3, F.Cu at (197.0, 53.0)
- added H2: 0, MountingHole:MountingHole_3.2mm_M3, F.Cu at (197.0, 127.0)
- added H3: 0, MountingHole:MountingHole_3.2mm_M3, F.Cu at (103.0, 53.0)
- added H4: 0, MountingHole:MountingHole_3.2mm_M3, F.Cu at (104.0, 126.0)
- C1: value C_Polarized -> 100uF
- C2, C3: value C_Polarized -> 22uF
- J2: value Screw_Terminal_01x09 -> parallel port
- J4: value Screw_Terminal_01x03 -> 5V Sel
- J6: value Screw_Terminal_01x05 -> I2C
- J7: value Screw_Terminal_01x09 -> keypad
- SW1: value SW_Push -> Reset
Routing:
- net /SDA: track 91.9 -> 97.5 mm
- net /SCL: track 90.2 -> 91.4 mm
Other:
- board text added: "PicoXpressSmdK version 2"

Commit message: 09:25 Arrakis.local
Parts:
- U5: footprint MCU_RaspberryPi_and_Boards:RPi_Pico_SMD_TH -> MCU_RaspberryPi_and_Boards:RP2040Pico
- turned U5 to 0 degrees
Routing:
- net Net-(J7-Pad1): track 13.8 -> 56.2 mm
- net /VSYS: track 24.9 -> 63.5 mm
- net /GND: track 319.6 -> 281.7 mm
- net Net-(J7-Pad2): track 13.8 -> 51.0 mm
- net /GP0: track 73.5 -> 36.7 mm
- net Net-(J7-Pad3): track 13.8 -> 45.5 mm
- net /RTS: track 66.4 -> 35.5 mm
- net /VBUS: track 39.1 -> 65.1 mm
- net Net-(J7-Pad4): track 13.8 -> 39.7 mm
- net /GP1: track 67.1 -> 43.8 mm
- net /RUN: track 118.0 -> 101.9 mm
- net Net-(J1-Pad3): track 46.1 -> 32.6 mm
- net /SCL: track 91.4 -> 103.9 mm
- net Net-(J7-Pad8): track 37.2 -> 26.8 mm
- net Net-(J7-Pad5): track 37.3 -> 27.1 mm
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
Commit message: 14:57 Arrakis.local
Parts:
- added U5: CAT24C256, Package_DIP:DIP-8_W7.62mm_LongPads, F.Cu at (152.1, 90.0)
- U3: footprint Package_TO_SOT_SMD:SuperSOT-8 -> Package_SO:SOIC-8_3.9x4.9mm_P1.27mm
- moved J5 21.2 mm to (141.1, 123.3)
- moved J4 16.0 mm to (133.3, 86.4)
- moved U4 15.2 mm to (121.8, 87.8)
- moved Q1 14.7 mm to (141.2, 87.1)
- moved J6 6.61 mm to (135.2, 112.4)
- moved J3 3.34 mm to (156.1, 123.2)
- renumbered U5 to U6
Routing:
- net /GND: track 281.7 -> 12.0 mm, vias 0 -> 7
- net /3V3: track 139.3 -> 173.6 mm, vias 2 -> 0
- net /VBUS: track 65.1 -> 79.2 mm
- net /SDA: track 89.2 -> 101.3 mm
- net /RUN: track 101.9 -> 113.2 mm
- net /5V: track 100.4 -> 92.9 mm, vias 1 -> 0
- net /GP1: track 43.8 -> 36.3 mm
- net /SCL: track 103.9 -> 99.6 mm
- net /RTS: track 35.5 -> 39.8 mm
- net Net-(J1-Pad3): track 32.6 -> 36.2 mm
- net Net-(J1-Pad4): track 33.0 -> 35.3 mm
- net /VSYS: track 63.5 -> 61.4 mm
- net /5Vopt: track 16.6 -> 15.0 mm
- net /12V: track 13.8 -> 15.2 mm
- net /GP0: track 36.7 -> 35.8 mm
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- added copper zone on B.Cu, net /GND
