File: PicoXpressSmdK/PicoXpressSmdK.kicad_pcb (KiCad board)
At the start: 2 copper layers, 100 x 80 mm, 28 parts, among them J1 6P6C, J2 parallel port, J3 I2C, J4 5V Sel, J5 I2C, J6 I2C, J7 keypad, Q1 DMG2305UX-7, SW1 Reset, U1 AMS1117-5.0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

Commit message: 18:34 Arrakis.local
Other:
- board text added: "PicoXpressSmdK version 3"
- board text removed: "PicoXpressSmdK version 2"
Changed lines of the file:
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@@
     (effects (font (size 1 1) (thickness 0.15)))
   )
-  (gr_text "PicoXpressSmdK version 2\n" (at 141 54) (layer "F.SilkS")
+  (gr_text "PicoXpressSmdK version 3\n" (at 141 54) (layer "F.SilkS")
     (effects (font (size 2 2) (thickness 0.15)))
   )
