File: PicoXpressSmdK/PicoXpressSmdK.kicad_sch (KiCad schematic)
At the start: 22 parts, among them J1 6P6C, J2 Screw_Terminal_01x09, J3 I2C, J4 Screw_Terminal_01x03, J5 I2C, J6 Screw_Terminal_01x09, Q1 DMG2305UX-7, SW1 SW_Push, U1 AMS1117-5.0, U2 MCP23008-xSO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

Commit message: 13:19 Arrakis.local
Parts:
- added J6: Screw_Terminal_01x05, Connector_PinHeader_2.54mm:PinHeader_1x05_P2.54mm_Vertical, symbol Connector:Screw_Terminal_01x05
- renumbered J6 to J7
Connections:
- net 3V3: now also J3.3, J5.3, J6.2 (Pin_2); no longer J3.2, J5.2
- net GND: now also J3.4, J5.4, J6.3 (Pin_3); no longer J3.1, J5.1
- net SCL: now also J3.1, J5.1, J6.4 (Pin_4); no longer J3.4, J5.4
- net SDA: now also J3.2, J5.2, J6.5 (Pin_5); no longer J3.3, J5.3
- no-connect marks 29 -> 30

Commit message: 19:27 Arrakis.local
Parts:
- added H1, H2, H3, H4: 0, MountingHole:MountingHole_3.2mm_M3, symbol Mechanical:MountingHole
- C1: value C_Polarized -> 100uF
- C2, C3: value C_Polarized -> 22uF
- J2: value Screw_Terminal_01x09 -> parallel port
- J4: value Screw_Terminal_01x03 -> 5V Sel
- J6: value Screw_Terminal_01x05 -> I2C
- J7: value Screw_Terminal_01x09 -> keypad
- SW1: value SW_Push -> Reset

Commit message: 09:25 Arrakis.local
Parts:
- U5: footprint MCU_RaspberryPi_and_Boards:RPi_Pico_SMD_TH -> MCU_RaspberryPi_and_Boards:RP2040Pico
Changed lines of the file:
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@@
     (property "Reference" "U5" (id 0) (at 240.0481 90.17 0))
     (property "Value" "Pico" (id 1) (at 240.0481 92.71 0))
-    (property "Footprint" "MCU_RaspberryPi_and_Boards:RPi_Pico_SMD_TH" (id 2) (at 240.0481 60.9873 90)
+    (property "Footprint" "MCU_RaspberryPi_and_Boards:RP2040Pico" (id 2) (at 240.0481 60.9873 90)
       (effects (font (size 1.27 1.27)) hide)
     )
@@
     )
     (path "/47e24da2-76f2-49b3-a05e-d1d7eec92d5c"
-      (reference "U5") (unit 1) (value "Pico") (footprint "MCU_RaspberryPi_and_Boards:RPi_Pico_SMD_TH")
-    )
-  )
+      (reference "U5") (unit 1) (value "Pico") (footprint "MCU_RaspberryPi_and_Boards:RP2040Pico")
+    )
+  )

Commit message: 14:57 Arrakis.local
Parts:
- added U5: CAT24C256, Package_DIP:DIP-8_W7.62mm_LongPads, symbol Memory_EEPROM:CAT24C256
- U3: footprint Package_TO_SOT_SMD:SuperSOT-8 -> Package_SO:SOIC-8_3.9x4.9mm_P1.27mm
- renumbered U5 to U6
Connections:
- net 3V3: now also U5.8 (VCC)
- net GND: now also U5.1 (A0), U5.2 (A1), U5.3 (A2), U5.4 (GND), U5.7 (WP)
- net SCL: now also U5.6 (SCL)
- net SDA: now also U5.5 (SDA)
Changed lines of the file:
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@@
   (junction (at 64.0163 72.8339) (diameter 0) (color 0 0 0 0)
   )
+  (junction (at 214.9438 126.1546) (diameter 0) (color 0 0 0 0)
+  )
   (junction (at 165.0932 118.5628) (diameter 0) (color 0 0 0 0)
   )
@@
   (junction (at 26.473 175.1236) (diameter 0) (color 0 0 0 0)
   )
+  (junction (at 201.8307 114.8779) (diameter 0) (color 0 0 0 0)
+  )
   (junction (at 165.0949 125.948) (diameter 0) (color 0 0 0 0)
   )
@@
   )
   (junction (at 43.0027 125.948) (diameter 0) (color 0 0 0 0)
+  )
+  (junction (at 201.8307 117.4179) (diameter 0) (color 0 0 0 0)
   )
   (junction (at 75.1542 123.1369) (diameter 0) (color 0 0 0 0)
@@
     (stroke (width 0) (type default) (color 0 0 0 0))
   )
+  (wire (pts (xy 225.2873 117.4179) (xy 225.1038 117.4179))
+    (stroke (width 0) (type default) (color 0 0 0 0))
+  )
   (wire (pts (xy 29.1396 60.1369) (xy 37.4416 60.1369))
     (stroke (width 0) (type default) (color 0 0 0 0))
@@
     (stroke (width 0) (type default) (color 0 0 0 0))
   )
+  (wire (pts (xy 230.5085 112.3379) (xy 230.5085 112.2001))
+    (stroke (width 0) (type default) (color 0 0 0 0))
+  )
+  (wire (pts (xy 201.8307 112.3379) (xy 201.8307 114.8779))
+    (stroke (width 0) (type default) (color 0 0 0 0))
+  )
   (wire (pts (xy 32.0213 106.1064) (xy 32.2766 106.1064))
     (stroke (width 0) (type default) (color 0 0 0 0))
@@
     (stroke (width 0) (type default) (color 0 0 0 0))
   )
+  (wire (pts (xy 201.8307 117.4179) (xy 204.7838 117.4179))
+    (stroke (width 0) (type default) (color 0 0 0 0))
+  )
   (wire (pts (xy 46.4082 60.1369) (xy 46.4082 65.2139))
     (stroke (width 0) (type default) (color 0 0 0 0))
@@
     (stroke (width 0) (type default) (color 0 0 0 0))
   )
+  (wire (pts (xy 225.1038 112.3379) (xy 230.5085 112.3379))
+    (stroke (width 0) (type default) (color 0 0 0 0))
+  )
   (wire (pts (xy 208.8276 33.3071) (xy 208.8276 33.2781))
     (stroke (width 0) (type default) (color 0 0 0 0))
@@
     (stroke (width 0) (type default) (color 0 0 0 0))
   )
+  (wire (pts (xy 201.8307 112.3379) (xy 204.7838 112.3379))
+    (stroke (width 0) (type default) (color 0 0 0 0))
+  )
   (wire (pts (xy 75.1507 115.5169) (xy 75.1542 115.5169))
     (stroke (width 0) (type default) (color 0 0 0 0))
@@
     (stroke (width 0) (type default) (color 0 0 0 0))
   )
+  (wire (pts (xy 201.8307 114.8779) (xy 201.8307 117.4179))
+    (stroke (width 0) (type default) (color 0 0 0 0))
+  )
   (wire (pts (xy 31.9198 125.948) (xy 31.9198 120.6533))
     (stroke (width 0) (type default) (color 0 0 0 0))
@@
     (stroke (width 0) (type default) (color 0 0 0 0))
   )
+  (wire (pts (xy 230.5085 114.8779) (xy 230.5085 114.9378))
+    (stroke (width 0) (type default) (color 0 0 0 0))
+  )
   (wire (pts (xy 48.3481 30.372) (xy 48.3481 40.617))
     (stroke (width 0) (type default) (color 0 0 0 0))
@@
     (stroke (width 0) (type default) (color 0 0 0 0))
   )
+  (wire (pts (xy 201.8307 117.4179) (xy 201.8307 126.1546))
+    (stroke (width 0) (type default) (color 0 0 0 0))
+  )
   (wire (pts (xy 48.1207 182.0554) (xy 55.4536 182.0554))
     (stroke (width 0) (type default) (color 0 0 0 0))
@@
     (stroke (width 0) (type default) (color 0 0 0 0))
   )
+  (wire (pts (xy 214.9438 126.1546) (xy 225.2873 126.1546))
+    (stroke (width 0) (type default) (color 0 0 0 0))
+  )
   (wire (pts (xy 128.5793 33.5006) (xy 128.5793 33.5916))
     (stroke (width 0) (type default) (color 0 0 0 0))
@@
     (stroke (width 0) (type default) (color 0 0 0 0))
   )
+  (wire (pts (xy 225.2873 126.1546) (xy 225.2873 117.4179))
+    (stroke (width 0) (type default) (color 0 0 0 0))
+  )
   (wire (pts (xy 57.2363 125.948) (xy 75.2236 125.948))
     (stroke (width 0) (type default) (color 0 0 0 0))
@@
     (stroke (width 0) (type default) (color 0 0 0 0))
   )
+  (wire (pts (xy 214.9438 107.2579) (xy 214.9438 103.1095))
+    (stroke (width 0) (type default) (color 0 0 0 0))
+  )
   (wire (pts (xy 205.1379 59.6272) (xy 210.8216 59.6272))
     (stroke (width 0) (type default) (color 0 0 0 0))
@@
     (stroke (width 0) (type default) (color 0 0 0 0))
   )
+  (wire (pts (xy 225.1038 114.8779) (xy 230.5085 114.8779))
+    (stroke (width 0) (type default) (color 0 0 0 0))
+  )
   (wire (pts (xy 152.1247 34.277) (xy 155.9024 34.277))
     (stroke (width 0) (type default) (color 0 0 0 0))
   )
+  (wire (pts (xy 214.9438 103.1095) (xy 214.9307 103.1095))
+    (stroke (width 0) (type default) (color 0 0 0 0))
+  )
   (wire (pts (xy 37.4416 55.8377) (xy 37.4416 60.1369))
     (stroke (width 0) (type default) (color 0 0 0 0))
@@
     (stroke (width 0) (type default) (color 0 0 0 0))
   )
+  (wire (pts (xy 201.8307 126.1546) (xy 214.9438 126.1546))
+    (stroke (width 0) (type default) (color 0 0 0 0))
+  )
   (wire (pts (xy 158.1538 105.7795) (xy 165.0561 105.7795))
     (stroke (width 0) (type default) (color 0 0 0 0))
@@
     (stroke (width 0) (type default) (color 0 0 0 0))
   )
+  (wire (pts (xy 214.9438 122.4979) (xy 214.9438 126.1546))
+    (stroke (width 0) (type default) (color 0 0 0 0))
+  )
   (wire (pts (xy 188.5329 59.6272) (xy 194.9779 59.6272))
     (stroke (width 0) (type default) (color 0 0 0 0))
@@
     (stroke (width 0) (type default) (color 0 0 0 0))
   )
+  (wire (pts (xy 201.8307 114.8779) (xy 204.7838 114.8779))
+    (stroke (width 0) (type default) (color 0 0 0 0))
+  )
   (wire (pts (xy 46.2116 95.6939) (xy 46.4082 95.6939))
     (stroke (width 0) (type default) (color 0 0 0 0))
@@
     (effects (font (size 1.27 1.27)) (justify left bottom))
   )
+  (label "SCL" (at 230.5085 114.9378 0)
+    (effects (font (size 1.27 1.27)) (justify left bottom))
+  )
   (label "GND" (at 14.4151 125.948 0)
     (effects (font (size 1.27 1.27)) (justify left bottom))
@@
     (effects (font (size 1.27 1.27)) (justify left bottom))
   )
+  (label "SDA" (at 230.5085 112.2001 0)
+    (effects (font (size 1.27 1.27)) (justify left bottom))
+  )
   (label "VBUS" (at 129.5384 85.533 0)
     (effects (font (size 1.27 1.27)) (justify left bottom))
@@
     (effects (font (size 1.27 1.27)) (justify left bottom))
   )
+  (label "3V3" (at 214.9307 103.1095 0)
+    (effects (font (size 1.27 1.27)) (justify left bottom))
+  )
   (label "SDA" (at 110.9975 28.2071 0)
     (effects (font (size 1.27 1.27)) (justify left bottom))
@@
   )
   (label "SCL" (at 110.9975 25.6828 0)
+    (effects (font (size 1.27 1.27)) (justify left bottom))
+  )
+  (label "GND" (at 214.9307 126.1546 0)
     (effects (font (size 1.27 1.27)) (justify left bottom))
   )
@@
   (symbol (lib_id "MCU_RaspberryPi_and_Boards:Pico") (at 240.0481 60.9873 180) (unit 1)
     (in_bom yes) (on_board yes) (fields_autoplaced)
-    (property "Reference" "U5" (id 0) (at 240.0481 90.17 0))
+    (property "Reference" "U6" (id 0) (at 240.0481 90.17 0))
     (property "Value" "Pico" (id 1) (at 240.0481 92.71 0))
     (property "Footprint" "MCU_RaspberryPi_and_Boards:RP2040Pico" (id 2) (at 240.0481 60.9873 90)
@@
     (pin "9")
   )
+  (symbol (lib_id "Memory_EEPROM:CAT24C256") (at 214.9438 114.8779 0) (unit 1)
+    (in_bom yes) (on_board yes) (fields_autoplaced)
+    (property "Reference" "U5" (id 0) (at 216.9632 104.14 0)
+      (effects (font (size 1.27 1.27)) (justify left))
+    )
+    (property "Value" "CAT24C256" (id 1) (at 216.9632 106.68 0)
+      (effects (font (size 1.27 1.27)) (justify left))
+    )
+    (property "Footprint" "Package_DIP:DIP-8_W7.62mm_LongPads" (id 2) (at 214.9438 114.8779 0)
+      (effects (font (size 1.27 1.27)) hide)
+    )
+    (property "Datasheet" "https://www.onsemi.cn/PowerSolutions/document/CAT24C256-D.PDF" (id 3) (at 214.9438 114.8779 0)
+      (effects (font (size 1.27 1.27)) hide)
+    )
+    (pin "1")
+    (pin "2")
+    (pin "3")
+    (pin "4")
+    (pin "5")
+    (pin "6")
+    (pin "7")
+    (pin "8")
+  )
   (symbol (lib_id "Interface_Expansion:MCP23008-xSO") (at 46.4082 80.4539 180) (unit 1)
     (in_bom yes) (on_board yes) (fields_autoplaced)
@@
       (effects (font (size 1.27 1.27)) (justify right))
     )
-    (property "Footprint" "Package_TO_SOT_SMD:SuperSOT-8" (id 2) (at 69.5861 53.3075 0)
+    (property "Footprint" "Package_SO:SOIC-8_3.9x4.9mm_P1.27mm" (id 2) (at 69.5861 53.3075 0)
       (effects (font (size 1.27 1.27)) hide)
     )
@@
     )
     (path "/792104c5-3e22-452a-89e8-4ea70a4f2fd3"
-      (reference "U3") (unit 1) (value "MAX3485") (footprint "Package_TO_SOT_SMD:SuperSOT-8")
+      (reference "U3") (unit 1) (value "MAX3485") (footprint "Package_SO:SOIC-8_3.9x4.9mm_P1.27mm")
     )
     (path "/633946f7-6171-45d7-9b79-cc8824467c30"
       (reference "U4") (unit 1) (value "AMS1117-3.3") (footprint "Package_TO_SOT_SMD:SOT-223-3_TabPin2")
     )
+    (path "/4d6515b2-e8bf-4a2f-92c9-f1af029d2b9d"
+      (reference "U5") (unit 1) (value "CAT24C256") (footprint "Package_DIP:DIP-8_W7.62mm_LongPads")
+    )
     (path "/47e24da2-76f2-49b3-a05e-d1d7eec92d5c"
-      (reference "U5") (unit 1) (value "Pico") (footprint "MCU_RaspberryPi_and_Boards:RP2040Pico")
-    )
-  )
+      (reference "U6") (unit 1) (value "Pico") (footprint "MCU_RaspberryPi_and_Boards:RP2040Pico")
+    )
+  )
