File: DCCStepperDrive2/DCCStepperDrive2.kicad_sch (KiCad schematic)
At the start: 33 parts, among them J1 12v, J2 CBUS, J3 5V select, J4 DCC, J5 Grove 2mm, J6 I2C, J7 Sensor, J8 Motor, J9 Mode Select, Q1 DMG2305UX-7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

Commit message: 19:58 Titan.local
Connections:
- net +5V is gone; now on net 3V3: J9.10 (Pin_10), J9.6 (Pin_6), J9.8 (Pin_8)
Changed lines of the file:
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@@
     (effects (font (size 1.27 1.27)) (justify left bottom))
   )
-  (label "+5V" (at 257.81 22.86 0)
+  (label "3V3" (at 257.81 22.86 0)
     (effects (font (size 1.27 1.27)) (justify left bottom))
   )
