File: DCCStepperDrive2/DCCStepperDrive2.kicad_pcb (KiCad board)
At the start: 2 copper layers, 100 x 100 mm, 35 parts, among them J1 12v, J2 CBUS, J3 5V select, J4 DCC, J5 Grove 2mm, J6 I2C, J7 Sensor, J8 Motor, J9 Mode Select, Q1 DMG2305UX-7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

Commit message: 19:58 Titan.local
Connections:
- J9 pad 10: /+5V -> /3V3
- J9 pad 6: /+5V -> /3V3
- J9 pad 8: /+5V -> /3V3
Routing:
- net /3V3: track 206.9 -> 240.7 mm
- net /DccIn: track 82.9 -> 62.3 mm
- net Net-(J7-Pad3): track 103.9 -> 83.5 mm
- net /5V: track 47.1 -> 34.9 mm
- net Net-(C2-Pad1): track 70.7 -> 80.8 mm, vias 1 -> 0
- net Net-(A1-Pad9): track 90.7 -> 98.8 mm
- net /+5V: track 5.08 -> 0.00 mm
- net Net-(R3-Pad1): track 38.4 -> 34.8 mm
- net /SDA: track 98.3 -> 101.1 mm
- net Net-(SW1-Pad2): track 46.2 -> 43.7 mm
- net /VSYS: track 78.2 -> 77.0 mm
- net /12V: track 85.1 -> 84.2 mm
- net Net-(A1-Pad15): track 79.8 -> 80.5 mm, vias 0 -> 1
- net GND: track 312.5 -> 311.7 mm
- net /SCL: track 100.2 -> 99.5 mm
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Other:
- board text added: "DCC"
- board text added: "GND"

Commit message: 09/09/25 09:18 Arrakis.local
Parts:
- removed NT1, NT2: NetTie_2, NetTie:NetTie-2_SMD_Pad0.5mm
- J5, J6: footprint OPL_Connector:HW4-2.0 -> OPL_Kicad_Library:HW4-2.0
- U4: footprint MCU_RaspberryPi_and_Boards:RP2040Pico -> Kicad-RP-Pico:RPi_Pico_SMD_TH
Routing:
- net GND: track 311.7 -> 0.00 mm
- net /3V3: track 240.7 -> 0.00 mm
- net /SDA: track 101.1 -> 0.00 mm
- net /SCL: track 99.5 -> 0.00 mm
- net Net-(A1-~{ENABLE}): track 98.8 -> 0.00 mm
- net /VBUS: track 85.1 -> 0.00 mm
- net /12V: track 84.2 -> 0.00 mm
- net Net-(J7-Pin_3): track 83.5 -> 0.00 mm
- net Net-(J4-Pin_2): track 80.8 -> 0.00 mm
- net Net-(A1-STEP): track 80.5 -> 0.00 mm, vias 1 -> 0
- net /VSYS: track 77.0 -> 0.00 mm, vias 1 -> 0
- net Net-(A1-DIR): track 76.6 -> 0.00 mm, vias 1 -> 0
- net /DccIn: track 62.3 -> 0.00 mm, vias 1 -> 0
- net Net-(D1-A): track 59.9 -> 0.00 mm
- net Net-(J7-Pin_2): track 57.8 -> 0.00 mm
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
Commit message: 09/09/25 10:15 Titan.local
Parts:
- moved U4 1.15 mm to (123.2, 83.8)
Routing:
- net GND: track 0.00 -> 336.0 mm, vias 0 -> 1
- net /3V3: track 0.00 -> 225.0 mm, vias 0 -> 2
- net /SDA: track 0.00 -> 115.1 mm
- net /SCL: track 0.00 -> 111.4 mm, vias 0 -> 1
- net Net-(A1-STEP): track 0.00 -> 97.3 mm, vias 0 -> 1
- net Net-(A1-DIR): track 0.00 -> 93.1 mm, vias 0 -> 1
- net Net-(A1-~{ENABLE}): track 0.00 -> 90.2 mm
- net Net-(J7-Pin_3): track 0.00 -> 88.8 mm
- net /VSYS: track 0.00 -> 87.3 mm, vias 0 -> 1
- net /12V: track 0.00 -> 85.8 mm
- net /VBUS: track 0.00 -> 81.7 mm
- net Net-(J4-Pin_2): track 0.00 -> 74.8 mm, vias 0 -> 1
- net Net-(D2-K): track 0.00 -> 69.3 mm, vias 0 -> 1
- net Net-(J7-Pin_2): track 0.00 -> 62.2 mm
- net /DccIn: track 0.00 -> 61.8 mm, vias 0 -> 1
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
Commit message: 09/09/25 11:50 Arrakis.local
Parts:
- U4: footprint Kicad-RP-Pico:RPi_Pico_SMD_TH -> RP-Pico Libraries:RP2040Pico

Commit message: 09/09/25 16:21 Titan.local
Parts:
- U4: footprint RP-Pico Libraries:RP2040Pico -> Kicad-RP-Pico:RPi_Pico_SMD_TH
