File: SingleRelay/SingleRelay.kicad_sch (KiCad schematic)
At the start: 2 parts, among them Q1 2N7002

Commit message: 15:58 Arrakis.local
Parts:
- added D2: LED, LED_THT:LED_D3.0mm_Clear, symbol Device:LED
- added J1: Logic In, TerminalBlock_Phoenix:TerminalBlock_Phoenix_PT-1,5-2-3.5-H_1x02_P3.50mm_Horizontal, symbol Connector:Screw_Terminal_01x02
- added J2: Relay Power, TerminalBlock_Phoenix:TerminalBlock_Phoenix_PT-1,5-2-3.5-H_1x02_P3.50mm_Horizontal, symbol Connector:Screw_Terminal_01x02
- added J3, J5: OUT1, TerminalBlock_Phoenix:TerminalBlock_Phoenix_PT-1,5-3-3.5-H_1x03_P3.50mm_Horizontal, symbol Connector:Screw_Terminal_01x03
- added J4: OUT2, TerminalBlock_Phoenix:TerminalBlock_Phoenix_PT-1,5-3-3.5-H_1x03_P3.50mm_Horizontal, symbol Connector:Screw_Terminal_01x03
- added K1: FINDER-36.11, Relay_THT:Relay_SPDT_Finder_36.11, symbol Relay:FINDER-36.11
- added R1, R2: 10k, Resistor_SMD:R_1206_3216Metric, symbol Device:R_US
- added RL1: G2RL-2-DC5, Relay_THT:Relay_DPDT_Omron_G2RL, symbol Relay:G2RL-2-DC5
Connections:
- net at Q1.1 (G): now also J1.2 (Pin_2), R1.1, R2.1
- net GND: now reaches Q1.2 (S)
- net GND: now also D2.1 (K), J1.1 (Pin_1), J2.1 (Pin_1), R2.2
- net at Q1.3 (D): now also D1.2 (A), K1.A2, RL1.8
- net +5V: now reaches D1.1 (K)
- net +5V: now also J2.2 (Pin_2), K1.A1, RL1.1
- new net: J4.1 (Pin_1), RL1.2
- new net: J4.2 (Pin_2), RL1.3
- new net: J4.3 (Pin_3), RL1.4
- new net: J3.3 (Pin_3), RL1.5
- new net: J3.2 (Pin_2), RL1.6
- new net: J3.1 (Pin_1), RL1.7
- new net: J5.2 (Pin_2), K1.11
- new net: J5.1 (Pin_1), K1.12
- new net: J5.3 (Pin_3), K1.14
- new net: D2.2 (A), R1.2
Other:
- note added: "Notes: 1. alternative relay types 2. SPDT is Songle SRD-05VDC-SL-C or similar 3. DPDT is DIP style"
- title: (none) -> Single Relay DPDT
- moved on the sheet: D1

Commit message: 19:58 Titan.local
Parts:
- added D3: LED, LED_THT:LED_D3.0mm_Clear, symbol Device:LED
- added D4: 1N4148W, Diode_SMD:D_SOD-123, symbol Diode:1N4148W
- added J6: Logic In, TerminalBlock_Phoenix:TerminalBlock_Phoenix_PT-1,5-2-3.5-H_1x02_P3.50mm_Horizontal, symbol Connector:Screw_Terminal_01x02
- added J7: Relay Power, TerminalBlock_Phoenix:TerminalBlock_Phoenix_PT-1,5-2-3.5-H_1x02_P3.50mm_Horizontal, symbol Connector:Screw_Terminal_01x02
- added Q2: 2N7002, Package_TO_SOT_SMD:SOT-23, symbol Transistor_FET:2N7002
- added R3, R4: 10k, Resistor_SMD:R_1206_3216Metric, symbol Device:R_US
Connections:
- net +5V: no longer K1.A1
- net at D1.2 (A), Q1.3 (D), RL1.8: no longer K1.A2
- net at K1.12: now also J5.3 (Pin_3); no longer J5.1 (Pin_1)
- net at K1.14: now also J5.1 (Pin_1); no longer J5.3 (Pin_3)
- new net: J6.2 (Pin_2), Q2.1 (G), R3.1, R4.1
- new net: D4.2 (A), K1.A2, Q2.3 (D)
- new net: D3.2 (A), R3.2
- new net 5V: D4.1 (K), J7.2 (Pin_2), K1.A1
- new net Gnd: D3.1 (K), J6.1 (Pin_1), J7.1 (Pin_1), Q2.2 (S), R4.2
Other:
- note added: "Notes: 1. alternative relay types 2. SPDT is Songle SRD-05VDC-SL-C or similar 3. DPDT is DIP style 4. Logic in to +5V to turn on"
- note removed: "Notes: 1. alternative relay types 2. SPDT is Songle SRD-05VDC-SL-C or similar 3. DPDT is DIP style"
- moved on the sheet: D1, D2, J1, J2, J3, J4, J5, K1, Q1, R1, R2, RL1
