File: RFBasicBoard/RFBasicBoard/RFBasicBoard.kicad_pcb (KiCad board)
At the start: 2 copper layers, 100 x 80 mm, 17 parts, among them J1 3.50 CBUS, J2 5V select, J3 Grove 2mm, J4 Receiver, J5 Transmitter, J6 Barrel_Jack, Q1 DMG2305UX-7, U1 AMS1117-5.0, U2 AMS1117-3.3, U3 Pico

Commit message: 08:44 Titan.local
Parts:
- moved J5 14.8 mm to (126.8, 52.3)
- moved J4 14.1 mm to (147.6, 50.9)
Connections:
- J4 pad 2: Net-(J4-Pad2) -> Net-(U3-Pad22)
- U3 pad 10: Net-(J4-Pad2) -> unconnected-(U3-Pad10)
- U3 pad 21: unconnected-(U3-Pad21) -> Net-(J5-Pad1)
- U3 pad 22: unconnected-(U3-Pad22) -> Net-(U3-Pad22)
- U3 pad 9: Net-(J5-Pad1) -> unconnected-(U3-Pad9)
Routing:
- net Net-(U3-Pad22): track 0.00 -> 45.0 mm
- net Net-(J5-Pad1): track 40.6 -> 67.2 mm
- net Net-(J4-Pad2): track 23.4 -> 0.00 mm
- net /VSYS: track 117.6 -> 111.6 mm
- net Net-(J4-Pad1): track 44.0 -> 41.1 mm
- net /VBUS: track 68.2 -> 69.6 mm
