File: RFBasicBoard/RFBasicBoard.kicad_sch (KiCad schematic)
At the start: 17 parts, among them J1 3.50 CBUS, J2 5V select, J3 Grove 2mm, J4 Receiver, J5 Transmitter, J6 Barrel_Jack, Q1 DMG2305UX-7, U1 AMS1117-5.0, U2 AMS1117-3.3, U3 Pico

Commit message: 20:53 Arrakis.local
Parts:
- removed C1: 22uF, Capacitor_THT:CP_Radial_Tantal_D7.0mm_P5.00mm, symbol Device:C_Polarized
- removed U2: AMS1117-3.3, Package_TO_SOT_SMD:SOT-223-3_TabPin2, symbol Regulator_Linear:AMS1117-3.3
- added Brd1: SSD1306, SSD1306:128x64OLED, symbol SSD1306-128x64_OLED:SSD1306
- added D2: CUS05540, Diode_SMD:D_SOD-123, symbol Diode:MBR0520
- renumbered C2 to C1, J6 to J4, J4 to J5, J5 to J6, U3 to U2
Connections:
- net 3V3: now also Brd1.2 (VCC)
- net 5V: now also D2.2 (A)
- net GND: now also Brd1.1 (GND)
- net SCL: now also Brd1.3 (SCL)
- net SDA: now also Brd1.4 (SDA)
- net VSYS: now also D2.1 (K)
