File: RaspberryPiExtension/RaspberryPiExtension.kicad_pcb (KiCad board)
At the start: 2 copper layers, 2 parts, among them J1 RASPBERRYPI-40-PIN-GPIO_PTH_N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, J2 Screw_Terminal_01x02

Commit message: 20:53 Arrakis.local
Parts:
- removed the J2 at (259.4, 45.7)
- added H1: MountingHole, MountingHole:MountingHole_2.5mm_Pad_TopBottom, F.Cu at (103.5, 111.5)
- added H2: MountingHole, MountingHole:MountingHole_2.5mm_Pad_TopBottom, F.Cu at (103.5, 53.5)
- added H3: MountingHole, MountingHole:MountingHole_2.5mm_Pad_TopBottom, F.Cu at (152.5, 53.5)
- added H4: MountingHole, MountingHole:MountingHole_2.5mm_Pad_TopBottom, F.Cu at (152.5, 111.5)
- added J3: RF Transmitter, Connector_PinHeader_2.54mm:PinHeader_1x03_P2.54mm_Vertical, F.Cu at (139.0, 56.5)
- added J4: RF Receiver, Connector_PinHeader_2.54mm:PinHeader_1x04_P2.54mm_Vertical, F.Cu at (145.0, 76.5)
- added J5: Somfy Transmitter, Connector_PinHeader_2.54mm:PinHeader_1x03_P2.54mm_Vertical, F.Cu at (130.5, 56.5)
- moved J2 142.4 mm to (104.8, 106.6), turned to 0 degrees
- renumbered J1 to J2
Connections:
- J2 pad 1: unconnected-(J1-Pad1) -> /3V3
- J2 pad 16: unconnected-(J1-Pad16) -> Net-(J2-Pad16)
- J2 pad 32: unconnected-(J1-Pad32) -> Net-(J2-Pad32)
- J2 pad 36: unconnected-(J1-Pad36) -> Net-(J3-Pad2)
Routing:
- net /3V3: track 0.00 -> 59.3 mm
- net /GND: track 25.9 -> 85.1 mm
- net Net-(J2-Pad16): track 0.00 -> 48.5 mm
- net /5V: track 25.9 -> 72.0 mm
- net Net-(J3-Pad2): track 0.00 -> 39.8 mm
- net Net-(J2-Pad32): track 0.00 -> 32.4 mm
- added copper zone on B.Cu, net /GND
Other:
- board outline added: 56 x 65 mm
- board text added: "Gnd"

Commit message: 08:55 Titan.local
Parts:
- H1, H2, H3, H4: footprint MountingHole:MountingHole_2.5mm_Pad_TopBottom -> MountingHole:MountingHole_2.7mm_M2.5_Pad
Other:
- board text added: "RF 433 MHz transmit receive v1.0"
Changed lines of the file:
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@@
   (net 37 "/3V3")
   (net 38 "Net-(J2-Pad16)")
-  (net 39 "Net-(J3-Pad2)")
+  (net 39 "Net-(J2-Pad36)")
   (net 40 "Net-(J2-Pad32)")
-  (footprint "MountingHole:MountingHole_2.5mm_Pad_TopBottom" (layer "F.Cu")
+  (footprint "MountingHole:MountingHole_2.7mm_M2.5_Pad" (layer "F.Cu")
     (at 103.5 111.5)
-    (descr "Mounting Hole 2.5mm")
-    (tags "mounting hole 2.5mm")
+    (descr "Mounting Hole 2.7mm, M2.5")
+    (tags "mounting hole 2.7mm m2.5")
     (property "Sheetfile" "RaspberryPiExtension.kicad_sch")
     (property "Sheetname" "")
     (attr exclude_from_pos_files)
-    (fp_text reference "H1" (at 0 -3.5) (layer "F.SilkS")
-      (effects (font (size 1 1) (thickness 0.15)))
-    )
-    (fp_text value "MountingHole" (at 0 3.5) (layer "F.Fab")
+    (fp_text reference "H1" (at 0 -3.7) (layer "F.SilkS")
+      (effects (font (size 1 1) (thickness 0.15)))
+    )
+    (fp_text value "MountingHole" (at 0 3.7) (layer "F.Fab")
       (effects (font (size 1 1) (thickness 0.15)))
     )
@@
       (effects (font (size 1 1) (thickness 0.15)))
     )
-    (fp_circle (center 0 0) (end 2.5 0) (layer "Cmts.User") (width 0.15) (fill none))
-    (fp_circle (center 0 0) (end 2.75 0) (layer "F.CrtYd") (width 0.05) (fill none))
-    (pad "1" thru_hole circle (at 0 0) (size 2.9 2.9) (drill 2.5) (layers *.Cu *.Mask))
-    (pad "1" connect circle (at 0 0) (size 5 5) (layers "B.Cu" "B.Mask"))
-    (pad "1" connect circle (at 0 0) (size 5 5) (layers "F.Cu" "F.Mask"))
+    (fp_circle (center 0 0) (end 2.7 0) (layer "Cmts.User") (width 0.15) (fill none))
+    (fp_circle (center 0 0) (end 2.95 0) (layer "F.CrtYd") (width 0.05) (fill none))
+    (pad "1" thru_hole circle (at 0 0) (size 5.4 5.4) (drill 2.7) (layers *.Cu *.Mask))
   )
   (footprint "Connector_PinHeader_2.54mm:PinHeader_1x03_P2.54mm_Vertical" (layer "F.Cu")
@@
     )
   )
-  (footprint "MountingHole:MountingHole_2.5mm_Pad_TopBottom" (layer "F.Cu")
+  (footprint "MountingHole:MountingHole_2.7mm_M2.5_Pad" (layer "F.Cu")
     (at 152.5 111.5)
-    (descr "Mounting Hole 2.5mm")
-    (tags "mounting hole 2.5mm")
+    (descr "Mounting Hole 2.7mm, M2.5")
+    (tags "mounting hole 2.7mm m2.5")
     (property "Sheetfile" "RaspberryPiExtension.kicad_sch")
     (property "Sheetname" "")
     (attr exclude_from_pos_files)
-    (fp_text reference "H4" (at 0 -3.5) (layer "F.SilkS")
-      (effects (font (size 1 1) (thickness 0.15)))
-    )
-    (fp_text value "MountingHole" (at 0 3.5) (layer "F.Fab")
+    (fp_text reference "H4" (at 0 -3.7) (layer "F.SilkS")
+      (effects (font (size 1 1) (thickness 0.15)))
+    )
+    (fp_text value "MountingHole" (at 0 3.7) (layer "F.Fab")
       (effects (font (size 1 1) (thickness 0.15)))
     )
@@
       (effects (font (size 1 1) (thickness 0.15)))
     )
-    (fp_circle (center 0 0) (end 2.5 0) (layer "Cmts.User") (width 0.15) (fill none))
-    (fp_circle (center 0 0) (end 2.75 0) (layer "F.CrtYd") (width 0.05) (fill none))
-    (pad "1" connect circle (at 0 0) (size 5 5) (layers "F.Cu" "F.Mask"))
-    (pad "1" connect circle (at 0 0) (size 5 5) (layers "B.Cu" "B.Mask"))
-    (pad "1" thru_hole circle (at 0 0) (size 2.9 2.9) (drill 2.5) (layers *.Cu *.Mask))
+    (fp_circle (center 0 0) (end 2.7 0) (layer "Cmts.User") (width 0.15) (fill none))
+    (fp_circle (center 0 0) (end 2.95 0) (layer "F.CrtYd") (width 0.05) (fill none))
+    (pad "1" thru_hole circle (at 0 0) (size 5.4 5.4) (drill 2.7) (layers *.Cu *.Mask))
   )
   (footprint "Connector_PinHeader_2.54mm:PinHeader_1x03_P2.54mm_Vertical" (layer "F.Cu")
@@
       (net 35 "/5V") (pinfunction "Pin_1") (pintype "passive"))
     (pad "2" thru_hole oval (at 0 2.54) (size 1.7 1.7) (drill 1) (layers *.Cu *.Mask)
-      (net 39 "Net-(J3-Pad2)") (pinfunction "Pin_2") (pintype "passive"))
+      (net 39 "Net-(J2-Pad36)") (pinfunction "Pin_2") (pintype "passive"))
     (pad "3" thru_hole oval (at 0 5.08) (size 1.7 1.7) (drill 1) (layers *.Cu *.Mask)
       (net 36 "/GND") (pinfunction "Pin_3") (pintype "passive"))
@@
     )
   )
-  (footprint "MountingHole:MountingHole_2.5mm_Pad_TopBottom" (layer "F.Cu")
+  (footprint "MountingHole:MountingHole_2.7mm_M2.5_Pad" (layer "F.Cu")
     (at 152.5 53.5)
-    (descr "Mounting Hole 2.5mm")
-    (tags "mounting hole 2.5mm")
+    (descr "Mounting Hole 2.7mm, M2.5")
+    (tags "mounting hole 2.7mm m2.5")
     (property "Sheetfile" "RaspberryPiExtension.kicad_sch")
     (property "Sheetname" "")
     (attr exclude_from_pos_files)
-    (fp_text reference "H3" (at 0 -3.5) (layer "F.SilkS")
-      (effects (font (size 1 1) (thickness 0.15)))
-    )
-    (fp_text value "MountingHole" (at 0 3.5) (layer "F.Fab")
+    (fp_text reference "H3" (at 0 -3.7) (layer "F.SilkS")
+      (effects (font (size 1 1) (thickness 0.15)))
+    )
+    (fp_text value "MountingHole" (at 0 3.7) (layer "F.Fab")
       (effects (font (size 1 1) (thickness 0.15)))
     )
@@
       (effects (font (size 1 1) (thickness 0.15)))
     )
-    (fp_circle (center 0 0) (end 2.5 0) (layer "Cmts.User") (width 0.15) (fill none))
-    (fp_circle (center 0 0) (end 2.75 0) (layer "F.CrtYd") (width 0.05) (fill none))
-    (pad "1" connect circle (at 0 0) (size 5 5) (layers "F.Cu" "F.Mask"))
-    (pad "1" thru_hole circle (at 0 0) (size 2.9 2.9) (drill 2.5) (layers *.Cu *.Mask))
-    (pad "1" connect circle (at 0 0) (size 5 5) (layers "B.Cu" "B.Mask"))
-  )
-  (footprint "MountingHole:MountingHole_2.5mm_Pad_TopBottom" (layer "F.Cu")
+    (fp_circle (center 0 0) (end 2.7 0) (layer "Cmts.User") (width 0.15) (fill none))
+    (fp_circle (center 0 0) (end 2.95 0) (layer "F.CrtYd") (width 0.05) (fill none))
+    (pad "1" thru_hole circle (at 0 0) (size 5.4 5.4) (drill 2.7) (layers *.Cu *.Mask))
+  )
+  (footprint "MountingHole:MountingHole_2.7mm_M2.5_Pad" (layer "F.Cu")
     (at 103.5 53.5)
-    (descr "Mounting Hole 2.5mm")
-    (tags "mounting hole 2.5mm")
+    (descr "Mounting Hole 2.7mm, M2.5")
+    (tags "mounting hole 2.7mm m2.5")
     (property "Sheetfile" "RaspberryPiExtension.kicad_sch")
     (property "Sheetname" "")
     (attr exclude_from_pos_files)
-    (fp_text reference "H2" (at 0 -3.5) (layer "F.SilkS")
-      (effects (font (size 1 1) (thickness 0.15)))
-    )
-    (fp_text value "MountingHole" (at 0 3.5) (layer "F.Fab")
+    (fp_text reference "H2" (at 0 -3.7) (layer "F.SilkS")
+      (effects (font (size 1 1) (thickness 0.15)))
+    )
+    (fp_text value "MountingHole" (at 0 3.7) (layer "F.Fab")
       (effects (font (size 1 1) (thickness 0.15)))
     )
@@
       (effects (font (size 1 1) (thickness 0.15)))
     )
-    (fp_circle (center 0 0) (end 2.5 0) (layer "Cmts.User") (width 0.15) (fill none))
-    (fp_circle (center 0 0) (end 2.75 0) (layer "F.CrtYd") (width 0.05) (fill none))
-    (pad "1" connect circle (at 0 0) (size 5 5) (layers "B.Cu" "B.Mask"))
-    (pad "1" thru_hole circle (at 0 0) (size 2.9 2.9) (drill 2.5) (layers *.Cu *.Mask))
-    (pad "1" connect circle (at 0 0) (size 5 5) (layers "F.Cu" "F.Mask"))
+    (fp_circle (center 0 0) (end 2.7 0) (layer "Cmts.User") (width 0.15) (fill none))
+    (fp_circle (center 0 0) (end 2.95 0) (layer "F.CrtYd") (width 0.05) (fill none))
+    (pad "1" thru_hole circle (at 0 0) (size 5.4 5.4) (drill 2.7) (layers *.Cu *.Mask))
   )
   (footprint "Connector_PinSocket_2.54mm:PinSocket_2x20_P2.54mm_Vertical" (layer "B.Cu")
@@
       (net 30 "unconnected-(J2-Pad35)") (pinfunction "GP19") (pintype "bidirectional+no_connect"))
     (pad "36" thru_hole oval (at -2.54 -43.18) (size 1.7 1.7) (drill 1) (layers *.Cu *.Mask)
-      (net 39 "Net-(J3-Pad2)") (pinfunction "GP16") (pintype "bidirectional"))
+      (net 39 "Net-(J2-Pad36)") (pinfunction "GP16") (pintype "bidirectional"))
     (pad "37" thru_hole oval (at 0 -45.72) (size 1.7 1.7) (drill 1) (layers *.Cu *.Mask)
       (net 31 "unconnected-(J2-Pad37)") (pinfunction "GP26") (pintype "bidirectional+no_connect"))
@@
     (effects (font (size 1 1) (thickness 0.15)))
   )
-  (dimension (type aligned) (layer "B.Cu")
+  (gr_text "RF 433 MHz transmit receive v1.0\n" (at 128.833085 51.874814) (layer "F.SilkS")
+    (effects (font (size 1.5 1.5) (thickness 0.3)))
+  )
+  (dimension (type aligned) (layer "Eco1.User")
     (pts (xy 103.5 53.5) (xy 103.5 111.5))
     (height 7)
-    (gr_text "58.0000 mm" (at 94.7 82.5 90) (layer "B.Cu")
+    (gr_text "58.0000 mm" (at 94.7 82.5 90) (layer "Eco1.User")
       (effects (font (size 1.5 1.5) (thickness 0.3)))
     )
@@
     (style (thickness 0.2) (arrow_length 1.27) (text_position_mode 0) (extension_height 0.58642) (extension_offset 0.5) keep_text_aligned)
   )
-  (dimension (type aligned) (layer "B.Cu")
+  (dimension (type aligned) (layer "Eco1.User")
     (pts (xy 103.5 53.5) (xy 152.5 53.5))
     (height -6.5)
-    (gr_text "49.0000 mm" (at 128 45.2) (layer "B.Cu")
+    (gr_text "49.0000 mm" (at 128 45.2) (layer "Eco1.User")
       (effects (font (size 1.5 1.5) (thickness 0.3)))
     )
@@
     (style (thickness 0.2) (arrow_length 1.27) (text_position_mode 0) (extension_height 0.58642) (extension_offset 0.5) keep_text_aligned)
   )
-  (dimension (type aligned) (layer "B.Cu")
+  (dimension (type aligned) (layer "Eco1.User")
     (pts (xy 152.5 53.5) (xy 156 53.5))
     (height -9)
-    (gr_text "3.5000 mm" (at 154.25 42.7) (layer "B.Cu")
+    (gr_text "3.5000 mm" (at 154.25 42.7) (layer "Eco1.User")
       (effects (font (size 1.5 1.5) (thickness 0.3)))
     )
