File: RaspberryPiExtension/RaspberryPiExtension.kicad_pcb (KiCad board)
At the start: 2 copper layers, 56 x 65 mm, 8 parts, among them J2 RASPBERRYPI-40-PIN-GPIO_PTH_N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, J3 RF Transmitter, J4 RF Receiver, J5 Somfy Transmitter

Commit message: 14:40 Arrakis.local
Parts:
- ?: renamed from H1; value MountingHole -> (none)
- ?: renamed from H4; value MountingHole -> (none)
- ?: renamed from H3; value MountingHole -> (none)
- ?: renamed from H2; value MountingHole -> (none)
