File: RaspberryPiExtension/RaspberryPiExtension.kicad_sch (KiCad schematic)
At the start: 2 parts, among them J1 RASPBERRYPI-40-PIN-GPIO_PTH_N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, J2 Screw_Terminal_01x02

Commit message: 20:53 Arrakis.local
Parts:
- removed J2: Screw_Terminal_01x02, TerminalBlock_Phoenix:TerminalBlock_Phoenix_MKDS-1,5-2_1x02_P5.00mm_Horizontal, symbol Connector:Screw_Terminal_01x02
- added H1, H2, H3, H4: MountingHole, MountingHole:MountingHole_2.5mm_Pad_TopBottom, symbol Mechanical:MountingHole
- added J3: RF Transmitter, Connector_PinHeader_2.54mm:PinHeader_1x03_P2.54mm_Vertical, symbol Connector:Screw_Terminal_01x03
- added J4: RF Receiver, Connector_PinHeader_2.54mm:PinHeader_1x04_P2.54mm_Vertical, symbol Connector:Screw_Terminal_01x04
- added J5: Somfy Transmitter, Connector_PinHeader_2.54mm:PinHeader_1x03_P2.54mm_Vertical, symbol Connector:Screw_Terminal_01x03
- renumbered J1 to J2
Connections:
- net 5V: now also J3.1 (Pin_1), J5.1 (Pin_1)
- net GND: now also J3.3 (Pin_3), J4.4 (Pin_4), J5.3 (Pin_3)
- net 3V3: now reaches J2.1 (3.3V)
- net 3V3: now also J4.1 (Pin_1)
- net at J2.16 (GP23): now also J4.2 (Pin_2), J4.3 (Pin_3)
- net at J2.32 (GP12): now also J5.2 (Pin_2)
- net at J2.36 (GP16): now also J3.2 (Pin_2)
- no-connect marks 0 -> 34

Commit message: 08:55 Titan.local
Parts:
- H1, H2, H3, H4: footprint MountingHole:MountingHole_2.5mm_Pad_TopBottom -> MountingHole:MountingHole_2.7mm_M2.5_Pad
Other:
- title: (none) -> Raspberry piExpansion Board for RF Receive Transmit
Changed lines of the file:
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@@
 (kicad_sch (version 20211123) (generator eeschema)
   (paper "A4")
+  (title_block
+    (title "Raspberry piExpansion Board for RF Receive Transmit")
+    (date "2024-07-09")
+    (rev "1.0")
+  )
   (junction (at 203.2 71.12) (diameter 0) (color 0 0 0 0)
   )
@@
       (effects (font (size 1.27 1.27)) (justify left))
     )
-    (property "Footprint" "MountingHole:MountingHole_2.5mm_Pad_TopBottom" (id 2) (at 38.1 177.8 0)
+    (property "Footprint" "MountingHole:MountingHole_2.7mm_M2.5_Pad" (id 2) (at 38.1 177.8 0)
       (effects (font (size 1.27 1.27)) hide)
     )
@@
       (effects (font (size 1.27 1.27)) (justify left))
     )
-    (property "Footprint" "MountingHole:MountingHole_2.5mm_Pad_TopBottom" (id 2) (at 38.1 165.1 0)
+    (property "Footprint" "MountingHole:MountingHole_2.7mm_M2.5_Pad" (id 2) (at 38.1 165.1 0)
       (effects (font (size 1.27 1.27)) hide)
     )
@@
       (effects (font (size 1.27 1.27)) (justify left))
     )
-    (property "Footprint" "MountingHole:MountingHole_2.5mm_Pad_TopBottom" (id 2) (at 50.8 166.37 0)
+    (property "Footprint" "MountingHole:MountingHole_2.7mm_M2.5_Pad" (id 2) (at 50.8 166.37 0)
       (effects (font (size 1.27 1.27)) hide)
     )
@@
       (effects (font (size 1.27 1.27)) (justify left))
     )
-    (property "Footprint" "MountingHole:MountingHole_2.5mm_Pad_TopBottom" (id 2) (at 50.8 177.8 0)
+    (property "Footprint" "MountingHole:MountingHole_2.7mm_M2.5_Pad" (id 2) (at 50.8 177.8 0)
       (effects (font (size 1.27 1.27)) hide)
     )
@@
     )
     (path "/19b28336-8a5d-4757-a46a-8fb0723c8931"
-      (reference "H1") (unit 1) (value "MountingHole") (footprint "MountingHole:MountingHole_2.5mm_Pad_TopBottom")
+      (reference "H1") (unit 1) (value "MountingHole") (footprint "MountingHole:MountingHole_2.7mm_M2.5_Pad")
     )
     (path "/173ee601-dbdc-4515-b950-40d3179401dc"
-      (reference "H2") (unit 1) (value "MountingHole") (footprint "MountingHole:MountingHole_2.5mm_Pad_TopBottom")
+      (reference "H2") (unit 1) (value "MountingHole") (footprint "MountingHole:MountingHole_2.7mm_M2.5_Pad")
     )
     (path "/54d29be9-0b3e-40c8-9852-faa7a490d23f"
-      (reference "H3") (unit 1) (value "MountingHole") (footprint "MountingHole:MountingHole_2.5mm_Pad_TopBottom")
+      (reference "H3") (unit 1) (value "MountingHole") (footprint "MountingHole:MountingHole_2.7mm_M2.5_Pad")
     )
     (path "/cf14c459-3a9f-427f-b55f-05be5de35091"
-      (reference "H4") (unit 1) (value "MountingHole") (footprint "MountingHole:MountingHole_2.5mm_Pad_TopBottom")
+      (reference "H4") (unit 1) (value "MountingHole") (footprint "MountingHole:MountingHole_2.7mm_M2.5_Pad")
     )
     (path "/4b5434d5-3510-416b-95e8-f0230607849f"
