File: PicoXpressSmdK3/PicoXpressSmdK3.kicad_pcb (KiCad board)
At the start: 2 copper layers, 100 x 80 mm, 28 parts, among them J1 6P6C, J2 parallel port, J3 I2C, J4 5V Sel, J5 I2C, J6 I2C, J7 keypad, Q1 DMG2305UX-7, SW1 Reset, U1 AMS1117-5.0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

Commit message: 14:40 Arrakis.local
Connections:
- U6 pad 6: /SCL -> unconnected-(U6-Pad6)
- U6 pad 7: /SDA -> unconnected-(U6-Pad7)
Routing:
- net /SCL: track 99.6 -> 64.8 mm
- net /SDA: track 101.3 -> 69.6 mm
- net Net-(J1-Pad4): track 35.3 -> 57.1 mm
- net /GP1: track 36.3 -> 48.4 mm
- net Net-(J1-Pad3): track 36.2 -> 32.5 mm
- net /RTS: track 39.8 -> 36.8 mm
- net /RUN: track 113.2 -> 111.5 mm
- net /12V: track 15.2 -> 13.8 mm
- net /3V3: track 173.6 -> 172.2 mm
- net /5V: track 92.9 -> 93.9 mm
- net Net-(D2-Pad2): track 9.96 -> 9.09 mm
- net /VBUS: track 79.2 -> 78.6 mm
Other:
- board text added: "0"
- board text added: "7"
- board text added: "EXT"
- board text added: "GND"
- board text added: "USB"
