File: PicoXpressSmdK3/PicoXpressSmdK3.kicad_sch (KiCad schematic)
At the start: 28 parts, among them J1 6P6C, J2 parallel port, J3 I2C, J4 5V Sel, J5 I2C, J6 I2C, J7 keypad, Q1 DMG2305UX-7, SW1 Reset, U1 AMS1117-5.0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

Commit message: 14:40 Arrakis.local
Connections:
- net SCL: no longer U6.6 (GPIO4)
- net SDA: no longer U6.7 (GPIO5)
Changed lines of the file:
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@@
   (junction (at 57.2363 112.6785) (diameter 0) (color 0 0 0 0)
-  )
-  (junction (at 257.8281 72.4173) (diameter 0) (color 0 0 0 0)
   )
   (junction (at 75.1679 106.139) (diameter 0) (color 0 0 0 0)
@@
     (stroke (width 0) (type default) (color 0 0 0 0))
   )
+  (wire (pts (xy 257.81 72.39) (xy 266.7 72.39))
+    (stroke (width 0) (type default) (color 0 0 0 0))
+  )
   (wire (pts (xy 38.9521 38.2651) (xy 38.9521 47.4486))
     (stroke (width 0) (type default) (color 0 0 0 0))
@@
     (stroke (width 0) (type default) (color 0 0 0 0))
   )
-  (wire (pts (xy 266.1702 69.6182) (xy 257.8281 69.6182))
-    (stroke (width 0) (type default) (color 0 0 0 0))
-  )
   (wire (pts (xy 38.9521 47.5552) (xy 38.9521 47.5835))
     (stroke (width 0) (type default) (color 0 0 0 0))
@@
     (stroke (width 0) (type default) (color 0 0 0 0))
   )
-  (wire (pts (xy 257.8281 69.6182) (xy 257.8281 69.8773))
-    (stroke (width 0) (type default) (color 0 0 0 0))
-  )
   (wire (pts (xy 210.9555 43.4671) (xy 210.9555 47.0173))
     (stroke (width 0) (type default) (color 0 0 0 0))
@@
     (stroke (width 0) (type default) (color 0 0 0 0))
   )
+  (wire (pts (xy 257.81 69.85) (xy 266.7 69.85))
+    (stroke (width 0) (type default) (color 0 0 0 0))
+  )
   (wire (pts (xy 108.6296 28.2533) (xy 110.9975 28.2533))
     (stroke (width 0) (type default) (color 0 0 0 0))
@@
     (stroke (width 0) (type default) (color 0 0 0 0))
   )
-  (wire (pts (xy 257.8281 72.4964) (xy 257.8281 72.4173))
-    (stroke (width 0) (type default) (color 0 0 0 0))
-  )
   (wire (pts (xy 38.9521 47.4486) (xy 38.9521 47.5552))
     (stroke (width 0) (type default) (color 0 0 0 0))
@@
     (stroke (width 0) (type default) (color 0 0 0 0))
   )
-  (wire (pts (xy 266.1702 72.4964) (xy 257.8281 72.4964))
-    (stroke (width 0) (type default) (color 0 0 0 0))
-  )
   (wire (pts (xy 206.6838 38.3871) (xy 206.6838 52.0973))
     (stroke (width 0) (type default) (color 0 0 0 0))
@@
     (stroke (width 0) (type default) (color 0 0 0 0))
   )
-  (label "SDA" (at 266.1702 69.6182 0)
+  (label "SDA" (at 266.7 72.39 0)
     (effects (font (size 1.27 1.27)) (justify left bottom))
   )
@@
     (effects (font (size 1.27 1.27)) (justify left bottom))
   )
-  (label "SCL" (at 266.1702 72.4964 0)
+  (label "SCL" (at 266.7 69.85 0)
     (effects (font (size 1.27 1.27)) (justify left bottom))
   )
