File: PicoXpressSmdK2/PicoXpressSmdK2.kicad_sch (KiCad schematic)
At the start: 28 parts, among them J1 6P6C, J2 parallel port, J3 I2C, J4 5V Sel, J5 I2C, J6 I2C, J7 keypad, Q1 DMG2305UX-7, SW1 Reset, U1 AMS1117-5.0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

Commit message: 20:06 Arrakis.local
Other:
- note added: "SDA/SCL reversed"
Changed lines of the file:
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@@
     (stroke (width 0) (type default) (color 0 0 0 0))
+  )
+  (text "SDA/SCL reversed\n" (at 190.5 81.28 0)
+    (effects (font (size 5.08 5.08)) (justify left bottom))
   )
   (label "SDA" (at 266.1702 69.6182 0)
