File: CanPicoBase/CanPicoBase.kicad_pcb (KiCad board)
At the start: 2 copper layers, 100 x 80 mm, 13 parts, among them J1 3.50 CBUS, J2 5V select, J3 Grove 2mm, Q1 DMG2305UX-7, U1 AMS1117-5.0, U2 AMS1117-3.3, U3 Pico

Commit message: 12:28 Arrakis.local
Parts:
- added D1: 1N4148, Diode_THT:D_DO-35_SOD27_P7.62mm_Horizontal, F.Cu at (114.0, 32.8)
- J3: footprint Connector_PinHeader_2.00mm:PinHeader_1x04_P2.00mm_Vertical -> OPL_Connector:HW4-2.0
- moved C1 4.31 mm to (131.9, 41.0)
- moved J3 3.16 mm to (105.0, 61.0), turned to 90 degrees
- moved C2 3.03 mm to (130.6, 28.0)
- moved J2 2.27 mm to (141.3, 38.5)
- moved U1 2.24 mm to (122.0, 28.0)
- moved U2 2.00 mm to (122.0, 41.0)
- moved Q1 1.95 mm to (140.9, 28.0)
Connections:
- net +5V renamed /5V
- net /5Voption renamed /5Vopt
- C1 pad 2: GND -> /GND
- C2 pad 2: GND -> /GND
- J1 pad 1: +12V -> Net-(J1-Pad1)
- J1 pad 4: GND -> /GND
- J3 pad 1: GND -> /SCL
- J3 pad 2: /3V3a -> /SDA
- J3 pad 3: /SDA -> /3V3a
- J3 pad 4: /SCL -> /GND
- U1 pad 1: GND -> /GND
- U1 pad 3: +12V -> /12V
- U2 pad 1: GND -> /GND
- U3 pad 3: GND -> /GND
Routing:
- net GND: track 110.5 -> 0.00 mm
- net +12V: track 11.0 -> 0.00 mm
- net Net-(J1-Pad1): track 0.00 -> 10.7 mm
- net /VSYS: track 54.9 -> 47.5 mm
- net /12V: track 0.00 -> 6.02 mm
- net /GND: track 0.00 -> 3.90 mm, vias 0 -> 2
- net /3V3a: track 38.5 -> 42.0 mm
- net /VBUS: track 72.3 -> 69.0 mm
- net /SCL: track 69.3 -> 70.3 mm
- net /SDA: track 69.6 -> 70.6 mm
- net /5V: track 38.1 -> 37.3 mm
- added copper zone on B.Cu, net /GND
- removed copper zone on B.Cu, net GND

Commit message: 09:25 Arrakis.local
Parts:
- U3: footprint MCU_RaspberryPi_and_Boards:RPi_Pico_SMD_TH -> MCU_RaspberryPi_and_Boards:RP2040Pico

Commit message: 19:39 Arrakis.local
Parts:
- moved U3 1.11 mm to (174.9, 53.0)
Connections:
- net /3V3a renamed /3V3
- net /GND renamed GND
Routing:
- net unconnected-(U3-Pad18): track 0.00 -> 94.3 mm
- net GND: track 3.90 -> 20.8 mm
- net /5Vopt: track 23.4 -> 28.8 mm
- net /VBUS: track 69.0 -> 67.5 mm
- net /5V: track 37.3 -> 38.6 mm
- net /VSYS: track 47.5 -> 46.3 mm
- net /SDA: track 70.6 -> 69.5 mm
- net /SCL: track 70.3 -> 69.2 mm

Commit message: 20:43 Titan.local
Parts:
- moved Q1 4.61 mm to (145.5, 27.2)
Routing:
- net unconnected-(U3-Pad18): track 94.3 -> 0.00 mm
- net /SDA: track 69.5 -> 0.00 mm
- net /SCL: track 69.2 -> 0.00 mm
- net /VBUS: track 67.5 -> 0.00 mm
- net /VSYS: track 46.3 -> 0.00 mm
- net /3V3: track 42.0 -> 0.00 mm
- net /5V: track 38.6 -> 0.00 mm
- net /5Vopt: track 28.8 -> 0.00 mm
- net GND: track 20.8 -> 0.00 mm, vias 2 -> 0
- net Net-(D1-Pad2): track 10.7 -> 0.00 mm
- net /12V: track 6.02 -> 0.00 mm
Other:
- board text added: "CanPicoBase v1.0 with ground plane so some GND wires not required"
- board text removed: "CanPicoBase v1.0"
Changed lines of the file:
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@@
   )
   (footprint "Package_TO_SOT_SMD:SOT-23" (layer "F.Cu")
-    (at 140.95 28)
+    (at 145.488624 27.181486)
     (descr "SOT, 3 Pin (https://www.jedec.org/system/files/docs/to-236h.pdf variant AB), generated with kicad-footprint-generator ipc_gullwing_generator.py")
     (tags "SOT TO_SOT_SMD")
@@
     (effects (font (size 1 1) (thickness 0.15)))
   )
-  (gr_text "CanPicoBase v1.0\n" (at 124 77) (layer "F.SilkS")
+  (gr_text "CanPicoBase v1.0\nwith ground plane\nso some GND wires not required\n" (at 138.2172 87.14837) (layer "F.SilkS")
     (effects (font (size 2 2) (thickness 0.15)))
   )
@@
     (style (thickness 0.15) (arrow_length 1.27) (text_position_mode 0) (extension_height 0.58642) (extension_offset 0.5) keep_text_aligned)
   )
-  (segment (start 125.15 27.9997) (end 125.15 27.9994) (width 0.254) (layer "F.Cu") (net 1))
-  (segment (start 141.8875 28) (end 141.1819 28) (width 0.254) (layer "F.Cu") (net 1))
-  (segment (start 138.8878 34.8617) (end 141.27 37.2439) (width 0.254) (layer "F.Cu") (net 1))
-  (segment (start 139.46 28) (end 138.8878 28.5722) (width 0.254) (layer "F.Cu") (net 1))
-  (segment (start 130.6147 28) (end 129.4336 28) (width 0.254) (layer "F.Cu") (net 1))
-  (segment (start 118.85 28) (end 120.2311 28) (width 0.254) (layer "F.Cu") (net 1))
-  (segment (start 125.15 27.9997) (end 129.4333 27.9997) (width 0.254) (layer "F.Cu") (net 1))
-  (segment (start 141.1819 28) (end 139.46 28) (width 0.254) (layer "F.Cu") (net 1))
-  (segment (start 120.2317 27.9994) (end 120.2311 28) (width 0.254) (layer "F.Cu") (net 1))
-  (segment (start 125.15 28) (end 125.15 27.9997) (width 0.254) (layer "F.Cu") (net 1))
-  (segment (start 141.1819 26.6929) (end 140.8473 26.3583) (width 0.254) (layer "F.Cu") (net 1))
-  (segment (start 141.27 38.475) (end 141.27 37.2439) (width 0.254) (layer "F.Cu") (net 1))
-  (segment (start 140.8473 26.3583) (end 133.4375 26.3583) (width 0.254) (layer "F.Cu") (net 1))
-  (segment (start 141.1819 28) (end 141.1819 26.6929) (width 0.254) (layer "F.Cu") (net 1))
-  (segment (start 138.8878 28.5722) (end 138.8878 34.8617) (width 0.254) (layer "F.Cu") (net 1))
-  (segment (start 130.6147 28) (end 131.7958 28) (width 0.254) (layer "F.Cu") (net 1))
-  (segment (start 133.4375 26.3583) (end 131.7958 28) (width 0.254) (layer "F.Cu") (net 1))
-  (segment (start 129.4333 27.9997) (end 129.4336 28) (width 0.254) (layer "F.Cu") (net 1))
-  (segment (start 125.15 27.9994) (end 120.2317 27.9994) (width 0.254) (layer "F.Cu") (net 1))
-  (segment (start 114 32.81) (end 115.1811 32.81) (width 0.254) (layer "F.Cu") (net 4))
-  (segment (start 117.4689 30.5222) (end 115.1811 32.81) (width 0.254) (layer "F.Cu") (net 4))
-  (segment (start 118.85 30.3) (end 117.4689 30.3) (width 0.254) (layer "F.Cu") (net 4))
-  (segment (start 117.4689 30.3) (end 117.4689 30.5222) (width 0.254) (layer "F.Cu") (net 4))
-  (segment (start 141.743 44.8236) (end 119.2425 44.8236) (width 0.254) (layer "F.Cu") (net 5))
-  (segment (start 119.2425 44.8236) (end 118.85 44.4311) (width 0.254) (layer "F.Cu") (net 5))
-  (segment (start 118.85 43.3) (end 118.85 44.4311) (width 0.254) (layer "F.Cu") (net 5))
-  (segment (start 142.5048 44.0618) (end 141.743 44.8236) (width 0.254) (layer "F.Cu") (net 5))
-  (segment (start 141.27 41.015) (end 142.5048 42.2498) (width 0.254) (layer "F.Cu") (net 5))
-  (segment (start 142.5048 42.2498) (end 142.5048 44.0618) (width 0.254) (layer "F.Cu") (net 5))
-  (segment (start 140.0125 27.05) (end 139.6532 27.05) (width 0.254) (layer "F.Cu") (net 6))
-  (segment (start 140.8083 42.3239) (end 141.27 42.3239) (width 0.254) (layer "F.Cu") (net 6))
-  (segment (start 141.27 43.555) (end 141.27 42.3239) (width 0.254) (layer "F.Cu") (net 6))
-  (segment (start 139.6532 27.05) (end 138.3797 28.3235) (width 0.254) (layer "F.Cu") (net 6))
-  (segment (start 138.3797 39.8953) (end 140.8083 42.3239) (width 0.254) (layer "F.Cu") (net 6))
-  (segment (start 138.3797 28.3235) (end 138.3797 39.8953) (width 0.254) (layer "F.Cu") (net 6))
-  (segment (start 183.78 28.87) (end 182.5489 28.87) (width 0.254) (layer "B.Cu") (net 6))
-  (segment (start 182.5489 28.87) (end 181.3178 30.1011) (width 0.254) (layer "B.Cu") (net 6))
-  (segment (start 181.3178 30.1011) (end 155.955 30.1011) (width 0.254) (layer "B.Cu") (net 6))
-  (segment (start 141.27 43.555) (end 142.5011 43.555) (width 0.254) (layer "B.Cu") (net 6))
-  (segment (start 155.955 30.1011) (end 142.5011 43.555) (width 0.254) (layer "B.Cu") (net 6))
-  (segment (start 183.78 31.41) (end 182.1759 31.41) (width 1) (layer "F.Cu") (net 7))
-  (segment (start 178.0317 27.2658) (end 144.815 27.2658) (width 1) (layer "F.Cu") (net 7))
-  (segment (start 140.2075 29.145) (end 140.0125 28.95) (width 1) (layer "F.Cu") (net 7))
-  (segment (start 182.1759 31.41) (end 178.0317 27.2658) (width 1) (layer "F.Cu") (net 7))
-  (segment (start 144.815 27.2658) (end 142.9358 29.145) (width 1) (layer "F.Cu") (net 7))
-  (segment (start 142.9358 29.145) (end 140.2075 29.145) (width 1) (layer "F.Cu") (net 7))
-  (segment (start 102 43.419) (end 104.419 41) (width 0.254) (layer "F.Cu") (net 22))
-  (segment (start 105.05 72.05) (end 102 69) (width 0.254) (layer "F.Cu") (net 22))
-  (segment (start 166 72.05) (end 105.05 72.05) (width 0.254) (layer "F.Cu") (net 22))
-  (segment (start 102 69) (end 102 43.419) (width 0.254) (layer "F.Cu") (net 22))
-  (segment (start 125.15 40.2885) (end 125.15 38.7189) (width 0.254) (layer "F.Cu") (net 45))
-  (segment (start 105 60.0018) (end 112.4783 52.5235) (width 0.254) (layer "F.Cu") (net 45))
-  (segment (start 120.9426 40.2885) (end 120.2311 41) (width 0.254) (layer "F.Cu") (net 45))
-  (segment (start 118.85 41) (end 120.2311 41) (width 0.254) (layer "F.Cu") (net 45))
-  (segment (start 112.4783 52.5235) (end 112.4783 47.3717) (width 0.254) (layer "F.Cu") (net 45))
-  (segment (start 125.15 41) (end 125.15 40.2885) (width 0.254) (layer "F.Cu") (net 45))
-  (segment (start 125.15 40.2885) (end 120.9426 40.2885) (width 0.254) (layer "F.Cu") (net 45))
-  (segment (start 112.4783 47.3717) (end 117.7189 42.1311) (width 0.254) (layer "F.Cu") (net 45))
-  (segment (start 131.8924 41) (end 130.7113 41) (width 0.254) (layer "F.Cu") (net 45))
-  (segment (start 128.4302 38.7189) (end 125.15 38.7189) (width 0.254) (layer "F.Cu") (net 45))
-  (segment (start 130.7113 41) (end 128.4302 38.7189) (width 0.254) (layer "F.Cu") (net 45))
-  (segment (start 118.85 41) (end 118.85 42.1311) (width 0.254) (layer "F.Cu") (net 45))
-  (segment (start 117.7189 42.1311) (end 118.85 42.1311) (width 0.254) (layer "F.Cu") (net 45))
-  (segment (start 166 41.57) (end 160.3283 41.57) (width 0.254) (layer "F.Cu") (net 46))
-  (segment (start 139.9001 61.9982) (end 105 61.9982) (width 0.254) (layer "F.Cu") (net 46))
-  (segment (start 160.3283 41.57) (end 139.9001 61.9982) (width 0.254) (layer "F.Cu") (net 46))
-  (segment (start 162.9689 44.11) (end 143.0792 63.9997) (width 0.254) (layer "F.Cu") (net 47))
-  (segment (start 166 44.11) (end 162.9689 44.11) (width 0.254) (layer "F.Cu") (net 47))
-  (segment (start 143.0792 63.9997) (end 105 63.9997) (width 0.254) (layer "F.Cu") (net 47))
-  (segment (start 106 31) (end 107.5811 31) (width 0.254) (layer "F.Cu") (net 48))
-  (segment (start 107.5811 31) (end 107.5811 30.4278) (width 0.254) (layer "F.Cu") (net 48))
-  (segment (start 107.5811 30.4278) (end 112.8189 25.19) (width 0.254) (layer "F.Cu") (net 48))
-  (segment (start 114 25.19) (end 112.8189 25.19) (width 0.254) (layer "F.Cu") (net 48))
-  (segment (start 117.1691 25.484) (end 117.2529 25.484) (width 0.254) (layer "F.Cu") (net 49))
-  (segment (start 106 57.0003) (end 105 58.0003) (width 0.254) (layer "F.Cu") (net 49))
-  (segment (start 118.2489 37.5689) (end 118.85 37.5689) (width 0.254) (layer "F.Cu") (net 49))
-  (segment (start 118.85 25.7) (end 117.4689 25.7) (width 0.254) (layer "F.Cu") (net 49))
-  (segment (start 117.9659 37.2859) (end 118.2489 37.5689) (width 0.254) (layer "F.Cu") (net 49))
-  (segment (start 118.85 38.7) (end 118.85 37.5689) (width 0.254) (layer "F.Cu") (net 49))
-  (segment (start 106 41.5) (end 106 57.0003) (width 0.254) (layer "F.Cu") (net 49))
-  (segment (start 117.2529 25.484) (end 117.4689 25.7) (width 0.254) (layer "F.Cu") (net 49))
-  (via (at 117.1691 25.484) (size 0.8) (drill 0.4) (layers "F.Cu" "B.Cu") (net 49))
-  (via (at 117.9659 37.2859) (size 0.8) (drill 0.4) (layers "F.Cu" "B.Cu") (net 49))
   (zone (net 49) (net_name "GND") (layer "B.Cu") (hatch edge 0.508)
     (connect_pads (clearance 0.508))

Commit message: 21:22 Arrakis.local
Parts:
- added D2: CUS05540, Diode_SMD:D_SOD-123, F.Cu at (162.6, 77.3)
- added J4: Conn_01x20_Male, Connector_PinHeader_2.54mm:PinHeader_1x20_P2.54mm_Vertical, F.Cu at (181.0, 77.0)
- added J5: Conn_01x20_Male, Connector_PinHeader_2.54mm:PinHeader_1x20_P2.54mm_Vertical, F.Cu at (169.0, 28.9)
Connections:
- J2 pad 2: /5Vopt -> /VSYS
- U2 pad 3: /5Vopt -> /VSYS
- U3 pad 1: unconnected-(U3-Pad1) -> Net-(U3-Pad1)
- U3 pad 10: unconnected-(U3-Pad10) -> Net-(U3-Pad10)
- U3 pad 11: unconnected-(U3-Pad11) -> Net-(U3-Pad11)
- U3 pad 12: unconnected-(U3-Pad12) -> Net-(U3-Pad12)
- U3 pad 14: unconnected-(U3-Pad14) -> Net-(U3-Pad14)
- U3 pad 15: unconnected-(U3-Pad15) -> Net-(U3-Pad15)
- U3 pad 16: unconnected-(U3-Pad16) -> Net-(U3-Pad16)
- U3 pad 17: unconnected-(U3-Pad17) -> Net-(U3-Pad17)
- U3 pad 19: unconnected-(U3-Pad19) -> Net-(U3-Pad19)
- U3 pad 2: unconnected-(U3-Pad2) -> Net-(U3-Pad2)
- U3 pad 20: unconnected-(U3-Pad20) -> Net-(U3-Pad20)
- U3 pad 21: unconnected-(U3-Pad21) -> Net-(U3-Pad21)
- U3 pad 22: unconnected-(U3-Pad22) -> Net-(U3-Pad22)
- U3 pad 24: unconnected-(U3-Pad24) -> Net-(U3-Pad24)
- U3 pad 25: unconnected-(U3-Pad25) -> Net-(U3-Pad25)
- U3 pad 26: unconnected-(U3-Pad26) -> Net-(U3-Pad26)
- U3 pad 27: unconnected-(U3-Pad27) -> Net-(U3-Pad27)
- U3 pad 29: unconnected-(U3-Pad29) -> Net-(U3-Pad29)
- U3 pad 30: unconnected-(U3-Pad30) -> Net-(U3-Pad30)
- U3 pad 31: unconnected-(U3-Pad31) -> Net-(U3-Pad31)
- U3 pad 32: unconnected-(U3-Pad32) -> Net-(U3-Pad32)
- U3 pad 34: unconnected-(U3-Pad34) -> Net-(U3-Pad34)
- U3 pad 4: unconnected-(U3-Pad4) -> Net-(U3-Pad4)
- U3 pad 5: unconnected-(U3-Pad5) -> Net-(U3-Pad5)
- U3 pad 9: unconnected-(U3-Pad9) -> Net-(U3-Pad9)

Commit message: 21:44 Titan.local
Parts:
- moved D2 51.0 mm to (139.3, 31.9), turned to 180 degrees
- moved J4 0.18 mm to (180.9, 77.1)
Routing:
- net /VSYS: track 0.00 -> 81.3 mm
- net /SDA: track 0.00 -> 72.5 mm
- net /SCL: track 0.00 -> 72.2 mm
- net /VBUS: track 0.00 -> 59.9 mm, vias 0 -> 1
- net /5V: track 0.00 -> 49.4 mm
- net /3V3: track 0.00 -> 42.0 mm
- net Net-(D1-Pad2): track 0.00 -> 10.7 mm
- net /12V: track 0.00 -> 6.02 mm
- net GND: track 0.00 -> 3.91 mm, vias 0 -> 2
- net Net-(U3-Pad20): track 0.00 -> 3.00 mm
- net Net-(U3-Pad9): track 0.00 -> 3.00 mm
- net Net-(U3-Pad14): track 0.00 -> 3.00 mm
- net Net-(U3-Pad10): track 0.00 -> 3.00 mm
- net Net-(U3-Pad2): track 0.00 -> 3.00 mm
- net Net-(U3-Pad1): track 0.00 -> 3.00 mm
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
Commit message: 20:38 Arrakis.local
Parts:
- J4, J5: footprint Connector_PinHeader_2.54mm:PinHeader_1x20_P2.54mm_Vertical -> Connector_PinSocket_2.54mm:PinSocket_1x20_P2.54mm_Vertical
- moved J5 10.5 mm to (158.5, 28.9)
- moved J4 10.1 mm to (191.0, 77.1)
Connections:
- net /3V3 renamed /3v3
Routing:
- net /VBUS: track 59.9 -> 67.2 mm
- net /VSYS: track 81.3 -> 87.2 mm
- net Net-(J5-Pad5): track 3.00 -> 7.49 mm
- net Net-(J5-Pad4): track 3.00 -> 7.49 mm
- net Net-(J5-Pad19): track 3.00 -> 7.49 mm
- net Net-(J5-Pad17): track 3.00 -> 7.49 mm
- net Net-(J5-Pad16): track 3.00 -> 7.49 mm
- net Net-(J5-Pad12): track 3.00 -> 7.49 mm
- net Net-(J5-Pad2): track 3.00 -> 7.49 mm
- net Net-(J5-Pad10): track 3.00 -> 7.49 mm
- net Net-(J5-Pad9): track 3.00 -> 7.49 mm
- net Net-(J5-Pad14): track 3.00 -> 7.49 mm
- net Net-(J5-Pad11): track 3.00 -> 7.49 mm
- net Net-(J5-Pad1): track 3.00 -> 7.49 mm
- net Net-(J5-Pad20): track 3.00 -> 7.49 mm
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
Commit message: 21:37 Titan.local
Connections:
- J4 pad 13: unconnected-(J4-Pad13) -> Net-(J4-Pad13)
- J4 pad 15: unconnected-(J4-Pad15) -> Net-(J4-Pad15)
- J4 pad 16: unconnected-(J4-Pad16) -> Net-(J4-Pad16)
- J4 pad 17: unconnected-(J4-Pad17) -> Net-(J4-Pad17)
- U3 pad 33: unconnected-(U3-Pad33) -> Net-(J4-Pad13)
- U3 pad 35: unconnected-(U3-Pad35) -> Net-(J4-Pad15)
- U3 pad 36: unconnected-(U3-Pad36) -> Net-(J4-Pad16)
- U3 pad 37: unconnected-(U3-Pad37) -> Net-(J4-Pad17)
Routing:
- net Net-(J4-Pad17): track 0.00 -> 7.21 mm
- net Net-(J4-Pad16): track 0.00 -> 7.21 mm
- net Net-(J4-Pad15): track 0.00 -> 7.21 mm
- net Net-(J4-Pad13): track 0.00 -> 7.21 mm
- net /VBUS: track 67.2 -> 69.1 mm
- net /5V: track 47.5 -> 49.3 mm
- net /VSYS: track 87.2 -> 88.5 mm
