File: CanPicoBase/CanPicoBase.kicad_sch (KiCad schematic)
At the start: 13 parts, among them J1 3.50 CBUS, J2 5V select, J3 Grove 2mm, Q1 DMG2305UX-7, U1 AMS1117-5.0, U2 AMS1117-3.3, U3 Pico

Commit message: 12:28 Arrakis.local
Parts:
- added D1: 1N4148, Diode_THT:D_DO-35_SOD27_P7.62mm_Horizontal, symbol Diode:1N4148
- J3: footprint Connector_PinHeader_2.00mm:PinHeader_1x04_P2.00mm_Vertical -> OPL_Connector:HW4-2.0
Connections:
- net 3V3a: now also J3.3 (Pin_3); no longer J3.2 (Pin_2)
- net GND: now also J3.4 (Pin_4); no longer J3.1 (Pin_1)
- net SCL: now also J3.1 (Pin_1); no longer J3.4 (Pin_4)
- net SDA: now also J3.2 (Pin_2); no longer J3.3 (Pin_3)
- net +12V: no longer names the net of J1.1 (Pin_1)
- net +12V: now also D1.2 (A); no longer U1.3 (VI)
- net +5V renamed 5V
- net 5Voption renamed 5Vopt
- new net 12V: D1.1 (K), U1.3 (VI)

Commit message: 09:25 Arrakis.local
Parts:
- U3: footprint MCU_RaspberryPi_and_Boards:RPi_Pico_SMD_TH -> MCU_RaspberryPi_and_Boards:RP2040Pico
Changed lines of the file:
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@@
     (property "Reference" "U3" (id 0) (at 232.41 92.71 0))
     (property "Value" "Pico" (id 1) (at 232.41 95.25 0))
-    (property "Footprint" "MCU_RaspberryPi_and_Boards:RPi_Pico_SMD_TH" (id 2) (at 232.41 63.5 90)
+    (property "Footprint" "MCU_RaspberryPi_and_Boards:RP2040Pico" (id 2) (at 232.41 63.5 90)
       (effects (font (size 1.27 1.27)) hide)
     )
@@
     )
     (path "/a0336853-30aa-4b51-9ed7-c3dc664197ab"
-      (reference "U3") (unit 1) (value "Pico") (footprint "MCU_RaspberryPi_and_Boards:RPi_Pico_SMD_TH")
+      (reference "U3") (unit 1) (value "Pico") (footprint "MCU_RaspberryPi_and_Boards:RP2040Pico")
     )
   )

Commit message: 19:39 Arrakis.local
Connections:
- net 3V3a renamed 3V3

Commit message: 20:53 Arrakis.local
Parts:
- added D2: CUS05540, Diode_SMD:D_SOD-123, symbol Diode:MBR0580
Connections:
- net 5V: now also D2.2 (A)
- net VSYS: now also D2.1 (K)
Changed lines of the file:
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@@
     (rev "1.0")
   )
+  (junction (at 62.23 48.26) (diameter 0) (color 0 0 0 0)
+  )
   (junction (at 80.01 87.63) (diameter 0) (color 0 0 0 0)
   )
@@
   )
   (junction (at 80.01 87.5771) (diameter 0) (color 0 0 0 0)
+  )
+  (junction (at 83.82 48.26) (diameter 0) (color 0 0 0 0)
   )
   (junction (at 57.15 100.2425) (diameter 0) (color 0 0 0 0)
@@
   (no_connect (at 250.19 57.15))
   (no_connect (at 250.19 41.91))
-  (wire (pts (xy 80.01 48.26) (xy 93.98 48.26))
+  (wire (pts (xy 80.01 48.26) (xy 83.82 48.26))
     (stroke (width 0) (type default) (color 0 0 0 0))
   )
@@
     (stroke (width 0) (type default) (color 0 0 0 0))
   )
+  (wire (pts (xy 62.23 48.26) (xy 64.77 48.26))
+    (stroke (width 0) (type default) (color 0 0 0 0))
+  )
   (wire (pts (xy 205.74 87.63) (xy 214.63 87.63))
     (stroke (width 0) (type default) (color 0 0 0 0))
@@
     (stroke (width 0) (type default) (color 0 0 0 0))
   )
+  (wire (pts (xy 69.85 33.02) (xy 62.23 33.02))
+    (stroke (width 0) (type default) (color 0 0 0 0))
+  )
   (wire (pts (xy 53.1444 62.23) (xy 58.42 62.23))
     (stroke (width 0) (type default) (color 0 0 0 0))
@@
     (stroke (width 0) (type default) (color 0 0 0 0))
   )
+  (wire (pts (xy 62.23 33.02) (xy 62.23 48.26))
+    (stroke (width 0) (type default) (color 0 0 0 0))
+  )
   (wire (pts (xy 57.15 87.63) (xy 80.01 87.63))
     (stroke (width 0) (type default) (color 0 0 0 0))
   )
+  (wire (pts (xy 83.82 33.02) (xy 83.82 48.26))
+    (stroke (width 0) (type default) (color 0 0 0 0))
+  )
   (wire (pts (xy 22.86 24.13) (xy 26.67 24.13))
     (stroke (width 0) (type default) (color 0 0 0 0))
@@
     (stroke (width 0) (type default) (color 0 0 0 0))
   )
+  (wire (pts (xy 77.47 33.02) (xy 83.82 33.02))
+    (stroke (width 0) (type default) (color 0 0 0 0))
+  )
   (wire (pts (xy 250.19 72.39) (xy 259.08 72.39))
     (stroke (width 0) (type default) (color 0 0 0 0))
@@
     (stroke (width 0) (type default) (color 0 0 0 0))
   )
+  (wire (pts (xy 83.82 48.26) (xy 93.98 48.26))
+    (stroke (width 0) (type default) (color 0 0 0 0))
+  )
   (wire (pts (xy 65.4745 180.6696) (xy 69.5486 180.6696))
     (stroke (width 0) (type default) (color 0 0 0 0))
@@
     (stroke (width 0) (type default) (color 0 0 0 0))
   )
-  (wire (pts (xy 58.42 48.26) (xy 64.77 48.26))
+  (wire (pts (xy 58.42 48.26) (xy 62.23 48.26))
     (stroke (width 0) (type default) (color 0 0 0 0))
   )
@@
       (effects (font (size 1.27 1.27)) hide)
     )
+  )
+  (symbol (lib_id "Diode:MBR0580") (at 73.66 33.02 0) (mirror y) (unit 1)
+    (in_bom yes) (on_board yes) (fields_autoplaced)
+    (property "Reference" "D2" (id 0) (at 73.9775 26.67 0))
+    (property "Value" "CUS05540" (id 1) (at 73.9775 29.21 0))
+    (property "Footprint" "Diode_SMD:D_SOD-123" (id 2) (at 73.66 37.465 0)
+      (effects (font (size 1.27 1.27)) hide)
+    )
+    (property "Datasheet" "http://www.mccsemi.com/up_pdf/MBR0520~MBR0580(SOD123).pdf" (id 3) (at 73.66 33.02 0)
+      (effects (font (size 1.27 1.27)) hide)
+    )
+    (pin "1")
+    (pin "2")
   )
   (symbol (lib_id "Connector:Screw_Terminal_01x04") (at 24.13 115.57 0) (mirror y) (unit 1)
@@
       (reference "D1") (unit 1) (value "1N4148") (footprint "Diode_THT:D_DO-35_SOD27_P7.62mm_Horizontal")
     )
+    (path "/416a663b-1e36-4493-91ac-7c3b13979834"
+      (reference "D2") (unit 1) (value "CUS05540") (footprint "Diode_SMD:D_SOD-123")
+    )
     (path "/3b040f86-6673-47ab-8508-722b36bf57e0"

Commit message: 21:22 Arrakis.local
Parts:
- added J4, J5: Conn_01x20_Male, Connector_PinHeader_2.54mm:PinHeader_1x20_P2.54mm_Vertical, symbol Connector:Conn_01x20_Male
Connections:
- net 5Vopt is gone; now on net VSYS: J2.2 (Pin_2), U2.3 (VI)
- net GND: now also J4.18 (Pin_18), J4.3 (Pin_3), J4.8 (Pin_8), J5.13 (Pin_13), J5.18 (Pin_18), J5.3 (Pin_3), J5.8 (Pin_8)
- net SCL: now also J5.7 (Pin_7)
- net SDA: now also J5.6 (Pin_6)
- net VBUS: now also J4.20 (Pin_20)
- net VSYS: now also J4.19 (Pin_19)
- net at U3.1 (GPIO0): now also J5.1 (Pin_1)
- net at U3.10 (GPIO7): now also J5.10 (Pin_10)
- net at U3.11 (GPIO8): now also J5.11 (Pin_11)
- net at U3.12 (GPIO9): now also J5.12 (Pin_12)
- net at U3.14 (GPIO10): now also J5.14 (Pin_14)
- net at U3.15 (GPIO11): now also J5.15 (Pin_15)
- net at U3.16 (GPIO12): now also J5.16 (Pin_16)
- net at U3.17 (GPIO13): now also J5.17 (Pin_17)
- net at U3.19 (GPIO14): now also J5.19 (Pin_19)
- net at U3.2 (GPIO1): now also J5.2 (Pin_2)
- net at U3.20 (GPIO15): now also J5.20 (Pin_20)
- net at U3.21 (GPIO16): now also J4.1 (Pin_1)
- net at U3.22 (GPIO17): now also J4.2 (Pin_2)
- net at U3.24 (GPIO18): now also J4.4 (Pin_4)
- net at U3.25 (GPIO19): now also J4.5 (Pin_5)
- net at U3.26 (GPIO20): now also J4.6 (Pin_6)
- net at U3.27 (GPIO21): now also J4.7 (Pin_7)
- net at U3.29 (GPIO22): now also J4.9 (Pin_9)
- net at U3.30 (RUN): now also J4.10 (Pin_10)
- net at U3.31 (GPIO26_ADC0): now also J4.11 (Pin_11)
- net at U3.32 (GPIO27_ADC1): now also J4.12 (Pin_12)
- net at U3.34 (GPIO28_ADC2): now also J4.14 (Pin_14)
- net at U3.4 (GPIO2): now also J5.4 (Pin_4)
- net at U3.5 (GPIO3): now also J5.5 (Pin_5)
- net at U3.9 (GPIO6): now also J5.9 (Pin_9)
- no-connect marks 40 -> 19

Commit message: 21:44 Titan.local
Connections:
- net 3V3 renamed 3v3
Changed lines of the file:
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@@
-    (stroke (width 0) (type default) (color 0 0 0 0))
-  )
-  (wire (pts (xy 96.52 177.8) (xy 96.52 180.34))
     (stroke (width 0) (type default) (color 0 0 0 0))
   )
@@
   (wire (pts (xy 58.42 48.26) (xy 62.23 48.26))
     (stroke (width 0) (type default) (color 0 0 0 0))
-  )
-  (label "3V3" (at 96.52 180.34 0)
-    (effects (font (size 1.27 1.27)) (justify left bottom))
   )
   (label "VBUS" (at 34.29 73.66 0)
@@
     (effects (font (size 1.27 1.27)) (justify right bottom))
   )
-  (label "3V3" (at 38.2808 118.0266 0)
+  (label "3v3" (at 38.2808 118.0266 0)
     (effects (font (size 1.27 1.27)) (justify left bottom))
   )
@@
     (effects (font (size 1.27 1.27)) (justify left bottom))
   )
-  (label "3V3" (at 68.58 87.63 0)
+  (label "3v3" (at 68.58 87.63 0)
     (effects (font (size 1.27 1.27)) (justify left bottom))
   )
@@
     (pin "8")
     (pin "9")
-  )
-  (symbol (lib_id "power:PWR_FLAG") (at 96.52 177.8 0) (unit 1)
-    (in_bom yes) (on_board yes) (fields_autoplaced)
-    (property "Reference" "#FLG05" (id 0) (at 96.52 175.895 0)
-      (effects (font (size 1.27 1.27)) hide)
-    )
-    (property "Value" "PWR_FLAG" (id 1) (at 96.52 172.3904 0))
-    (property "Footprint" "" (id 2) (at 96.52 177.8 0)
-      (effects (font (size 1.27 1.27)) hide)
-    )
-    (property "Datasheet" "~" (id 3) (at 96.52 177.8 0)
-      (effects (font (size 1.27 1.27)) hide)
-    )
-    (pin "1")
   )
   (symbol (lib_id "Connector:Screw_Terminal_01x04") (at 24.13 115.57 0) (mirror y) (unit 1)
@@
       (reference "#FLG04") (unit 1) (value "PWR_FLAG") (footprint "")
     )
-    (path "/50dae00c-1440-4296-a3cf-40b54d3df5ea"
-      (reference "#FLG05") (unit 1) (value "PWR_FLAG") (footprint "")
-    )
     (path "/25d52506-8d92-4dfa-bd69-530ed70b2860"

Commit message: 20:38 Arrakis.local
Parts:
- J4, J5: footprint Connector_PinHeader_2.54mm:PinHeader_1x20_P2.54mm_Vertical -> Connector_PinSocket_2.54mm:PinSocket_1x20_P2.54mm_Vertical
Changed lines of the file:
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@@
     (property "Reference" "J4" (id 0) (at 191.135 34.29 0))
     (property "Value" "Conn_01x20_Male" (id 1) (at 191.135 36.83 0))
-    (property "Footprint" "Connector_PinHeader_2.54mm:PinHeader_1x20_P2.54mm_Vertical" (id 2) (at 190.5 62.23 0)
+    (property "Footprint" "Connector_PinSocket_2.54mm:PinSocket_1x20_P2.54mm_Vertical" (id 2) (at 190.5 62.23 0)
       (effects (font (size 1.27 1.27)) hide)
     )
@@
       (effects (font (size 1.27 1.27)) (justify right))
     )
-    (property "Footprint" "Connector_PinHeader_2.54mm:PinHeader_1x20_P2.54mm_Vertical" (id 2) (at 273.05 64.77 0)
+    (property "Footprint" "Connector_PinSocket_2.54mm:PinSocket_1x20_P2.54mm_Vertical" (id 2) (at 273.05 64.77 0)
       (effects (font (size 1.27 1.27)) hide)
     )
@@
     )
     (path "/1a850953-e696-40b6-a1fc-7a92a62063d4"
-      (reference "J4") (unit 1) (value "Conn_01x20_Male") (footprint "Connector_PinHeader_2.54mm:PinHeader_1x20_P2.54mm_Vertical")
+      (reference "J4") (unit 1) (value "Conn_01x20_Male") (footprint "Connector_PinSocket_2.54mm:PinSocket_1x20_P2.54mm_Vertical")
     )
     (path "/508c1793-b3ac-4a28-93d9-e73559a97305"
-      (reference "J5") (unit 1) (value "Conn_01x20_Male") (footprint "Connector_PinHeader_2.54mm:PinHeader_1x20_P2.54mm_Vertical")
+      (reference "J5") (unit 1) (value "Conn_01x20_Male") (footprint "Connector_PinSocket_2.54mm:PinSocket_1x20_P2.54mm_Vertical")
     )
     (path "/37118974-3a56-4fcc-9031-fa4d14c74939"

Commit message: 21:37 Titan.local
Connections:
- net at J4.13 (Pin_13): now also U3.33 (AGND)
- net at J4.15 (Pin_15): now also U3.35 (ADC_VREF)
- net at J4.16 (Pin_16): now also U3.36 (3V3)
- net at J4.17 (Pin_17): now also U3.37 (3V3_EN)
- no-connect marks 19 -> 11
Changed lines of the file:
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@@
   (junction (at 267.97 82.55) (diameter 0) (color 0 0 0 0)
   )
+  (junction (at 195.58 77.3836) (diameter 0) (color 0 0 0 0)
+  )
   (junction (at 34.065 120.5719) (diameter 0) (color 0 0 0 0)
   )
+  (junction (at 195.58 74.9115) (diameter 0) (color 0 0 0 0)
+  )
   (junction (at 58.42 62.1444) (diameter 0) (color 0 0 0 0)
   )
@@
   (junction (at 214.63 41.91) (diameter 0) (color 0 0 0 0)
   )
+  (junction (at 195.58 74.93) (diameter 0) (color 0 0 0 0)
+  )
   (junction (at 257.81 57.15) (diameter 0) (color 0 0 0 0)
   )
@@
   (junction (at 57.15 100.2425) (diameter 0) (color 0 0 0 0)
   )
+  (junction (at 195.58 77.47) (diameter 0) (color 0 0 0 0)
+  )
   (junction (at 203.2 44.45) (diameter 0) (color 0 0 0 0)
   )
+  (junction (at 195.58 69.85) (diameter 0) (color 0 0 0 0)
+  )
   (no_connect (at 250.19 69.85))
-  (no_connect (at 214.63 80.01))
-  (no_connect (at 195.58 69.85))
   (no_connect (at 214.63 82.55))
-  (no_connect (at 195.58 80.01))
   (no_connect (at 234.95 34.29))
   (no_connect (at 250.19 57.15))
@@
   (no_connect (at 22.86 29.21))
   (no_connect (at 229.87 34.29))
-  (no_connect (at 214.63 77.47))
-  (no_connect (at 195.58 74.93))
-  (no_connect (at 214.63 69.85))
   (no_connect (at 214.63 44.45))
-  (no_connect (at 214.63 74.93))
-  (no_connect (at 195.58 77.47))
   (no_connect (at 214.63 57.15))
   (wire (pts (xy 250.19 82.55) (xy 257.81 82.55))
@@
     (stroke (width 0) (type default) (color 0 0 0 0))
   )
+  (wire (pts (xy 188.379 69.85) (xy 195.58 69.85))
+    (stroke (width 0) (type default) (color 0 0 0 0))
+  )
   (wire (pts (xy 58.42 48.26) (xy 58.42 52.07))
     (stroke (width 0) (type default) (color 0 0 0 0))
@@
     (stroke (width 0) (type default) (color 0 0 0 0))
   )
+  (wire (pts (xy 195.58 77.3836) (xy 195.58 77.47))
+    (stroke (width 0) (type default) (color 0 0 0 0))
+  )
   (wire (pts (xy 250.19 41.91) (xy 267.97 41.91))
     (stroke (width 0) (type default) (color 0 0 0 0))
@@
     (stroke (width 0) (type default) (color 0 0 0 0))
   )
+  (wire (pts (xy 185.9652 74.9115) (xy 195.58 74.9115))
+    (stroke (width 0) (type default) (color 0 0 0 0))
+  )
   (wire (pts (xy 203.2 44.45) (xy 203.2 57.15))
     (stroke (width 0) (type default) (color 0 0 0 0))
@@
     (stroke (width 0) (type default) (color 0 0 0 0))
   )
+  (wire (pts (xy 195.58 74.93) (xy 214.63 74.93))
+    (stroke (width 0) (type default) (color 0 0 0 0))
+  )
   (wire (pts (xy 83.82 33.02) (xy 83.82 48.26))
     (stroke (width 0) (type default) (color 0 0 0 0))
@@
     (stroke (width 0) (type default) (color 0 0 0 0))
   )
+  (wire (pts (xy 176.4825 77.3828) (xy 195.58 77.3836))
+    (stroke (width 0) (type default) (color 0 0 0 0))
+  )
   (wire (pts (xy 29.21 120.65) (xy 34.065 120.65))
     (stroke (width 0) (type default) (color 0 0 0 0))
@@
     (stroke (width 0) (type default) (color 0 0 0 0))
   )
+  (wire (pts (xy 195.58 74.9115) (xy 195.58 74.93))
+    (stroke (width 0) (type default) (color 0 0 0 0))
+  )
   (wire (pts (xy 195.58 59.69) (xy 214.63 59.69))
     (stroke (width 0) (type default) (color 0 0 0 0))
@@
     (stroke (width 0) (type default) (color 0 0 0 0))
   )
+  (wire (pts (xy 195.58 77.47) (xy 214.63 77.47))
+    (stroke (width 0) (type default) (color 0 0 0 0))
+  )
   (wire (pts (xy 250.19 46.99) (xy 267.97 46.99))
     (stroke (width 0) (type default) (color 0 0 0 0))
@@
     (stroke (width 0) (type default) (color 0 0 0 0))
   )
+  (wire (pts (xy 195.58 80.01) (xy 214.63 80.01))
+    (stroke (width 0) (type default) (color 0 0 0 0))
+  )
   (wire (pts (xy 69.5486 180.6696) (xy 69.5486 180.8186))
+    (stroke (width 0) (type default) (color 0 0 0 0))
+  )
+  (wire (pts (xy 188.379 69.85) (xy 188.379 69.6241))
+    (stroke (width 0) (type default) (color 0 0 0 0))
+  )
+  (wire (pts (xy 195.58 69.85) (xy 214.63 69.85))
     (stroke (width 0) (type default) (color 0 0 0 0))
   )
@@
     (pin "1")
   )
+  (symbol (lib_id "power:PWR_FLAG") (at 185.9652 74.9115 0) (unit 1)
+    (in_bom yes) (on_board yes) (fields_autoplaced)
+    (property "Reference" "#FLG05" (id 0) (at 185.9652 73.0065 0)
+      (effects (font (size 1.27 1.27)) hide)
+    )
+    (property "Value" "PWR_FLAG" (id 1) (at 185.9652 69.85 0))
+    (property "Footprint" "" (id 2) (at 185.9652 74.9115 0)
+      (effects (font (size 1.27 1.27)) hide)
+    )
+    (property "Datasheet" "~" (id 3) (at 185.9652 74.9115 0)
+      (effects (font (size 1.27 1.27)) hide)
+    )
+    (pin "1")
+  )
   (symbol (lib_id "power:PWR_FLAG") (at 102.87 43.18 0) (unit 1)
     (in_bom yes) (on_board yes) (fields_autoplaced)
@@
     (pin "4")
   )
+  (symbol (lib_id "power:PWR_FLAG") (at 176.4825 77.3828 0) (unit 1)
+    (in_bom yes) (on_board yes) (fields_autoplaced)
+    (property "Reference" "#FLG02" (id 0) (at 176.4825 75.4778 0)
+      (effects (font (size 1.27 1.27)) hide)
+    )
+    (property "Value" "PWR_FLAG" (id 1) (at 176.4825 72.3892 0))
+    (property "Footprint" "" (id 2) (at 176.4825 77.3828 0)
+      (effects (font (size 1.27 1.27)) hide)
+    )
+    (property "Datasheet" "~" (id 3) (at 176.4825 77.3828 0)
+      (effects (font (size 1.27 1.27)) hide)
+    )
+    (pin "1")
+  )
   (symbol (lib_id "Connector:Screw_Terminal_01x04") (at 17.78 26.67 0) (mirror y) (unit 1)
     (in_bom yes) (on_board yes)
@@
     )
     (property "Datasheet" "" (id 3) (at 27.4135 31.9563 0)
+      (effects (font (size 1.27 1.27)) hide)
+    )
+    (pin "1")
+  )
+  (symbol (lib_id "power:PWR_FLAG") (at 188.379 69.6241 0) (unit 1)
+    (in_bom yes) (on_board yes) (fields_autoplaced)
+    (property "Reference" "#FLG07" (id 0) (at 188.379 67.7191 0)
+      (effects (font (size 1.27 1.27)) hide)
+    )
+    (property "Value" "PWR_FLAG" (id 1) (at 188.379 64.77 0))
+    (property "Footprint" "" (id 2) (at 188.379 69.6241 0)
+      (effects (font (size 1.27 1.27)) hide)
+    )
+    (property "Datasheet" "~" (id 3) (at 188.379 69.6241 0)
       (effects (font (size 1.27 1.27)) hide)
     )
@@
       (reference "#FLG01") (unit 1) (value "PWR_FLAG") (footprint "")
     )
+    (path "/576b0112-b207-4bf3-8c1d-a5c23dcda14e"
+      (reference "#FLG02") (unit 1) (value "PWR_FLAG") (footprint "")
+    )
     (path "/29410c01-763d-4c52-8a72-4db199a9dfe7"
       (reference "#FLG03") (unit 1) (value "PWR_FLAG") (footprint "")
@@
       (reference "#FLG04") (unit 1) (value "PWR_FLAG") (footprint "")
     )
+    (path "/2112fe59-d187-4c42-afed-65235cd0d021"
+      (reference "#FLG05") (unit 1) (value "PWR_FLAG") (footprint "")
+    )
     (path "/25d52506-8d92-4dfa-bd69-530ed70b2860"
       (reference "#FLG06") (unit 1) (value "PWR_FLAG") (footprint "")
     )
+    (path "/97181b30-8464-4d71-943e-45f9bae00245"
+      (reference "#FLG07") (unit 1) (value "PWR_FLAG") (footprint "")
+    )
     (path "/95f09844-5459-48d5-92f4-372322dbe922"
