File: DccDecoder/DccDecoder.kicad_sch (KiCad schematic)
At the start: 9 parts, among them Q1 2N7002K, U1 HT7533-1-SOT89

Commit message: 22:30 Titan.local
Parts:
- C1, C2: footprint Capacitor_SMD:C_0603_1608Metric_Pad1.08x0.95mm_HandSolder -> Capacitor_SMD:C_1206_3216Metric_Pad1.33x1.80mm_HandSolder
- J1: renamed from J?; footprint (none) -> TerminalBlock_Phoenix:TerminalBlock_Phoenix_PT-1,5-2-3.5-H_1x02_P3.50mm_Horizontal
- U2: renamed from U?; footprint RPi_Pico:RPi_Pico_SMD_TH -> MCU_RaspberryPi_and_Boards:RP2040Pico
Changed lines of the file:
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@@
       (effects (font (size 1.27 1.27)) (justify left))
     )
-    (property "Footprint" "Capacitor_SMD:C_0603_1608Metric_Pad1.08x0.95mm_HandSolder" (id 2) (at 50.4952 45.72 0)
+    (property "Footprint" "Capacitor_SMD:C_1206_3216Metric_Pad1.33x1.80mm_HandSolder" (id 2) (at 50.4952 45.72 0)
       (effects (font (size 1.27 1.27)) hide)
     )
@@
   (symbol (lib_id "OPL_Connector:SCREW-TERMINAL-GREEN_2P-3.5_") (at 15.24 31.75 180) (unit 1)
     (in_bom yes) (on_board yes) (fields_autoplaced)
-    (property "Reference" "J?" (id 0) (at 15.24 21.59 0)
+    (property "Reference" "J1" (id 0) (at 15.24 21.59 0)
       (effects (font (size 1.143 1.143)))
     )
@@
       (effects (font (size 1.143 1.143)))
     )
-    (property "Footprint" "" (id 2) (at 15.24 31.75 0)
+    (property "Footprint" "TerminalBlock_Phoenix:TerminalBlock_Phoenix_PT-1,5-2-3.5-H_1x02_P3.50mm_Horizontal" (id 2) (at 15.24 31.75 0)
       (effects (font (size 1.27 1.27)) hide)
     )
@@
       (effects (font (size 1.27 1.27)) (justify left))
     )
-    (property "Footprint" "Capacitor_SMD:C_0603_1608Metric_Pad1.08x0.95mm_HandSolder" (id 2) (at 27.6352 45.72 0)
+    (property "Footprint" "Capacitor_SMD:C_1206_3216Metric_Pad1.33x1.80mm_HandSolder" (id 2) (at 27.6352 45.72 0)
       (effects (font (size 1.27 1.27)) hide)
     )
@@
   (symbol (lib_id "MCU_RaspberryPi_and_Boards:Pico") (at 185.42 49.53 0) (unit 1)
     (in_bom yes) (on_board yes) (fields_autoplaced)
-    (property "Reference" "U?" (id 0) (at 185.42 17.78 0))
+    (property "Reference" "U2" (id 0) (at 185.42 17.78 0))
     (property "Value" "Pico" (id 1) (at 185.42 20.32 0))
-    (property "Footprint" "RPi_Pico:RPi_Pico_SMD_TH" (id 2) (at 185.42 49.53 90)
+    (property "Footprint" "MCU_RaspberryPi_and_Boards:RP2040Pico" (id 2) (at 185.42 49.53 90)
       (effects (font (size 1.27 1.27)) hide)
     )
@@
     )
     (path "/f28b9939-5d27-4e25-afa5-7656c7b2ae7c"
-      (reference "C1") (unit 1) (value "10u") (footprint "Capacitor_SMD:C_0603_1608Metric_Pad1.08x0.95mm_HandSolder")
+      (reference "C1") (unit 1) (value "10u") (footprint "Capacitor_SMD:C_1206_3216Metric_Pad1.33x1.80mm_HandSolder")
     )
     (path "/4bc60d4f-7124-49f4-8545-74f33f432b07"
-      (reference "C2") (unit 1) (value "10u") (footprint "Capacitor_SMD:C_0603_1608Metric_Pad1.08x0.95mm_HandSolder")
+      (reference "C2") (unit 1) (value "10u") (footprint "Capacitor_SMD:C_1206_3216Metric_Pad1.33x1.80mm_HandSolder")
     )
     (path "/52bebcff-fb7a-49c3-a22b-e159983b2adf"
@@
     )
     (path "/d2fb4cee-b325-4041-a1c1-2577771ec70c"
-      (reference "J?") (unit 1) (value "SCREW-TERMINAL-GREEN_2P-3.5_") (footprint "")
+      (reference "J1") (unit 1) (value "SCREW-TERMINAL-GREEN_2P-3.5_") (footprint "TerminalBlock_Phoenix:TerminalBlock_Phoenix_PT-1,5-2-3.5-H_1x02_P3.50mm_Horizontal")
     )
     (path "/b9283763-a7ad-4ac4-9704-a7d5cfce6853"
@@
     )
     (path "/fc46393a-0e65-4fa4-b436-9a4249989bdd"
-      (reference "U?") (unit 1) (value "Pico") (footprint "RPi_Pico:RPi_Pico_SMD_TH")
-    )
-  )
+      (reference "U2") (unit 1) (value "Pico") (footprint "MCU_RaspberryPi_and_Boards:RP2040Pico")
+    )
+  )

Commit message: 14:17 Titan.local
Parts:
- removed J1: SCREW-TERMINAL-GREEN_2P-3.5_, TerminalBlock_Phoenix:TerminalBlock_Phoenix_PT-1,5-2-3.5-H_1x02_P3.50mm_Horizontal, symbol OPL_Connector:SCREW-TERMINAL-GREEN_2P-3.5_
- removed Q1: 2N7002K, Package_TO_SOT_SMD:SOT-23, symbol Transistor_FET:2N7002K
- added J2: +V, TestPoint:TestPoint_Pad_D2.0mm, symbol Connector:Conn_01x01_Male
- added J3: M_OUT_B, TestPoint:TestPoint_Pad_D2.0mm, symbol Connector:Conn_01x01_Male
- added J4: M_OUT_A, TestPoint:TestPoint_Pad_D2.0mm, symbol Connector:Conn_01x01_Male
- added J5: GND, TestPoint:TestPoint_Pad_D2.0mm, symbol Connector:Conn_01x01_Male
- added J6: DCC, TerminalBlock_Phoenix:TerminalBlock_Phoenix_PT-1,5-2-3.5-H_1x02_P3.50mm_Horizontal, symbol Connector:Screw_Terminal_01x02
- added Q1: T2N7002BK, Package_TO_SOT_SMD:SOT-23, symbol RP2040-Decoder_Additional_Symbols:T2N7002BK
- added R3, R5: 6k8, Resistor_SMD:R_1206_3216Metric_Pad1.30x1.75mm_HandSolder, symbol Device:R
- added R4, R6: 1k, RP2040-Decoder_Additional_Footprints:R_0603_1608Metric, symbol Device:R
- added U3: BDR6133, RP2040-Decoder_Additional_Footprints:SOIC-8-1EP_3.9x4.9mm_P1.27mm_EP2.41x3.3mm_ThermalVias, symbol RP2040-Decoder_Additional_Symbols:BDR6133
- D1: value D_Bridge_+-AA -> KMB24F
- R1, R2: footprint Resistor_SMD:R_1206_3216Metric -> Resistor_SMD:R_1206_3216Metric_Pad1.30x1.75mm_HandSolder
Connections:
- net +V: now also D1.3, R1.1, J2.1 (Pin_1), J6.2 (Pin_2), U3.3 (VM)
- net GND: now also J5.1 (Pin_1), Q1.2 (S), R4.1, R6.1, U3.1 (GND), U3.9 (GND)
- net +3V3: now reaches C1.1, U1.3 (VOUT)
- net +3V3: now also U3.2 (VCC)
- net at D1.4: now also J6.1 (Pin_1)
- net at R1.2, R2.1: now also Q1.1 (G)
- new net ADC_EMF_A: R3.1, R4.2
- new net ADC_EMF_B: R5.1, R6.2
- new net GPIO22: U3.7 (INB)
- new net GPIO23: U3.6 (INA)
- new net MOTOR_OUT_A: R3.2, U3.4 (OUTA)
- new net MOTOR_OUT_B: R5.2, U3.5 (OUTB)
Other:
- note added: "Motor Driver"

Commit message: 16:26 Titan.local
Parts:
- removed D1: KMB24F, Package_TO_SOT_SMD:TO-269AA, symbol Device:D_Bridge_+-AA
- removed J6: DCC, TerminalBlock_Phoenix:TerminalBlock_Phoenix_PT-1,5-2-3.5-H_1x02_P3.50mm_Horizontal, symbol Connector:Screw_Terminal_01x02
- removed R3: 6k8, Resistor_SMD:R_1206_3216Metric_Pad1.30x1.75mm_HandSolder, symbol Device:R
- removed U1: HT7533-1-SOT89, Package_TO_SOT_SMD:SOT-23, symbol Regulator_Linear:HT75xx-1-SOT89
- removed U2: Pico, MCU_RaspberryPi_and_Boards:RP2040Pico, symbol MCU_RaspberryPi_and_Boards:Pico
- removed U3: BDR6133, RP2040-Decoder_Additional_Footprints:SOIC-8-1EP_3.9x4.9mm_P1.27mm_EP2.41x3.3mm_ThermalVias, symbol RP2040-Decoder_Additional_Symbols:BDR6133
- added C15: 100n, RP2040-Decoder_Additional_Footprints:C_0603_1608Metric, symbol Device:C
- added D1: KMB24F, Package_TO_SOT_SMD:TO-269AA, symbol RP2040-Decoder_Additional_Symbols:KMB24F
- added J1: T0, TestPoint:TestPoint_Pad_D2.0mm, symbol Connector:Conn_01x01_Male
- added J14: +V, TestPoint:TestPoint_Pad_D2.0mm, symbol Connector:Conn_01x01_Male
- added J15: M_OUT_B, TestPoint:TestPoint_Pad_D2.0mm, symbol Connector:Conn_01x01_Male
- added J16: M_OUT_A, TestPoint:TestPoint_Pad_D2.0mm, symbol Connector:Conn_01x01_Male
- added J17: GND, TestPoint:TestPoint_Pad_D2.0mm, symbol Connector:Conn_01x01_Male
- added J6: 3, TestPoint:TestPoint_Pad_D2.0mm, symbol Connector:Conn_01x01_Male
- added J7: +3V3, TestPoint:TestPoint_Pad_D2.0mm, symbol Connector:Conn_01x01_Male
- added Q2, Q3, Q4, Q5: T2N7002BK, Package_TO_SOT_SMD:SOT-23, symbol RP2040-Decoder_Additional_Symbols:T2N7002BK
- added R7, R8: 1k, RP2040-Decoder_Additional_Footprints:R_0603_1608Metric, symbol Device:R
- added U1: HT7533S, Package_TO_SOT_SMD:SOT-23, symbol RP2040-Decoder_Additional_Symbols:HT7533S
- added U2: BDR6133, RP2040-Decoder_Additional_Footprints:SOIC-8-1EP_3.9x4.9mm_P1.27mm_EP2.41x3.3mm_ThermalVias, symbol RP2040-Decoder_Additional_Symbols:BDR6133
- added U3: W25Q64JVSSIQ, RP2040-Decoder_Additional_Footprints:SOIC-8_5.23x5.23mm_P1.27mm, symbol RP2040-Decoder_Additional_Symbols:W25Q64JVSSIQ
- added U4: Pico, RPi_Pico:RPi_Pico_SMD_TH, symbol MCU_RaspberryPi_and_Boards:Pico
- C1, C2: footprint Capacitor_SMD:C_1206_3216Metric_Pad1.33x1.80mm_HandSolder -> RP2040-Decoder_Additional_Footprints:C_0603_1608Metric
- J2: value +V -> T1
- J3: value M_OUT_B -> 0
- J4: value M_OUT_A -> 1
- J5: value GND -> 2
- R1, R2, R5: footprint Resistor_SMD:R_1206_3216Metric_Pad1.30x1.75mm_HandSolder -> RP2040-Decoder_Additional_Footprints:R_0603_1608Metric
- R4: value 1k -> DNF
- R6: value 1k -> 6k8
Connections:
- net +3V3: now also R4.2, C15.1, J7.1 (Pin_1), U1.2 (VOUT), U2.2 (VCC), U3.8 (VCC), U4.36 (3V3)
- net +V: now also C2.1, D1.3 (+), J14.1 (Pin_1), U1.3 (VIN), U2.3 (VM); no longer J2.1 (Pin_1), R1.1
- net ADC_EMF_A: now also R5.1, R7.2; no longer R4.2
- net ADC_EMF_B: now also R6.1, R8.2; no longer R5.1, R6.2
- net GND: now also R2.1, C15.2, D1.4 (-), J17.1 (Pin_1), Q2.2 (S), Q3.2 (S), Q4.2 (S), Q5.2 (S), R7.1, R8.1, U1.1 (GND), U2.1 (GND), U2.9 (GND), U3.4 (GND), U4.42 (GND); no longer J5.1 (Pin_1), R2.2, R4.1, R6.1
- net GPIO22: now also U2.7 (INB)
- net GPIO23: now also U2.6 (INA)
- net MOTOR_OUT_A: now also R5.2, J15.1 (Pin_1), U2.4 (OUTA)
- net MOTOR_OUT_B: now also R6.2, J16.1 (Pin_1), U2.5 (OUTB); no longer R5.2
- net GPIO21: now reaches Q1.3 (D)
- net at J3.1 (Pin_1): now also Q2.3 (D)
- net at J4.1 (Pin_1): now also Q3.3 (D)
- new net: R4.1, U3.1 (~{CS})
- new net: Q1.1 (G), R1.1, R2.2
- new net: J5.1 (Pin_1), Q4.3 (D)
- new net: D1.1, J1.1 (Pin_1), R1.2
- new net: D1.2, J2.1 (Pin_1)
- new net: J6.1 (Pin_1), Q5.3 (D)
- new net GPIO24: Q2.1 (G)
- new net GPIO25: Q3.1 (G)
- new net GPIO26: Q4.1 (G)
- new net GPIO27: Q5.1 (G)
Other:
- note added: "Aux Outputs"
- note added: "Flash Memory"
- note added: "GPIO21 is pulled up internally in RP2040"
- note added: "Gates are pulled down using RP2040 pull-down resistors"
- note added: "Input Stage"
- note removed: "J"
- note removed: "K"

Commit message: 16:43 Titan.local
Connections:
- net GPIO22 is gone; now on net GPIO15: U2.7 (INB)
- net GPIO23 is gone; now on net GPIO14: U2.6 (INA)
- net GPIO14: now reaches U4.19 (GPIO14)
- net GPIO15: now reaches U4.20 (GPIO15)
Changed lines of the file:
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@@
+    (stroke (width 0) (type default))
+  )
+  (wire (pts (xy 95.25 138.43) (xy 109.22 138.43))
     (stroke (width 0) (type default))
   )
@@
   )
   (wire (pts (xy 83.82 38.1) (xy 83.82 48.26))
+    (stroke (width 0) (type default))
+  )
+  (wire (pts (xy 95.25 140.97) (xy 109.22 140.97))
     (stroke (width 0) (type default))
   )
@@
     (effects (font (size 1.27 1.27)) (justify right bottom))
   )
-  (label "GPIO23" (at 215.9 105.41 0) (fields_autoplaced)
+  (label "GPIO14" (at 95.25 138.43 180) (fields_autoplaced)
+    (effects (font (size 1.27 1.27)) (justify right bottom))
+  )
+  (label "GPIO14" (at 215.9 105.41 0) (fields_autoplaced)
     (effects (font (size 1.27 1.27)) (justify left bottom))
   )
@@
     (effects (font (size 1.27 1.27)) (justify left bottom))
   )
+  (label "GPIO15" (at 95.25 140.97 180) (fields_autoplaced)
+    (effects (font (size 1.27 1.27)) (justify right bottom))
+  )
   (label "MOTOR_OUT_A" (at 280.67 142.24 180) (fields_autoplaced)
     (effects (font (size 1.27 1.27)) (justify right bottom))
   )
-  (label "GPIO22" (at 251.46 105.41 180) (fields_autoplaced)
-    (effects (font (size 1.27 1.27)) (justify right bottom))
-  )
+  (label "GPIO15" (at 251.46 105.41 180) (fields_autoplaced)
+    (effects (font (size 1.27 1.27)) (justify right bottom))
+  )

Commit message: 17:14 Arrakis.local
Parts:
- removed J1: T0, TestPoint:TestPoint_Pad_D2.0mm, symbol Connector:Conn_01x01_Male
- removed J2: T1, TestPoint:TestPoint_Pad_D2.0mm, symbol Connector:Conn_01x01_Male
- removed J7: +3V3, TestPoint:TestPoint_Pad_D2.0mm, symbol Connector:Conn_01x01_Male
- added J8: DCC, TerminalBlock_Phoenix:TerminalBlock_Phoenix_PT-1,5-2-3.5-H_1x02_P3.50mm_Horizontal, symbol Connector:Screw_Terminal_01x02
- C1, C15, C2: footprint RP2040-Decoder_Additional_Footprints:C_0603_1608Metric -> Capacitor_SMD:C_1206_3216Metric_Pad1.33x1.80mm_HandSolder
- R1, R2, R4, R5, R6, R7, R8: footprint RP2040-Decoder_Additional_Footprints:R_0603_1608Metric -> Resistor_SMD:R_1206_3216Metric_Pad1.30x1.75mm_HandSolder
- U2: footprint RP2040-Decoder_Additional_Footprints:SOIC-8-1EP_3.9x4.9mm_P1.27mm_EP2.41x3.3mm_ThermalVias -> Package_SO:SOIC-8-1EP_3.9x4.9mm_P1.27mm_EP2.41x3.3mm_ThermalVias
- U3: footprint RP2040-Decoder_Additional_Footprints:SOIC-8_5.23x5.23mm_P1.27mm -> Package_SO:SOIC-8_5.23x5.23mm_P1.27mm
- U4: footprint RPi_Pico:RPi_Pico_SMD_TH -> MCU_RaspberryPi_and_Boards:RP2040Pico
Connections:
- net at D1.1, R1.2: now also J8.2 (Pin_2)
- net at D1.2: now also J8.1 (Pin_1)
Changed lines of the file:
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@@
   (junction (at 99.06 48.26) (diameter 0) (color 0 0 0 0)
   )
+  (junction (at 233.68 132.08) (diameter 0) (color 0 0 0 0)
+  )
   (junction (at 83.82 20.32) (diameter 0) (color 0 0 0 0)
   )
-  (junction (at 233.68 132.08) (diameter 0) (color 0 0 0 0)
-  )
   (junction (at 50.8 30.48) (diameter 0) (color 0 0 0 0)
   )
@@
     (stroke (width 0) (type default))
   )
+  (wire (pts (xy 34.29 48.26) (xy 34.29 22.86))
+    (stroke (width 0) (type default))
+  )
   (wire (pts (xy 93.98 30.48) (xy 93.98 48.26))
     (stroke (width 0) (type default))
@@
     (stroke (width 0) (type default))
   )
+  (wire (pts (xy 33.02 20.32) (xy 83.82 20.32))
+    (stroke (width 0) (type default))
+  )
   (wire (pts (xy 220.98 111.76) (xy 223.52 111.76))
     (stroke (width 0) (type default))
@@
     (stroke (width 0) (type default))
   )
-  (wire (pts (xy 33.02 20.32) (xy 83.82 20.32))
+  (wire (pts (xy 34.29 22.86) (xy 33.02 22.86))
     (stroke (width 0) (type default))
   )
@@
     (stroke (width 0) (type default))
   )
-  (wire (pts (xy 33.02 22.86) (xy 34.29 22.86))
-    (stroke (width 0) (type default))
-  )
   (wire (pts (xy 236.22 93.98) (xy 236.22 95.25))
     (stroke (width 0) (type default))
@@
     (stroke (width 0) (type default))
   )
-  (wire (pts (xy 49.53 30.48) (xy 50.8 30.48))
-    (stroke (width 0) (type default))
-  )
   (wire (pts (xy 280.67 144.78) (xy 265.43 144.78))
     (stroke (width 0) (type default))
@@
   )
   (wire (pts (xy 246.38 130.81) (xy 246.38 132.08))
-    (stroke (width 0) (type default))
-  )
-  (wire (pts (xy 34.29 22.86) (xy 34.29 48.26))
     (stroke (width 0) (type default))
   )
@@
       (effects (font (size 1.27 1.27)) (justify left))
     )
-    (property "Footprint" "RP2040-Decoder_Additional_Footprints:C_0603_1608Metric" (at 25.781 116.6114 0)
+    (property "Footprint" "Capacitor_SMD:C_1206_3216Metric_Pad1.33x1.80mm_HandSolder" (at 25.781 116.6114 0)
       (effects (font (size 1.27 1.27)) (justify left) hide)
     )
@@
       (effects (font (size 1.27 1.27)))
     )
-    (property "Footprint" "RP2040-Decoder_Additional_Footprints:R_0603_1608Metric" (at 44.45 101.092 90)
+    (property "Footprint" "Resistor_SMD:R_1206_3216Metric_Pad1.30x1.75mm_HandSolder" (at 44.45 101.092 90)
       (effects (font (size 1.27 1.27)) hide)
     )
@@
       (effects (font (size 1.27 1.27)) (justify left))
     )
-    (property "Footprint" "RP2040-Decoder_Additional_Footprints:C_0603_1608Metric" (at 71.4248 40.64 0)
+    (property "Footprint" "Capacitor_SMD:C_1206_3216Metric_Pad1.33x1.80mm_HandSolder" (at 71.4248 40.64 0)
       (effects (font (size 1.27 1.27)) hide)
     )
@@
       (effects (font (size 1.27 1.27)) (justify left))
     )
-    (property "Footprint" "RP2040-Decoder_Additional_Footprints:C_0603_1608Metric" (at 49.8348 40.64 0)
+    (property "Footprint" "Capacitor_SMD:C_1206_3216Metric_Pad1.33x1.80mm_HandSolder" (at 49.8348 40.64 0)
       (effects (font (size 1.27 1.27)) hide)
     )
@@
       (effects (font (size 1.27 1.27)))
     )
-    (property "Footprint" "RP2040-Decoder_Additional_Footprints:R_0603_1608Metric" (at 248.158 116.84 90)
+    (property "Footprint" "Resistor_SMD:R_1206_3216Metric_Pad1.30x1.75mm_HandSolder" (at 248.158 116.84 90)
       (effects (font (size 1.27 1.27)) hide)
     )
@@
       (effects (font (size 1.27 1.27)))
     )
-    (property "Footprint" "RP2040-Decoder_Additional_Footprints:R_0603_1608Metric" (at 248.158 127 90)
+    (property "Footprint" "Resistor_SMD:R_1206_3216Metric_Pad1.30x1.75mm_HandSolder" (at 248.158 127 90)
       (effects (font (size 1.27 1.27)) hide)
     )
@@
       (effects (font (size 1.27 1.27)))
     )
-    (property "Footprint" "RP2040-Decoder_Additional_Footprints:R_0603_1608Metric" (at 222.758 127 90)
+    (property "Footprint" "Resistor_SMD:R_1206_3216Metric_Pad1.30x1.75mm_HandSolder" (at 222.758 127 90)
       (effects (font (size 1.27 1.27)) hide)
     )
@@
       (effects (font (size 1.27 1.27)))
     )
-    (property "Footprint" "RP2040-Decoder_Additional_Footprints:R_0603_1608Metric" (at 222.758 116.84 90)
+    (property "Footprint" "Resistor_SMD:R_1206_3216Metric_Pad1.30x1.75mm_HandSolder" (at 222.758 116.84 90)
       (effects (font (size 1.27 1.27)) hide)
     )
@@
       (effects (font (size 1.27 1.27)))
     )
-    (property "Footprint" "RP2040-Decoder_Additional_Footprints:R_0603_1608Metric" (at 100.838 39.37 90)
+    (property "Footprint" "Resistor_SMD:R_1206_3216Metric_Pad1.30x1.75mm_HandSolder" (at 100.838 39.37 90)
       (effects (font (size 1.27 1.27)) hide)
     )
@@
       (effects (font (size 1.27 1.27)))
     )
-    (property "Footprint" "RPi_Pico:RPi_Pico_SMD_TH" (at 127 116.84 90)
+    (property "Footprint" "MCU_RaspberryPi_and_Boards:RP2040Pico" (at 127 116.84 90)
       (effects (font (size 1.27 1.27)) hide)
     )
@@
       (effects (font (size 1.27 1.27)))
     )
-    (property "Footprint" "RP2040-Decoder_Additional_Footprints:SOIC-8_5.23x5.23mm_P1.27mm" (at 45.72 128.27 0)
+    (property "Footprint" "Package_SO:SOIC-8_5.23x5.23mm_P1.27mm" (at 45.72 128.27 0)
       (effects (font (size 1.27 1.27)) hide)
     )
@@
     )
   )
+  (symbol (lib_id "Connector:Screw_Terminal_01x02") (at 27.94 22.86 180) (unit 1)
+    (in_bom yes) (on_board yes) (dnp no)
+    (property "Reference" "J8" (at 24.13 22.86 0)
+      (effects (font (size 1.27 1.27)))
+    )
+    (property "Value" "DCC" (at 24.13 20.32 0)
+      (effects (font (size 1.27 1.27)))
+    )
+    (property "Footprint" "TerminalBlock_Phoenix:TerminalBlock_Phoenix_PT-1,5-2-3.5-H_1x02_P3.50mm_Horizontal" (at 27.94 22.86 0)
+      (effects (font (size 1.27 1.27)) hide)
+    )
+    (property "Datasheet" "~" (at 27.94 22.86 0)
+      (effects (font (size 1.27 1.27)) hide)
+    )
+    (pin "1")
+    (pin "2")
+    (instances
+      (project "DccDecoder"
+        (path "/68a87a67-79ef-42dd-968e-a1e235d63e5c"
+          (reference "J8") (unit 1)
+        )
+      )
+    )
+  )
   (symbol (lib_id "RP2040-Decoder_Additional_Symbols:T2N7002BK") (at 109.22 33.02 0) (unit 1)
     (in_bom yes) (on_board yes) (dnp no)
@@
       (effects (font (size 1.27 1.27)))
     )
-    (property "Footprint" "RP2040-Decoder_Additional_Footprints:R_0603_1608Metric" (at 100.838 26.67 90)
+    (property "Footprint" "Resistor_SMD:R_1206_3216Metric_Pad1.30x1.75mm_HandSolder" (at 100.838 26.67 90)
       (effects (font (size 1.27 1.27)) hide)
     )
@@
         (path "/68a87a67-79ef-42dd-968e-a1e235d63e5c"
           (reference "R1") (unit 1)
-        )
-      )
-    )
-  )
-  (symbol (lib_name "Conn_01x01_Male_2") (lib_id "Connector:Conn_01x01_Male") (at 27.94 22.86 0) (unit 1)
-    (in_bom yes) (on_board yes) (dnp no)
-    (property "Reference" "J2" (at 26.67 22.86 0)
-      (effects (font (size 1.27 1.27)))
-    )
-    (property "Value" "T1" (at 22.86 22.86 0)
-      (effects (font (size 1.27 1.27)))
-    )
-    (property "Footprint" "TestPoint:TestPoint_Pad_D2.0mm" (at 27.94 22.86 0)
-      (effects (font (size 1.27 1.27)) hide)
-    )
-    (property "Datasheet" "~" (at 27.94 22.86 0)
-      (effects (font (size 1.27 1.27)) hide)
-    )
-    (pin "1")
-    (instances
-      (project "RP2040-Decoder"
-        (path "/11d18738-0f49-4d63-b61c-22a93efd5959"
-          (reference "J2") (unit 1)
-        )
-      )
-      (project "DccDecoder"
-        (path "/68a87a67-79ef-42dd-968e-a1e235d63e5c"
-          (reference "J2") (unit 1)
         )
       )
@@
     )
   )
-  (symbol (lib_name "Conn_01x01_Male_1") (lib_id "Connector:Conn_01x01_Male") (at 27.94 20.32 0) (unit 1)
-    (in_bom yes) (on_board yes) (dnp no)
-    (property "Reference" "J1" (at 26.67 20.32 0)
-      (effects (font (size 1.27 1.27)))
-    )
-    (property "Value" "T0" (at 22.86 20.32 0)
-      (effects (font (size 1.27 1.27)))
-    )
-    (property "Footprint" "TestPoint:TestPoint_Pad_D2.0mm" (at 27.94 20.32 0)
-      (effects (font (size 1.27 1.27)) hide)
-    )
-    (property "Datasheet" "~" (at 27.94 20.32 0)
-      (effects (font (size 1.27 1.27)) hide)
-    )
-    (pin "1")
-    (instances
-      (project "RP2040-Decoder"
-        (path "/11d18738-0f49-4d63-b61c-22a93efd5959"
-          (reference "J1") (unit 1)
-        )
-      )
-      (project "DccDecoder"
-        (path "/68a87a67-79ef-42dd-968e-a1e235d63e5c"
-          (reference "J1") (unit 1)
-        )
-      )
-    )
-  )
   (symbol (lib_id "power:GND") (at 127 152.4 0) (unit 1)
     (in_bom yes) (on_board yes) (dnp no)
@@
         (path "/68a87a67-79ef-42dd-968e-a1e235d63e5c"
           (reference "J6") (unit 1)
-        )
-      )
-    )
-  )
-  (symbol (lib_id "Connector:Conn_01x01_Male") (at 44.45 30.48 0) (unit 1)
-    (in_bom yes) (on_board yes) (dnp no)
-    (property "Reference" "J7" (at 43.18 30.48 0)
-      (effects (font (size 1.27 1.27)))
-    )
-    (property "Value" "+3V3" (at 38.1 30.48 0)
-      (effects (font (size 1.27 1.27)))
-    )
-    (property "Footprint" "TestPoint:TestPoint_Pad_D2.0mm" (at 44.45 30.48 0)
-      (effects (font (size 1.27 1.27)) hide)
-    )
-    (property "Datasheet" "~" (at 44.45 30.48 0)
-      (effects (font (size 1.27 1.27)) hide)
-    )
-    (pin "1")
-    (instances
-      (project "RP2040-Decoder"
-        (path "/11d18738-0f49-4d63-b61c-22a93efd5959"
-          (reference "J7") (unit 1)
-        )
-      )
-      (project "DccDecoder"
-        (path "/68a87a67-79ef-42dd-968e-a1e235d63e5c"
-          (reference "J7") (unit 1)
         )
       )
@@
       (effects (font (size 1.27 1.27)) (justify left))
     )
-    (property "Footprint" "RP2040-Decoder_Additional_Footprints:SOIC-8-1EP_3.9x4.9mm_P1.27mm_EP2.41x3.3mm_ThermalVias" (at 233.68 129.54 0)
-      (effects (font (size 1.27 1.27)) hide)
-    )
+    (property "Footprint" "Package_SO:SOIC-8-1EP_3.9x4.9mm_P1.27mm_EP2.41x3.3mm_ThermalVias" (at 233.68 129.54 0)
+      (effects (font (size 1.27 1.27)) hide)
+    )
