File: DccDecoder/DccDecoder.kicad_sch (KiCad schematic)
At the start: 29 parts, among them J14 +V, J15 M_OUT_B, J16 M_OUT_A, J17 GND, J3 0, J4 1, J5 2, J6 3, J8 DCC, Q1 T2N7002BK, Q2 T2N7002BK, Q3 T2N7002BK, Q4 T2N7002BK, Q5 T2N7002BK, U1 HT7533S, U2 BDR6133, U3 W25Q64JVSSIQ, U4 Pico

Commit message: 17:48 Arrakis.local
Parts:
- added SW1: SW_Push, Button_Switch_SMD:SW_Tactile_SPST_NO_Straight_CK_PTS636Sx25SMTRLFS, symbol Switch:SW_Push
Connections:
- net ADC_EMF_A: now also U4.31 (GPIO26_ADC0)
- net ADC_EMF_B: now also U4.32 (GPIO27_ADC1)
- net GND: now also SW1.2
- net GPIO21: now also U4.27 (GPIO21)
- net at U4.30 (RUN): now also SW1.1
- no-connect marks 0 -> 41
Changed lines of the file:
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@@
   (junction (at 72.39 30.48) (diameter 0) (color 0 0 0 0)
   )
+  (no_connect (at 109.22 113.03))
+  (no_connect (at 144.78 130.81))
+  (no_connect (at 73.66 123.19))
+  (no_connect (at 144.78 135.89))
+  (no_connect (at 109.22 133.35))
+  (no_connect (at 109.22 123.19))
+  (no_connect (at 109.22 95.25))
+  (no_connect (at 109.22 92.71))
+  (no_connect (at 144.78 107.95))
+  (no_connect (at 109.22 97.79))
+  (no_connect (at 144.78 100.33))
+  (no_connect (at 144.78 95.25))
+  (no_connect (at 73.66 114.3))
+  (no_connect (at 109.22 128.27))
+  (no_connect (at 109.22 130.81))
+  (no_connect (at 73.66 107.95))
+  (no_connect (at 109.22 102.87))
+  (no_connect (at 144.78 123.19))
+  (no_connect (at 144.78 133.35))
+  (no_connect (at 109.22 118.11))
+  (no_connect (at 109.22 115.57))
+  (no_connect (at 144.78 97.79))
+  (no_connect (at 124.46 146.05))
+  (no_connect (at 144.78 140.97))
+  (no_connect (at 109.22 105.41))
+  (no_connect (at 109.22 110.49))
+  (no_connect (at 109.22 135.89))
+  (no_connect (at 144.78 110.49))
+  (no_connect (at 144.78 92.71))
+  (no_connect (at 109.22 125.73))
+  (no_connect (at 73.66 116.84))
+  (no_connect (at 73.66 111.76))
+  (no_connect (at 144.78 128.27))
+  (no_connect (at 144.78 120.65))
+  (no_connect (at 129.54 146.05))
+  (no_connect (at 109.22 107.95))
+  (no_connect (at 144.78 138.43))
+  (no_connect (at 73.66 119.38))
+  (no_connect (at 109.22 120.65))
+  (no_connect (at 109.22 100.33))
+  (no_connect (at 144.78 105.41))
   (wire (pts (xy 246.38 113.03) (xy 246.38 111.76))
     (stroke (width 0) (type default))
@@
     (stroke (width 0) (type default))
   )
-  (wire (pts (xy 92.71 190.5) (xy 92.71 191.77))
-    (stroke (width 0) (type default))
-  )
   (wire (pts (xy 34.29 48.26) (xy 83.82 48.26))
     (stroke (width 0) (type default))
@@
     (stroke (width 0) (type default))
   )
+  (wire (pts (xy 144.78 125.73) (xy 154.94 125.73))
+    (stroke (width 0) (type default))
+  )
   (wire (pts (xy 214.63 29.21) (xy 214.63 33.02))
     (stroke (width 0) (type default))
@@
     (stroke (width 0) (type default))
   )
+  (wire (pts (xy 144.78 113.03) (xy 153.67 113.03))
+    (stroke (width 0) (type default))
+  )
   (wire (pts (xy 31.75 110.49) (xy 22.86 110.49))
     (stroke (width 0) (type default))
@@
     (stroke (width 0) (type default))
   )
+  (wire (pts (xy 144.78 115.57) (xy 162.56 115.57))
+    (stroke (width 0) (type default))
+  )
   (wire (pts (xy 99.06 20.32) (xy 99.06 22.86))
     (stroke (width 0) (type default))
@@
   )
   (wire (pts (xy 83.82 38.1) (xy 83.82 48.26))
+    (stroke (width 0) (type default))
+  )
+  (wire (pts (xy 144.78 118.11) (xy 175.26 118.11))
     (stroke (width 0) (type default))
   )
@@
     (effects (font (size 1.27 1.27)) (justify left bottom))
   )
+  (label "GPIO21" (at 154.94 125.73 0) (fields_autoplaced)
+    (effects (font (size 1.27 1.27)) (justify left bottom))
+  )
   (label "GPIO24" (at 157.48 39.37 0) (fields_autoplaced)
     (effects (font (size 1.27 1.27)) (justify left bottom))
@@
     (effects (font (size 1.27 1.27)) (justify right bottom))
   )
+  (label "ADC_EMF_B" (at 153.67 113.03 0) (fields_autoplaced)
+    (effects (font (size 1.27 1.27)) (justify left bottom))
+  )
   (label "GPIO15" (at 251.46 105.41 180) (fields_autoplaced)
     (effects (font (size 1.27 1.27)) (justify right bottom))
@@
   )
   (label "ADC_EMF_B" (at 257.81 121.92 0) (fields_autoplaced)
+    (effects (font (size 1.27 1.27)) (justify left bottom))
+  )
+  (label "ADC_EMF_A" (at 162.56 115.57 0) (fields_autoplaced)
     (effects (font (size 1.27 1.27)) (justify left bottom))
   )
@@
     )
   )
+  (symbol (lib_id "Switch:SW_Push") (at 180.34 118.11 0) (unit 1)
+    (in_bom yes) (on_board yes) (dnp no)
+    (property "Reference" "SW1" (at 180.34 111.76 0)
+      (effects (font (size 1.27 1.27)))
+    )
+    (property "Value" "SW_Push" (at 180.34 114.3 0)
+      (effects (font (size 1.27 1.27)))
+    )
+    (property "Footprint" "Button_Switch_SMD:SW_Tactile_SPST_NO_Straight_CK_PTS636Sx25SMTRLFS" (at 180.34 113.03 0)
+      (effects (font (size 1.27 1.27)) hide)
+    )
+    (property "Datasheet" "~" (at 180.34 113.03 0)
+      (effects (font (size 1.27 1.27)) hide)
+    )
+    (pin "1")
+    (pin "2")
+    (instances
+      (project "DccDecoder"
+        (path "/68a87a67-79ef-42dd-968e-a1e235d63e5c"
+          (reference "SW1") (unit 1)
+        )
+      )
+    )
+  )
   (symbol (lib_id "Connector:Screw_Terminal_01x02") (at 27.94 22.86 180) (unit 1)
     (in_bom yes) (on_board yes) (dnp no)
@@
     )
   )
-  (symbol (lib_id "power:GND") (at 92.71 191.77 0) (unit 1)
-    (in_bom yes) (on_board yes) (dnp no)
-    (property "Reference" "#PWR023" (at 92.71 198.12 0)
-      (effects (font (size 1.27 1.27)) hide)
-    )
-    (property "Value" "GND" (at 92.71 195.58 0)
-      (effects (font (size 1.27 1.27)))
-    )
-    (property "Footprint" "" (at 92.71 191.77 0)
-      (effects (font (size 1.27 1.27)) hide)
-    )
-    (property "Datasheet" "" (at 92.71 191.77 0)
-      (effects (font (size 1.27 1.27)) hide)
-    )
+  (symbol (lib_id "power:GND") (at 185.42 118.11 0) (unit 1)
+    (in_bom yes) (on_board yes) (dnp no)
+    (property "Reference" "#PWR023" (at 185.42 124.46 0)
+      (effects (font (size 1.27 1.27)) hide)
+    )
+    (property "Value" "GND" (at 185.42 121.92 0)
+      (effects (font (size 1.27 1.27)))
+    )
+    (property "Footprint" "" (at 185.42 118.11 0)
+      (effects (font (size 1.27 1.27)) hide)
+    )
+    (property "Datasheet" "" (at 185.42 118.11 0)
+      (effects (font (size 1.27 1.27)) hide)
+    )

Commit message: 20:04 Arrakis.local
Connections:
- net GPIO24 is gone; now on net GPIO16: Q2.1 (G)
- net GPIO25 is gone; now on net GPIO17: Q3.1 (G)
- net GPIO26 is gone; now on net GPIO18: Q4.1 (G)
- net GPIO27 is gone; now on net GPIO19: Q5.1 (G)
- net GPIO16: now reaches U4.21 (GPIO16)
- net GPIO17: now reaches U4.22 (GPIO17)
- net GPIO18: now reaches U4.24 (GPIO18)
- net GPIO19: now reaches U4.25 (GPIO19)
- no-connect marks 41 -> 37
Changed lines of the file:
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@@
   )
   (no_connect (at 109.22 113.03))
-  (no_connect (at 144.78 130.81))
   (no_connect (at 73.66 123.19))
-  (no_connect (at 144.78 135.89))
   (no_connect (at 109.22 133.35))
   (no_connect (at 109.22 123.19))
@@
   (no_connect (at 109.22 130.81))
   (no_connect (at 73.66 107.95))
+  (no_connect (at 144.78 135.89))
   (no_connect (at 109.22 102.87))
   (no_connect (at 144.78 123.19))
-  (no_connect (at 144.78 133.35))
   (no_connect (at 109.22 118.11))
   (no_connect (at 109.22 115.57))
   (no_connect (at 144.78 97.79))
   (no_connect (at 124.46 146.05))
-  (no_connect (at 144.78 140.97))
   (no_connect (at 109.22 105.41))
   (no_connect (at 109.22 110.49))
@@
   (no_connect (at 129.54 146.05))
   (no_connect (at 109.22 107.95))
-  (no_connect (at 144.78 138.43))
   (no_connect (at 73.66 119.38))
   (no_connect (at 109.22 120.65))
@@
     (stroke (width 0) (type default))
   )
+  (wire (pts (xy 144.78 130.81) (xy 162.56 130.81))
+    (stroke (width 0) (type default))
+  )
   (wire (pts (xy 34.29 48.26) (xy 34.29 22.86))
     (stroke (width 0) (type default))
@@
     (stroke (width 0) (type default))
   )
+  (wire (pts (xy 144.78 138.43) (xy 162.56 138.43))
+    (stroke (width 0) (type default))
+  )
   (wire (pts (xy 201.93 33.02) (xy 214.63 33.02))
     (stroke (width 0) (type default))
@@
     (stroke (width 0) (type default))
   )
+  (wire (pts (xy 144.78 133.35) (xy 162.56 133.35))
+    (stroke (width 0) (type default))
+  )
   (wire (pts (xy 95.25 140.97) (xy 109.22 140.97))
     (stroke (width 0) (type default))
@@
   )
   (wire (pts (xy 50.8 30.48) (xy 50.8 27.94))
+    (stroke (width 0) (type default))
+  )
+  (wire (pts (xy 144.78 140.97) (xy 162.56 140.97))
     (stroke (width 0) (type default))
   )
@@
     (effects (font (size 1.27 1.27)) (justify left bottom))
   )
-  (label "GPIO27" (at 245.11 39.37 0) (fields_autoplaced)
+  (label "GPIO19" (at 245.11 39.37 0) (fields_autoplaced)
     (effects (font (size 1.27 1.27)) (justify left bottom))
   )
@@
     (effects (font (size 1.27 1.27)) (justify left bottom))
   )
-  (label "GPIO24" (at 157.48 39.37 0) (fields_autoplaced)
-    (effects (font (size 1.27 1.27)) (justify left bottom))
-  )
-  (label "GPIO26" (at 215.9 39.37 0) (fields_autoplaced)
+  (label "GPIO16" (at 157.48 39.37 0) (fields_autoplaced)
+    (effects (font (size 1.27 1.27)) (justify left bottom))
+  )
+  (label "GPIO18" (at 215.9 39.37 0) (fields_autoplaced)
     (effects (font (size 1.27 1.27)) (justify left bottom))
   )
@@
     (effects (font (size 1.27 1.27)) (justify right bottom))
   )
+  (label "GPIO19" (at 162.56 130.81 0) (fields_autoplaced)
+    (effects (font (size 1.27 1.27)) (justify left bottom))
+  )
   (label "ADC_EMF_B" (at 153.67 113.03 0) (fields_autoplaced)
     (effects (font (size 1.27 1.27)) (justify left bottom))
   )
+  (label "GPIO17" (at 162.56 138.43 0) (fields_autoplaced)
+    (effects (font (size 1.27 1.27)) (justify left bottom))
+  )
   (label "GPIO15" (at 251.46 105.41 180) (fields_autoplaced)
     (effects (font (size 1.27 1.27)) (justify right bottom))
   )
+  (label "GPIO16" (at 162.56 140.97 0) (fields_autoplaced)
+    (effects (font (size 1.27 1.27)) (justify left bottom))
+  )
   (label "MOTOR_OUT_A" (at 212.09 111.76 180) (fields_autoplaced)
     (effects (font (size 1.27 1.27)) (justify right bottom))
@@
     (effects (font (size 1.27 1.27)) (justify left bottom))
   )
+  (label "GPIO18" (at 162.56 133.35 0) (fields_autoplaced)
+    (effects (font (size 1.27 1.27)) (justify left bottom))
+  )
   (label "MOTOR_OUT_B" (at 280.67 144.78 180) (fields_autoplaced)
     (effects (font (size 1.27 1.27)) (justify right bottom))
   )
-  (label "GPIO25" (at 186.69 39.37 0) (fields_autoplaced)
-    (effects (font (size 1.27 1.27)) (justify left bottom))
-  )
+  (label "GPIO17" (at 186.69 39.37 0) (fields_autoplaced)
+    (effects (font (size 1.27 1.27)) (justify left bottom))
+  )

Commit message: 20:57 Titan.local
Parts:
- removed C15: 100n, Capacitor_SMD:C_1206_3216Metric_Pad1.33x1.80mm_HandSolder, symbol Device:C
- removed R4: DNF, Resistor_SMD:R_1206_3216Metric_Pad1.30x1.75mm_HandSolder, symbol Device:R
- removed U3: W25Q64JVSSIQ, Package_SO:SOIC-8_5.23x5.23mm_P1.27mm, symbol RP2040-Decoder_Additional_Symbols:W25Q64JVSSIQ
Connections:
- no-connect marks 37 -> 31
Other:
- note removed: "Flash Memory"
