File: DccDecoder/DccDecoder.kicad_sch (KiCad schematic)
At the start: 27 parts, among them J14 +V, J15 M_OUT_B, J16 M_OUT_A, J17 GND, J3 0, J4 1, J5 2, J6 3, J8 DCC, Q1 T2N7002BK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

Commit message: 14:34 Titan.local
Parts:
- U2: footprint Package_SO:SOIC-8-1EP_3.9x4.9mm_P1.27mm_EP2.41x3.3mm_ThermalVias -> RP2040-Decoder_Additional_Footprints:SOIC-8-1EP_3.9x4.9mm_P1.27mm_EP2.41x3.3mm_ThermalVias
Changed lines of the file:
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@@
       (effects (font (size 1.27 1.27)) (justify left))
     )
-    (property "Footprint" "Package_SO:SOIC-8-1EP_3.9x4.9mm_P1.27mm_EP2.41x3.3mm_ThermalVias" (at 233.68 129.54 0)
+    (property "Footprint" "RP2040-Decoder_Additional_Footprints:SOIC-8-1EP_3.9x4.9mm_P1.27mm_EP2.41x3.3mm_ThermalVias" (at 233.68 129.54 0)
       (effects (font (size 1.27 1.27)) hide)
     )

Commit message: 14:24 Titan.local
Parts:
- added J1: 3v3, Connector_PinHeader_2.54mm:PinHeader_1x02_P2.54mm_Vertical, symbol Connector:Conn_01x02_Pin
- U1: value HT7533S -> HT7550S
Connections:
- net +3V3: no longer C1.1, U1.2 (VOUT)
- net GND: now also U4.23 (GND); no longer U4.42 (GND)
- net VSYS: now reaches U4.39 (VSYS)
- net VSYS: now also J1.2 (Pin_2)
- new net 5V: C1.1, J1.1 (Pin_1), U1.2 (VOUT)
Other:
- title: (none) -> Pico DCC Decoder
