File: DccDecoder/DccDecoder.kicad_pcb (KiCad board)
At the start: 2 copper layers, 88.9 x 33 mm, 0 parts

Commit message: 20:57 Titan.local
Parts:
- added C1: 10u, Capacitor_SMD:C_1206_3216Metric_Pad1.33x1.80mm_HandSolder, F.Cu at (184.4, 78.5)
- added C2: 10u, Capacitor_SMD:C_1206_3216Metric_Pad1.33x1.80mm_HandSolder, F.Cu at (184.1, 74.7)
- added D1: KMB24F, Package_TO_SOT_SMD:TO-269AA, F.Cu at (175.0, 56.6)
- added J14: +V, TestPoint:TestPoint_Pad_D2.0mm, F.Cu at (87.7, 65.9)
- added J15: M_OUT_B, TestPoint:TestPoint_Pad_D2.0mm, F.Cu at (91.8, 65.9)
- added J16: M_OUT_A, TestPoint:TestPoint_Pad_D2.0mm, F.Cu at (87.7, 61.9)
- added J17: GND, TestPoint:TestPoint_Pad_D2.0mm, F.Cu at (91.8, 61.9)
- added J3: 0, TestPoint:TestPoint_Pad_D2.0mm, F.Cu at (87.7, 74.0)
- added J4: 1, TestPoint:TestPoint_Pad_D2.0mm, F.Cu at (91.8, 74.0)
- added J5: 2, TestPoint:TestPoint_Pad_D2.0mm, F.Cu at (87.7, 70.0)
- added J6: 3, TestPoint:TestPoint_Pad_D2.0mm, F.Cu at (91.8, 70.0)
- added J8: DCC, TerminalBlock_Phoenix:TerminalBlock_Phoenix_PT-1,5-2-3.5-H_1x02_P3.50mm_Horizontal, F.Cu at (186.5, 68.8)
- added Q1: T2N7002BK, Package_TO_SOT_SMD:SOT-23, F.Cu at (163.9, 75.9)
- added Q2: T2N7002BK, Package_TO_SOT_SMD:SOT-23, F.Cu at (79.7, 77.9)
- added Q3: T2N7002BK, Package_TO_SOT_SMD:SOT-23, F.Cu at (79.4, 59.8)
- added Q4: T2N7002BK, Package_TO_SOT_SMD:SOT-23, F.Cu at (79.4, 66.5)
- added Q5: T2N7002BK, Package_TO_SOT_SMD:SOT-23, F.Cu at (79.7, 72.1)
- added R1: 6k8, Resistor_SMD:R_1206_3216Metric_Pad1.30x1.75mm_HandSolder, F.Cu at (163.6, 63.0)
- added R2: 6k8, Resistor_SMD:R_1206_3216Metric_Pad1.30x1.75mm_HandSolder, F.Cu at (164.1, 69.6)
- added R5: 6k8, Resistor_SMD:R_1206_3216Metric_Pad1.30x1.75mm_HandSolder, F.Cu at (169.7, 61.7)
- added R6: 6k8, Resistor_SMD:R_1206_3216Metric_Pad1.30x1.75mm_HandSolder, F.Cu at (169.7, 65.0)
- added R7: 1k, Resistor_SMD:R_1206_3216Metric_Pad1.30x1.75mm_HandSolder, F.Cu at (169.7, 68.3)
- added R8: 1k, Resistor_SMD:R_1206_3216Metric_Pad1.30x1.75mm_HandSolder, F.Cu at (169.7, 71.6)
- added SW1: SW_Push, Button_Switch_SMD:SW_Tactile_SPST_NO_Straight_CK_PTS636Sx25SMTRLFS, F.Cu at (176.5, 66.0)
- added U1: HT7533S, Package_TO_SOT_SMD:SOT-23, F.Cu at (163.6, 58.2)
- added U2: BDR6133, Package_SO:SOIC-8-1EP_3.9x4.9mm_P1.27mm_EP2.41x3.3mm_ThermalVias, F.Cu at (174.6, 76.3)
- added U4: Pico, MCU_RaspberryPi_and_Boards:RP2040Pico, F.Cu at (129.0, 67.3)
Other:
- board size 88.9 x 33 mm -> 116.8 x 35.6 mm

Commit message: 21:39 Arrakis.local
Parts:
- SW1: value SW_Push -> Reset
- moved SW1 13.5 mm to (185.4, 55.9)
- moved R6 5.80 mm to (175.3, 63.5)
- moved R7 5.59 mm to (175.3, 68.6)
- moved R8 3.65 mm to (167.6, 68.6)
- moved R2 3.24 mm to (161.0, 68.6)
- moved U1 3.24 mm to (163.5, 54.9)
- moved R5 2.68 mm to (167.6, 63.5)
- moved R1 2.59 mm to (161.0, 63.5)
Routing:
- net GND: track 0.00 -> 211.5 mm, vias 0 -> 1
- net +V: track 0.00 -> 148.8 mm
- net /MOTOR_OUT_B: track 0.00 -> 115.1 mm
- net /MOTOR_OUT_A: track 0.00 -> 113.4 mm, vias 0 -> 2
- net +3V3: track 0.00 -> 90.6 mm, vias 0 -> 3
- net /GPIO16: track 0.00 -> 85.3 mm, vias 0 -> 1
- net /GPIO17: track 0.00 -> 76.5 mm
- net /GPIO18: track 0.00 -> 72.5 mm, vias 0 -> 1
- net /GPIO19: track 0.00 -> 71.5 mm, vias 0 -> 1
- net Net-(U4-RUN): track 0.00 -> 60.5 mm
- net /ADC_EMF_A: track 0.00 -> 60.0 mm
- net /ADC_EMF_B: track 0.00 -> 57.3 mm, vias 0 -> 1
- net Net-(J4-Pin_1): track 0.00 -> 39.2 mm
- net /GPIO21: track 0.00 -> 34.6 mm, vias 0 -> 1
- net /GPIO14: track 0.00 -> 31.8 mm, vias 0 -> 1
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
Commit message: 14:34 Titan.local
Parts:
- SW1: value Reset -> SW_Push
- U2: footprint Package_SO:SOIC-8-1EP_3.9x4.9mm_P1.27mm_EP2.41x3.3mm_ThermalVias -> RP2040-Decoder_Additional_Footprints:SOIC-8-1EP_3.9x4.9mm_P1.27mm_EP2.41x3.3mm_ThermalVias
Changed lines of the file:
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@@
   (net 2 "GND")
   (net 3 "+V")
-  (net 4 "Net-(J8-Pin_2)")
-  (net 5 "Net-(J8-Pin_1)")
+  (net 4 "Net-(#FLG02-pwr)")
+  (net 5 "Net-(#FLG01-pwr)")
   (net 6 "Net-(J3-Pin_1)")
   (net 7 "Net-(J4-Pin_1)")
@@
     )
   )
-  (footprint "Package_SO:SOIC-8-1EP_3.9x4.9mm_P1.27mm_EP2.41x3.3mm_ThermalVias" (layer "F.Cu")
+  (footprint "RP2040-Decoder_Additional_Footprints:SOIC-8-1EP_3.9x4.9mm_P1.27mm_EP2.41x3.3mm_ThermalVias" (layer "F.Cu")
     (at 174.563 76.327)
     (descr "SOIC, 8 Pin (http://www.allegromicro.com/~/media/Files/Datasheets/A4950-Datasheet.ashx#page=8), generated with kicad-footprint-generator ipc_gullwing_generator.py")
@@
     (property "ki_keywords" "half bridge driver")
     (attr smd)
-    (fp_text reference "U2" (at 0 -3.4) (layer "F.SilkS")
+    (fp_text reference "U2" (at -0.2 -4.3) (layer "F.SilkS")
         (effects (font (size 1 1) (thickness 0.15)))
     )
@@
         (effects (font (size 0.98 0.98) (thickness 0.15)))
     )
-    (fp_line (start 0 -2.56) (end -3.45 -2.56)
-      (stroke (width 0.12) (type solid)) (layer "F.SilkS"))
-    (fp_line (start 0 -2.56) (end 1.95 -2.56)
-      (stroke (width 0.12) (type solid)) (layer "F.SilkS"))
-    (fp_line (start 0 2.56) (end -1.95 2.56)
-      (stroke (width 0.12) (type solid)) (layer "F.SilkS"))
-    (fp_line (start 0 2.56) (end 1.95 2.56)
+    (fp_line (start -1.55 -2.56) (end -3.4 -2.56)
+      (stroke (width 0.12) (type solid)) (layer "F.SilkS"))
+    (fp_line (start -1.55 2.56) (end -3.4 2.56)
+      (stroke (width 0.12) (type solid)) (layer "F.SilkS"))
+    (fp_line (start 1.55 -2.56) (end 3.4 -2.56)
+      (stroke (width 0.12) (type solid)) (layer "F.SilkS"))
+    (fp_line (start 1.55 2.56) (end 3.4 2.56)
       (stroke (width 0.12) (type solid)) (layer "F.SilkS"))
     (fp_line (start -3.7 -2.7) (end -3.7 2.7)
@@
     (pad "9" thru_hole circle (at 0.7 1.2) (size 0.5 0.5) (drill 0.2) (layers "*.Cu")
       (net 2 "GND") (pinfunction "GND") (pintype "passive"))
-    (model "${KICAD6_3DMODEL_DIR}/Package_SO.3dshapes/SOIC-8-1EP_3.9x4.9mm_P1.27mm_EP2.41x3.3mm.wrl"
+    (model "${KICAD6_3DMODEL_DIR}/Package_SO.3dshapes/SOIC-8_3.9x4.9mm_P1.27mm.wrl"
       (offset (xyz 0 0 0))
       (scale (xyz 1 1 1))
@@
       (stroke (width 0.1) (type solid)) (fill none) (layer "F.Fab"))
     (pad "1" thru_hole rect (at 0 0 90) (size 2.4 2.4) (drill 1.2) (layers "*.Cu" "*.Mask")
-      (net 5 "Net-(J8-Pin_1)") (pinfunction "Pin_1") (pintype "passive"))
+      (net 5 "Net-(#FLG01-pwr)") (pinfunction "Pin_1") (pintype "passive"))
     (pad "2" thru_hole circle (at 3.5 0 90) (size 2.4 2.4) (drill 1.2) (layers "*.Cu" "*.Mask")
-      (net 4 "Net-(J8-Pin_2)") (pinfunction "Pin_2") (pintype "passive"))
+      (net 4 "Net-(#FLG02-pwr)") (pinfunction "Pin_2") (pintype "passive"))
     (model "${KICAD6_3DMODEL_DIR}/TerminalBlock_Phoenix.3dshapes/TerminalBlock_Phoenix_PT-1,5-2-3.5-H_1x02_P3.50mm_Horizontal.wrl"
       (offset (xyz 0 0 0))
@@
       (net 12 "Net-(Q1-G)") (pintype "passive"))
     (pad "2" smd roundrect (at 1.55 0) (size 1.3 1.75) (layers "F.Cu" "F.Paste" "F.Mask") (roundrect_rratio 0.192308)
-      (net 4 "Net-(J8-Pin_2)") (pintype "passive"))
+      (net 4 "Net-(#FLG02-pwr)") (pintype "passive"))
     (model "${KICAD6_3DMODEL_DIR}/Resistor_SMD.3dshapes/R_1206_3216Metric.wrl"
       (offset (xyz 0 0 0))
@@
       (stroke (width 0.12) (type solid)) (layer "F.Fab"))
     (pad "1" smd rect (at -3.075 -1.27) (size 1 0.8) (layers "F.Cu" "F.Paste" "F.Mask")
-      (net 4 "Net-(J8-Pin_2)") (pintype "power_in"))
+      (net 4 "Net-(#FLG02-pwr)") (pintype "power_in"))
     (pad "2" smd rect (at -3.075 1.27) (size 1 0.8) (layers "F.Cu" "F.Paste" "F.Mask")
-      (net 5 "Net-(J8-Pin_1)") (pintype "power_in"))
+      (net 5 "Net-(#FLG01-pwr)") (pintype "power_in"))
     (pad "3" smd rect (at 3.075 1.27) (size 1 0.8) (layers "F.Cu" "F.Paste" "F.Mask")
       (net 3 "+V") (pinfunction "+") (pintype "power_out"))
@@
         (effects (font (size 1 1) (thickness 0.15)))
     )
-    (fp_text value "Reset" (at 0 3 90 unlocked) (layer "F.Fab")
-        (effects (font (size 1 1) (thickness 0.15)))
-    )
+    (fp_text value "SW_Push" (at 0 3 90 unlocked) (layer "F.Fab")
+        (effects (font (size 1 1) (thickness 0.15)))
+    )

Commit message: 16:27 Arrakis.local
Routing:
- net /MOTOR_OUT_A: track 113.4 -> 94.2 mm, vias 2 -> 3
- net Net-(J4-Pin_1): track 39.2 -> 20.9 mm, vias 0 -> 2
- net Net-(J8-Pin_2): track 31.5 -> 47.8 mm
- net +V: track 148.8 -> 135.5 mm, vias 0 -> 3
- net GND: track 211.5 -> 220.1 mm, vias 1 -> 0
- net /GPIO18: track 72.5 -> 80.8 mm, vias 1 -> 0
- net /ADC_EMF_B: track 57.3 -> 64.0 mm, vias 1 -> 0
- net /GPIO15: track 29.2 -> 33.9 mm, vias 1 -> 0
- net /ADC_EMF_A: track 60.0 -> 64.5 mm, vias 0 -> 1
- net Net-(U4-RUN): track 60.5 -> 56.7 mm
- net +3V3: track 90.6 -> 87.9 mm, vias 3 -> 2
- net /GPIO16: track 85.3 -> 82.7 mm
- net /GPIO17: track 76.5 -> 79.1 mm
- net /GPIO14: track 31.8 -> 33.9 mm, vias 1 -> 0
- net /GPIO21: track 34.6 -> 35.9 mm
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