File: DccDecoder2/DccDecoder2.kicad_pcb (KiCad board)
At the start: 2 copper layers, 94 x 35.6 mm, 28 parts, among them J14 +V, J15 M_OUT_B, J16 M_OUT_A, J17 GND, J3 0, J4 1, J5 2, J6 3, J8 DCC, Q1 T2N7002BK, Q2 T2N7002BK, Q3 T2N7002BK, Q4 T2N7002BK, Q5 T2N7002BK, SW1 SW_Push, U1 HT7550S, U2 BDR6133, U4 Pico

Commit message: 30/11/24 19:40 Titan.local
Parts:
- removed the U1 at (169.2, 55.9)
- added C2: 100n, Capacitor_SMD:C_1206_3216Metric_Pad1.33x1.80mm_HandSolder, F.Cu at (187.0, 55.9)
- added D1: CUHS20F30, Diode_SMD:D_1206_3216Metric, F.Cu at (161.4, 53.3)
- added IC1: AP64060QWU-7, Package_TO_SOT_SMD:TSOT-23-6, F.Cu at (169.0, 54.3)
- added L1: 10uH, Inductor_SMD_Wurth:L_Wurth_WE-LQSH-2010, F.Cu at (187.2, 50.8)
- added R1: 115k, Resistor_SMD:R_1206_3216Metric_Pad1.30x1.75mm_HandSolder, F.Cu at (187.0, 61.0)
- added R2: 22k1, Resistor_SMD:R_1206_3216Metric_Pad1.30x1.75mm_HandSolder, F.Cu at (168.6, 58.4)
- C3: renamed from C2; value 10u -> 2.2uF/25V
- moved SW1 71.8 mm to (114.3, 66.0)
- renumbered D1 to D2, J8 to J1, J3 to J2, J4 to J3, J5 to J4, J6 to J5, J14 to J6, J15 to J7, J16 to J8, J17 to J9, R1 to R3, R2 to R4, R7 to R6, R6 to R7, U4 to U1
Routing:
- net GND: track 201.9 -> 0.00 mm
- net +V: track 121.8 -> 0.00 mm, vias 2 -> 0
- net /GPIO15: track 80.5 -> 0.00 mm
- net /MOTOR_OUT_B: track 77.7 -> 0.00 mm, vias 2 -> 0
- net /GPIO14: track 75.7 -> 0.00 mm
- net /ADC_EMF_B: track 70.6 -> 0.00 mm
- net /MOTOR_OUT_A: track 69.4 -> 0.00 mm, vias 3 -> 0
- net /ADC_EMF_A: track 62.0 -> 0.00 mm, vias 1 -> 0
- net Net-(U1-RUN): track 60.6 -> 0.00 mm
- net /5V: track 56.3 -> 0.00 mm
- net /GPIO21: track 52.9 -> 0.00 mm, vias 1 -> 0
- net /GPIO17: track 43.0 -> 0.00 mm
- net /GPIO18: track 39.7 -> 0.00 mm, vias 1 -> 0
- net /GPIO16: track 39.5 -> 0.00 mm
- net +3V3: track 37.0 -> 0.00 mm, vias 1 -> 0
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
Commit message: 30/11/24 22:26 Arrakis.local
Routing:
- net GND: track 0.00 -> 167.2 mm, vias 0 -> 1
- net +V: track 0.00 -> 123.0 mm
- net /MOTOR_OUT_B: track 0.00 -> 82.7 mm
- net /GPIO15: track 0.00 -> 80.5 mm
- net /5V: track 0.00 -> 77.9 mm
- net /GPIO14: track 0.00 -> 75.7 mm
- net /MOTOR_OUT_A: track 0.00 -> 64.6 mm, vias 0 -> 3
- net /ADC_EMF_A: track 0.00 -> 59.7 mm
- net /GPIO21: track 0.00 -> 56.2 mm
- net /ADC_EMF_B: track 0.00 -> 50.3 mm
- net Net-(U1-RUN): track 0.00 -> 43.5 mm
- net /GPIO17: track 0.00 -> 43.0 mm
- net Net-(IC1-BST): track 0.00 -> 42.6 mm
- net +3V3: track 0.00 -> 42.2 mm, vias 0 -> 1
- net /GPIO18: track 0.00 -> 39.7 mm, vias 0 -> 1
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
Commit message: 01/12/24 09:58 Titan.local
Parts:
- D1: footprint Diode_SMD:D_1206_3216Metric -> CUHS20F30:CUHS20F30H3F
Changed lines of the file:
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@@
       (net 52 "/VSYS") (pinfunction "B") (pintype "passive"))
   )
-  (footprint "Diode_SMD:D_1206_3216Metric" (layer "F.Cu")
+  (footprint "CUHS20F30:CUHS20F30H3F" (layer "F.Cu")
     (at 161.42 53.34)
-    (descr "Diode SMD 1206 (3216 Metric), square (rectangular) end terminal, IPC_7351 nominal, (Body size source: http://www.tortai-tech.com/upload/download/2011102023233369053.pdf), generated with kicad-footprint-generator")
-    (tags "diode")
+    (descr "US2H")
+    (tags "Schottky Diode")
     (property "Sheetfile" "DccDecoder2.kicad_sch")
     (property "Sheetname" "")
@@
     (property "ki_keywords" "diode")
     (attr smd)
-    (fp_text reference "D1" (at 0 -1.82) (layer "F.SilkS")
-        (effects (font (size 1 1) (thickness 0.15)))
+    (fp_text reference "D1" (at 0 0) (layer "F.SilkS")
+        (effects (font (size 1.27 1.27) (thickness 0.254)))
     )
-    (fp_text value "CUHS20F30" (at 0 1.82) (layer "F.Fab")
-        (effects (font (size 1 1) (thickness 0.15)))
+    (fp_text value "CUHS20F30" (at 0 0) (layer "F.SilkS") hide
+        (effects (font (size 1.27 1.27) (thickness 0.254)))
     )
     (fp_text user "${REFERENCE}" (at 0 0) (layer "F.Fab")
-        (effects (font (size 0.8 0.8) (thickness 0.12)))
+        (effects (font (size 1.27 1.27) (thickness 0.254)))
     )
-    (fp_line (start -2.285 -1.135) (end -2.285 1.135)
-      (stroke (width 0.12) (type solid)) (layer "F.SilkS"))
-    (fp_line (start -2.285 1.135) (end 1.6 1.135)
-      (stroke (width 0.12) (type solid)) (layer "F.SilkS"))
-    (fp_line (start 1.6 -1.135) (end -2.285 -1.135)
-      (stroke (width 0.12) (type solid)) (layer "F.SilkS"))
-    (fp_line (start -2.28 -1.12) (end 2.28 -1.12)
-      (stroke (width 0.05) (type solid)) (layer "F.CrtYd"))
-    (fp_line (start -2.28 1.12) (end -2.28 -1.12)
-      (stroke (width 0.05) (type solid)) (layer "F.CrtYd"))
-    (fp_line (start 2.28 -1.12) (end 2.28 1.12)
-      (stroke (width 0.05) (type solid)) (layer "F.CrtYd"))
-    (fp_line (start 2.28 1.12) (end -2.28 1.12)
-      (stroke (width 0.05) (type solid)) (layer "F.CrtYd"))
-    (fp_line (start -1.6 -0.4) (end -1.6 0.8)
+    (fp_line (start -2.3 0) (end -2.3 0)
+      (stroke (width 0.1) (type solid)) (layer "F.SilkS"))
+    (fp_line (start -2.2 0) (end -2.2 0)
+      (stroke (width 0.1) (type solid)) (layer "F.SilkS"))
+    (fp_arc (start -2.3 0) (mid -2.25 -0.05) (end -2.2 0)
+      (stroke (width 0.1) (type solid)) (layer "F.SilkS"))
+    (fp_arc (start -2.2 0) (mid -2.25 0.05) (end -2.3 0)
+      (stroke (width 0.1) (type solid)) (layer "F.SilkS"))
+    (fp_line (start -2.65 -1.7) (end 2.65 -1.7)
+      (stroke (width 0.1) (type solid)) (layer "F.CrtYd"))
+    (fp_line (start -2.65 1.7) (end -2.65 -1.7)
+      (stroke (width 0.1) (type solid)) (layer "F.CrtYd"))
+    (fp_line (start 2.65 -1.7) (end 2.65 1.7)
+      (stroke (width 0.1) (type solid)) (layer "F.CrtYd"))
+    (fp_line (start 2.65 1.7) (end -2.65 1.7)
+      (stroke (width 0.1) (type solid)) (layer "F.CrtYd"))
+    (fp_line (start -1 -0.7) (end 1 -0.7)
       (stroke (width 0.1) (type solid)) (layer "F.Fab"))
-    (fp_line (start -1.6 0.8) (end 1.6 0.8)
+    (fp_line (start -1 0.7) (end -1 -0.7)
       (stroke (width 0.1) (type solid)) (layer "F.Fab"))
-    (fp_line (start -1.2 -0.8) (end -1.6 -0.4)
+    (fp_line (start 1 -0.7) (end 1 0.7)
       (stroke (width 0.1) (type solid)) (layer "F.Fab"))
-    (fp_line (start 1.6 -0.8) (end -1.2 -0.8)
+    (fp_line (start 1 0.7) (end -1 0.7)
       (stroke (width 0.1) (type solid)) (layer "F.Fab"))
-    (fp_line (start 1.6 0.8) (end 1.6 -0.8)
-      (stroke (width 0.1) (type solid)) (layer "F.Fab"))
-    (pad "1" smd roundrect (at -1.4 0) (size 1.25 1.75) (layers "F.Cu" "F.Paste" "F.Mask") (roundrect_rratio 0.2)
+    (pad "1" smd rect (at -0.65 0 90) (size 1.1 2) (layers "F.Cu" "F.Paste" "F.Mask")
       (net 3 "+V") (pinfunction "K") (pintype "passive"))
-    (pad "2" smd roundrect (at 1.4 0) (size 1.25 1.75) (layers "F.Cu" "F.Paste" "F.Mask") (roundrect_rratio 0.2)
+    (pad "2" smd rect (at 1.25 0) (size 0.8 1.1) (layers "F.Cu" "F.Paste" "F.Mask")
       (net 3 "+V") (pinfunction "A") (pintype "passive"))
-    (model "${KICAD6_3DMODEL_DIR}/Diode_SMD.3dshapes/D_1206_3216Metric.wrl"
+    (model "/Users/colinc/Downloads/LIB_CUHS20F30,H3F/CUHS20F30,H3F/3D/CUHS20F30,H3F.stp"
       (offset (xyz 0 0 0))
       (scale (xyz 1 1 1))
-      (rotate (xyz 0 0 0))
+      (rotate (xyz 0 0 -90))
     )
   )
