File: DccDecoder2/DccDecoder2.kicad_sch (KiCad schematic)
At the start: 28 parts, among them J14 +V, J15 M_OUT_B, J16 M_OUT_A, J17 GND, J3 0, J4 1, J5 2, J6 3, J8 DCC, Q1 T2N7002BK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

Commit message: 30/11/24 17:42 Arrakis.local
Parts:
- added IC1: AP64060QWU-7, Package_TO_SOT_SMD:TSOT-23-6, symbol AP64060QWU-7:AP64060QWU-7
Changed lines of the file:
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@@
+    )
+  )
+  (symbol (lib_id "AP64060QWU-7:AP64060QWU-7") (at 53.34 80.01 0) (unit 1)
+    (in_bom yes) (on_board yes) (dnp no) (fields_autoplaced)
+    (property "Reference" "IC1" (at 66.04 73.66 0)
+      (effects (font (size 1.27 1.27)))
+    )
+    (property "Value" "AP64060QWU-7" (at 66.04 76.2 0)
+      (effects (font (size 1.27 1.27)))
+    )
+    (property "Footprint" "Package_TO_SOT_SMD:TSOT-23-6" (at 74.93 174.93 0)
+      (effects (font (size 1.27 1.27)) (justify left top) hide)
+    )
+    (property "Datasheet" "https://www.diodes.com//assets/Datasheets/AP64060.pdf" (at 74.93 274.93 0)
+      (effects (font (size 1.27 1.27)) (justify left top) hide)
+    )
+    (property "Height" "1" (at 74.93 474.93 0)
+      (effects (font (size 1.27 1.27)) (justify left top) hide)
+    )
+    (property "Mouser Part Number" "621-AP64060QWU-7" (at 74.93 574.93 0)
+      (effects (font (size 1.27 1.27)) (justify left top) hide)
+    )
+    (property "Mouser Price/Stock" "https://www.mouser.co.uk/ProductDetail/Diodes-Incorporated/AP64060QWU-7?qs=Li%252BoUPsLEnvtPycFvZmEcQ%3D%3D" (at 74.93 674.93 0)
+      (effects (font (size 1.27 1.27)) (justify left top) hide)
+    )
+    (property "Manufacturer_Name" "Diodes Incorporated" (at 74.93 774.93 0)
+      (effects (font (size 1.27 1.27)) (justify left top) hide)
+    )
+    (property "Manufacturer_Part_Number" "AP64060QWU-7" (at 74.93 874.93 0)
+      (effects (font (size 1.27 1.27)) (justify left top) hide)
+    )
+    (pin "1")
+    (pin "2")
+    (pin "3")
+    (pin "4")
+    (pin "5")
+    (pin "6")
+    (instances
+      (project "DccDecoder2"
+        (path "/68a87a67-79ef-42dd-968e-a1e235d63e5c"
+          (reference "IC1") (unit 1)
+        )
+      )
     )
   )

Commit message: 30/11/24 19:40 Titan.local
Parts:
- removed U1: HT7550S, Package_TO_SOT_SMD:SOT-23, symbol RP2040-Decoder_Additional_Symbols:HT7533S
- added C1: 100n, Capacitor_SMD:C_1206_3216Metric_Pad1.33x1.80mm_HandSolder, symbol Device:C
- added D1: CUHS20F30, Diode_SMD:D_1206_3216Metric, symbol Device:D_Zener
- added L1: 10uH, Inductor_SMD_Wurth:L_Wurth_WE-LQSH-2010, symbol Device:L
- added R1: 115k, Resistor_SMD:R_1206_3216Metric_Pad1.30x1.75mm_HandSolder, symbol Device:R
- added R1: 22k1, Resistor_SMD:R_1206_3216Metric_Pad1.30x1.75mm_HandSolder, symbol Device:R
- C2: value 10u -> 2.2uF/25V
- renumbered J8 to J1, U4 to U1
Connections:
- net +V: now also IC1.4 (EN), IC1.5 (VIN), D1.1 (K), D1.2 (A)
- net 5V: now also L1.1, R1.2
- net GND: now also IC1.2 (GND), R1.1
- net at IC1.1 (BST): now also C1.2
- net at IC1.3 (FB): now also R1.1, R1.2
- net at IC1.6 (SW): now also C1.1, L1.2
Other:
- moved on the sheet: C1, C2, D1, IC1, JP1, Q1, R1, R2

Commit message: 01/12/24 09:58 Titan.local
Parts:
- D1: footprint Diode_SMD:D_1206_3216Metric -> CUHS20F30:CUHS20F30H3F
Changed lines of the file:
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@@
       (effects (font (size 1.27 1.27)))
     )
-    (property "Footprint" "Diode_SMD:D_1206_3216Metric" (at 105.41 35.56 0)
+    (property "Footprint" "CUHS20F30:CUHS20F30H3F" (at 105.41 35.56 0)
       (effects (font (size 1.27 1.27)) hide)
     )

Commit message: 04/12/24 22:17 Titan.local
Connections:
- net +V: no longer D1.2 (A), D1.3 (+)
- new net: D1.2 (A), D1.3 (+)
Changed lines of the file:
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@@
   (junction (at 113.03 20.32) (diameter 0) (color 0 0 0 0)
-  )
-  (junction (at 109.22 30.48) (diameter 0) (color 0 0 0 0)
   )
   (junction (at 113.03 63.5) (diameter 0) (color 0 0 0 0)
@@
     (stroke (width 0) (type default))
   )
-  (wire (pts (xy 109.22 30.48) (xy 109.22 27.94))
-    (stroke (width 0) (type default))
-  )
   (wire (pts (xy 265.43 147.32) (xy 266.7 147.32))
     (stroke (width 0) (type default))
@@
         )
       )
-    )
-  )
-  (symbol (lib_id "RP2040-Decoder_Additional_Symbols:+V") (at 109.22 27.94 0) (unit 1)
-    (in_bom yes) (on_board yes) (dnp no)
-    (property "Reference" "#PWR02" (at 109.22 31.75 0)
-      (effects (font (size 1.27 1.27)) hide)
-    )
-    (property "Value" "+VP" (at 109.22 24.13 0)
-      (effects (font (size 1.27 1.27)))
-    )
-    (property "Footprint" "" (at 109.22 27.94 0)
-      (effects (font (size 1.27 1.27)) hide)
-    )
-    (property "Datasheet" "" (at 109.22 27.94 0)
-      (effects (font (size 1.27 1.27)) hide)
-    )
-    (pin "1")
-    (instances
-      (project "RP2040-Decoder"
-        (path "/11d18738-0f49-4d63-b61c-22a93efd5959"
-          (reference "#PWR02") (unit 1)
-        )
-      )
-      (project "DccDecoder2"
-        (path "/68a87a67-79ef-42dd-968e-a1e235d63e5c"
-          (reference "#PWR03") (unit 1)
-        )
-      )

Commit message: 09/12/24 17:09 Arrakis.local
Parts:
- removed JP1: Jumper_2_Open, Jumper:SolderJumper-2_P1.3mm_Open_Pad1.0x1.5mm, symbol Jumper:Jumper_2_Bridged
- added Q6: DMG2305UX-7, SOT96P240X110-3N, symbol DMG2305UX-7:DMG2305UX-7
- R1: value 115k -> 69k8
Connections:
- net 5V is gone; now on net +3V3: C1.1, L1.1, R1.2
- net +3V3: now also Q6.3; no longer U1.36 (3V3)
- net VSYS: now also Q6.2
- net at U1.40 (VBUS): now also Q6.1
- no-connect marks 31 -> 32

Commit message: 09/12/24 22:16 Arrakis.local
Parts:
- D1: footprint CUHS20F30:CUHS20F30H3F -> Diode_SMD:D_1206_3216Metric
- L1: footprint Inductor_SMD_Wurth:L_Wurth_WE-LQSH-2010 -> Inductor_SMD:L_1206_3216Metric
Changed lines of the file:
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@@
       (effects (font (size 1.27 1.27)))
     )
-    (property "Footprint" "CUHS20F30:CUHS20F30H3F" (at 105.41 35.56 0)
+    (property "Footprint" "Diode_SMD:D_1206_3216Metric" (at 105.41 35.56 0)
       (effects (font (size 1.27 1.27)) hide)
     )
@@
       (effects (font (size 1.27 1.27)))
     )
-    (property "Footprint" "Inductor_SMD_Wurth:L_Wurth_WE-LQSH-2010" (at 66.04 24.13 0)
+    (property "Footprint" "Inductor_SMD:L_1206_3216Metric" (at 66.04 24.13 0)
       (effects (font (size 1.27 1.27)) hide)
     )
