File: DccDecoder2/DccDecoder2.kicad_sch (KiCad schematic)
At the start: 33 parts, among them IC1 AP64060QWU-7, J1 DCC, J14 +V, J15 M_OUT_B, J16 M_OUT_A, J17 GND, J3 0, J4 1, J5 2, J6 3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

Commit message: 10/12/24 16:11 Arrakis.local
Changed lines of the file:
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@@
   (junction (at 134.62 33.02) (diameter 0) (color 0 0 0 0)
-  )
-  (junction (at 113.03 20.32) (diameter 0) (color 0 0 0 0)
-  )
-  (junction (at 113.03 63.5) (diameter 0) (color 0 0 0 0)
   )
   (junction (at 246.38 121.92) (diameter 0) (color 0 0 0 0)
@@
     (stroke (width 0) (type default))
   )
-  (wire (pts (xy 34.29 63.5) (xy 113.03 63.5))
-    (stroke (width 0) (type default))
-  )
   (wire (pts (xy 157.48 39.37) (xy 165.1 39.37))
     (stroke (width 0) (type default))
@@
     (stroke (width 0) (type default))
   )
-  (wire (pts (xy 33.02 20.32) (xy 113.03 20.32))
-    (stroke (width 0) (type default))
-  )
   (wire (pts (xy 50.8 24.13) (xy 50.8 30.48))
     (stroke (width 0) (type default))
@@
     (stroke (width 0) (type default))
   )
-  (wire (pts (xy 113.03 63.5) (xy 119.38 63.5))
+  (wire (pts (xy 34.29 63.5) (xy 119.38 63.5))
     (stroke (width 0) (type default))
   )
@@
     (stroke (width 0) (type default))
   )
-  (wire (pts (xy 113.03 20.32) (xy 119.38 20.32))
+  (wire (pts (xy 33.02 20.32) (xy 119.38 20.32))
     (stroke (width 0) (type default))
   )
@@
     (stroke (width 0) (type default))
   )
-  (wire (pts (xy 113.03 17.78) (xy 113.03 20.32))
-    (stroke (width 0) (type default))
-  )
   (wire (pts (xy 153.67 92.71) (xy 153.67 83.82))
     (stroke (width 0) (type default))
@@
   )
   (wire (pts (xy 134.62 46.99) (xy 134.62 49.53))
-    (stroke (width 0) (type default))
-  )
-  (wire (pts (xy 113.03 60.96) (xy 113.03 63.5))
     (stroke (width 0) (type default))
   )
@@
   (label "GPIO17" (at 186.69 39.37 0) (fields_autoplaced)
     (effects (font (size 1.27 1.27)) (justify left bottom))
-  )
-  (netclass_flag "" (length 2.54) (shape round) (at 41.91 20.32 0) (fields_autoplaced)
-    (effects (font (size 1.27 1.27)) (justify left bottom))
-    (property "Netclass" "power" (at 42.6085 17.78 0)
-      (effects (font (size 1.27 1.27) italic) (justify left) hide)
-    )
-  )
-  (netclass_flag "" (length 2.54) (shape round) (at 68.58 63.5 0) (fields_autoplaced)
-    (effects (font (size 1.27 1.27)) (justify left bottom))
-    (property "Netclass" "power" (at 69.2785 60.96 0)
-      (effects (font (size 1.27 1.27) italic) (justify left))
-    )
   )
   (symbol (lib_id "Device:C") (at 106.68 46.99 0) (mirror y) (unit 1)
@@
     )
   )
-  (symbol (lib_id "power:PWR_FLAG") (at 113.03 17.78 0) (unit 1)
-    (in_bom yes) (on_board yes) (dnp no)
-    (property "Reference" "#FLG02" (at 113.03 15.875 0)
-      (effects (font (size 1.27 1.27)) hide)
-    )
-    (property "Value" "PWR_FLAG" (at 113.03 13.97 0)
-      (effects (font (size 1.27 1.27)))
-    )
-    (property "Footprint" "" (at 113.03 17.78 0)
-      (effects (font (size 1.27 1.27)) hide)
-    )
-    (property "Datasheet" "~" (at 113.03 17.78 0)
-      (effects (font (size 1.27 1.27)) hide)
-    )
-    (pin "1")
-    (instances
-      (project "DccDecoder2"
-        (path "/68a87a67-79ef-42dd-968e-a1e235d63e5c"
-          (reference "#FLG02") (unit 1)
-        )
-      )
-    )
-  )
   (symbol (lib_id "power:GND") (at 201.93 45.72 0) (unit 1)
     (in_bom yes) (on_board yes) (dnp no)
@@
         )
       )
-    )
-  )
-  (symbol (lib_id "power:PWR_FLAG") (at 113.03 60.96 0) (unit 1)
-    (in_bom yes) (on_board yes) (dnp no)
-    (property "Reference" "#FLG03" (at 113.03 59.055 0)
-      (effects (font (size 1.27 1.27)) hide)
-    )
-    (property "Value" "PWR_FLAG" (at 113.03 57.15 0)
-      (effects (font (size 1.27 1.27)))
-    )
-    (property "Footprint" "" (at 113.03 60.96 0)
-      (effects (font (size 1.27 1.27)) hide)
-    )
-    (property "Datasheet" "~" (at 113.03 60.96 0)
-      (effects (font (size 1.27 1.27)) hide)
-    )
-    (pin "1")
-    (instances
-      (project "DccDecoder2"
-        (path "/68a87a67-79ef-42dd-968e-a1e235d63e5c"
-          (reference "#FLG03") (unit 1)
-        )
-      )
