File: PowerFromDcc/PowerFromDcc.kicad_sch (KiCad schematic)
At the start: 12 parts, among them IC1 AP64060QWU-7, J3 5V

Commit message: 01/12/24 16:56 Titan.local
Parts:
- removed D2: CUHS20F30,H3F, CUHS20F30H3F, symbol CUHS20F30:CUHS20F30,H3F
- added D3: CUHS20F30, Diode_SMD:D_1206_3216Metric, symbol Device:D_Schottky
- added J1: DCC/J, TestPoint:TestPoint_Pad_D2.0mm, symbol Connector:TestPoint
- added J2: DCC/K, TestPoint:TestPoint_Pad_D2.0mm, symbol Connector:TestPoint
- added J5: DCC, TerminalBlock_Phoenix:TerminalBlock_Phoenix_PT-1,5-2-3.5-H_1x02_P3.50mm_Horizontal, symbol Connector:Screw_Terminal_01x02
- J3: footprint TestPoint:TestPoint_Pad_D2.0mm -> DMG2305UX-7.lib
- J4: renamed from JJ4; footprint TestPoint:TestPoint_Pad_D2.0mm -> DMG2305UX-7.mod
- L1: footprint Inductor_SMD_Wurth:L_Wurth_WE-LQSH-3012 -> DMG2305UX-7.kicad_sym
Connections:
- net +V: now also D3.1 (K)
- net at D1.3 (+): now also D3.2 (A)
- net DCC/J: no longer names the net of D1.1
- net DCC/J: now also J1.1, J5.2 (Pin_2)
- net DCC/K: no longer names the net of D1.2
- net DCC/K: now also J2.1, J5.1 (Pin_1)

Commit message: 01/12/24 22:40 Titan.local
Parts:
- J3: footprint DMG2305UX-7.lib -> TestPoint:TestPoint_Pad_D2.0mm
- J4: footprint DMG2305UX-7.mod -> TestPoint:TestPoint_Pad_D2.0mm
- L1: footprint DMG2305UX-7.kicad_sym -> Inductor_SMD_Wurth:L_Wurth_WE-LQSH-4020
Changed lines of the file:
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@@
       (effects (font (size 1.27 1.27)) (justify left))
     )
-    (property "Footprint" "DMG2305UX-7.mod" (at 52.07 74.93 0)
+    (property "Footprint" "TestPoint:TestPoint_Pad_D2.0mm" (at 52.07 74.93 0)
       (effects (font (size 1.27 1.27)) hide)
     )
@@
       (effects (font (size 1.27 1.27)))
     )
-    (property "Footprint" "DMG2305UX-7.kicad_sym" (at 114.3 33.02 0)
+    (property "Footprint" "Inductor_SMD_Wurth:L_Wurth_WE-LQSH-4020" (at 114.3 33.02 0)
       (effects (font (size 1.27 1.27)) hide)
     )
@@
       (effects (font (size 1.27 1.27)) (justify left))
     )
-    (property "Footprint" "DMG2305UX-7.lib" (at 54.61 33.02 0)
+    (property "Footprint" "TestPoint:TestPoint_Pad_D2.0mm" (at 54.61 33.02 0)
       (effects (font (size 1.27 1.27)) hide)
     )

Commit message: 02/12/24 08:43 Titan.local
Parts:
- IC1: footprint SOT95P280X100-6N -> Package_TO_SOT_SMD:SOT-23-6
- L1: footprint Inductor_SMD_Wurth:L_Wurth_WE-LQSH-4020 -> Inductor_SMD_Wurth:L_Wurth_WE-LQSH-2010
Changed lines of the file:
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@@
       (effects (font (size 1.27 1.27)))
     )
-    (property "Footprint" "SOT95P280X100-6N" (at 123.19 141.91 0)
+    (property "Footprint" "Package_TO_SOT_SMD:SOT-23-6" (at 123.19 141.91 0)
       (effects (font (size 1.27 1.27)) (justify left top) hide)
     )
@@
       (effects (font (size 1.27 1.27)))
     )
-    (property "Footprint" "Inductor_SMD_Wurth:L_Wurth_WE-LQSH-4020" (at 114.3 33.02 0)
+    (property "Footprint" "Inductor_SMD_Wurth:L_Wurth_WE-LQSH-2010" (at 114.3 33.02 0)
       (effects (font (size 1.27 1.27)) hide)
     )

Commit message: 04/12/24 19:52 Titan.local
Parts:
- renumbered D3 to D2
Changed lines of the file:
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@@
   (symbol (lib_id "Device:D_Schottky") (at 148.59 52.07 0) (unit 1)
     (in_bom yes) (on_board yes) (dnp no) (fields_autoplaced)
-    (property "Reference" "D3" (at 148.2725 46.99 0)
+    (property "Reference" "D2" (at 148.2725 45.72 0)
       (effects (font (size 1.27 1.27)))
     )
-    (property "Value" "CUHS20F30" (at 148.2725 49.53 0)
+    (property "Value" "CUHS20F30" (at 148.2725 48.26 0)
       (effects (font (size 1.27 1.27)))
     )
@@
       (project "PowerFromDcc"
         (path "/682eb615-157b-497c-a26b-f536ca133095"
-          (reference "D3") (unit 1)
+          (reference "D2") (unit 1)
         )
       )

Commit message: 04/12/24 20:52 Arrakis.local
Parts:
- removed C1: 2.2uF/25V, Capacitor_SMD:C_1206_3216Metric, symbol Device:C
- removed C3: 100n, Capacitor_SMD:C_1206_3216Metric, symbol Device:C
- removed C4: 10uF/6.3V, Capacitor_SMD:C_1206_3216Metric, symbol Device:C
- removed D1: KMB24F, Package_TO_SOT_SMD:TO-269AA, symbol Additional:KMB24F
- removed D2: CUHS20F30, Diode_SMD:D_1206_3216Metric, symbol Device:D_Schottky
- removed J1: DCC/J, TestPoint:TestPoint_Pad_D2.0mm, symbol Connector:TestPoint
- removed J2: DCC/K, TestPoint:TestPoint_Pad_D2.0mm, symbol Connector:TestPoint
- removed J3: 5V, TestPoint:TestPoint_Pad_D2.0mm, symbol Connector:TestPoint
- removed J4: Gnd, TestPoint:TestPoint_Pad_D2.0mm, symbol Connector:TestPoint
- removed J5: DCC, TerminalBlock_Phoenix:TerminalBlock_Phoenix_PT-1,5-2-3.5-H_1x02_P3.50mm_Horizontal, symbol Connector:Screw_Terminal_01x02
- removed R1: 115k, Resistor_SMD:R_1206_3216Metric, symbol Device:R
- removed R2: 22k1, Resistor_SMD:R_1206_3216Metric, symbol Device:R
- added C1: 10u, Capacitor_SMD:C_1206_3216Metric_Pad1.33x1.80mm_HandSolder, symbol Device:C
- added C1: 100n, Capacitor_SMD:C_1206_3216Metric_Pad1.33x1.80mm_HandSolder, symbol Device:C
- added D1: KMB24F, Package_TO_SOT_SMD:TO-269AA, symbol RP2040-Decoder_Additional_Symbols:KMB24F
- added D1: CUHS20F30, CUHS20F30:CUHS20F30H3F, symbol Device:D_Zener
- added J1: DCC, TerminalBlock_Phoenix:TerminalBlock_Phoenix_PT-1,5-2-3.5-H_1x02_P3.50mm_Horizontal, symbol Connector:Screw_Terminal_01x02
- added R1: 115k, Resistor_SMD:R_1206_3216Metric_Pad1.30x1.75mm_HandSolder, symbol Device:R
- added R1: 22k1, Resistor_SMD:R_1206_3216Metric_Pad1.30x1.75mm_HandSolder, symbol Device:R
- C2: value 10uF/6.3V -> 2.2uF/25V; footprint Capacitor_SMD:C_1206_3216Metric -> Capacitor_SMD:C_1206_3216Metric_Pad1.33x1.80mm_HandSolder
- IC1: footprint Package_TO_SOT_SMD:SOT-23-6 -> Package_TO_SOT_SMD:TSOT-23-6
Connections:
- net +V: now also C2.1, D1.1 (K), D1.2 (A), D1.3 (+)
- net GND: now also C1.2, D1.4 (-), R1.1
- net at IC1.1 (BST): now also C1.2
- net at IC1.3 (FB): now also R1.1, R1.2
- net at IC1.6 (SW): now also L1.2, C1.1; no longer L1.1
- removed net +5V: C2.1, L1.2
- new net: D1.1, J1.2 (Pin_2)
- new net: D1.2, J1.1 (Pin_1)
- new net 5V: C1.1, L1.1, R1.2
Other:
- title: DC powerfrom DCC -> (none)

Commit message: 04/12/24 21:07 Titan.local
Changed lines of the file:
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@@
       (project "PowerFromDcc"
         (path "/ce5bbdfd-6719-4170-a6f6-5cd4493cec2b"
-          (reference "D2") (unit 1)
+          (reference "D1") (unit 1)
         )
       )
@@
   (symbol (lib_id "Device:D_Zener") (at 111.76 41.91 0) (unit 1)
     (in_bom yes) (on_board yes) (dnp no) (fields_autoplaced)
-    (property "Reference" "D1" (at 111.76 36.83 0)
-      (effects (font (size 1.27 1.27)))
-    )
-    (property "Value" "CUHS20F30" (at 111.76 39.37 0)
+    (property "Reference" "D1" (at 111.76 35.56 0)
+      (effects (font (size 1.27 1.27)))
+    )
+    (property "Value" "CUHS20F30" (at 111.76 38.1 0)
       (effects (font (size 1.27 1.27)))
     )
@@
       (project "PowerFromDcc"
         (path "/ce5bbdfd-6719-4170-a6f6-5cd4493cec2b"
-          (reference "D1") (unit 1)
-        )
-      )
+          (reference "D2") (unit 1)
+        )
+      )

Commit message: 04/12/24 22:17 Titan.local
Parts:
- added J3: 5V, TestPoint:TestPoint_Pad_D2.0mm, symbol Connector:TestPoint
- added j2: Gnd, TestPoint:TestPoint_Pad_D2.0mm, symbol Connector:TestPoint
- added j4: +V, TestPoint:TestPoint_Pad_D2.0mm, symbol Connector:TestPoint
Connections:
- net +V: now also j4.1; no longer D1.2 (A), D1.3 (+)
- net 5V: now also J3.1
- net GND: now also j2.1
- new net VP: D1.2 (A), D1.3 (+)

Commit message: 05/12/24 09:43 Titan.local
Changed lines of the file:
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@@
 (kicad_sch (version 20230121) (generator eeschema)
   (paper "A4")
-  (junction (at 67.31 60.96) (diameter 0) (color 0 0 0 0)
-  )
   (junction (at 63.5 45.72) (diameter 0) (color 0 0 0 0)
   )
@@
   (junction (at 101.6 45.72) (diameter 0) (color 0 0 0 0)
   )
+  (junction (at 81.28 60.96) (diameter 0) (color 0 0 0 0)
+  )
   (junction (at 104.14 45.72) (diameter 0) (color 0 0 0 0)
   )
@@
   (junction (at 107.95 45.72) (diameter 0) (color 0 0 0 0)
   )
+  (wire (pts (xy 81.28 60.96) (xy 113.03 60.96))
+    (stroke (width 0) (type default))
+  )
   (wire (pts (xy 76.2 40.64) (xy 76.2 39.37))
     (stroke (width 0) (type default))
@@
     (stroke (width 0) (type default))
   )
+  (wire (pts (xy 81.28 60.96) (xy 81.28 63.5))
+    (stroke (width 0) (type default))
+  )
   (wire (pts (xy 63.5 57.15) (xy 63.5 60.96))
     (stroke (width 0) (type default))
@@
     (stroke (width 0) (type default))
   )
-  (wire (pts (xy 67.31 60.96) (xy 67.31 62.23))
-    (stroke (width 0) (type default))
-  )
   (wire (pts (xy 57.15 36.83) (xy 57.15 50.8))
     (stroke (width 0) (type default))
@@
     (stroke (width 0) (type default))
   )
-  (wire (pts (xy 63.5 60.96) (xy 67.31 60.96))
+  (wire (pts (xy 63.5 60.96) (xy 72.39 60.96))
     (stroke (width 0) (type default))
   )
@@
     (stroke (width 0) (type default))
   )
-  (wire (pts (xy 72.39 60.96) (xy 113.03 60.96))
+  (wire (pts (xy 72.39 60.96) (xy 81.28 60.96))
     (stroke (width 0) (type default))
   )
@@
   )
   (wire (pts (xy 101.6 45.72) (xy 104.14 45.72))
-    (stroke (width 0) (type default))
-  )
-  (wire (pts (xy 67.31 60.96) (xy 72.39 60.96))
     (stroke (width 0) (type default))
   )
@@
     )
   )
+  (symbol (lib_id "power:GND") (at 81.28 63.5 0) (unit 1)
+    (in_bom yes) (on_board yes) (dnp no) (fields_autoplaced)
+    (property "Reference" "#PWR01" (at 81.28 69.85 0)
+      (effects (font (size 1.27 1.27)) hide)
+    )
+    (property "Value" "GND" (at 81.28 68.58 0)
+      (effects (font (size 1.27 1.27)))
+    )
+    (property "Footprint" "" (at 81.28 63.5 0)
+      (effects (font (size 1.27 1.27)) hide)
+    )
+    (property "Datasheet" "" (at 81.28 63.5 0)
+      (effects (font (size 1.27 1.27)) hide)
+    )
+    (pin "1")
+    (instances
+      (project "PowerFromDcc"
+        (path "/ce5bbdfd-6719-4170-a6f6-5cd4493cec2b"
+          (reference "#PWR01") (unit 1)
+        )
+      )
+    )
+  )
   (symbol (lib_id "Connector:TestPoint") (at 53.34 36.83 0) (unit 1)
     (in_bom yes) (on_board yes) (dnp no)
@@
         )
       )
-    )
-  )
-  (symbol (lib_id "power:GND") (at 67.31 62.23 0) (unit 1)
-    (in_bom yes) (on_board yes) (dnp no)
-    (property "Reference" "#PWR03" (at 67.31 68.58 0)
-      (effects (font (size 1.27 1.27)) hide)
-    )
-    (property "Value" "GND" (at 67.31 67.31 0)
-      (effects (font (size 1.27 1.27)))
-    )
-    (property "Footprint" "" (at 67.31 62.23 0)
-      (effects (font (size 1.27 1.27)) hide)
-    )
-    (property "Datasheet" "" (at 67.31 62.23 0)
-      (effects (font (size 1.27 1.27)) hide)
-    )
-    (pin "1")
-    (instances
-      (project "RP2040-Decoder"
-        (path "/11d18738-0f49-4d63-b61c-22a93efd5959"
-          (reference "#PWR03") (unit 1)
-        )
-      )
-      (project "DccDecoder2"
-        (path "/68a87a67-79ef-42dd-968e-a1e235d63e5c"
-          (reference "#PWR01") (unit 1)
-        )
-      )
-      (project "PowerFromDcc"
-        (path "/ce5bbdfd-6719-4170-a6f6-5cd4493cec2b"
-          (reference "#PWR01") (unit 1)
-        )
-      )
