File: DccDecoder3/DccDecoder3.kicad_pcb (KiCad board)
At the start: 2 copper layers, 94 x 35.6 mm, 34 parts, among them J1 DCC, J2 0, J3 1, J4 2, J5 3, J6 +V, J7 M_OUT_B, J8 M_OUT_A, J9 GND, Q1 T2N7002BK, Q2 T2N7002BK, Q3 T2N7002BK, Q4 T2N7002BK, Q5 T2N7002BK, Q6 DMG2305UX-7, SW1 SW_Push, U1 Pico, U2 BDR6133, U3 AP7384-33Y

Commit message: 19/01/25 19:37 Arrakis.local
Parts:
- added Q1: 2N7002K, Package_TO_SOT_SMD:SOT-23_Handsoldering, B.Cu at (151.4, 60.0)
- added Q2: 2N7002K, Package_TO_SOT_SMD:SOT-23_Handsoldering, B.Cu at (151.4, 61.9)
- added Q4: 2N7002K, Package_TO_SOT_SMD:SOT-23_Handsoldering, B.Cu at (151.4, 71.0)
- Q3, Q5: value T2N7002BK -> 2N7002K; footprint Package_TO_SOT_SMD:SOT-23 -> Package_TO_SOT_SMD:SOT-23_Handsoldering; moved to B.Cu
- moved Q5 17.4 mm to (151.4, 75.6), turned to 180 degrees
- moved Q3 5.95 mm to (151.4, 67.0), turned to 180 degrees
- turned U1 to -90 degrees
Connections:
- Q3 pad 1: /GPIO17 -> /GPIO18
- Q3 pad 3: Net-(J3-Pin_1) -> Net-(J4-Pin_1)
- Q5 pad 1: /GPIO19 -> /GPIO16
- Q5 pad 3: Net-(J5-Pin_1) -> Net-(J2-Pin_1)
Routing:
- net GND: track 225.1 -> 0.00 mm, vias 1 -> 0
- net /MOTOR_OUT_B: track 73.7 -> 0.00 mm, vias 2 -> 0
- net /MOTOR_OUT_A: track 72.3 -> 0.00 mm, vias 3 -> 0
- net /GPIO15: track 69.5 -> 0.00 mm
- net /ADC_EMF_A: track 68.8 -> 0.00 mm, vias 2 -> 0
- net /GPIO14: track 64.6 -> 0.00 mm
- net /GPIO21: track 62.4 -> 0.00 mm
- net /ADC_EMF_B: track 49.6 -> 0.00 mm, vias 2 -> 0
- net /GPIO18: track 49.6 -> 0.00 mm, vias 1 -> 0
- net Net-(U3-VO): track 44.4 -> 0.00 mm, vias 3 -> 0
- net /GPIO17: track 43.1 -> 0.00 mm
- net Net-(D1-A): track 42.8 -> 0.00 mm, vias 1 -> 0
- net /GPIO16: track 39.6 -> 0.00 mm
- net +V: track 37.2 -> 0.00 mm
- net Net-(D1-K): track 32.9 -> 0.00 mm
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Other:
- board size 94 x 35.6 mm -> 94 x 50.8 mm

Commit message: 19/01/25 22:12 Titan.local
Parts:
- removed the Q1 at (174.9, 72.1)
- removed the Q2 at (141.3, 68.6)
- removed the Q4 at (148.3, 69.5)
- moved J1 93.3 mm to (98.4, 68.6)
- moved D1 78.2 mm to (109.2, 60.3)
- moved D4 76.4 mm to (109.2, 71.8)
- moved D3 74.4 mm to (109.2, 67.9)
- moved D2 74.3 mm to (109.2, 64.1)
- moved U3 55.5 mm to (120.7, 61.0)
- moved SW1 32.4 mm to (135.3, 41.3)
- moved Q1 26.7 mm to (129.9, 75.9)
- moved U2 25.4 mm to (141.7, 62.2)
- moved U1 24.1 mm to (128.9, 41.9)
- moved J5 20.9 mm to (150.5, 71.1)
- moved J4 19.4 mm to (150.5, 67.5)
- moved J9 17.7 mm to (143.5, 69.8)
- moved J2 17.3 mm to (150.5, 59.7)
- moved J3 15.4 mm to (150.5, 63.5)
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
Commit message: 20/01/25 13:14 Arrakis.local
Parts:
- removed the R1 at (167.9, 53.3)
- removed the R2 at (160.9, 53.3)
- added J2: PAD, TestPoint:TestPoint_Pad_2.5x2.5mm, F.Cu at (101.6, 66.0)
- J1: value DCC -> PAD; footprint TerminalBlock_Phoenix:TerminalBlock_Phoenix_PT-1,5-2-3.5-H_1x02_P3.50mm_Horizontal -> TestPoint:TestPoint_Pad_2.5x2.5mm
- J10: renamed from J9; footprint TestPoint:TestPoint_Pad_D2.0mm -> TestPoint:TestPoint_Pad_2.5x2.5mm
- J3: renamed from J2; footprint TestPoint:TestPoint_Pad_D2.0mm -> TestPoint:TestPoint_Pad_2.5x2.5mm
- J4: renamed from J3; footprint TestPoint:TestPoint_Pad_D2.0mm -> TestPoint:TestPoint_Pad_2.5x2.5mm
- J5: renamed from J4; footprint TestPoint:TestPoint_Pad_D2.0mm -> TestPoint:TestPoint_Pad_2.5x2.5mm
- J6: renamed from J5; footprint TestPoint:TestPoint_Pad_D2.0mm -> TestPoint:TestPoint_Pad_2.5x2.5mm
- J7: renamed from J6; footprint TestPoint:TestPoint_Pad_D2.0mm -> TestPoint:TestPoint_Pad_2.5x2.5mm
- J8: renamed from J7; footprint TestPoint:TestPoint_Pad_D2.0mm -> TestPoint:TestPoint_Pad_2.5x2.5mm
- J9: renamed from J8; footprint TestPoint:TestPoint_Pad_D2.0mm -> TestPoint:TestPoint_Pad_2.5x2.5mm
- Q1: renamed from Q6; moved to B.Cu
- R1: renamed from R3; footprint Resistor_SMD:R_1206_3216Metric_Pad1.30x1.75mm_HandSolder -> Resistor_SMD:R_0805_2012Metric_Pad1.20x1.40mm_HandSolder; moved to B.Cu
- R2: renamed from R4; footprint Resistor_SMD:R_1206_3216Metric_Pad1.30x1.75mm_HandSolder -> Resistor_SMD:R_0805_2012Metric_Pad1.20x1.40mm_HandSolder; moved to B.Cu
- R3: renamed from R5; footprint Resistor_SMD:R_1206_3216Metric_Pad1.30x1.75mm_HandSolder -> Resistor_SMD:R_0805_2012Metric_Pad1.20x1.40mm_HandSolder; moved to B.Cu
- R4: renamed from R6; footprint Resistor_SMD:R_1206_3216Metric_Pad1.30x1.75mm_HandSolder -> Resistor_SMD:R_0805_2012Metric_Pad1.20x1.40mm_HandSolder; moved to B.Cu
- R5: renamed from R7; footprint Resistor_SMD:R_1206_3216Metric_Pad1.30x1.75mm_HandSolder -> Resistor_SMD:R_0805_2012Metric_Pad1.20x1.40mm_HandSolder; moved to B.Cu
- R6: renamed from R8; footprint Resistor_SMD:R_1206_3216Metric_Pad1.30x1.75mm_HandSolder -> Resistor_SMD:R_0805_2012Metric_Pad1.20x1.40mm_HandSolder; moved to B.Cu
- moved C1 74.8 mm to (101.6, 71.1), turned to -90 degrees
- moved C3 57.8 mm to (116.8, 62.2), turned to 90 degrees
- moved Q1 57.0 mm to (105.4, 68.6), turned to 180 degrees
- moved R1 53.1 mm to (108.0, 64.8), turned to 180 degrees
- moved C2 52.9 mm to (121.9, 62.2), turned to 90 degrees
- moved R2 46.9 mm to (114.3, 64.8), turned to 180 degrees
- moved R5 46.8 mm to (121.9, 68.6), turned to 180 degrees
- moved R3 45.5 mm to (122.2, 64.8), turned to 180 degrees
- moved R4 42.7 mm to (128.3, 68.6), turned to 180 degrees
- moved R6 39.6 mm to (128.3, 64.8), turned to 180 degrees
- moved SW1 30.4 mm to (141.0, 71.1)
- moved U2 24.3 mm to (125.7, 66.0)
- moved Q2 18.2 mm to (113.3, 68.6)
- moved U1 10.2 mm to (119.4, 71.1), turned to 180 degrees
- moved J7 9.86 mm to (129.5, 72.4)
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- renumbered C3 to C1, C1 to C2, C2 to C3, D3 to D2, D4 to D3, D2 to D4, Q1 to Q2, Q5 to Q3, Q2 to Q4, Q3 to Q5, Q4 to Q6, U3 to U1, U1 to U2, U2 to U3
Connections:
- C1 pad 1: Net-(U3-VO) -> +3V3
- C2 pad 1: Net-(D1-K) -> +V
- C3 pad 1: Net-(D1-K) -> +V
- D1 pad 1: Net-(D1-K) -> +V
- D3 pad 1: Net-(D2-A) -> Net-(D3-K)
- D4 pad 1: Net-(D1-K) -> +V
- D4 pad 2: Net-(D2-A) -> Net-(D3-K)
- J1 pad 1: Net-(D2-A) -> Net-(D1-A)
- Q1 pad 3: Net-(U3-VO) -> +3V3
- U1 pad 1: Net-(U3-VO) -> +3V3
- U1 pad 3: Net-(D1-K) -> +V
Routing:
- net GND: track 0.00 -> 145.0 mm, vias 0 -> 2
- net +3V3: track 0.00 -> 66.7 mm, vias 0 -> 2
- net +V: track 0.00 -> 48.9 mm
- net /GPIO21: track 0.00 -> 32.7 mm
- net /MOTOR_OUT_A: track 0.00 -> 28.8 mm, vias 0 -> 2
- net Net-(D1-A): track 0.00 -> 22.6 mm, vias 0 -> 1
- net /MOTOR_OUT_B: track 0.00 -> 22.1 mm, vias 0 -> 1
- net /GPIO18: track 0.00 -> 20.4 mm
- net /ADC_EMF_A: track 0.00 -> 18.1 mm
- net Net-(D3-K): track 0.00 -> 18.0 mm
- net /GPIO15: track 0.00 -> 15.9 mm
- net Net-(U2-RUN): track 0.00 -> 15.8 mm
- net Net-(J3-Pin_1): track 0.00 -> 15.2 mm, vias 0 -> 1
- net /ADC_EMF_B: track 0.00 -> 12.7 mm
- net /GPIO14: track 0.00 -> 9.90 mm
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Other:
- board size 94 x 50.8 mm -> 94 x 55.9 mm

Commit message: 20/01/25 13:46 Titan.local
Parts:
- U2: value Pico -> Pico_RaspberryPico; footprint MCU_RaspberryPi_and_Boards:RP2040Pico -> PicoNoSwd:RaspberryPico_TH_NoSWD
- moved U2 26.3 mm to (101.0, 57.1)
- moved SW1 4.49 mm to (137.8, 67.9), turned to 0 degrees
- moved Q6 3.82 mm to (147.6, 67.9)
- moved Q4 3.81 mm to (147.6, 60.0)
- moved Q5 3.81 mm to (147.6, 64.1)
- moved Q3 3.65 mm to (147.7, 71.8)
- moved J3 3.24 mm to (147.3, 60.3)
- moved J5 3.18 mm to (147.3, 67.3)
- moved J4 3.18 mm to (147.3, 63.5)
- moved J6 3.18 mm to (147.3, 71.1)
- moved C1 0.64 mm to (101.6, 70.5), turned to 90 degrees
Connections:
- Q1 pad 1: unconnected-(Q1-Pad1) -> Net-(U2-VBUS)
- U2 pad 23: GND -> unconnected-(U2-GND-Pad23)
- U2 pad 3: unconnected-(U2-GND-Pad3) -> GND
- U2 pad 40: unconnected-(Q1-Pad1) -> Net-(U2-VBUS)
Routing:
- net GND: track 145.0 -> 0.00 mm, vias 2 -> 0
- net +3V3: track 66.7 -> 0.00 mm, vias 2 -> 0
- net +V: track 48.9 -> 0.00 mm
- net /GPIO21: track 32.7 -> 0.00 mm
- net /MOTOR_OUT_A: track 28.8 -> 0.00 mm, vias 2 -> 0
- net Net-(D1-A): track 22.6 -> 0.00 mm, vias 1 -> 0
- net /MOTOR_OUT_B: track 22.1 -> 0.00 mm, vias 1 -> 0
- net /GPIO18: track 20.4 -> 0.00 mm
- net /ADC_EMF_A: track 18.1 -> 0.00 mm
- net Net-(D3-K): track 18.0 -> 0.00 mm
- net /GPIO15: track 15.9 -> 0.00 mm
- net Net-(U2-RUN): track 15.8 -> 0.00 mm
- net Net-(J3-Pin_1): track 15.2 -> 0.00 mm, vias 1 -> 0
- net /ADC_EMF_B: track 12.7 -> 0.00 mm
- net /GPIO14: track 9.90 -> 0.00 mm
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
Commit message: 20/01/25 19:41 Arrakis.local
Parts:
- Q1, Q2: moved to F.Cu
- SW1: moved to B.Cu
- moved Q1 24.1 mm to (128.3, 61.0), turned to 0 degrees
- moved Q2 15.2 mm to (128.3, 66.0), turned to 0 degrees
- moved J7 13.7 mm to (142.2, 67.3)
- moved SW1 10.0 mm to (128.3, 71.1)
- moved J8 9.92 mm to (137.2, 67.3)
- moved J9 9.16 mm to (137.2, 71.1)
- moved J10 7.73 mm to (142.2, 71.1)
- moved D2 7.62 mm to (109.2, 60.3)
- moved D1 3.81 mm to (109.2, 64.1), turned to 180 degrees
- moved D4 3.81 mm to (109.2, 67.9), turned to 180 degrees
- moved R4 1.27 mm to (128.3, 67.3)
- moved U3 1.14 mm to (139.0, 62.2)
- moved J4 0.64 mm to (147.3, 64.1)
- moved U2 0.64 mm to (100.3, 57.1)
- moved J5 0.63 mm to (147.3, 67.9)
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Routing:
- net GND: track 0.00 -> 159.9 mm
- net +V: track 0.00 -> 61.9 mm, vias 0 -> 2
- net +3V3: track 0.00 -> 53.4 mm, vias 0 -> 2
- net /MOTOR_OUT_B: track 0.00 -> 46.6 mm, vias 0 -> 1
- net Net-(U2-VBUS): track 0.00 -> 38.1 mm, vias 0 -> 1
- net /VSYS: track 0.00 -> 34.1 mm, vias 0 -> 1
- net Net-(J3-Pin_1): track 0.00 -> 26.0 mm, vias 0 -> 1
- net /GPIO17: track 0.00 -> 24.5 mm
- net /MOTOR_OUT_A: track 0.00 -> 21.6 mm, vias 0 -> 1
- net Net-(J4-Pin_1): track 0.00 -> 19.0 mm, vias 0 -> 1
- net /ADC_EMF_A: track 0.00 -> 18.7 mm
- net Net-(Q2-G): track 0.00 -> 18.6 mm, vias 0 -> 1
- net /GPIO19: track 0.00 -> 18.5 mm
- net /GPIO18: track 0.00 -> 17.4 mm
- net Net-(D1-A): track 0.00 -> 13.8 mm, vias 0 -> 1
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Other:
- board size 94 x 55.9 mm -> 54.6 x 24.8 mm

Commit message: 20/01/25 20:01 Titan.local
Routing:
- net /MOTOR_OUT_B: track 46.6 -> 48.3 mm
Changed lines of the file:
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@@
     (property "ki_keywords" "R res resistor")
     (attr smd)
-    (fp_text reference "R4" (at 0 1.65) (layer "B.SilkS")
+    (fp_text reference "R4" (at -2.54 1.27) (layer "B.SilkS")
         (effects (font (size 1 1) (thickness 0.15)) (justify mirror))
     )
@@
     (style (thickness 0.15) (arrow_length 1.27) (text_position_mode 0) (extension_height 0.58642) (extension_offset 0.5) keep_text_aligned)
   )
+  (segment (start 130.8068 61.5425) (end 130.2243 60.96) (width 0.3048) (layer "F.Cu") (net 1))
+  (segment (start 106.5731 73.5531) (end 106.68 73.66) (width 0.3048) (layer "F.Cu") (net 1))
+  (segment (start 106.68 73.66) (end 106.68 75.7478) (width 0.3048) (layer "F.Cu") (net 1))
+  (segment (start 101.6 72.0475) (end 103.1056 73.5531) (width 0.3048) (layer "F.Cu") (net 1))
+  (segment (start 132.29 61.595) (end 132.2375 61.5425) (width 0.3048) (layer "F.Cu") (net 1))
+  (segment (start 114.3 74.1163) (end 115.7963 72.62) (width 0.3048) (layer "F.Cu") (net 1))
+  (segment (start 106.68 75.7478) (end 107.2612 76.329) (width 0.3048) (layer "F.Cu") (net 1))
+  (segment (start 129.32 60.96) (end 130.2243 60.96) (width 0.3048) (layer "F.Cu") (net 1))
   (segment (start 114.3 75.738) (end 114.3 74.1163) (width 0.3048) (layer "F.Cu") (net 1))
-  (segment (start 130.8068 61.5425) (end 130.2243 60.96) (width 0.3048) (layer "F.Cu") (net 1))
-  (segment (start 132.29 61.595) (end 132.2375 61.5425) (width 0.3048) (layer "F.Cu") (net 1))
-  (segment (start 106.0949 73.5531) (end 106.68 74.1382) (width 0.3048) (layer "F.Cu") (net 1))
-  (segment (start 129.32 60.96) (end 130.2243 60.96) (width 0.3048) (layer "F.Cu") (net 1))
-  (segment (start 106.68 75.7478) (end 107.2612 76.329) (width 0.3048) (layer "F.Cu") (net 1))
-  (segment (start 106.68 74.1382) (end 106.68 75.7478) (width 0.3048) (layer "F.Cu") (net 1))
   (segment (start 132.2375 61.5425) (end 130.8068 61.5425) (width 0.3048) (layer "F.Cu") (net 1))
   (segment (start 115.7963 72.62) (end 121.83 72.62) (width 0.3048) (layer "F.Cu") (net 1))
-  (segment (start 103.1056 73.5531) (end 106.0949 73.5531) (width 0.3048) (layer "F.Cu") (net 1))
   (segment (start 121.83 72.62) (end 127.3098 72.62) (width 0.3048) (layer "F.Cu") (net 1))
   (segment (start 127.3098 72.62) (end 129.9795 69.9503) (width 0.3048) (layer "F.Cu") (net 1))
+  (segment (start 113.709 76.329) (end 114.3 75.738) (width 0.3048) (layer "F.Cu") (net 1))
   (segment (start 136.525 61.595) (end 132.29 61.595) (width 0.3048) (layer "F.Cu") (net 1))
-  (segment (start 101.6 72.0475) (end 103.1056 73.5531) (width 0.3048) (layer "F.Cu") (net 1))
-  (segment (start 114.3 74.1163) (end 115.7963 72.62) (width 0.3048) (layer "F.Cu") (net 1))
+  (segment (start 103.1056 73.5531) (end 106.5731 73.5531) (width 0.3048) (layer "F.Cu") (net 1))
   (segment (start 107.2612 76.329) (end 113.709 76.329) (width 0.3048) (layer "F.Cu") (net 1))
-  (segment (start 113.709 76.329) (end 114.3 75.738) (width 0.3048) (layer "F.Cu") (net 1))
   (segment (start 129.9795 69.9503) (end 132.6502 69.9503) (width 0.3048) (layer "F.Cu") (net 1))
   (via (at 132.2375 61.5425) (size 0.8) (drill 0.4) (layers "F.Cu" "B.Cu") (net 1))
@@
   (segment (start 143.9043 65.9732) (end 143.9043 72.5322) (width 0.3048) (layer "F.Cu") (net 8))
   (segment (start 137.16 71.12) (end 138.7643 71.12) (width 0.3048) (layer "F.Cu") (net 8))
-  (segment (start 137.16 71.12) (end 135.5557 71.12) (width 0.3048) (layer "F.Cu") (net 8))
-  (segment (start 135.5557 71.12) (end 129.9394 71.12) (width 0.3048) (layer "F.Cu") (net 8))
+  (segment (start 134.62 71.12) (end 135.5557 71.12) (width 0.3048) (layer "F.Cu") (net 8))
   (segment (start 142.0661 64.135) (end 143.9043 65.9732) (width 0.3048) (layer "F.Cu") (net 8))
+  (segment (start 135.5557 71.12) (end 137.16 71.12) (width 0.3048) (layer "F.Cu") (net 8))
   (segment (start 141.475 64.135) (end 142.0661 64.135) (width 0.3048) (layer "F.Cu") (net 8))
   (segment (start 143.7122 72.7243) (end 140.3686 72.7243) (width 0.3048) (layer "F.Cu") (net 8))
   (segment (start 143.9043 72.5322) (end 143.7122 72.7243) (width 0.3048) (layer "F.Cu") (net 8))
-  (via (at 129.9394 71.12) (size 0.8) (drill 0.4) (layers "F.Cu" "B.Cu") (net 8))
-  (segment (start 120.4424 76.8574) (end 125.8806 76.8574) (width 0.3048) (layer "B.Cu") (net 8))
-  (segment (start 125.8806 76.8574) (end 127 75.738) (width 0.3048) (layer "B.Cu") (net 8))
-  (segment (start 119.4942 75.9092) (end 120.4424 76.8574) (width 0.3048) (layer "B.Cu") (net 8))
-  (segment (start 127 74.0594) (end 129.9394 71.12) (width 0.3048) (layer "B.Cu") (net 8))
-  (segment (start 119.4942 70.0058) (end 119.4942 75.9092) (width 0.3048) (layer "B.Cu") (net 8))
-  (segment (start 120.92 68.58) (end 119.4942 70.0058) (width 0.3048) (layer "B.Cu") (net 8))
-  (segment (start 127 75.738) (end 127 74.0594) (width 0.3048) (layer "B.Cu") (net 8))
+  (via (at 134.62 71.12) (size 0.8) (drill 0.4) (layers "F.Cu" "B.Cu") (net 8))
+  (segment (start 134.62 71.12) (end 134.62 75.724054) (width 0.3048) (layer "B.Cu") (net 8))
+  (segment (start 120.4424 76.8574) (end 119.4942 75.9092) (width 0.3048) (layer "B.Cu") (net 8))
+  (segment (start 119.4942 70.0058) (end 120.92 68.58) (width 0.3048) (layer "B.Cu") (net 8))
+  (segment (start 119.4942 75.9092) (end 119.4942 70.0058) (width 0.3048) (layer "B.Cu") (net 8))
+  (segment (start 133.486654 76.8574) (end 120.4424 76.8574) (width 0.3048) (layer "B.Cu") (net 8))
+  (segment (start 134.62 75.724054) (end 133.486654 76.8574) (width 0.3048) (layer "B.Cu") (net 8))
   (segment (start 101.6 66.04) (end 104.815 66.04) (width 0.3048) (layer "F.Cu") (net 9))
   (segment (start 106.72 71.755) (end 106.72 67.945) (width 0.3048) (layer "F.Cu") (net 9))
