File: DccDecoder3/DccDecoder3.kicad_sch (KiCad schematic)
At the start: 32 parts, among them J1 DCC, J14 +V, J15 M_OUT_B, J16 M_OUT_A, J17 GND, J3 0, J4 1, J5 2, J6 3, Q1 T2N7002BK, Q2 T2N7002BK, Q3 T2N7002BK, Q4 T2N7002BK, Q5 T2N7002BK, Q6 DMG2305UX-7, SW1 SW_Push, U1 Pico, U2 BDR6133, U3 AP7384-33Y

Commit message: 19/01/25 19:37 Arrakis.local
Parts:
- removed Q1, Q2, Q3, Q4, Q5: T2N7002BK, Package_TO_SOT_SMD:SOT-23, symbol RP2040-Decoder_Additional_Symbols:T2N7002BK
- added Q1, Q2, Q3, Q4, Q5: 2N7002K, Package_TO_SOT_SMD:SOT-23_Handsoldering, symbol Transistor_FET:2N7002K
Connections:
- net GND: now also Q1.2 (S), Q2.2 (S), Q3.2 (S), Q4.2 (S), Q5.2 (S)
- net GPIO16: now also Q5.1 (G)
- net GPIO17: now also Q2.1 (G)
- net GPIO18: now also Q3.1 (G)
- net GPIO19: now also Q4.1 (G)
- net GPIO21: now also Q1.3 (D)
- net at R1.1, R2.2: now also Q1.1 (G)
- net at J5.1 (Pin_1): now also Q3.3 (D)
- net at J3.1 (Pin_1): now also Q5.3 (D)
- net at J6.1 (Pin_1): now also Q4.3 (D)
- net at J4.1 (Pin_1): now also Q2.3 (D)

Commit message: 20/01/25 13:14 Arrakis.local
Parts:
- removed J1: DCC, TerminalBlock_Phoenix:TerminalBlock_Phoenix_PT-1,5-2-3.5-H_1x02_P3.50mm_Horizontal, symbol Connector:Screw_Terminal_01x02
- added J1, J2: PAD, TestPoint:TestPoint_Pad_2.5x2.5mm, symbol Connector:Conn_01x01_Pin
- J14, J15, J16, J17, J3, J4, J5, J6: footprint TestPoint:TestPoint_Pad_D2.0mm -> TestPoint:TestPoint_Pad_2.5x2.5mm
- R1, R2, R5, R6, R7, R8: footprint Resistor_SMD:R_1206_3216Metric_Pad1.30x1.75mm_HandSolder -> Resistor_SMD:R_0805_2012Metric_Pad1.20x1.40mm_HandSolder
- renumbered C3 to C1, C1 to C2, C2 to C3, D3 to D2, D4 to D3, D2 to D4, Q6 to Q1, Q1 to Q2, Q5 to Q3, Q2 to Q4, Q3 to Q5, Q4 to Q6, U3 to U1, U1 to U2
Connections:
- net +3V3: now also C1.1, Q1.3, U1.1 (VO)
- net +V: now also C2.1, C3.1, D1.1 (K), D4.1 (K), U1.3 (VI)
- net at D3.1 (K), D4.2 (A): now also J2.1 (Pin_1)
- net at D1.2 (A), D2.1 (K), R1.2: now also J1.1 (Pin_1)
Other:
- note added: "Other possible diodes B340LA-13-F"
- note added: "Size 2412 Vishay 593D106X9025C2TE3"

Commit message: 20/01/25 13:46 Titan.local
Parts:
- removed U2: Pico, MCU_RaspberryPi_and_Boards:RP2040Pico, symbol MCU_RaspberryPi_and_Boards:Pico
- added U2: Pico_RaspberryPico, PicoNoSwd:RaspberryPico_TH_NoSWD, symbol PicoNoSwd:RaspberryPico-Pico
Connections:
- net ADC_EMF_A: now also U2.31 (GPIO26)
- net ADC_EMF_B: now also U2.32 (GPIO27)
- net GND: now also U2.3 (GND)
- net GPIO14: now also U2.19 (GPIO14)
- net GPIO15: now also U2.20 (GPIO15)
- net GPIO16: now also U2.21 (GPIO16)
- net GPIO17: now also U2.22 (GPIO17)
- net GPIO18: now also U2.24 (GPIO18)
- net GPIO19: now also U2.25 (GPIO19)
- net GPIO21: now also U2.27 (GPIO21)
- net VSYS: now also U2.39 (VSYS)
- net at SW1.1: now also U2.30 (RUN)
- net at Q1.1: now also U2.40 (VBUS)
- no-connect marks 32 -> 27
Other:
- moved on the sheet: SW1

Commit message: 20/01/25 19:41 Arrakis.local
Other:
- title: Pico DCC Decoder -  -> Pico DCC Decoder - Duaghter board
Changed lines of the file:
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@@
   (paper "A4")
   (title_block
-    (title "Pico DCC Decoder - ")
+    (title "Pico DCC Decoder - Duaghter board")
     (date "2024-10-26")
     (rev "3.0")
