File: DccDecoder4/DCCDecoder4/DCCDecoder4.kicad_pcb (KiCad board)
At the start: 2 copper layers, 52 x 25 mm, 0 parts

Commit message: 20/01/25 21:44 Titan.local
Parts:
- added C1: 10uf/16V, Capacitor_SMD:C_1206_3216Metric_Pad1.33x1.80mm_HandSolder, F.Cu at (40.1, 23.9)
- added C2: 10uF/25V, Capacitor_Tantalum_SMD:CP_EIA-6032-20_AVX-F_Pad2.25x2.35mm_HandSolder, F.Cu at (37.3, 42.8)
- added C3: 10uF/25v, Capacitor_Tantalum_SMD:CP_EIA-6032-20_AVX-F_Pad2.25x2.35mm_HandSolder, F.Cu at (37.3, 47.6)
- added D1: RBR3L60AD, Diode_SMD:D_SMA_Handsoldering, F.Cu at (27.3, 24.5)
- added D2: RBR3L60AD, Diode_SMD:D_SMA_Handsoldering, F.Cu at (27.3, 29.1)
- added D3: RBR3L60AD, Diode_SMD:D_SMA_Handsoldering, F.Cu at (27.3, 33.6)
- added D4: RBR3L60AD, Diode_SMD:D_SMA_Handsoldering, F.Cu at (27.3, 38.2)
- added J1: PAD, TestPoint:TestPoint_Pad_2.5x2.5mm, F.Cu at (24.5, 1.77)
- added J10: GND, TestPoint:TestPoint_Pad_2.5x2.5mm, F.Cu at (29.0, 20.0)
- added J2: PAD, TestPoint:TestPoint_Pad_2.5x2.5mm, F.Cu at (24.5, 6.33)
- added J3: 0, TestPoint:TestPoint_Pad_2.5x2.5mm, F.Cu at (24.5, 10.9)
- added J4: 1, TestPoint:TestPoint_Pad_2.5x2.5mm, F.Cu at (24.5, 15.4)
- added J5: 2, TestPoint:TestPoint_Pad_2.5x2.5mm, F.Cu at (24.5, 20.0)
- added J6: 3, TestPoint:TestPoint_Pad_2.5x2.5mm, F.Cu at (29.0, 1.77)
- added J7: +V, TestPoint:TestPoint_Pad_2.5x2.5mm, F.Cu at (29.0, 6.33)
- added J8: M_OUT_B, TestPoint:TestPoint_Pad_2.5x2.5mm, F.Cu at (29.0, 10.9)
- added J9: M_OUT_A, TestPoint:TestPoint_Pad_2.5x2.5mm, F.Cu at (29.0, 15.4)
- added Q1: DMG2305UX-7, DMG2305UX-7:SOT96P240X110-3N, F.Cu at (39.4, 27.9)
- added Q2: 2N7002K, Package_TO_SOT_SMD:SOT-23_Handsoldering, F.Cu at (34.5, 1.77)
- added Q3: 2N7002K, Package_TO_SOT_SMD:SOT-23_Handsoldering, F.Cu at (34.5, 6.33)
- added Q4: 2N7002K, Package_TO_SOT_SMD:SOT-23_Handsoldering, F.Cu at (34.5, 10.9)
- added Q5: 2N7002K, Package_TO_SOT_SMD:SOT-23_Handsoldering, F.Cu at (34.5, 15.4)
- added Q6: 2N7002K, Package_TO_SOT_SMD:SOT-23_Handsoldering, F.Cu at (34.5, 20.0)
- added R1: 6k8, Resistor_SMD:R_0805_2012Metric_Pad1.20x1.40mm_HandSolder, F.Cu at (34.7, 23.7)
- added R2: 6k8, Resistor_SMD:R_0805_2012Metric_Pad1.20x1.40mm_HandSolder, F.Cu at (34.7, 26.7)
- added R3: 6k8, Resistor_SMD:R_0805_2012Metric_Pad1.20x1.40mm_HandSolder, F.Cu at (34.7, 29.6)
- added R4: 1k, Resistor_SMD:R_0805_2012Metric_Pad1.20x1.40mm_HandSolder, F.Cu at (34.7, 32.6)
- added R5: 6k8, Resistor_SMD:R_0805_2012Metric_Pad1.20x1.40mm_HandSolder, F.Cu at (34.7, 35.5)
- added R6: 1k, Resistor_SMD:R_0805_2012Metric_Pad1.20x1.40mm_HandSolder, F.Cu at (34.7, 38.5)
- added SW1: SW_Push, Button_Switch_SMD:SW_Tactile_SPST_NO_Straight_CK_PTS636Sx25SMTRLFS, F.Cu at (27.5, 43.1)
- added U1: AP7384-33Y, Package_TO_SOT_SMD:SOT-89-3_Handsoldering, F.Cu at (26.6, 48.7)
- added U2: Pico_RaspberryPico, PicoNoSwd:RaspberryPico_TH_NoSWD, F.Cu at (2.60, 2.60)
- added U3: BDR6133, Package_TO_SOT_SMD:SC-70-8, F.Cu at (39.3, 32.0)
