File: DccDecoder4/DCCDecoder4/DCCDecoder4.kicad_sch (KiCad schematic)
At the start: 33 parts, among them J1 PAD, J14 +V, J15 M_OUT_B, J16 M_OUT_A, J17 GND, J2 PAD, J3 0, J4 1, J5 2, J6 3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

Commit message: 20/01/25 21:44 Titan.local
Parts:
- U2: footprint RP2040-Decoder_Additional_Footprints:SOIC-8-1EP_3.9x4.9mm_P1.27mm_EP2.41x3.3mm_ThermalVias -> Package_TO_SOT_SMD:SC-70-8
Changed lines of the file:
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@@
       (effects (font (size 1.27 1.27)) (justify left))
     )
-    (property "Footprint" "RP2040-Decoder_Additional_Footprints:SOIC-8-1EP_3.9x4.9mm_P1.27mm_EP2.41x3.3mm_ThermalVias" (at 231.14 139.7 0)
+    (property "Footprint" "Package_TO_SOT_SMD:SC-70-8" (at 231.14 139.7 0)
       (effects (font (size 1.27 1.27)) hide)
     )
