File: DccDecoder4/DCCDecoder4.kicad_pcb (KiCad board)
At the start: 2 copper layers, 51.1 x 20.6 mm, 33 parts, among them J1 PAD, J10 GND, J2 PAD, J3 0, J4 1, J5 2, J6 3, J7 +V, J8 M_OUT_B, J9 M_OUT_A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

Commit message: 21/01/25 18:52 Arrakis.local
Parts:
- Q2, Q3, Q4, Q5, Q6: value 2N7002K -> 2N7002BK
Other:
- board text added: "Dcc Decoder 4 2025"
Changed lines of the file:
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@@
         (effects (font (size 1 1) (thickness 0.15)))
     )
-    (fp_text value "2N7002K" (at 0 2.5) (layer "F.Fab")
+    (fp_text value "2N7002BK" (at 0 2.5) (layer "F.Fab")
         (effects (font (size 1 1) (thickness 0.15)))
     )
@@
         (effects (font (size 1 1) (thickness 0.15)))
     )
-    (fp_text value "2N7002K" (at 0 2.5) (layer "F.Fab")
+    (fp_text value "2N7002BK" (at 0 2.5) (layer "F.Fab")
         (effects (font (size 1 1) (thickness 0.15)))
     )
@@
         (effects (font (size 1 1) (thickness 0.15)))
     )
-    (fp_text value "2N7002K" (at 0 2.5) (layer "F.Fab")
+    (fp_text value "2N7002BK" (at 0 2.5) (layer "F.Fab")
         (effects (font (size 1 1) (thickness 0.15)))
     )
@@
         (effects (font (size 1 1) (thickness 0.15)))
     )
+    (fp_text user "${REFERENCE}" (at 0 0) (layer "F.Fab")
+        (effects (font (size 0.4 0.4) (thickness 0.06)))
+    )
     (fp_line (start 0 -1.56) (end -1.8 -1.56)
       (stroke (width 0.12) (type solid)) (layer "F.SilkS"))
@@
         (effects (font (size 1 1) (thickness 0.15)))
     )
-    (fp_text value "2N7002K" (at -0.889 2.54) (layer "F.Fab")
+    (fp_text value "2N7002BK" (at -0.889 2.54) (layer "F.Fab")
         (effects (font (size 0.8001 0.8001) (thickness 0.15)))
     )
@@
     (property "Sheetfile" "DCCDecoder4.kicad_sch")
     (property "Sheetname" "")
-    (attr through_hole exclude_from_pos_files exclude_from_bom)
+    (attr through_hole exclude_from_pos_files)
     (fp_text reference "U2" (at 15.5575 -0.508 90) (layer "F.SilkS")
         (effects (font (size 1 1) (thickness 0.15)))
@@
         (effects (font (size 1 1) (thickness 0.15)))
     )
-    (fp_text value "2N7002K" (at 0 2.5) (layer "F.Fab")
+    (fp_text value "2N7002BK" (at 0 2.5) (layer "F.Fab")
         (effects (font (size 1 1) (thickness 0.15)))
     )
@@
     (property "ki_description" "Generic connector, single row, 01x01, script generated")
     (property "ki_keywords" "connector")
-    (attr exclude_from_pos_files exclude_from_bom)
+    (attr exclude_from_pos_files)
     (fp_text reference "J2" (at 2.54 0) (layer "B.SilkS")
         (effects (font (size 1 1) (thickness 0.15)) (justify mirror))
@@
     (property "ki_description" "Generic connector, single row, 01x01, script generated")
     (property "ki_keywords" "connector")
-    (attr exclude_from_pos_files exclude_from_bom)
+    (attr exclude_from_pos_files)
     (fp_text reference "J1" (at 0 2.148) (layer "B.SilkS")
         (effects (font (size 1 1) (thickness 0.15)) (justify mirror))
@@
     (property "ki_description" "Generic connector, single row, 01x01, script generated (kicad-library-utils/schlib/autogen/connector/)")
     (property "ki_keywords" "connector")
-    (attr exclude_from_pos_files exclude_from_bom)
+    (attr exclude_from_pos_files)
     (fp_text reference "J6" (at 0 2.148) (layer "B.SilkS")
         (effects (font (size 1 1) (thickness 0.15)) (justify mirror))
@@
     (property "ki_description" "Generic connector, single row, 01x01, script generated (kicad-library-utils/schlib/autogen/connector/)")
     (property "ki_keywords" "connector")
-    (attr exclude_from_pos_files exclude_from_bom)
+    (attr exclude_from_pos_files)
     (fp_text reference "J7" (at 0 2.148) (layer "B.SilkS") hide
         (effects (font (size 1 1) (thickness 0.15)) (justify mirror))
@@
     (property "ki_description" "Push button switch, generic, two pins")
     (property "ki_keywords" "switch normally-open pushbutton push-button")
-    (attr smd exclude_from_pos_files exclude_from_bom)
+    (attr smd exclude_from_pos_files)
     (fp_text reference "SW1" (at 0 3 unlocked) (layer "B.SilkS") hide
         (effects (font (size 1 1) (thickness 0.15)) (justify mirror))
@@
     (property "ki_description" "Generic connector, single row, 01x01, script generated (kicad-library-utils/schlib/autogen/connector/)")
     (property "ki_keywords" "connector")
-    (attr exclude_from_pos_files exclude_from_bom)
+    (attr exclude_from_pos_files)
     (fp_text reference "J10" (at 0 2.148) (layer "B.SilkS") hide
         (effects (font (size 1 1) (thickness 0.15)) (justify mirror))
@@
     (property "ki_description" "Generic connector, single row, 01x01, script generated (kicad-library-utils/schlib/autogen/connector/)")
     (property "ki_keywords" "connector")
-    (attr exclude_from_pos_files exclude_from_bom)
+    (attr exclude_from_pos_files)
     (fp_text reference "J3" (at 2.54 0) (layer "B.SilkS")
         (effects (font (size 1 1) (thickness 0.15)) (justify mirror))
@@
     (property "ki_description" "Generic connector, single row, 01x01, script generated (kicad-library-utils/schlib/autogen/connector/)")
     (property "ki_keywords" "connector")
-    (attr exclude_from_pos_files exclude_from_bom)
+    (attr exclude_from_pos_files)
     (fp_text reference "J9" (at -0.635 2.54) (layer "B.SilkS") hide
         (effects (font (size 1 1) (thickness 0.15)) (justify mirror))
@@
     (property "ki_description" "Generic connector, single row, 01x01, script generated (kicad-library-utils/schlib/autogen/connector/)")
     (property "ki_keywords" "connector")
-    (attr exclude_from_pos_files exclude_from_bom)
+    (attr exclude_from_pos_files)
     (fp_text reference "J4" (at 2.54 0) (layer "B.SilkS")
         (effects (font (size 1 1) (thickness 0.15)) (justify mirror))
@@
     (property "ki_description" "Generic connector, single row, 01x01, script generated (kicad-library-utils/schlib/autogen/connector/)")
     (property "ki_keywords" "connector")
-    (attr exclude_from_pos_files exclude_from_bom)
+    (attr exclude_from_pos_files)
     (fp_text reference "J8" (at 0 2.148) (layer "B.SilkS") hide
         (effects (font (size 1 1) (thickness 0.15)) (justify mirror))
@@
     (property "ki_description" "Generic connector, single row, 01x01, script generated (kicad-library-utils/schlib/autogen/connector/)")
     (property "ki_keywords" "connector")
-    (attr exclude_from_pos_files exclude_from_bom)
+    (attr exclude_from_pos_files)
     (fp_text reference "J5" (at 2.54 0) (layer "B.SilkS")
         (effects (font (size 1 1) (thickness 0.15)) (justify mirror))
@@
   (gr_line (start 111.252 117.348) (end 111.252 137.922)
     (stroke (width 0.1) (type default)) (layer "Edge.Cuts"))
+  (gr_text "Dcc Decoder 4 2025" (at 83.185 122.555) (layer "B.SilkS")
+    (effects (font (size 1 1) (thickness 0.15)) (justify left bottom mirror))
+  )
   (gr_text "Motor B" (at 98.425 128.27) (layer "B.SilkS")
     (effects (font (size 1 1) (thickness 0.15)) (justify left bottom mirror))
@@
     (effects (font (size 1 1) (thickness 0.15)) (justify left bottom mirror))
   )
+  (dimension (type aligned) (layer "User.1")
+    (pts (xy 111.252 117.348) (xy 60.198 117.348))
+    (height 4.952999)
+    (gr_text "51.0540 mm" (at 85.725 111.245001) (layer "User.1")
+      (effects (font (size 1 1) (thickness 0.15)))
+    )
+    (format (prefix "") (suffix "") (units 2) (units_format 1) (precision 4))
+    (style (thickness 0.15) (arrow_length 1.27) (text_position_mode 0) (extension_height 0.58642) (extension_offset 0.5) keep_text_aligned)
+  )
+  (dimension (type aligned) (layer "User.1")
+    (pts (xy 60.198 117.348) (xy 60.198 137.922))
+    (height 6.223)
+    (gr_text "20.5740 mm" (at 52.825 127.635 90) (layer "User.1")
+      (effects (font (size 1 1) (thickness 0.15)))
+    )
+    (format (prefix "") (suffix "") (units 2) (units_format 1) (precision 4))
+    (style (thickness 0.15) (arrow_length 1.27) (text_position_mode 0) (extension_height 0.58642) (extension_offset 0.5) keep_text_aligned)
+  )
   (segment (start 77.56 129.945) (end 80.1308 129.945) (width 0.25) (layer "F.Cu") (net 1))

Commit message: 11/05/25 09:47 Arrakis.local
Parts:
- removed U3: BDR6133, RP2040-Decoder_Additional_Footprints:SOIC-8-1EP_3.9x4.9mm_P1.27mm_EP2.41x3.3mm_ThermalVias
- added IC1: BD62321HFP-TR, Package_TO_SOT_SMD:Rohm_HRP7, F.Cu at (99.7, 127.6)
- moved J8 1.27 mm to (94.0, 125.1)
- moved J9 1.27 mm to (94.0, 130.2)
- moved R4 0.91 mm to (91.4, 127.2)
- moved R5 0.91 mm to (91.4, 130.2)
- moved R6 0.76 mm to (91.4, 133.1)
Connections:
- net +3V3 renamed /+3V3
Routing:
- net Net-(J6-Pin_1): track 59.7 -> 0.00 mm, vias 1 -> 0
- net GND: track 134.6 -> 177.6 mm, vias 3 -> 4
- net /GPIO15: track 16.8 -> 0.00 mm, vias 1 -> 0
- net /GPIO14: track 14.1 -> 0.00 mm, vias 1 -> 0
- net /GPIO18: track 13.6 -> 0.00 mm, vias 1 -> 0
- net /ADC_EMF_A: track 25.4 -> 38.5 mm, vias 2 -> 1
- net /+3V3: track 34.3 -> 22.6 mm
- net Net-(J4-Pin_1): track 10.4 -> 0.00 mm, vias 1 -> 0
- net /GPIO17: track 9.67 -> 0.00 mm
- net Net-(J5-Pin_1): track 8.96 -> 0.00 mm, vias 1 -> 0
- net +V: track 68.4 -> 76.7 mm, vias 2 -> 5
- net Net-(J3-Pin_1): track 8.23 -> 0.00 mm, vias 1 -> 0
- net /GPIO19: track 21.0 -> 28.6 mm
- net /MOTOR_OUT_B: track 14.5 -> 7.85 mm
- net Net-(D3-K): track 56.5 -> 61.2 mm, vias 3 -> 1
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