File: DccDecoder4/DCCDecoder4.kicad_pcb (KiCad board)
At the start: 2 copper layers, 115.6 x 29.8 mm, 32 parts, among them IC1 BD62321HFP-TR, J1 Screw_Terminal_01x02, J2 0, J3 1, J4 2, J5 3, J6 +V, J7 M_OUT_B, J8 M_OUT_A, J9 GND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

Commit message: 12/05/25 20:40 Arrakis.local
Connections:
- U1 pad 1: unconnected-(U1-VO-Pad1) -> /+3V3
- U1 pad 3: /+3V3 -> +V
Routing:
- net PWM_F: track 49.2 -> 58.7 mm, vias 0 -> 2
- net ADC_EMF_B: track 53.2 -> 44.6 mm, vias 1 -> 0
- net +V: track 92.8 -> 101.2 mm, vias 3 -> 1
- net DCC_IN: track 65.1 -> 72.9 mm
- net Net-(D1-A): track 56.7 -> 64.5 mm, vias 1 -> 2
- net Net-(U2-VBUS): track 81.1 -> 75.0 mm
- net Net-(U2-RUN): track 58.4 -> 52.7 mm, vias 2 -> 0
- net PWM_R: track 55.9 -> 60.8 mm, vias 0 -> 2
- net FUNC_C: track 56.2 -> 60.8 mm, vias 0 -> 1
- net GND: track 280.5 -> 285.0 mm, vias 4 -> 5
- net Net-(Q2-G): track 17.4 -> 14.6 mm, vias 2 -> 0
- net FUNC_D: track 51.9 -> 54.4 mm
- net Net-(J5-Pin_1): track 24.0 -> 21.7 mm
- net /VSYS: track 70.4 -> 71.9 mm, vias 0 -> 3
- net /MOTOR_OUT_A: track 53.4 -> 52.1 mm
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
Commit message: 12/05/25 20:56 Arrakis.local
Other:
- board text added: "DccDecoder 4.1"
- board text removed: "DccDecoder 4"
Changed lines of the file:
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@@
     (effects (font (size 1 1) (thickness 0.15)) (justify left bottom mirror))
   )
-  (gr_text "DccDecoder 4" (at 171.45 92.075) (layer "F.SilkS")
+  (gr_text "DccDecoder 4.1" (at 171.45 92.075) (layer "F.SilkS")
     (effects (font (size 1 1) (thickness 0.15)) (justify left bottom))
   )
