File: DccDecoder4/DCCDecoder4.kicad_sch (KiCad schematic)
At the start: 33 parts, among them J1 PAD, J14 +V, J15 M_OUT_B, J16 M_OUT_A, J17 GND, J2 PAD, J3 0, J4 1, J5 2, J6 3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

Commit message: 21/01/25 18:52 Arrakis.local
Parts:
- Q1: footprint SOT96P240X110-3N -> Package_TO_SOT_SMD:SOT-23-3
- Q2, Q3, Q4, Q5, Q6: value 2N7002K -> 2N7002BK
Changed lines of the file:
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@@
       (effects (font (size 1.27 1.27)) (justify left))
     )
-    (property "Value" "2N7002K" (at 148.59 45.085 0)
+    (property "Value" "2N7002BK" (at 148.59 45.085 0)
       (effects (font (size 1.27 1.27)) (justify left))
     )
@@
       (effects (font (size 1.27 1.27)) (justify left))
     )
-    (property "Value" "2N7002K" (at 173.99 51.435 0)
+    (property "Value" "2N7002BK" (at 173.99 51.435 0)
       (effects (font (size 1.27 1.27)) (justify left))
     )
@@
       (effects (font (size 1.27 1.27)) (justify left))
     )
-    (property "Value" "2N7002K" (at 232.41 51.435 0)
+    (property "Value" "2N7002BK" (at 232.41 51.435 0)
       (effects (font (size 1.27 1.27)) (justify left))
     )
@@
       (effects (font (size 1.27 1.27)) (justify left))
     )
-    (property "Value" "2N7002K" (at 203.2 51.435 0)
+    (property "Value" "2N7002BK" (at 203.2 51.435 0)
       (effects (font (size 1.27 1.27)) (justify left))
     )
@@
       (effects (font (size 1.27 1.27)))
     )
-    (property "Footprint" "SOT96P240X110-3N" (at 69.85 82.55 0)
+    (property "Footprint" "Package_TO_SOT_SMD:SOT-23-3" (at 69.85 82.55 0)
       (effects (font (size 1.27 1.27)) (justify left) hide)
     )
@@
       (effects (font (size 1.27 1.27)) (justify left))
     )
-    (property "Value" "2N7002K" (at 261.62 51.435 0)
+    (property "Value" "2N7002BK" (at 261.62 51.435 0)
       (effects (font (size 1.27 1.27)) (justify left))
     )

Commit message: 11/05/25 09:47 Arrakis.local
Parts:
- removed U2: BDR6133, RP2040-Decoder_Additional_Footprints:SOIC-8-1EP_3.9x4.9mm_P1.27mm_EP2.41x3.3mm_ThermalVias, symbol RP2040-Decoder_Additional_Symbols:BDR6133
- added IC1: BD62321HFP-TR, Package_TO_SOT_SMD:Rohm_HRP7, symbol BD623xx:BD62321HFP-TR
Connections:
- net +V: now also IC1.1 (VCC_1), IC1.7 (VCC_2)
- net GND: now also IC1.4 (GND_1), IC1.8 (GND_2)
- net GPIO14: now also IC1.5 (RIN)
- net GPIO15: now also IC1.3 (FIN)
- net MOTOR_OUT_A: now also IC1.2 (OUT1)
- net MOTOR_OUT_B: now also IC1.6 (OUT2)
