File: DccDecoder4/DCCDecoder4.kicad_sch (KiCad schematic)
At the start: 32 parts, among them IC1 BD62321HFP-TR, J1 Screw_Terminal_01x02, J14 +V, J15 M_OUT_B, J16 M_OUT_A, J17 GND, J3 0, J4 1, J5 2, J6 3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

Commit message: 12/05/25 20:40 Arrakis.local
Connections:
- net +3V3: now also U1.1 (VO); no longer U1.3 (VI)
- net +V: now also U1.3 (VI)
Changed lines of the file:
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@@
   (junction (at 86.36 40.64) (diameter 0) (color 0 0 0 0)
+  )
+  (junction (at 73.66 40.64) (diameter 0) (color 0 0 0 0)
   )
   (junction (at 105.41 53.34) (diameter 0) (color 0 0 0 0)
@@
   )
   (wire (pts (xy 124.46 116.84) (xy 139.7 116.84))
+    (stroke (width 0) (type default))
+  )
+  (wire (pts (xy 68.58 40.64) (xy 73.66 40.64))
     (stroke (width 0) (type default))
   )
@@
     )
   )
-  (symbol (lib_id "Regulator_Linear:AP7384-50Y") (at 60.96 40.64 0) (unit 1)
+  (symbol (lib_id "Regulator_Linear:AP7384-50Y") (at 60.96 40.64 0) (mirror y) (unit 1)
     (in_bom yes) (on_board yes) (dnp no)
     (property "Reference" "U1" (at 60.96 34.29 0)

Commit message: 12/05/25 20:56 Arrakis.local
Other:
- note added: "Notes 1 now using same pin outs as Benoit's Merg scheme 2 Corrected earlier error AP73B4 reversed"
- note removed: "Notes 1 now using same pin outs as Benoit's Merg scheme"
Changed lines of the file:
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@@
     (effects (font (size 1.27 1.27)) (justify left bottom))
   )
-  (text "Notes\n1 now using same pin outs as Benoit's Merg scheme"
+  (text "Notes\n1 now using same pin outs as Benoit's Merg scheme\n2 Corrected earlier error AP73B4 reversed"
     (at 76.2 185.42 0)
     (effects (font (size 1.27 1.27)) (justify left bottom))
