File: DecoderMergCopy/PicoDecoder.kicad_pcb (KiCad board)
At the start: 2 copper layers, 51 x 20 mm, 33 parts, among them J1 PAD, J10 PAD, J2 PAD, J3 PAD, J4 PAD, J5 PAD, J6 PAD, J7 PAD, J8 PAD, J9 PAD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

Commit message: 11/05/25 20:19 Arrakis.local
Other:
- net class Default removed
