File: DCCDecoder4a/DCCDecoder4a.kicad_pcb (KiCad board)
At the start: 2 copper layers, 115.6 x 29.8 mm, 32 parts, among them IC1 BD62321HFP-TR, J1 Screw_Terminal_01x02, J2 0, J3 1, J4 2, J5 3, J6 +V, J7 M_OUT_B, J8 M_OUT_A, J9 GND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

Commit message: 12/05/25 20:40 Arrakis.local
Parts:
- moved R6 3.17 mm to (141.0, 113.0)
- moved R3 2.54 mm to (141.0, 93.3)
- moved IC1 2.29 mm to (130.9, 97.2)
- moved R5 1.91 mm to (141.0, 106.7)
- moved R4 0.64 mm to (141.0, 99.7)
Connections:
- net Net-(D1-A) renamed /DCC1
- net Net-(D3-K) renamed /DCC2
- U1 pad 1: unconnected-(U1-VO-Pad1) -> /+3V3
- U1 pad 3: /+3V3 -> +V
Routing:
- net GND: track 280.5 -> 26.8 mm, vias 4 -> 16
- net PWM_F: track 49.2 -> 0.00 mm
- net ADC_EMF_B: track 53.2 -> 80.1 mm
- net Net-(U2-VBUS): track 81.1 -> 70.1 mm, vias 2 -> 0
- net /MOTOR_OUT_A: track 53.4 -> 47.3 mm
- net /MOTOR_OUT_B: track 44.0 -> 48.9 mm, vias 1 -> 3
- net +V: track 92.8 -> 87.9 mm, vias 3 -> 1
- net Net-(U2-RUN): track 58.4 -> 54.2 mm, vias 2 -> 1
- net PWM_R: track 55.9 -> 52.0 mm, vias 0 -> 1
- net /ADC_EMF_A: track 41.3 -> 44.2 mm
- net /DCC1: track 56.7 -> 54.5 mm, vias 1 -> 2
- net Net-(Q2-G): track 17.4 -> 15.2 mm, vias 2 -> 0
- net /VSYS: track 70.4 -> 68.7 mm
- net FUNC_D: track 51.9 -> 53.4 mm, vias 0 -> 1
- net DCC_IN: track 65.1 -> 66.5 mm
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- added copper zone on B.Cu, net GND

Commit message: 12/05/25 20:56 Arrakis.local
Other:
- board text added: "DccDecoder 4.1"
- board text removed: "DccDecoder 4"
Changed lines of the file:
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@@
     (effects (font (size 1 1) (thickness 0.15)) (justify left bottom mirror))
   )
-  (gr_text "DccDecoder 4" (at 171.45 92.075) (layer "F.SilkS")
+  (gr_text "DccDecoder 4.1\n" (at 171.45 92.075) (layer "F.SilkS")
     (effects (font (size 1 1) (thickness 0.15)) (justify left bottom))
   )

Commit message: 12/05/25 21:51 Titan.local
Parts:
- moved J6 24.8 mm to (179.1, 107.3)
- moved J9 24.8 mm to (179.1, 100.3)
- moved J7 21.0 mm to (183.5, 107.3)
- moved J8 21.0 mm to (183.5, 100.3)
- moved J4 12.1 mm to (188.6, 107.3)
- moved J2 11.4 mm to (188.0, 100.3)
- moved J3 8.91 mm to (192.4, 100.3)
- moved J5 8.89 mm to (192.4, 107.3)
Routing:
- net PWM_F: track 0.00 -> 46.4 mm
- net /MOTOR_OUT_A: track 47.3 -> 82.3 mm, vias 1 -> 3
- net ADC_EMF_B: track 80.1 -> 50.2 mm, vias 1 -> 3
- net /MOTOR_OUT_B: track 48.9 -> 69.5 mm
- net +V: track 87.9 -> 106.0 mm
- net /DCC1: track 54.5 -> 66.8 mm
- net Net-(J4-Pin_1): track 25.5 -> 13.7 mm
- net Net-(J2-Pin_1): track 27.8 -> 16.4 mm
- net Net-(J5-Pin_1): track 22.8 -> 13.2 mm
- net PWM_R: track 52.0 -> 61.3 mm, vias 1 -> 3
- net Net-(J3-Pin_1): track 18.9 -> 10.9 mm
- net /VSYS: track 68.7 -> 75.4 mm
- net /ADC_EMF_A: track 44.2 -> 48.9 mm
- net Net-(U2-RUN): track 54.2 -> 58.0 mm
- net FUNC_C: track 56.2 -> 58.3 mm
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