File: DCCDecoder4a/DCCDecoder4a.kicad_pcb (KiCad board)
At the start: 2 copper layers, 115.6 x 29.8 mm, 32 parts, among them IC1 BD62321HFP-TR, J1 Screw_Terminal_01x02, J2 0, J3 1, J4 2, J5 3, J6 +V, J7 M_OUT_B, J8 M_OUT_A, J9 GND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

Commit message: 20/05/25 20:56 Arrakis.local
Parts:
- added R3: 10k, Resistor_SMD:R_1206_3216Metric_Pad1.30x1.75mm_HandSolder, F.Cu at (156.8, 109.2)
- added R4: 10k, Resistor_SMD:R_1206_3216Metric_Pad1.30x1.75mm_HandSolder, F.Cu at (150.5, 109.2)
- added TP1: TestPoint, TestPoint:TestPoint_Pad_2.0x2.0mm, F.Cu at (120.7, 108.0)
- added TP2: TestPoint, TestPoint:TestPoint_Pad_2.0x2.0mm, F.Cu at (120.7, 113.0)
- R1, R2: footprint Resistor_SMD:R_0805_2012Metric_Pad1.20x1.40mm_HandSolder -> Resistor_SMD:R_1206_3216Metric_Pad1.30x1.75mm_HandSolder
- R5: renamed from R3; footprint Resistor_SMD:R_0805_2012Metric_Pad1.20x1.40mm_HandSolder -> Resistor_SMD:R_1206_3216Metric_Pad1.30x1.75mm_HandSolder
- R6: renamed from R4; footprint Resistor_SMD:R_0805_2012Metric_Pad1.20x1.40mm_HandSolder -> Resistor_SMD:R_1206_3216Metric_Pad1.30x1.75mm_HandSolder
- R7: renamed from R5; footprint Resistor_SMD:R_0805_2012Metric_Pad1.20x1.40mm_HandSolder -> Resistor_SMD:R_1206_3216Metric_Pad1.30x1.75mm_HandSolder
- R8: renamed from R6; footprint Resistor_SMD:R_0805_2012Metric_Pad1.20x1.40mm_HandSolder -> Resistor_SMD:R_1206_3216Metric_Pad1.30x1.75mm_HandSolder
- moved SW1 21.9 mm to (95.9, 112.4)
- moved R7 16.1 mm to (156.8, 104.1)
- moved R6 15.9 mm to (156.8, 99.1)
- moved R8 13.0 mm to (150.5, 104.1)
- moved R5 11.1 mm to (150.5, 99.1)
- moved C1 8.89 mm to (114.9, 113.7), turned to 180 degrees
- moved U1 6.54 mm to (114.3, 108.0)
- moved Q2 4.49 mm to (132.7, 110.5)
- moved R2 4.24 mm to (138.4, 113.7), turned to 180 degrees
- moved Q1 4.15 mm to (126.4, 110.5)
- moved R1 2.84 mm to (138.4, 108.6), turned to 180 degrees
- moved IC1 2.58 mm to (132.7, 99.1)
- moved J6 2.54 mm to (176.5, 107.3)
- moved J9 2.54 mm to (176.5, 100.3)
Connections:
- net /+3V3 renamed +5V
- IC1 pad 3: PWM_F -> Net-(IC1-FIN)
- IC1 pad 5: PWM_R -> Net-(IC1-RIN)
- U2 pad 13: unconnected-(U2-GND-Pad13) -> GND
- U2 pad 5: unconnected-(U2-GPIO3-Pad5) -> DCC_IN
- U2 pad 7: DCC_IN -> unconnected-(U2-GPIO5-Pad7)
- U2 pad 8: unconnected-(U2-GND-Pad8) -> GND
Routing:
- net Net-(IC1-FIN): track 0.00 -> 41.0 mm, vias 0 -> 2
- net PWM_R: track 61.3 -> 30.1 mm, vias 3 -> 1
- net Net-(IC1-RIN): track 0.00 -> 28.8 mm, vias 0 -> 2
- net PWM_F: track 46.4 -> 19.0 mm, vias 0 -> 1
- net Net-(U2-RUN): track 58.0 -> 75.2 mm
- net /DCC1: track 66.8 -> 52.0 mm
- net /ADC_EMF_A: track 48.9 -> 35.2 mm
- net ADC_EMF_B: track 50.2 -> 40.4 mm, vias 3 -> 1
- net /MOTOR_OUT_B: track 69.5 -> 61.8 mm, vias 3 -> 1
- net Net-(Q2-G): track 13.4 -> 20.7 mm
- net +5V: track 14.7 -> 20.2 mm
- net FUNC_D: track 51.7 -> 56.1 mm
- net /MOTOR_OUT_A: track 82.3 -> 78.6 mm, vias 3 -> 2
- net DCC_IN: track 66.1 -> 63.0 mm
- net Net-(U2-VBUS): track 71.6 -> 73.4 mm, vias 1 -> 0
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Other:
- board text added: "bridge 5V"
