File: DCCDecoder4a/DCCDecoder4a.kicad_sch (KiCad schematic)
At the start: 32 parts, among them IC1 BD62321HFP-TR, J1 Screw_Terminal_01x02, J14 +V, J15 M_OUT_B, J16 M_OUT_A, J17 GND, J3 0, J4 1, J5 2, J6 3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

Commit message: 12/05/25 20:40 Arrakis.local
Connections:
- net +3V3: now also U1.1 (VO); no longer U1.3 (VI)
- net +V: now also U1.3 (VI)
- net DCC1: now reaches D1.2 (A), D2.1 (K), J1.1 (Pin_1), R1.2
- net DCC2: now reaches D3.1 (K), D4.2 (A), J1.2 (Pin_2)
Other:
- note added: "Notes 1 now using same pin outs as Benoit's Merg scheme 2 Added ground plane and wider power traces"
- note removed: "Notes 1 now using same pin outs as Benoit's Merg scheme"
- title: DCC Decoder 4 - modified PCB -> DCC Decoder 4a - modified PCB - As 4 but with ground plane
Changed lines of the file:
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@@
   (paper "A4")
   (title_block
-    (title "DCC Decoder 4 - modified PCB")
+    (title "DCC Decoder 4a - modified PCB - As 4 but with ground plane")
     (date "2025-01-20")
     (rev "4.0")
@@
   )
   (junction (at 73.66 53.34) (diameter 0) (color 0 0 0 0)
+  )
+  (junction (at 73.66 40.64) (diameter 0) (color 0 0 0 0)
   )
   (junction (at 116.84 40.64) (diameter 0) (color 0 0 0 0)
@@
     (stroke (width 0) (type default))
   )
+  (wire (pts (xy 68.58 40.64) (xy 73.66 40.64))
+    (stroke (width 0) (type default))
+  )
   (wire (pts (xy 91.44 93.98) (xy 91.44 104.14))
     (stroke (width 0) (type default))
@@
     (effects (font (size 1.27 1.27)) (justify left bottom))
   )
-  (text "Notes\n1 now using same pin outs as Benoit's Merg scheme"
+  (text "Notes\n1 now using same pin outs as Benoit's Merg scheme\n2 Added ground plane and wider power traces"
     (at 76.2 185.42 0)
     (effects (font (size 1.27 1.27)) (justify left bottom))
@@
     (effects (font (size 1.27 1.27)) (justify right bottom))
   )
+  (label "DCC1" (at 44.45 30.48 0) (fields_autoplaced)
+    (effects (font (size 1.27 1.27)) (justify left bottom))
+  )
   (label "ADC_EMF_A" (at 142.24 162.56 0) (fields_autoplaced)
     (effects (font (size 1.27 1.27)) (justify left bottom))
@@
   (label "PWM_F" (at 189.23 91.44 180) (fields_autoplaced)
     (effects (font (size 1.27 1.27)) (justify right bottom))
+  )
+  (label "DCC2" (at 31.75 41.91 0) (fields_autoplaced)
+    (effects (font (size 1.27 1.27)) (justify left bottom))
   )
   (label "+V" (at 91.44 35.56 0) (fields_autoplaced)
@@
         )
       )
-      (project "DCCDecoder4"
+      (project "DCCDecoder4a"
         (path "/6ae54932-6757-4715-a65b-f855d09f7054"
           (reference "R3") (unit 1)
@@
         )
       )
-      (project "DCCDecoder4"
+      (project "DCCDecoder4a"
         (path "/6ae54932-6757-4715-a65b-f855d09f7054"
           (reference "D2") (unit 1)
@@
         )
       )
-      (project "DCCDecoder4"
+      (project "DCCDecoder4a"
         (path "/6ae54932-6757-4715-a65b-f855d09f7054"
           (reference "D4") (unit 1)
@@
         )
       )
-      (project "DCCDecoder4"
+      (project "DCCDecoder4a"
         (path "/6ae54932-6757-4715-a65b-f855d09f7054"
           (reference "#PWR03") (unit 1)
@@
         )
       )
-      (project "DCCDecoder4"
+      (project "DCCDecoder4a"
         (path "/6ae54932-6757-4715-a65b-f855d09f7054"
           (reference "J9") (unit 1)
@@
         )
       )
-      (project "DCCDecoder4"
+      (project "DCCDecoder4a"
         (path "/6ae54932-6757-4715-a65b-f855d09f7054"
           (reference "#PWR02") (unit 1)
@@
     (pin "1")
     (instances
-      (project "DCCDecoder4"
+      (project "DCCDecoder4a"
         (path "/6ae54932-6757-4715-a65b-f855d09f7054"
           (reference "#FLG02") (unit 1)
@@
         )
       )
-      (project "DCCDecoder4"
+      (project "DCCDecoder4a"
         (path "/6ae54932-6757-4715-a65b-f855d09f7054"
           (reference "Q2") (unit 1)
@@
         )
       )
-      (project "DCCDecoder4"
+      (project "DCCDecoder4a"
         (path "/6ae54932-6757-4715-a65b-f855d09f7054"
           (reference "D3") (unit 1)
@@
         )
       )
-      (project "DCCDecoder4"
+      (project "DCCDecoder4a"
         (path "/6ae54932-6757-4715-a65b-f855d09f7054"
           (reference "R6") (unit 1)
@@
         )
       )
-      (project "DCCDecoder4"
+      (project "DCCDecoder4a"
         (path "/6ae54932-6757-4715-a65b-f855d09f7054"
           (reference "#PWR011") (unit 1)
@@
         )
       )
-      (project "DCCDecoder4"
+      (project "DCCDecoder4a"
         (path "/6ae54932-6757-4715-a65b-f855d09f7054"
           (reference "#PWR06") (unit 1)
@@
         )
       )
-      (project "DCCDecoder4"
+      (project "DCCDecoder4a"
         (path "/6ae54932-6757-4715-a65b-f855d09f7054"
           (reference "J8") (unit 1)
@@
         )
       )
-      (project "DCCDecoder4"
+      (project "DCCDecoder4a"
         (path "/6ae54932-6757-4715-a65b-f855d09f7054"
           (reference "Q3") (unit 1)
@@
         )
       )
-      (project "DCCDecoder4"
+      (project "DCCDecoder4a"
         (path "/6ae54932-6757-4715-a65b-f855d09f7054"
           (reference "U2") (unit 1)
@@
     )
   )
-  (symbol (lib_id "Regulator_Linear:AP7384-50Y") (at 60.96 40.64 0) (unit 1)
+  (symbol (lib_id "Regulator_Linear:AP7384-50Y") (at 60.96 40.64 0) (mirror y) (unit 1)
     (in_bom yes) (on_board yes) (dnp no)
     (property "Reference" "U1" (at 60.96 34.29 0)
@@
     (pin "3")
     (instances
-      (project "DCCDecoder4"
+      (project "DCCDecoder4a"
         (path "/6ae54932-6757-4715-a65b-f855d09f7054"
           (reference "U1") (unit 1)
@@
         )
       )
-      (project "DCCDecoder4"
+      (project "DCCDecoder4a"
         (path "/6ae54932-6757-4715-a65b-f855d09f7054"
           (reference "J6") (unit 1)
@@
         )
       )
-      (project "DCCDecoder4"
+      (project "DCCDecoder4a"
         (path "/6ae54932-6757-4715-a65b-f855d09f7054"
           (reference "R1") (unit 1)
@@
         )
       )
-      (project "DCCDecoder4"
+      (project "DCCDecoder4a"
         (path "/6ae54932-6757-4715-a65b-f855d09f7054"
           (reference "#PWR04") (unit 1)
@@
         )
       )
-      (project "DCCDecoder4"
+      (project "DCCDecoder4a"
         (path "/6ae54932-6757-4715-a65b-f855d09f7054"
           (reference "#PWR010") (unit 1)
@@
         )
       )
-      (project "DCCDecoder4"
+      (project "DCCDecoder4a"
         (path "/6ae54932-6757-4715-a65b-f855d09f7054"
           (reference "J7") (unit 1)
@@
         )
       )
-      (project "DCCDecoder4"
+      (project "DCCDecoder4a"
         (path "/6ae54932-6757-4715-a65b-f855d09f7054"
           (reference "Q5") (unit 1)
@@
         )
       )
-      (project "DCCDecoder4"
+      (project "DCCDecoder4a"
         (path "/6ae54932-6757-4715-a65b-f855d09f7054"
           (reference "R4") (unit 1)
@@
         )
       )
-      (project "DCCDecoder4"
+      (project "DCCDecoder4a"
         (path "/6ae54932-6757-4715-a65b-f855d09f7054"
           (reference "R5") (unit 1)
@@
         )
       )
-      (project "DCCDecoder4"
+      (project "DCCDecoder4a"
         (path "/6ae54932-6757-4715-a65b-f855d09f7054"
           (reference "R2") (unit 1)
@@
         )
       )
-      (project "DCCDecoder4"
+      (project "DCCDecoder4a"
         (path "/6ae54932-6757-4715-a65b-f855d09f7054"
           (reference "Q4") (unit 1)
@@
         )
       )
-      (project "DCCDecoder4"
+      (project "DCCDecoder4a"
         (path "/6ae54932-6757-4715-a65b-f855d09f7054"
           (reference "SW1") (unit 1)
@@
         )
       )
-      (project "DCCDecoder4"
+      (project "DCCDecoder4a"
         (path "/6ae54932-6757-4715-a65b-f855d09f7054"
           (reference "J4") (unit 1)
@@
     (pin "1")
     (instances
-      (project "DCCDecoder4"
+      (project "DCCDecoder4a"
         (path "/6ae54932-6757-4715-a65b-f855d09f7054"
           (reference "#FLG01") (unit 1)
@@
         )
       )
-      (project "DCCDecoder4"
+      (project "DCCDecoder4a"
         (path "/6ae54932-6757-4715-a65b-f855d09f7054"
           (reference "D1") (unit 1)
@@
         )
       )
-      (project "DCCDecoder4"
+      (project "DCCDecoder4a"
         (path "/6ae54932-6757-4715-a65b-f855d09f7054"
           (reference "J2") (unit 1)
@@
         )
       )
-      (project "DCCDecoder4"
+      (project "DCCDecoder4a"
         (path "/6ae54932-6757-4715-a65b-f855d09f7054"
           (reference "#PWR01") (unit 1)
@@
     (pin "8")
     (instances
-      (project "DCCDecoder4"
+      (project "DCCDecoder4a"
         (path "/6ae54932-6757-4715-a65b-f855d09f7054"
           (reference "IC1") (unit 1)
@@
         )
       )
-      (project "DCCDecoder4"
+      (project "DCCDecoder4a"
         (path "/6ae54932-6757-4715-a65b-f855d09f7054"
           (reference "#PWR09") (unit 1)
@@
         )
       )
-      (project "DCCDecoder4"
+      (project "DCCDecoder4a"
         (path "/6ae54932-6757-4715-a65b-f855d09f7054"
           (reference "#PWR05") (unit 1)
@@
         )
       )
-      (project "DCCDecoder4"
+      (project "DCCDecoder4a"
         (path "/6ae54932-6757-4715-a65b-f855d09f7054"
           (reference "C1") (unit 1)
@@
         )
       )
-      (project "DCCDecoder4"
+      (project "DCCDecoder4a"
         (path "/6ae54932-6757-4715-a65b-f855d09f7054"
           (reference "J5") (unit 1)
@@
         )
       )
-      (project "DCCDecoder4"
+      (project "DCCDecoder4a"
         (path "/6ae54932-6757-4715-a65b-f855d09f7054"
           (reference "#PWR07") (unit 1)
@@
         )
       )
-      (project "DCCDecoder4"
+      (project "DCCDecoder4a"
         (path "/6ae54932-6757-4715-a65b-f855d09f7054"
           (reference "J3") (unit 1)
@@
     (pin "2")
     (instances
-      (project "DCCDecoder4"
+      (project "DCCDecoder4a"
         (path "/6ae54932-6757-4715-a65b-f855d09f7054"
           (reference "J1") (unit 1)
@@
         )
       )
-      (project "DCCDecoder4"
+      (project "DCCDecoder4a"
         (path "/6ae54932-6757-4715-a65b-f855d09f7054"
           (reference "Q1") (unit 1)
@@
         )
       )
-      (project "DCCDecoder4"
+      (project "DCCDecoder4a"
         (path "/6ae54932-6757-4715-a65b-f855d09f7054"
           (reference "Q6") (unit 1)
@@
         )
       )
-      (project "DCCDecoder4"
+      (project "DCCDecoder4a"
         (path "/6ae54932-6757-4715-a65b-f855d09f7054"
           (reference "C3") (unit 1)
@@
         )
       )
-      (project "DCCDecoder4"
+      (project "DCCDecoder4a"
         (path "/6ae54932-6757-4715-a65b-f855d09f7054"
           (reference "C2") (unit 1)
@@
         )
       )
-      (project "DCCDecoder4"
+      (project "DCCDecoder4a"
         (path "/6ae54932-6757-4715-a65b-f855d09f7054"
           (reference "#PWR08") (unit 1)

Commit message: 20/05/25 20:56 Arrakis.local
Parts:
- added R2 (x2): 10k, Resistor_SMD:R_1206_3216Metric_Pad1.30x1.75mm_HandSolder, symbol Device:R
- added TP1, TP2: TestPoint, TestPoint:TestPoint_Pad_2.0x2.0mm, symbol Connector:TestPoint
- R1, R2, R5, R6, R7, R8: footprint Resistor_SMD:R_0805_2012Metric_Pad1.20x1.40mm_HandSolder -> Resistor_SMD:R_1206_3216Metric_Pad1.30x1.75mm_HandSolder
Connections:
- net DCC_IN: now also U2.5 (GPIO3); no longer U2.7 (GPIO5)
- net GND: now also U2.13 (GND), U2.8 (GND)
- net PWM_F: now also R2.2; no longer IC1.3 (FIN)
- net PWM_R: now also R2.2; no longer IC1.5 (RIN)
- net VSYS: now also TP2.1
- net +3V3 renamed +5V
- net +5V: now also TP1.1
- new net: IC1.3 (FIN), R2.1
- new net: IC1.5 (RIN), R2.1
- no-connect marks 27 -> 25
Other:
- note added: "5v bypass - without DMG2305"
- note added: "GPIO3 is pulled up internally in RP2040"
- note removed: "GPIO21 is pulled up internally in RP2040"
