File: DCCDecoder4a/DCCDecoder4a.kicad_sch (KiCad schematic)
At the start: 36 parts, among them IC1 BD62321HFP-TR, J1 Screw_Terminal_01x02, J14 +V, J15 M_OUT_B, J16 M_OUT_A, J17 GND, J3 0, J4 1, J5 2, J6 3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

Commit message: 06/09/25 21:49 Titan.local
Parts:
- Q1: footprint Package_TO_SOT_SMD:SOT-23-3 -> Package_TO_SOT_SMD:SOT-23
Changed lines of the file:
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@@
       (effects (font (size 1.27 1.27)))
     )
-    (property "Footprint" "Package_TO_SOT_SMD:SOT-23-3" (at 69.85 82.55 0)
+    (property "Footprint" "Package_TO_SOT_SMD:SOT-23" (at 69.85 82.55 0)
       (effects (font (size 1.27 1.27)) (justify left) hide)
     )
