File: newPower/newPower.kicad_sch (KiCad schematic)
At the start: 12 parts, among them J1 Screw_Terminal_01x02, Q2 2N7002BK, U1 AP7384-50Y

Commit message: 16/05/25 09:45 Arrakis.local
Parts:
- added TP1, TP2, TP3: TestPoint, TestPoint:TestPoint_Pad_2.5x2.5mm, symbol Connector:TestPoint
Connections:
- net +V: now also U1.3 (VI); no longer U1.1 (VO)
- net DCC_IN: now also TP1.1
- net GND: now also TP2.1
- net +3V3 renamed +5V
- net +5V: now also U1.1 (VO), TP3.1; no longer U1.3 (VI)
Other:
- title: (none) -> Power from DCC
Changed lines of the file:
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@@
 (kicad_sch (version 20230121) (generator eeschema)
   (paper "A4")
+  (title_block
+    (title "Power from DCC")
+    (date "2025-05-15")
+    (rev "1.0")
+  )
   (junction (at 172.72 116.84) (diameter 0) (color 0 0 0 0)
   )
   (junction (at 129.54 91.44) (diameter 0) (color 0 0 0 0)
   )
+  (junction (at 207.01 107.95) (diameter 0) (color 0 0 0 0)
+  )
   (junction (at 142.24 91.44) (diameter 0) (color 0 0 0 0)
   )
@@
   (junction (at 142.24 104.14) (diameter 0) (color 0 0 0 0)
   )
+  (junction (at 200.66 107.95) (diameter 0) (color 0 0 0 0)
+  )
   (junction (at 129.54 104.14) (diameter 0) (color 0 0 0 0)
   )
@@
     (stroke (width 0) (type default))
   )
+  (wire (pts (xy 200.66 107.95) (xy 207.01 107.95))
+    (stroke (width 0) (type default))
+  )
   (wire (pts (xy 101.6 91.44) (xy 101.6 93.98))
     (stroke (width 0) (type default))
@@
     (stroke (width 0) (type default))
   )
-  (wire (pts (xy 200.66 81.28) (xy 214.63 81.28))
-    (stroke (width 0) (type default))
-  )
   (wire (pts (xy 161.29 100.33) (xy 161.29 104.14))
     (stroke (width 0) (type default))
@@
     (stroke (width 0) (type default))
   )
-  (wire (pts (xy 95.25 137.16) (xy 114.3 137.16))
+  (wire (pts (xy 207.01 107.95) (xy 214.63 107.95))
+    (stroke (width 0) (type default))
+  )
+  (wire (pts (xy 95.25 137.16) (xy 128.27 137.16))
+    (stroke (width 0) (type default))
+  )
+  (wire (pts (xy 200.66 81.28) (xy 222.25 81.28))
     (stroke (width 0) (type default))
   )
@@
     (effects (font (size 1.27 1.27)) (justify right bottom))
   )
-  (label "+3V3" (at 99.06 111.76 0) (fields_autoplaced)
+  (label "+5V" (at 99.06 111.76 0) (fields_autoplaced)
+    (effects (font (size 1.27 1.27)) (justify left bottom))
+  )
+  (label "GND" (at 121.92 104.14 0) (fields_autoplaced)
     (effects (font (size 1.27 1.27)) (justify left bottom))
   )
@@
     )
   )
-  (symbol (lib_id "Regulator_Linear:AP7384-50Y") (at 116.84 91.44 0) (unit 1)
+  (symbol (lib_id "Regulator_Linear:AP7384-50Y") (at 116.84 91.44 0) (mirror y) (unit 1)
     (in_bom yes) (on_board yes) (dnp no)
     (property "Reference" "U1" (at 116.84 85.09 0)
@@
     )
   )
+  (symbol (lib_id "power:PWR_FLAG") (at 207.01 107.95 0) (unit 1)
+    (in_bom yes) (on_board yes) (dnp no) (fields_autoplaced)
+    (property "Reference" "#FLG02" (at 207.01 106.045 0)
+      (effects (font (size 1.27 1.27)) hide)
+    )
+    (property "Value" "PWR_FLAG" (at 207.01 104.14 0)
+      (effects (font (size 1.27 1.27)))
+    )
+    (property "Footprint" "" (at 207.01 107.95 0)
+      (effects (font (size 1.27 1.27)) hide)
+    )
+    (property "Datasheet" "~" (at 207.01 107.95 0)
+      (effects (font (size 1.27 1.27)) hide)
+    )
+    (pin "1")
+    (instances
+      (project "newPower"
+        (path "/7d4f522c-2668-45df-bec0-b4805c24e4cc"
+          (reference "#FLG02") (unit 1)
+        )
+      )
+    )
+  )
+  (symbol (lib_id "Connector:TestPoint") (at 128.27 137.16 270) (unit 1)
+    (in_bom yes) (on_board yes) (dnp no) (fields_autoplaced)
+    (property "Reference" "TP3" (at 133.35 136.525 90)
+      (effects (font (size 1.27 1.27)) (justify left))
+    )
+    (property "Value" "TestPoint" (at 133.35 139.065 90)
+      (effects (font (size 1.27 1.27)) (justify left))
+    )
+    (property "Footprint" "TestPoint:TestPoint_Pad_2.5x2.5mm" (at 128.27 142.24 0)
+      (effects (font (size 1.27 1.27)) hide)
+    )
+    (property "Datasheet" "~" (at 128.27 142.24 0)
+      (effects (font (size 1.27 1.27)) hide)
+    )
+    (pin "1")
+    (instances
+      (project "newPower"
+        (path "/7d4f522c-2668-45df-bec0-b4805c24e4cc"
+          (reference "TP3") (unit 1)
+        )
+      )
+    )
+  )
   (symbol (lib_id "power:PWR_FLAG") (at 135.89 86.36 0) (unit 1)
     (in_bom yes) (on_board yes) (dnp no) (fields_autoplaced)
@@
         )
       )
+    )
+  )
+  (symbol (lib_id "Connector:TestPoint") (at 214.63 107.95 270) (unit 1)
+    (in_bom yes) (on_board yes) (dnp no) (fields_autoplaced)
+    (property "Reference" "TP2" (at 219.71 107.315 90)
+      (effects (font (size 1.27 1.27)) (justify left))
+    )
+    (property "Value" "TestPoint" (at 219.71 109.855 90)
+      (effects (font (size 1.27 1.27)) (justify left))
+    )
+    (property "Footprint" "TestPoint:TestPoint_Pad_2.5x2.5mm" (at 214.63 113.03 0)
+      (effects (font (size 1.27 1.27)) hide)
+    )
+    (property "Datasheet" "~" (at 214.63 113.03 0)
+      (effects (font (size 1.27 1.27)) hide)
+    )
+    (pin "1")
+    (instances
+      (project "newPower"
+        (path "/7d4f522c-2668-45df-bec0-b4805c24e4cc"
+          (reference "TP2") (unit 1)
+        )
+      )
+    )
+  )
+  (symbol (lib_id "Connector:TestPoint") (at 222.25 81.28 270) (unit 1)
+    (in_bom yes) (on_board yes) (dnp no) (fields_autoplaced)
+    (property "Reference" "TP1" (at 227.33 80.645 90)
+      (effects (font (size 1.27 1.27)) (justify left))
+    )
+    (property "Value" "TestPoint" (at 227.33 83.185 90)
+      (effects (font (size 1.27 1.27)) (justify left))
+    )
+    (property "Footprint" "TestPoint:TestPoint_Pad_2.5x2.5mm" (at 222.25 86.36 0)
+      (effects (font (size 1.27 1.27)) hide)
+    )
+    (property "Datasheet" "~" (at 222.25 86.36 0)
+      (effects (font (size 1.27 1.27)) hide)
+    )
+    (pin "1")
+    (instances
+      (project "newPower"
+        (path "/7d4f522c-2668-45df-bec0-b4805c24e4cc"
+          (reference "TP1") (unit 1)
+        )
+      )
