File: PicoBleCentral/PicoBleCentral.kicad_sch (KiCad schematic)
At the start: 10 parts, among them IC2 VREG-OKI-78SR-3.3/1.5-W36, J5 Sel Vreg In, Q3 DMG2305UX-7, U2 R-78E5.0-1.0

Commit message: 26/05/25 20:18 Titan.local
Parts:
- removed C1: 100uF, PicoCanSmd31:E5-8,5, symbol PicoCanSmd31-eagle-import:CPOL-EUE5-8.5
- removed C2: 4.7uF, PicoCanSmd31:E5-8,5, symbol PicoCanSmd31-eagle-import:CPOL-EUE5-8.5
- removed C3: 100nF, PicoCanSmd31:C025-024X044, symbol PicoCanSmd31-eagle-import:C-EU025-024X044
- removed D1: CUS05S40,H3F, PicoCanSmd31:1SS357TPH3F, symbol PicoCanSmd31-eagle-import:CUS05S40,H3F
- removed D3: 5V, PicoCanSmd31:LED_3MM, symbol PicoCanSmd31-eagle-import:LED3MM
- removed IC2: VREG-OKI-78SR-3.3/1.5-W36, PicoCanSmd31:OKI-78SR, symbol PicoCanSmd31-eagle-import:VREG-OKI-78SR-3.3/1.5-W36
- removed J5: Sel Vreg In, PicoCanSmd31:1X03, symbol PicoCanSmd31-eagle-import:CONN_03
- removed Q3: DMG2305UX-7, PicoCanSmd31:SOT96P240X110-3N, symbol PicoCanSmd31-eagle-import:DMG2305UX-7
- removed R6: 1k, PicoCanSmd31:C1206, symbol PicoCanSmd31-eagle-import:RESISTOR-1206
- removed U2: R-78E5.0-1.0, PicoCanSmd31:DC-DC_CONVERTER_78XX, symbol PicoCanSmd31-eagle-import:R-78E5.0-1.0
- added Q2: DMG2305UX-7, Package_TO_SOT_SMD:SOT-23-3, symbol DMG2305UX-7:DMG2305UX-7
- added SW1: SW_Push, Button_Switch_SMD:SW_Tactile_SPST_NO_Straight_CK_PTS636Sx25SMTRLFS, symbol Switch:SW_Push
- added TP1, TP2: TestPoint, TestPoint:TestPoint_Pad_2.0x2.0mm, symbol Connector:TestPoint
- added U2: Pico_RaspberryPico, PicoNoSwd:RaspberryPico_TH_NoSWD, symbol PicoNoSwd:RaspberryPico-Pico
Connections:
- net GND: now also SW1.2
- net VSYS: now also Q2.2, TP2.1, U2.39 (VSYS)
- new net: Q2.1, U2.40 (VBUS)
- new net: Q2.3, TP1.1
- new net: SW1.1, U2.30 (RUN)
- new net: U2.13 (GND), U2.3 (GND), U2.8 (GND)
- new net ADC_EMF_A: U2.31 (GPIO26)
- new net ADC_EMF_B: U2.34 (GPIO28)
- new net DCC_IN: U2.5 (GPIO3)
- new net FUNC_A: U2.19 (GPIO14)
- new net FUNC_B: U2.20 (GPIO15)
- new net FUNC_C: U2.21 (GPIO16)
- new net FUNC_D: U2.22 (GPIO17)
- new net PWM_F: U2.12 (GPIO9)
- new net PWM_R: U2.11 (GPIO8)
- no-connect marks 0 -> 25
Other:
- note added: "5v bypass - without DMG2305"

Commit message: 26/05/25 20:40 Titan.local
Parts:
- removed Q2: DMG2305UX-7, Package_TO_SOT_SMD:SOT-23-3, symbol DMG2305UX-7:DMG2305UX-7
- added C1: 10uf/16V, Capacitor_SMD:C_1206_3216Metric_Pad1.33x1.80mm_HandSolder, symbol Device:C
- added C2: 10uF/25V, Capacitor_Tantalum_SMD:CP_EIA-6032-20_AVX-F_Pad2.25x2.35mm_HandSolder, symbol Device:C_Polarized
- added C3: 10uF/25v, Capacitor_Tantalum_SMD:CP_EIA-6032-20_AVX-F_Pad2.25x2.35mm_HandSolder, symbol Device:C_Polarized
- added D1, D2, D3, D4: RBR3L60AD, Diode_SMD:D_SMA_Handsoldering, symbol Device:D_Schottky
- added J1: Screw_Terminal_01x02, TerminalBlock_Phoenix:TerminalBlock_Phoenix_PT-1,5-2-3.5-H_1x02_P3.50mm_Horizontal, symbol Connector:Screw_Terminal_01x02
- added Q1: DMG2305UX-7, Package_TO_SOT_SMD:SOT-23-3, symbol DMG2305UX-7:DMG2305UX-7
- added U1: AP7384-50Y, Package_TO_SOT_SMD:SOT-89-3, symbol Regulator_Linear:AP7384-50Y
Connections:
- net GND: now also U2.13 (GND), U2.3 (GND), U2.8 (GND), C1.2, C2.2, C3.2, D2.2 (A), D3.2 (A), U1.2 (GND)
- net VSYS: now also Q1.2
- net at U2.40 (VBUS): now also Q1.1
- net +5V: now reaches TP1.1
- net +5V: now also C1.1, Q1.3, U1.1 (VO)
- new net +V: C2.1, C3.1, D1.1 (K), D4.1 (K), U1.3 (VI)
- new net DCC1: D1.2 (A), D2.1 (K), J1.1 (Pin_1)
- new net DCC2: D3.1 (K), D4.2 (A), J1.2 (Pin_2)
Other:
- note added: "Input Stage"
- note added: "Notes 1 now using same pin outs as Benoit's Merg scheme 2 Added ground plane and wider power traces"
- note added: "Other possible diodes B340LA-13-F"
- note added: "Size 2412 Vishay 593D106X9025C2TE3"
- title: (none) -> DCC Decoder 4a - modified PCB - As 4 but with ground plane

Commit message: 26/05/25 22:33 Titan.local
Parts:
- added J2: 3V3 Sel, Connector_PinHeader_2.54mm:PinHeader_1x03_P2.54mm_Vertical, symbol Connector:Conn_01x03_Pin
- added J3: keypad, Connector_PinHeader_2.54mm:PinHeader_1x08_P2.54mm_Vertical, symbol Connector:Conn_01x08_Pin
- added R10, R8, R9: 1k, Resistor_SMD:R_1206_3216Metric_Pad1.30x1.75mm_HandSolder, symbol PicoCanSmd31-eagle-import:RESISTOR-1206
- added R7: 10k, Resistor_SMD:R_1206_3216Metric_Pad1.30x1.75mm_HandSolder, symbol PicoCanSmd31-eagle-import:RESISTOR-1206
- added S1: ENCODER-RGB-SWITCH, Sparkfun switch:ENCODER_LED_3_KIT, symbol PicoCanSmd31-eagle-import:ENCODER-RGB-SWITCH
- added U3: MCP23008-xSO, Package_SO:SOIC-18W_7.5x11.6mm_P1.27mm, symbol Interface_Expansion:MCP23008-xSO
- added U4: AMS1117-3.3, Package_TO_SOT_SMD:SOT-223-3_TabPin2, symbol Regulator_Linear:AMS1117-3.3
Connections:
- net +5V: now also U4.3 (VI)
- net GND: now also S1.C, U3.3 (A2), U3.4 (A1), U3.5 (A0)
- net PINB: now reaches U2.16 (GPIO12)
- net PINB: now also S1.B
- net PINA: now reaches U2.17 (GPIO13)
- net PINA: now also S1.A
- net BTN: now reaches U2.29 (GPIO22)
- net BTN: now also R7.2
- net RUN: now reaches SW1.1, U2.30 (RUN)
- net RUN: now also U3.6 (~{RESET})
- net 3V3_OUT: now reaches U2.36 (3V3_OUT)
- net 3V3_OUT: now also J2.1 (Pin_1)
- net SDA: now reaches U2.6 (GPIO4)
- net SDA: now also U3.2 (SDA)
- net SCL: now reaches U2.7 (GPIO5)
- net SCL: now also U3.1 (SCL)
- net ADC_EMF_A: no longer names the net of U2.31 (GPIO26)
- net ADC_EMF_B: no longer names the net of U2.34 (GPIO28)
- net DCC_IN: no longer names the net of U2.5 (GPIO3)
- net FUNC_A: no longer names the net of U2.19 (GPIO14)
- net FUNC_B renamed BLUE
- net BLUE: now also R8.2
- net FUNC_C: no longer names the net of U2.21 (GPIO16)
- net FUNC_D: no longer names the net of U2.22 (GPIO17)
- net PWM_F renamed GREEN
- net GREEN: now also R9.2
- net PWM_R renamed RED
- net RED: now also R10.2
- new net: R10.1, S1.1 (-R)
- new net: R9.1, S1.2 (-G)
- new net: R7.1, S1.3 (SW)
- new net: R8.1, S1.4 (-B)
- new net: J3.1 (Pin_1), U3.10 (GP0)
- new net: J3.2 (Pin_2), U3.11 (GP1)
- new net: J3.3 (Pin_3), U3.12 (GP2)
- new net: J3.4 (Pin_4), U3.13 (GP3)
- new net: J3.5 (Pin_5), U3.14 (GP4)
- new net: J3.6 (Pin_6), U3.15 (GP5)
- new net: J3.7 (Pin_7), U3.16 (GP6)
- new net: J3.8 (Pin_8), U3.17 (GP7)
- new net 3V3: J2.2 (Pin_2), S1.5 (+)
- new net 3V3a: J2.3 (Pin_3), U4.2 (VO)
- no-connect marks 25 -> 26
Other:
- title: DCC Decoder 4a - modified PCB - As 4 but with ground plane -> Pico Ble Central for loco 

Commit message: 27/05/25 08:45 Arrakis.local
Parts:
- added J4: grove 2mm, symbol Connector:Screw_Terminal_01x04
- added J5: i2c, symbol Connector:Screw_Terminal_01x04
Connections:
- net 3V3: now also U3.18 (VDD)
- net GND: now also U3.9 (VSS)
Changed lines of the file:
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@@
+    )
+  )
+  (global_label "GND" (shape input) (at 204.47 63.5 270) (fields_autoplaced)
+    (effects (font (size 1.27 1.27)) (justify right))
+    (property "Intersheetrefs" "${INTERSHEET_REFS}" (at 204.47 70.2763 90)
+      (effects (font (size 1.27 1.27)) (justify right) hide)
     )
   )
@@
     )
   )
+  (global_label "3V3" (shape input) (at 204.47 33.02 90) (fields_autoplaced)
+    (effects (font (size 1.27 1.27)) (justify left))
+    (property "Intersheetrefs" "${INTERSHEET_REFS}" (at 204.47 26.6066 90)
+      (effects (font (size 1.27 1.27)) (justify left) hide)
+    )
+  )
   (global_label "BLUE" (shape bidirectional) (at 262.89 102.87 0) (fields_autoplaced)
     (effects (font (size 1.2446 1.2446)) (justify left))
@@
         (path "/6ae54932-6757-4715-a65b-f855d09f7054"
           (reference "D3") (unit 1)
+        )
+      )
+    )
+  )
+  (symbol (lib_id "Connector:Screw_Terminal_01x04") (at 199.39 124.46 0) (unit 1)
+    (in_bom yes) (on_board yes) (dnp no)
+    (property "Reference" "J4" (at 201.93 125.095 0)
+      (effects (font (size 1.27 1.27)) (justify left))
+    )
+    (property "Value" "grove 2mm" (at 195.58 133.35 0)
+      (effects (font (size 1.27 1.27)) (justify left))
+    )
+    (property "Footprint" "" (at 199.39 124.46 0)
+      (effects (font (size 1.27 1.27)) hide)
+    )
+    (property "Datasheet" "~" (at 199.39 124.46 0)
+      (effects (font (size 1.27 1.27)) hide)
+    )
+    (pin "1")
+    (pin "2")
+    (pin "3")
+    (pin "4")
+    (instances
+      (project "PicoBleCentral"
+        (path "/6ae54932-6757-4715-a65b-f855d09f7054"
+          (reference "J4") (unit 1)
         )
       )
@@
         )
       )
+    )
+  )
+  (symbol (lib_id "Connector:Screw_Terminal_01x04") (at 223.52 124.46 0) (unit 1)
+    (in_bom yes) (on_board yes) (dnp no)
+    (property "Reference" "J5" (at 226.06 125.095 0)
+      (effects (font (size 1.27 1.27)) (justify left))
+    )
+    (property "Value" "i2c" (at 222.25 133.35 0)
+      (effects (font (size 1.27 1.27)) (justify left))
+    )
+    (property "Footprint" "" (at 223.52 124.46 0)
+      (effects (font (size 1.27 1.27)) hide)
+    )
+    (property "Datasheet" "~" (at 223.52 124.46 0)
+      (effects (font (size 1.27 1.27)) hide)
+    )
+    (pin "1")
+    (pin "2")
+    (pin "3")
+    (pin "4")
+    (instances
+      (project "PicoBleCentral"
+        (path "/6ae54932-6757-4715-a65b-f855d09f7054"
+          (reference "J5") (unit 1)
+        )
+      )

Commit message: 27/05/25 09:08 Arrakis.local
Parts:
- J4, J5: footprint (none) -> Seed Grove etc:HW4-SMD-2.0
Connections:
- net 3V3: now also J4.3 (Pin_3), J5.3 (Pin_3)
- net GND: now also J4.4 (Pin_4), J5.4 (Pin_4)
- net SCL: now also J4.1 (Pin_1), J5.1 (Pin_1)
- net SDA: now also J4.2 (Pin_2), J5.2 (Pin_2)
Changed lines of the file:
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@@
+    )
+  )
+  (global_label "3V3" (shape input) (at 218.44 127 180) (fields_autoplaced)
+    (effects (font (size 1.27 1.27)) (justify right))
+    (property "Intersheetrefs" "${INTERSHEET_REFS}" (at 212.0266 127 0)
+      (effects (font (size 1.27 1.27)) (justify right) hide)
     )
   )
@@
     (effects (font (size 1.27 1.27)) (justify right))
     (property "Intersheetrefs" "${INTERSHEET_REFS}" (at 170.0372 40.64 0)
+      (effects (font (size 1.27 1.27)) (justify right) hide)
+    )
+  )
+  (global_label "SCL" (shape input) (at 194.31 121.92 180) (fields_autoplaced)
+    (effects (font (size 1.27 1.27)) (justify right))
+    (property "Intersheetrefs" "${INTERSHEET_REFS}" (at 187.8966 121.92 0)
       (effects (font (size 1.27 1.27)) (justify right) hide)
     )
@@
     )
   )
+  (global_label "3V3" (shape input) (at 194.31 127 180) (fields_autoplaced)
+    (effects (font (size 1.27 1.27)) (justify right))
+    (property "Intersheetrefs" "${INTERSHEET_REFS}" (at 187.8966 127 0)
+      (effects (font (size 1.27 1.27)) (justify right) hide)
+    )
+  )
   (global_label "+5V" (shape input) (at 128.27 36.83 180) (fields_autoplaced)
     (effects (font (size 1.27 1.27)) (justify right))
@@
     )
   )
+  (global_label "SDA" (shape input) (at 194.31 124.46 180) (fields_autoplaced)
+    (effects (font (size 1.27 1.27)) (justify right))
+    (property "Intersheetrefs" "${INTERSHEET_REFS}" (at 187.8361 124.46 0)
+      (effects (font (size 1.27 1.27)) (justify right) hide)
+    )
+  )
   (global_label "PINA" (shape input) (at 140.97 137.16 0) (fields_autoplaced)
     (effects (font (size 1.27 1.27)) (justify left))
@@
     )
   )
+  (global_label "GND" (shape input) (at 218.44 129.54 180) (fields_autoplaced)
+    (effects (font (size 1.27 1.27)) (justify right))
+    (property "Intersheetrefs" "${INTERSHEET_REFS}" (at 211.6637 129.54 0)
+      (effects (font (size 1.27 1.27)) (justify right) hide)
+    )
+  )
   (global_label "RUN" (shape input) (at 82.55 147.32 0) (fields_autoplaced)
     (effects (font (size 1.27 1.27)) (justify left))
@@
     )
   )
+  (global_label "SDA" (shape input) (at 218.44 124.46 180) (fields_autoplaced)
+    (effects (font (size 1.27 1.27)) (justify right))
+    (property "Intersheetrefs" "${INTERSHEET_REFS}" (at 211.9661 124.46 0)
+      (effects (font (size 1.27 1.27)) (justify right) hide)
+    )
+  )
+  (global_label "SCL" (shape input) (at 218.44 121.92 180) (fields_autoplaced)
+    (effects (font (size 1.27 1.27)) (justify right))
+    (property "Intersheetrefs" "${INTERSHEET_REFS}" (at 212.0266 121.92 0)
+      (effects (font (size 1.27 1.27)) (justify right) hide)
+    )
+  )
   (global_label "3V3_OUT" (shape input) (at 161.29 72.39 0) (fields_autoplaced)
     (effects (font (size 1.27 1.27)) (justify left))
     (property "Intersheetrefs" "${INTERSHEET_REFS}" (at 172.379 72.39 0)
       (effects (font (size 1.27 1.27)) (justify left) hide)
+    )
+  )
+  (global_label "GND" (shape input) (at 194.31 129.54 180) (fields_autoplaced)
+    (effects (font (size 1.27 1.27)) (justify right))
+    (property "Intersheetrefs" "${INTERSHEET_REFS}" (at 187.5337 129.54 0)
+      (effects (font (size 1.27 1.27)) (justify right) hide)
     )
   )
@@
       (effects (font (size 1.27 1.27)) (justify left))
     )
-    (property "Footprint" "" (at 199.39 124.46 0)
+    (property "Footprint" "Seed Grove etc:HW4-SMD-2.0" (at 199.39 124.46 0)
       (effects (font (size 1.27 1.27)) hide)
     )
@@
       (effects (font (size 1.27 1.27)) (justify left))
     )
-    (property "Footprint" "" (at 223.52 124.46 0)
-      (effects (font (size 1.27 1.27)) hide)
-    )
+    (property "Footprint" "Seed Grove etc:HW4-SMD-2.0" (at 223.52 124.46 0)
+      (effects (font (size 1.27 1.27)) hide)
+    )

Commit message: 27/05/25 10:06 Arrakis.local
Parts:
- added TP3: +V, TestPoint:TestPoint_Pad_2.5x2.5mm, symbol Connector:TestPoint
- added TP4: GND, TestPoint:TestPoint_Pad_2.5x2.5mm, symbol Connector:TestPoint
- J4, J5: footprint Seed Grove etc:HW4-SMD-2.0 -> Seed Grove etc:HW4-2.0
- R10, R8, R9: value 1k -> 330
- S1: footprint Sparkfun switch:ENCODER_LED_3_KIT -> sparkfun switch:ENCODER_LED_3
Connections:
- net +V: now also TP3.1
- net GND: now also TP4.1
Changed lines of the file:
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@@
+    )
+  )
+  (global_label "+V" (shape input) (at 214.63 143.51 180) (fields_autoplaced)
+    (effects (font (size 1.27 1.27)) (justify right))
+    (property "Intersheetrefs" "${INTERSHEET_REFS}" (at 209.0632 143.51 0)
+      (effects (font (size 1.27 1.27)) (justify right) hide)
     )
   )
@@
     )
   )
+  (global_label "GND" (shape input) (at 215.9 152.4 180) (fields_autoplaced)
+    (effects (font (size 1.27 1.27)) (justify right))
+    (property "Intersheetrefs" "${INTERSHEET_REFS}" (at 209.1237 152.4 0)
+      (effects (font (size 1.27 1.27)) (justify right) hide)
+    )
+  )
   (global_label "3V3_OUT" (shape input) (at 161.29 72.39 0) (fields_autoplaced)
     (effects (font (size 1.27 1.27)) (justify left))
@@
       (effects (font (size 1.27 1.27)) (justify left))
     )
-    (property "Footprint" "Seed Grove etc:HW4-SMD-2.0" (at 199.39 124.46 0)
+    (property "Footprint" "Seed Grove etc:HW4-2.0" (at 199.39 124.46 0)
       (effects (font (size 1.27 1.27)) hide)
     )
@@
       (effects (font (size 1.778 1.778)) (justify left top) hide)
     )
-    (property "Footprint" "Sparkfun switch:ENCODER_LED_3_KIT" (at 209.55 97.79 0)
+    (property "Footprint" "sparkfun switch:ENCODER_LED_3" (at 209.55 97.79 0)
       (effects (font (size 1.27 1.27)) hide)
     )
@@
     )
   )
+  (symbol (lib_id "Connector:TestPoint") (at 215.9 152.4 270) (unit 1)
+    (in_bom yes) (on_board yes) (dnp no) (fields_autoplaced)
+    (property "Reference" "TP4" (at 220.98 151.765 90)
+      (effects (font (size 1.27 1.27)) (justify left))
+    )
+    (property "Value" "GND" (at 220.98 154.305 90)
+      (effects (font (size 1.27 1.27)) (justify left))
+    )
+    (property "Footprint" "TestPoint:TestPoint_Pad_2.5x2.5mm" (at 215.9 157.48 0)
+      (effects (font (size 1.27 1.27)) hide)
+    )
+    (property "Datasheet" "~" (at 215.9 157.48 0)
+      (effects (font (size 1.27 1.27)) hide)
+    )
+    (pin "1")
+    (instances
+      (project "PicoBleCentral"
+        (path "/6ae54932-6757-4715-a65b-f855d09f7054"
+          (reference "TP4") (unit 1)
+        )
+      )
+    )
+  )
   (symbol (lib_id "PicoCanSmd31-eagle-import:RESISTOR-1206") (at 237.49 105.41 0) (unit 1)
     (in_bom yes) (on_board yes) (dnp no)
@@
     )
   )
+  (symbol (lib_id "Connector:TestPoint") (at 214.63 143.51 270) (unit 1)
+    (in_bom yes) (on_board yes) (dnp no) (fields_autoplaced)
+    (property "Reference" "TP3" (at 219.71 142.875 90)
+      (effects (font (size 1.27 1.27)) (justify left))
+    )
+    (property "Value" "+V" (at 219.71 145.415 90)
+      (effects (font (size 1.27 1.27)) (justify left))
+    )
+    (property "Footprint" "TestPoint:TestPoint_Pad_2.5x2.5mm" (at 214.63 148.59 0)
+      (effects (font (size 1.27 1.27)) hide)
+    )
+    (property "Datasheet" "~" (at 214.63 148.59 0)
+      (effects (font (size 1.27 1.27)) hide)
+    )
+    (pin "1")
+    (instances
+      (project "PicoBleCentral"
+        (path "/6ae54932-6757-4715-a65b-f855d09f7054"
+          (reference "TP3") (unit 1)
+        )
+      )
+    )
+  )
   (symbol (lib_id "PicoCanSmd31-eagle-import:RESISTOR-1206") (at 242.57 102.87 0) (unit 1)
     (in_bom yes) (on_board yes) (dnp no)
@@
       (effects (font (size 1.778 1.5113)) (justify bottom))
     )
-    (property "Value" "1k" (at 242.57 104.14 0)
+    (property "Value" "330" (at 242.57 104.14 0)
       (effects (font (size 1.778 1.5113)) (justify top))
     )
@@
       (effects (font (size 1.778 1.5113)) (justify bottom))
     )
-    (property "Value" "1k" (at 252.73 99.06 0)
+    (property "Value" "330" (at 252.73 99.06 0)
       (effects (font (size 1.778 1.5113)) (justify top))
     )
@@
       (effects (font (size 1.27 1.27)) (justify left))
     )
-    (property "Footprint" "Seed Grove etc:HW4-SMD-2.0" (at 223.52 124.46 0)
+    (property "Footprint" "Seed Grove etc:HW4-2.0" (at 223.52 124.46 0)
       (effects (font (size 1.27 1.27)) hide)
     )
@@
       (effects (font (size 1.778 1.5113)) (justify bottom))
     )
-    (property "Value" "1k" (at 247.65 101.6 0)
+    (property "Value" "330" (at 247.65 101.6 0)
       (effects (font (size 1.778 1.5113)) (justify top))
     )

Commit message: 27/05/25 12:17 Titan.local
Parts:
- added J6: 12V, TerminalBlock_Phoenix:TerminalBlock_Phoenix_PT-1,5-2-3.5-H_1x02_P3.50mm_Horizontal, symbol Connector:Screw_Terminal_01x02
- J1: value Screw_Terminal_01x02 -> DCC
Connections:
- net DCC1: now also J6.2 (Pin_2)
- net GND: now also J6.1 (Pin_1)
Other:
- note removed: "Input Stage"
- note removed: "Notes 1 now using same pin outs as Benoit's Merg scheme 2 Added ground plane and wider power traces"
- moved on the sheet: C1, C2, C3, D1, D2, D3, D4, J1, J2, J3, J4, J5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

Commit message: 28/05/25 13:45 Arrakis.local
Parts:
- added Brd1: SSD1306, SSD1306:128x64OLED, symbol SSD1306:SSD1306
Connections:
- net 3V3: now also Brd1.2 (VCC)
- net GND: now also Brd1.1 (GND)
- net SCL: now also Brd1.3 (SCL)
- net SDA: now also Brd1.4 (SDA)
Changed lines of the file:
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@@
     (effects (font (size 1.27 1.27)) (justify left bottom))
   )
-  (text "Other possible diodes\nB340LA-13-F" (at 128.27 83.82 0)
+  (text "Other possible diodes\nB340LA-13-F" (at 77.47 76.2 0)
     (effects (font (size 1.27 1.27)) (justify left bottom))
   )
@@
     (property "Intersheetrefs" "${INTERSHEET_REFS}" (at 191.2038 46.99 0)
       (effects (font (size 1.27 1.27)) (justify right) hide)
+    )
+  )
+  (global_label "GND" (shape input) (at 270.51 50.8 0) (fields_autoplaced)
+    (effects (font (size 1.27 1.27)) (justify left))
+    (property "Intersheetrefs" "${INTERSHEET_REFS}" (at 277.2863 50.8 0)
+      (effects (font (size 1.27 1.27)) (justify left) hide)
     )
   )
@@
     )
   )
+  (global_label "3V3" (shape input) (at 270.51 53.34 0) (fields_autoplaced)
+    (effects (font (size 1.27 1.27)) (justify left))
+    (property "Intersheetrefs" "${INTERSHEET_REFS}" (at 276.9234 53.34 0)
+      (effects (font (size 1.27 1.27)) (justify left) hide)
+    )
+  )
   (global_label "BTN" (shape bidirectional) (at 269.24 114.3 0) (fields_autoplaced)
     (effects (font (size 1.2446 1.2446)) (justify left))
@@
     )
   )
+  (global_label "SDA" (shape input) (at 270.51 58.42 0) (fields_autoplaced)
+    (effects (font (size 1.27 1.27)) (justify left))
+    (property "Intersheetrefs" "${INTERSHEET_REFS}" (at 276.9839 58.42 0)
+      (effects (font (size 1.27 1.27)) (justify left) hide)
+    )
+  )
   (global_label "PINB" (shape bidirectional) (at 193.04 111.76 180) (fields_autoplaced)
     (effects (font (size 1.2446 1.2446)) (justify right))
@@
     (property "Intersheetrefs" "${INTERSHEET_REFS}" (at 218.3161 133.35 0)
       (effects (font (size 1.27 1.27)) (justify right) hide)
+    )
+  )
+  (global_label "SCL" (shape input) (at 270.51 55.88 0) (fields_autoplaced)
+    (effects (font (size 1.27 1.27)) (justify left))
+    (property "Intersheetrefs" "${INTERSHEET_REFS}" (at 276.9234 55.88 0)
+      (effects (font (size 1.27 1.27)) (justify left) hide)
     )
   )
@@
         )
       )
+    )
+  )
+  (symbol (lib_id "SSD1306:SSD1306") (at 261.62 54.61 270) (unit 1)
+    (in_bom yes) (on_board yes) (dnp no) (fields_autoplaced)
+    (property "Reference" "Brd1" (at 261.62 44.45 90)
+      (effects (font (size 1.27 1.27)))
+    )
+    (property "Value" "SSD1306" (at 261.62 46.99 90)
+      (effects (font (size 1.27 1.27)))
+    )
+    (property "Footprint" "SSD1306:128x64OLED" (at 267.97 54.61 0)
+      (effects (font (size 1.27 1.27)) hide)
+    )
+    (property "Datasheet" "" (at 267.97 54.61 0)
+      (effects (font (size 1.27 1.27)) hide)
+    )
+    (pin "1")
+    (pin "2")
+    (pin "3")
+    (pin "4")
+    (instances
+      (project "PicoBleCentral"
+        (path "/6ae54932-6757-4715-a65b-f855d09f7054"
+          (reference "Brd1") (unit 1)
+        )
+      )
