File: PicoBleCentral/PicoBleCentral.kicad_sch (KiCad schematic)
At the start: 29 parts, among them J1 DCC, J2 3V3 Sel, J3 keypad, J4 grove 2mm, J5 i2c, J6 12V, Q1 DMG2305UX-7, SW1 SW_Push, U1 AP7384-50Y, U2 Pico_RaspberryPico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

Commit message: 30/05/25 09:30 Arrakis.local
Parts:
- Q1: footprint Package_TO_SOT_SMD:SOT-23-3 -> Package_TO_SOT_SMD:SOT-23_Handsoldering
- U4: footprint Package_TO_SOT_SMD:SOT-223-3_TabPin2 -> Package_TO_SOT_SMD:SOT-23_Handsoldering
Changed lines of the file:
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@@
       (effects (font (size 1.27 1.27)))
     )
-    (property "Footprint" "Package_TO_SOT_SMD:SOT-223-3_TabPin2" (at 149.86 40.64 0)
+    (property "Footprint" "Package_TO_SOT_SMD:SOT-23_Handsoldering" (at 149.86 40.64 0)
       (effects (font (size 1.27 1.27)) hide)
     )
@@
       (effects (font (size 1.27 1.27)))
     )
-    (property "Footprint" "Package_TO_SOT_SMD:SOT-23-3" (at 76.2 91.44 0)
+    (property "Footprint" "Package_TO_SOT_SMD:SOT-23_Handsoldering" (at 76.2 91.44 0)
       (effects (font (size 1.27 1.27)) (justify left) hide)
     )
