File: PicoBleCentral/PicoBleCentral.kicad_pcb (KiCad board)
At the start: 2 copper layers, 115.6 x 29.8 mm, 16 parts, among them J1 Screw_Terminal_01x02, J6 +V, J9 GND, Q1 DMG2305UX-7, SW1 SW_Push, U1 AP7384-50Y, U2 Pico_RaspberryPico

Commit message: 26/05/25 22:33 Titan.local
Parts:
- added J2: 3V3 Sel, Connector_PinHeader_2.54mm:PinHeader_1x03_P2.54mm_Vertical, F.Cu at (152.2, 102.3)
- added R1: 10k, Resistor_SMD:R_1206_3216Metric_Pad1.30x1.75mm_HandSolder, F.Cu at (140.3, 98.8)
- added R2: 1k, Resistor_SMD:R_1206_3216Metric_Pad1.30x1.75mm_HandSolder, F.Cu at (140.3, 102.1)
- added R3: 1k, Resistor_SMD:R_1206_3216Metric_Pad1.30x1.75mm_HandSolder, F.Cu at (140.3, 105.4)
- added R4: 1k, Resistor_SMD:R_1206_3216Metric_Pad1.30x1.75mm_HandSolder, F.Cu at (140.3, 108.7)
- added S1: ENCODER-RGB-SWITCH, Sparkfun switch:ENCODER_LED_3_KIT, F.Cu at (128.3, 79.4)
- added U3: MCP23008-xSO, Package_SO:SOIC-18W_7.5x11.6mm_P1.27mm, F.Cu at (154.9, 81.3)
- added U4: AMS1117-3.3, Package_TO_SOT_SMD:SOT-223-3_TabPin2, F.Cu at (159.4, 104.1)
Connections:
- U2 pad 11: PWM_R -> RED
- U2 pad 12: PWM_F -> GREEN
- U2 pad 16: unconnected-(U2-GPIO12-Pad16) -> PINB
- U2 pad 17: unconnected-(U2-GPIO13-Pad17) -> PINA
- U2 pad 19: FUNC_A -> unconnected-(U2-GPIO14-Pad19)
- U2 pad 20: FUNC_B -> BLUE
- U2 pad 21: FUNC_C -> unconnected-(U2-GPIO16-Pad21)
- U2 pad 22: FUNC_D -> unconnected-(U2-GPIO17-Pad22)
- U2 pad 29: unconnected-(U2-GPIO22-Pad29) -> BTN
- U2 pad 31: /ADC_EMF_A -> unconnected-(U2-GPIO26-Pad31)
- U2 pad 34: ADC_EMF_B -> unconnected-(U2-GPIO28-Pad34)
- U2 pad 36: unconnected-(U2-3V3_OUT-Pad36) -> 3V3_OUT
- U2 pad 5: DCC_IN -> unconnected-(U2-GPIO3-Pad5)
- U2 pad 6: unconnected-(U2-GPIO4-Pad6) -> SDA
- U2 pad 7: unconnected-(U2-GPIO5-Pad7) -> SCL
Routing:
- removed copper zone on B.Cu, net GND
Other:
- board size 115.6 x 29.8 mm -> 115.6 x 55.2 mm

Commit message: 27/05/25 08:45 Arrakis.local
Parts:
- added J3: keypad, Connector_PinHeader_2.54mm:PinHeader_1x08_P2.54mm_Vertical, F.Cu at (167.0, 88.9)
Connections:
- SW1 pad 1: Net-(U2-RUN) -> RUN
- U2 pad 30: Net-(U2-RUN) -> RUN
- U3 pad 10: unconnected-(U3-GP0-Pad10) -> Net-(J3-Pin_1)
- U3 pad 11: unconnected-(U3-GP1-Pad11) -> Net-(J3-Pin_2)
- U3 pad 12: unconnected-(U3-GP2-Pad12) -> Net-(J3-Pin_3)
- U3 pad 13: unconnected-(U3-GP3-Pad13) -> Net-(J3-Pin_4)
- U3 pad 14: unconnected-(U3-GP4-Pad14) -> Net-(J3-Pin_5)
- U3 pad 15: unconnected-(U3-GP5-Pad15) -> Net-(J3-Pin_6)
- U3 pad 16: unconnected-(U3-GP6-Pad16) -> Net-(J3-Pin_7)
- U3 pad 17: unconnected-(U3-GP7-Pad17) -> Net-(J3-Pin_8)
- U3 pad 18: unconnected-(U3-VDD-Pad18) -> 3V3
- U3 pad 3: unconnected-(U3-A2-Pad3) -> GND
- U3 pad 4: unconnected-(U3-A1-Pad4) -> GND
- U3 pad 5: unconnected-(U3-A0-Pad5) -> GND
- U3 pad 6: unconnected-(U3-~{RESET}-Pad6) -> RUN
- U3 pad 9: unconnected-(U3-VSS-Pad9) -> GND
Routing:
- net GND: track 0.00 -> 159.1 mm
- net RUN: track 0.00 -> 133.8 mm, vias 0 -> 1
- net Net-(#FLG03-pwr): track 0.00 -> 75.4 mm
- net /VSYS: track 0.00 -> 72.7 mm
- net 3V3: track 0.00 -> 62.8 mm, vias 0 -> 1
- net +5V: track 0.00 -> 51.3 mm
- net Net-(S1--R): track 0.00 -> 50.3 mm, vias 0 -> 1
- net Net-(S1--G): track 0.00 -> 47.8 mm, vias 0 -> 1
- net 3V3_OUT: track 0.00 -> 45.4 mm, vias 0 -> 1
- net SCL: track 0.00 -> 42.2 mm, vias 0 -> 1
- net SDA: track 0.00 -> 40.6 mm
- net BTN: track 0.00 -> 40.2 mm, vias 0 -> 1
- net Net-(S1--B): track 0.00 -> 36.2 mm, vias 0 -> 1
- net Net-(S1-SW): track 0.00 -> 35.8 mm, vias 0 -> 1
- net RED: track 0.00 -> 32.8 mm
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
Commit message: 27/05/25 09:08 Arrakis.local
Parts:
- added J4: grove 2mm, Seed Grove etc:HW4-SMD-2.0, F.Cu at (189.4, 71.9)
- added J5: i2c, Seed Grove etc:HW4-SMD-2.0, F.Cu at (189.4, 80.6)
Changed lines of the file:
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@@
     )
+  )
+  (footprint "Seed Grove etc:HW4-SMD-2.0" (layer "F.Cu")
+    (at 189.37 71.93416)
+    (property "Sheetfile" "PicoBleCentral.kicad_sch")
+    (property "Sheetname" "")
+    (property "ki_description" "Generic screw terminal, single row, 01x04, script generated (kicad-library-utils/schlib/autogen/connector/)")
+    (property "ki_keywords" "screw terminal")
+    (attr smd)
+    (fp_text reference "J4" (at -0.025 -3.325) (layer "F.SilkS")
+        (effects (font (size 1 1) (thickness 0.15)))
+    )
+    (fp_text value "grove 2mm" (at -0.025 6.45) (layer "F.Fab")
+        (effects (font (size 1 1) (thickness 0.15)))
+    )
+    (fp_text user "${REFERENCE}" (at 0 0) (layer "F.Fab")
+        (effects (font (size 1 1) (thickness 0.15)))
+    )
+    (fp_line (start -6 -2.15) (end -6 -1.4395)
+      (stroke (width 0.127) (type solid)) (layer "F.SilkS"))
+    (fp_line (start -6 -2.15) (end 6 -2.15)
+      (stroke (width 0.127) (type solid)) (layer "F.SilkS"))
+    (fp_line (start -6 1.45) (end -6 3.35)
+      (stroke (width 0.127) (type solid)) (layer "F.SilkS"))
+    (fp_line (start -6 3.35) (end -3.8 3.35)
+      (stroke (width 0.127) (type solid)) (layer "F.SilkS"))
+    (fp_line (start -3.8 3.35) (end -3.8 2.06)
+      (stroke (width 0.127) (type solid)) (layer "F.SilkS"))
+    (fp_line (start -2.3485 2.06062) (end -1.65 2.06062)
+      (stroke (width 0.127) (type solid)) (layer "F.SilkS"))
+    (fp_line (start -0.3485 2.06062) (end 0.35 2.06062)
+      (stroke (width 0.127) (type solid)) (layer "F.SilkS"))
+    (fp_line (start 1.64896 2.06062) (end 2.35 2.06062)
+      (stroke (width 0.127) (type solid)) (layer "F.SilkS"))
+    (fp_line (start 3.8 2.06062) (end 3.8 3.35)
+      (stroke (width 0.127) (type solid)) (layer "F.SilkS"))
+    (fp_line (start 3.8 3.35) (end 6 3.35)
+      (stroke (width 0.127) (type solid)) (layer "F.SilkS"))
+    (fp_line (start 6 -2.15) (end 6 -1.4395)
+      (stroke (width 0.127) (type solid)) (layer "F.SilkS"))
+    (fp_line (start 6 1.425) (end 6 3.35)
+      (stroke (width 0.127) (type solid)) (layer "F.SilkS"))
+    (fp_line (start -6.6 -2.4) (end -6.6 5.25)
+      (stroke (width 0.05) (type solid)) (layer "F.CrtYd"))
+    (fp_line (start -6.6 5.25) (end 6.6 5.25)
+      (stroke (width 0.05) (type solid)) (layer "F.CrtYd"))
+    (fp_line (start 6.6 -2.4) (end -6.6 -2.4)
+      (stroke (width 0.05) (type solid)) (layer "F.CrtYd"))
+    (fp_line (start 6.6 5.25) (end 6.6 -2.4)
+      (stroke (width 0.05) (type solid)) (layer "F.CrtYd"))
+    (fp_line (start -6 -2.15) (end -6 3.35)
+      (stroke (width 0.1) (type solid)) (layer "F.Fab"))
+    (fp_line (start -6 -2.15) (end 6 -2.15)
+      (stroke (width 0.1) (type solid)) (layer "F.Fab"))
+    (fp_line (start -6 3.35) (end -3.8 3.35)
+      (stroke (width 0.1) (type solid)) (layer "F.Fab"))
+    (fp_line (start -3.8 2.06062) (end 3.8 2.06062)
+      (stroke (width 0.1) (type solid)) (layer "F.Fab"))
+    (fp_line (start -3.8 3.35) (end -3.8 2.06)
+      (stroke (width 0.1) (type solid)) (layer "F.Fab"))
+    (fp_line (start 3.8 2.06062) (end 3.8 3.35)
+      (stroke (width 0.1) (type solid)) (layer "F.Fab"))
+    (fp_line (start 3.8 3.35) (end 6 3.35)
+      (stroke (width 0.1) (type solid)) (layer "F.Fab"))
+    (fp_line (start 6 -2.15) (end 6 3.35)
+      (stroke (width 0.1) (type solid)) (layer "F.Fab"))
+    (pad "1" smd rect (at -3 3.5 90) (size 3 1) (layers "F.Cu" "F.Paste" "F.Mask")
+      (net 49 "SCL") (pinfunction "Pin_1") (pintype "passive"))
+    (pad "2" smd rect (at -1 3.5 90) (size 3 1) (layers "F.Cu" "F.Paste" "F.Mask")
+      (net 48 "SDA") (pinfunction "Pin_2") (pintype "passive"))
+    (pad "3" smd rect (at 1 3.5 90) (size 3 1) (layers "F.Cu" "F.Paste" "F.Mask")
+      (net 23 "3V3") (pinfunction "Pin_3") (pintype "passive"))
+    (pad "4" smd rect (at 3 3.5 90) (size 3 1) (layers "F.Cu" "F.Paste" "F.Mask")
+      (net 1 "GND") (pinfunction "Pin_4") (pintype "passive"))
+    (pad "5" smd rect (at -5.575 0.01084 90) (size 2.6 1.55) (layers "F.Cu" "F.Paste" "F.Mask"))
+    (pad "6" smd rect (at 5.575 0.01084 90) (size 2.6 1.55) (layers "F.Cu" "F.Paste" "F.Mask"))
   )
   (footprint "PicoNoSwd:RaspberryPico_TH_NoSWD" (layer "F.Cu")
@@
     )
   )
+  (footprint "Seed Grove etc:HW4-SMD-2.0" (layer "F.Cu")
+    (at 189.37 80.63416)
+    (property "Sheetfile" "PicoBleCentral.kicad_sch")
+    (property "Sheetname" "")
+    (property "ki_description" "Generic screw terminal, single row, 01x04, script generated (kicad-library-utils/schlib/autogen/connector/)")
+    (property "ki_keywords" "screw terminal")
+    (attr smd)
+    (fp_text reference "J5" (at -0.025 -3.325) (layer "F.SilkS")
+        (effects (font (size 1 1) (thickness 0.15)))
+    )
+    (fp_text value "i2c" (at -0.025 6.45) (layer "F.Fab")
+        (effects (font (size 1 1) (thickness 0.15)))
+    )
+    (fp_text user "${REFERENCE}" (at 0 0) (layer "F.Fab")
+        (effects (font (size 1 1) (thickness 0.15)))
+    )
+    (fp_line (start -6 -2.15) (end -6 -1.4395)
+      (stroke (width 0.127) (type solid)) (layer "F.SilkS"))
+    (fp_line (start -6 -2.15) (end 6 -2.15)
+      (stroke (width 0.127) (type solid)) (layer "F.SilkS"))
+    (fp_line (start -6 1.45) (end -6 3.35)
+      (stroke (width 0.127) (type solid)) (layer "F.SilkS"))
+    (fp_line (start -6 3.35) (end -3.8 3.35)
+      (stroke (width 0.127) (type solid)) (layer "F.SilkS"))
+    (fp_line (start -3.8 3.35) (end -3.8 2.06)
+      (stroke (width 0.127) (type solid)) (layer "F.SilkS"))
+    (fp_line (start -2.3485 2.06062) (end -1.65 2.06062)
+      (stroke (width 0.127) (type solid)) (layer "F.SilkS"))
+    (fp_line (start -0.3485 2.06062) (end 0.35 2.06062)
+      (stroke (width 0.127) (type solid)) (layer "F.SilkS"))
+    (fp_line (start 1.64896 2.06062) (end 2.35 2.06062)
+      (stroke (width 0.127) (type solid)) (layer "F.SilkS"))
+    (fp_line (start 3.8 2.06062) (end 3.8 3.35)
+      (stroke (width 0.127) (type solid)) (layer "F.SilkS"))
+    (fp_line (start 3.8 3.35) (end 6 3.35)
+      (stroke (width 0.127) (type solid)) (layer "F.SilkS"))
+    (fp_line (start 6 -2.15) (end 6 -1.4395)
+      (stroke (width 0.127) (type solid)) (layer "F.SilkS"))
+    (fp_line (start 6 1.425) (end 6 3.35)
+      (stroke (width 0.127) (type solid)) (layer "F.SilkS"))
+    (fp_line (start -6.6 -2.4) (end -6.6 5.25)
+      (stroke (width 0.05) (type solid)) (layer "F.CrtYd"))
+    (fp_line (start -6.6 5.25) (end 6.6 5.25)
+      (stroke (width 0.05) (type solid)) (layer "F.CrtYd"))
+    (fp_line (start 6.6 -2.4) (end -6.6 -2.4)
+      (stroke (width 0.05) (type solid)) (layer "F.CrtYd"))
+    (fp_line (start 6.6 5.25) (end 6.6 -2.4)
+      (stroke (width 0.05) (type solid)) (layer "F.CrtYd"))
+    (fp_line (start -6 -2.15) (end -6 3.35)
+      (stroke (width 0.1) (type solid)) (layer "F.Fab"))
+    (fp_line (start -6 -2.15) (end 6 -2.15)
+      (stroke (width 0.1) (type solid)) (layer "F.Fab"))
+    (fp_line (start -6 3.35) (end -3.8 3.35)
+      (stroke (width 0.1) (type solid)) (layer "F.Fab"))
+    (fp_line (start -3.8 2.06062) (end 3.8 2.06062)
+      (stroke (width 0.1) (type solid)) (layer "F.Fab"))
+    (fp_line (start -3.8 3.35) (end -3.8 2.06)
+      (stroke (width 0.1) (type solid)) (layer "F.Fab"))
+    (fp_line (start 3.8 2.06062) (end 3.8 3.35)
+      (stroke (width 0.1) (type solid)) (layer "F.Fab"))
+    (fp_line (start 3.8 3.35) (end 6 3.35)
+      (stroke (width 0.1) (type solid)) (layer "F.Fab"))
+    (fp_line (start 6 -2.15) (end 6 3.35)
+      (stroke (width 0.1) (type solid)) (layer "F.Fab"))
+    (pad "1" smd rect (at -3 3.5 90) (size 3 1) (layers "F.Cu" "F.Paste" "F.Mask")
+      (net 49 "SCL") (pinfunction "Pin_1") (pintype "passive"))
+    (pad "2" smd rect (at -1 3.5 90) (size 3 1) (layers "F.Cu" "F.Paste" "F.Mask")
+      (net 48 "SDA") (pinfunction "Pin_2") (pintype "passive"))
+    (pad "3" smd rect (at 1 3.5 90) (size 3 1) (layers "F.Cu" "F.Paste" "F.Mask")
+      (net 23 "3V3") (pinfunction "Pin_3") (pintype "passive"))
+    (pad "4" smd rect (at 3 3.5 90) (size 3 1) (layers "F.Cu" "F.Paste" "F.Mask")
+      (net 1 "GND") (pinfunction "Pin_4") (pintype "passive"))
+    (pad "5" smd rect (at -5.575 0.01084 90) (size 2.6 1.55) (layers "F.Cu" "F.Paste" "F.Mask"))
+    (pad "6" smd rect (at 5.575 0.01084 90) (size 2.6 1.55) (layers "F.Cu" "F.Paste" "F.Mask"))
+  )
   (footprint "Diode_SMD:D_SMA_Handsoldering" (layer "F.Cu")

Commit message: 27/05/25 10:06 Arrakis.local
Parts:
- removed J6: +V, TestPoint:TestPoint_Pad_2.5x2.5mm
- removed J9: GND, TestPoint:TestPoint_Pad_2.5x2.5mm
- added +V: +V, TestPoint:TestPoint_Pad_2.5x2.5mm, F.Cu at (172.7, 101.0)
- added GND: GND, TestPoint:TestPoint_Pad_2.5x2.5mm, F.Cu at (172.7, 107.3)
- J4, J5: footprint Seed Grove etc:HW4-SMD-2.0 -> Seed Grove etc:HW4-2.0
- S1: footprint Sparkfun switch:ENCODER_LED_3_KIT -> sparkfun switch:ENCODER_LED_3
- moved J5 2.55 mm to (189.4, 83.2)
Connections:
- C2 pad 1: /+V -> +V
- C3 pad 1: /+V -> +V
- D1 pad 1: /+V -> +V
- D4 pad 1: /+V -> +V
- U1 pad 3: /+V -> +V
Routing:
- net GND: track 159.1 -> 21.9 mm, vias 0 -> 11
- net +V: track 0.00 -> 83.0 mm
- net 3V3: track 62.8 -> 119.3 mm
- net SDA: track 40.6 -> 70.2 mm
- net /+V: track 25.8 -> 0.00 mm
- net SCL: track 42.2 -> 67.5 mm, vias 1 -> 0
- net RUN: track 133.8 -> 113.1 mm
- net RED: track 32.8 -> 47.5 mm, vias 0 -> 1
- net BTN: track 40.2 -> 30.6 mm
- net +5V: track 51.3 -> 58.0 mm
- net Net-(U2-VBUS): track 75.4 -> 70.8 mm
- net 3V3_OUT: track 45.4 -> 40.9 mm
- net BLUE: track 10.7 -> 15.0 mm, vias 0 -> 1
- net Net-(S1--G): track 47.8 -> 43.8 mm
- net Net-(S1-SW): track 35.8 -> 33.2 mm
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- added copper zone on B.Cu, net GND
Other:
- board text added: "3V3"
- board text added: "3V3 sel"
- board text added: "3V3a"
- board text added: "GND"
- board text added: "Pico"
- board text added: "PicoBleCentral 1.0"
- board text added: "SCL"
- board text added: "SDA"
- board text added: "bridge 5V direct to Vsys"
- board text removed: "DccDecoder 4.1"
- board text removed: "Gnd"
- board text removed: "V+"
- board text removed: "bridge 5V"

Commit message: 27/05/25 12:17 Titan.local
Parts:
- added J6: 12V, TerminalBlock_Phoenix:TerminalBlock_Phoenix_PT-1,5-2-3.5-H_1x02_P3.50mm_Horizontal, F.Cu at (95.2, 90.5)
- J1: value Screw_Terminal_01x02 -> DCC
- R2, R3, R4: value 1k -> 330
- renumbered +V to TP3, GND to TP4
Changed lines of the file:
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@@
+    )
+  )
+  (footprint "TerminalBlock_Phoenix:TerminalBlock_Phoenix_PT-1,5-2-3.5-H_1x02_P3.50mm_Horizontal" (layer "F.Cu")
+    (at 95.25 90.48 -90)
+    (descr "Terminal Block Phoenix PT-1,5-2-3.5-H, 2 pins, pitch 3.5mm, size 7x7.6mm^2, drill diamater 1.2mm, pad diameter 2.4mm, see , script-generated using https://github.com/pointhi/kicad-footprint-generator/scripts/TerminalBlock_Phoenix")
+    (tags "THT Terminal Block Phoenix PT-1,5-2-3.5-H pitch 3.5mm size 7x7.6mm^2 drill 1.2mm pad 2.4mm")
+    (property "Sheetfile" "PicoBleCentral.kicad_sch")
+    (property "Sheetname" "")
+    (property "ki_description" "Generic screw terminal, single row, 01x02, script generated (kicad-library-utils/schlib/autogen/connector/)")
+    (property "ki_keywords" "screw terminal")
+    (attr through_hole)
+    (fp_text reference "J6" (at 1.75 -4.16 90) (layer "F.SilkS")
+        (effects (font (size 1 1) (thickness 0.15)))
+    )
+    (fp_text value "12V" (at 1.75 5.56 90) (layer "F.Fab")
+        (effects (font (size 1 1) (thickness 0.15)))
+    )
+    (fp_text user "${REFERENCE}" (at 1.75 2.4 90) (layer "F.Fab")
+        (effects (font (size 1 1) (thickness 0.15)))
+    )
+    (fp_line (start -2.05 4.16) (end -2.05 4.8)
+      (stroke (width 0.12) (type solid)) (layer "F.SilkS"))
+    (fp_line (start -2.05 4.8) (end -1.65 4.8)
+      (stroke (width 0.12) (type solid)) (layer "F.SilkS"))
+    (fp_line (start -1.81 -3.16) (end -1.81 4.56)
+      (stroke (width 0.12) (type solid)) (layer "F.SilkS"))
+    (fp_line (start -1.81 -3.16) (end 5.31 -3.16)
+      (stroke (width 0.12) (type solid)) (layer "F.SilkS"))
+    (fp_line (start -1.81 3) (end 5.31 3)
+      (stroke (width 0.12) (type solid)) (layer "F.SilkS"))
+    (fp_line (start -1.81 4.1) (end 5.31 4.1)
+      (stroke (width 0.12) (type solid)) (layer "F.SilkS"))
+    (fp_line (start -1.81 4.56) (end 5.31 4.56)
+      (stroke (width 0.12) (type solid)) (layer "F.SilkS"))
+    (fp_line (start 2.355 0.941) (end 2.226 1.069)
+      (stroke (width 0.12) (type solid)) (layer "F.SilkS"))
+    (fp_line (start 2.525 1.181) (end 2.431 1.274)
+      (stroke (width 0.12) (type solid)) (layer "F.SilkS"))
+    (fp_line (start 4.57 -1.275) (end 4.476 -1.181)
+      (stroke (width 0.12) (type solid)) (layer "F.SilkS"))
+    (fp_line (start 4.775 -1.069) (end 4.646 -0.941)
+      (stroke (width 0.12) (type solid)) (layer "F.SilkS"))
+    (fp_line (start 5.31 -3.16) (end 5.31 4.56)
+      (stroke (width 0.12) (type solid)) (layer "F.SilkS"))
+    (fp_arc (start -1.425358 0.889894) (mid -1.680286 0.014012) (end -1.44 -0.866)
+      (stroke (width 0.12) (type solid)) (layer "F.SilkS"))
+    (fp_arc (start -0.889894 -1.425358) (mid -0.014012 -1.680286) (end 0.866 -1.44)
+      (stroke (width 0.12) (type solid)) (layer "F.SilkS"))
+    (fp_arc (start 0.028674 1.680099) (mid -0.435535 1.622918) (end -0.866 1.44)
+      (stroke (width 0.12) (type solid)) (layer "F.SilkS"))
+    (fp_arc (start 0.890264 1.424721) (mid 0.463071 1.61492) (end 0 1.68)
+      (stroke (width 0.12) (type solid)) (layer "F.SilkS"))
+    (fp_arc (start 1.425504 -0.890193) (mid 1.680626 0.000476) (end 1.425 0.891)
+      (stroke (width 0.12) (type solid)) (layer "F.SilkS"))
+    (fp_circle (center 3.5 0) (end 5.18 0)
+      (stroke (width 0.12) (type solid)) (fill none) (layer "F.SilkS"))
+    (fp_line (start -2.25 -3.6) (end -2.25 5)
+      (stroke (width 0.05) (type solid)) (layer "F.CrtYd"))
+    (fp_line (start -2.25 5) (end 5.75 5)
+      (stroke (width 0.05) (type solid)) (layer "F.CrtYd"))
+    (fp_line (start 5.75 -3.6) (end -2.25 -3.6)
+      (stroke (width 0.05) (type solid)) (layer "F.CrtYd"))
+    (fp_line (start 5.75 5) (end 5.75 -3.6)
+      (stroke (width 0.05) (type solid)) (layer "F.CrtYd"))
+    (fp_line (start -1.75 -3.1) (end 5.25 -3.1)
+      (stroke (width 0.1) (type solid)) (layer "F.Fab"))
+    (fp_line (start -1.75 3) (end 5.25 3)
+      (stroke (width 0.1) (type solid)) (layer "F.Fab"))
+    (fp_line (start -1.75 4.1) (end -1.75 -3.1)
+      (stroke (width 0.1) (type solid)) (layer "F.Fab"))
+    (fp_line (start -1.75 4.1) (end 5.25 4.1)
+      (stroke (width 0.1) (type solid)) (layer "F.Fab"))
+    (fp_line (start -1.35 4.5) (end -1.75 4.1)
+      (stroke (width 0.1) (type solid)) (layer "F.Fab"))
+    (fp_line (start 0.955 -1.138) (end -1.138 0.955)
+      (stroke (width 0.1) (type solid)) (layer "F.Fab"))
+    (fp_line (start 1.138 -0.955) (end -0.955 1.138)
+      (stroke (width 0.1) (type solid)) (layer "F.Fab"))
+    (fp_line (start 4.455 -1.138) (end 2.363 0.955)
+      (stroke (width 0.1) (type solid)) (layer "F.Fab"))
+    (fp_line (start 4.638 -0.955) (end 2.546 1.138)
+      (stroke (width 0.1) (type solid)) (layer "F.Fab"))
+    (fp_line (start 5.25 -3.1) (end 5.25 4.5)
+      (stroke (width 0.1) (type solid)) (layer "F.Fab"))
+    (fp_line (start 5.25 4.5) (end -1.35 4.5)
+      (stroke (width 0.1) (type solid)) (layer "F.Fab"))
+    (fp_circle (center 0 0) (end 1.5 0)
+      (stroke (width 0.1) (type solid)) (fill none) (layer "F.Fab"))
+    (fp_circle (center 3.5 0) (end 5 0)
+      (stroke (width 0.1) (type solid)) (fill none) (layer "F.Fab"))
+    (pad "1" thru_hole rect (at 0 0 270) (size 2.4 2.4) (drill 1.2) (layers "*.Cu" "*.Mask")
+      (net 1 "GND") (pinfunction "Pin_1") (pintype "passive"))
+    (pad "2" thru_hole circle (at 3.5 0 270) (size 2.4 2.4) (drill 1.2) (layers "*.Cu" "*.Mask")
+      (net 3 "/DCC1") (pinfunction "Pin_2") (pintype "passive"))
+    (model "${KICAD6_3DMODEL_DIR}/TerminalBlock_Phoenix.3dshapes/TerminalBlock_Phoenix_PT-1,5-2-3.5-H_1x02_P3.50mm_Horizontal.wrl"
+      (offset (xyz 0 0 0))
+      (scale (xyz 1 1 1))
+      (rotate (xyz 0 0 0))
     )
   )
@@
         (effects (font (size 1 1) (thickness 0.15)))
     )
-    (fp_text value "1k" (at 0 1.82) (layer "F.Fab")
+    (fp_text value "330" (at 0 1.82) (layer "F.Fab")
         (effects (font (size 1 1) (thickness 0.15)))
     )
@@
     (property "ki_keywords" "test point tp")
     (attr exclude_from_pos_files)
-    (fp_text reference "GND" (at 0 -2.148) (layer "F.SilkS")
+    (fp_text reference "TP4" (at 0 -2.148) (layer "F.SilkS")
         (effects (font (size 1 1) (thickness 0.15)))
     )
@@
     (property "ki_keywords" "test point tp")
     (attr exclude_from_pos_files)
-    (fp_text reference "+V" (at 0 -2.148) (layer "F.SilkS")
+    (fp_text reference "TP3" (at 0 -2.148) (layer "F.SilkS")
         (effects (font (size 1 1) (thickness 0.15)))
     )
@@
         (effects (font (size 1 1) (thickness 0.15)))
     )
-    (fp_text value "1k" (at 0 1.82) (layer "F.Fab")
+    (fp_text value "330" (at 0 1.82) (layer "F.Fab")
         (effects (font (size 1 1) (thickness 0.15)))
     )
@@
         (effects (font (size 1 1) (thickness 0.15)))
     )
-    (fp_text value "Screw_Terminal_01x02" (at 1.75 5.56 90) (layer "F.Fab") hide
+    (fp_text value "DCC" (at 1.75 5.56 90) (layer "F.Fab") hide
         (effects (font (size 1 1) (thickness 0.15)))
     )
@@
         (effects (font (size 1 1) (thickness 0.15)))
     )
-    (fp_text value "1k" (at 0 1.82) (layer "F.Fab")
+    (fp_text value "330" (at 0 1.82) (layer "F.Fab")
         (effects (font (size 1 1) (thickness 0.15)))
     )
@@
     (fp_arc (start -5.39242 6.69798) (mid -5.961768 6.462148) (end -6.1976 5.8928)
       (stroke (width 0.2032) (type solid)) (layer "F.SilkS"))
-    (fp_arc (start 5.39242 -6.69798) (mid 5.961768 -6.462148) (end 6.1976 -5.8928)
+    (fp_arc (start 5.39242 -6.69798) (mid 5.961755 -6.462141) (end 6.1976 -5.8928)
       (stroke (width 0.2032) (type solid)) (layer "F.SilkS"))
-    (fp_arc (start 6.1976 5.8928) (mid 5.961768 6.462148) (end 5.39242 6.69798)
+    (fp_arc (start 6.1976 5.8928) (mid 5.961769 6.462155) (end 5.39242 6.69798)
       (stroke (width 0.2032) (type solid)) (layer "F.SilkS"))
     (fp_circle (center 0 0) (end 0 -2.99974)

Commit message: 28/05/25 13:45 Arrakis.local
Parts:
- added Brd1: SSD1306, SSD1306:128x64OLED, F.Cu at (186.1, 79.4)
- U2: moved to B.Cu
- moved J4 80.2 mm to (109.2, 72.4)
- moved J5 80.2 mm to (109.2, 83.2)
- moved U2 47.6 mm to (146.7, 95.9)
- moved R1 12.8 mm to (128.9, 93.1)
- moved R2 12.8 mm to (128.9, 96.4)
- moved R3 12.8 mm to (128.9, 99.7)
- moved R4 12.8 mm to (128.9, 103.0)
- moved J2 10.0 mm to (142.2, 101.0)
Routing:
- net BLUE: track 15.0 -> 68.6 mm, vias 1 -> 0
- net SCL: track 67.5 -> 120.6 mm, vias 0 -> 2
- net Net-(U2-VBUS): track 70.8 -> 23.2 mm
- net /VSYS: track 72.7 -> 31.3 mm
- net BTN: track 30.6 -> 66.5 mm
- net PINA: track 31.6 -> 66.4 mm
- net PINB: track 29.2 -> 57.7 mm
- net 3V3: track 119.3 -> 142.5 mm, vias 1 -> 0
- net 3V3_OUT: track 40.9 -> 19.9 mm, vias 1 -> 0
- net GREEN: track 29.7 -> 48.0 mm, vias 1 -> 0
- net SDA: track 70.2 -> 85.6 mm, vias 0 -> 2
- net Net-(S1--R): track 49.9 -> 34.7 mm
- net /DCC1: track 13.1 -> 25.1 mm
- net Net-(S1--G): track 43.8 -> 32.0 mm
- net +5V: track 58.0 -> 48.5 mm, vias 0 -> 2
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