File: PicoBleCentral/PicoBleCentral.kicad_pcb (KiCad board)
At the start: 2 copper layers, 115.6 x 55.2 mm, 29 parts, among them J1 DCC, J2 3V3 Sel, J3 keypad, J4 grove 2mm, J5 i2c, J6 12V, Q1 DMG2305UX-7, SW1 SW_Push, U1 AP7384-50Y, U2 Pico_RaspberryPico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

Commit message: 30/05/25 09:30 Arrakis.local
Parts:
- GND: renamed from TP4; moved to B.Cu
- Q1: footprint Package_TO_SOT_SMD:SOT-23-3 -> Package_TO_SOT_SMD:SOT-23_Handsoldering
- U4: footprint Package_TO_SOT_SMD:SOT-223-3_TabPin2 -> Package_TO_SOT_SMD:SOT-23_Handsoldering
- V+: renamed from TP3; moved to B.Cu
- moved S1 1.42 mm to (128.9, 78.1), turned to -90 degrees
- turned GND to 180 degrees
- turned V+ to 180 degrees
Routing:
- net SDA: track 85.6 -> 120.5 mm
- net SCL: track 120.6 -> 138.2 mm
- net +5V: track 48.5 -> 62.7 mm, vias 2 -> 0
- net PINB: track 57.7 -> 69.7 mm
- net 3V3: track 142.5 -> 132.4 mm, vias 0 -> 1
- net RED: track 44.6 -> 54.3 mm
- net 3V3a: track 24.3 -> 16.1 mm
- net PINA: track 66.4 -> 74.3 mm
- net Net-(S1--B): track 29.0 -> 21.6 mm
- net Net-(S1-SW): track 24.9 -> 18.9 mm
- net Net-(S1--G): track 32.0 -> 36.1 mm
- net +V: track 86.2 -> 83.1 mm, vias 0 -> 1
- net GND: track 22.0 -> 20.1 mm
- net GREEN: track 48.0 -> 46.4 mm
- net Net-(S1--R): track 34.7 -> 33.2 mm
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