File: PicoRfid/PicoRfd.kicad_pcb (KiCad board)
At the start: 2 copper layers, 100 x 100 mm, 23 parts, among them J1 12v, J2 CBUS, J3 5V select, J5 Grove 2mm, Q1 DMG2305UX-7, SW1 SW_Push, U1 AMS1117-3.3, U2 AMS1117-5.0, U3 Pico_RaspberryPico, U5 CAT24C256

Commit message: 07/09/25 10:05 Arrakis.local
Parts:
- removed the C2 at (146.1, 121.2)
- removed D2: 1N4148, Diode_THT:D_DO-35_SOD27_P7.62mm_Horizontal
- removed NT1, NT2: NetTie_2, NetTie:NetTie-2_SMD_Pad0.5mm
- added J5: Grove 2mm, Seed Grove etc:HW4-2.0, F.Cu at (159.0, 61.0)
- added J6: IDC_A, Connector_IDC:IDC-Header_2x04_P2.54mm_Vertical, F.Cu at (178.8, 95.3)
- added J7: IDC_B, Connector_IDC:IDC-Header_2x04_P2.54mm_Vertical, F.Cu at (179.1, 107.4)
- added J8: IDC_C, Connector_IDC:IDC-Header_2x04_P2.54mm_Vertical, F.Cu at (179.7, 120.0)
- added J9: IDC_D, Connector_IDC:IDC-Header_2x04_P2.54mm_Vertical, F.Cu at (179.7, 133.3)
- moved SW1 21.2 mm to (144.1, 77.5), turned to 90 degrees
- renumbered C3 to C2, C4 to C3, J5 to J4, U5 to U3, U3 to U4
Connections:
- SW1 pad 2: Net-(SW1-Pad2) -> Net-(U4-RUN)
- U4 pad 11: unconnected-(U3-GPIO8-Pad11) -> /CSB
- U4 pad 12: unconnected-(U3-GPIO9-Pad12) -> /CSC
- U4 pad 14: unconnected-(U3-GPIO10-Pad14) -> /CSD
- U4 pad 20: unconnected-(U3-GPIO15-Pad20) -> /RST
- U4 pad 21: unconnected-(U3-GPIO16-Pad21) -> /MOSI
- U4 pad 22: unconnected-(U3-GPIO17-Pad22) -> /SCK
- U4 pad 24: unconnected-(U3-GPIO18-Pad24) -> /CSA
- U4 pad 25: unconnected-(U3-GPIO19-Pad25) -> /MISO
- U4 pad 30: Net-(U3-RUN) -> Net-(U4-RUN)
Routing:
- net GND: track 257.3 -> 0.00 mm
- net /3V3: track 174.7 -> 0.00 mm, vias 3 -> 0
- net /SCL: track 111.9 -> 0.00 mm, vias 1 -> 0
- net /SDA: track 108.6 -> 0.00 mm, vias 1 -> 0
- net /VSYS: track 83.6 -> 0.00 mm, vias 1 -> 0
- net /VBUS: track 79.1 -> 0.00 mm
- net /5V: track 49.5 -> 0.00 mm, vias 1 -> 0
- net Net-(D1-A): track 31.8 -> 0.00 mm
- net Net-(C2-Pad2): track 30.2 -> 0.00 mm
- net /5Vopt: track 29.5 -> 0.00 mm, vias 1 -> 0
- net /12V: track 21.5 -> 0.00 mm

Commit message: 07/09/25 10:39 Titan.local
Parts:
- removed U3: CAT24C256, Package_DIP:DIP-8_W7.62mm_LongPads
Connections:
- U4 pad 20: /RST -> unconnected-(U4-GPIO15-Pad20)
- U4 pad 26: unconnected-(U4-GPIO20-Pad26) -> /RST
Routing:
- net GND: track 0.00 -> 297.0 mm, vias 0 -> 2
- net /3V3: track 0.00 -> 206.2 mm
- net /CSD: track 0.00 -> 103.4 mm, vias 0 -> 1
- net /RST: track 0.00 -> 102.5 mm
- net /CSC: track 0.00 -> 100.3 mm, vias 0 -> 1
- net /MISO: track 0.00 -> 100.0 mm
- net /MOSI: track 0.00 -> 96.6 mm
- net /SCK: track 0.00 -> 93.5 mm
- net /CSB: track 0.00 -> 88.8 mm, vias 0 -> 1
- net /SDA: track 0.00 -> 85.4 mm, vias 0 -> 1
- net /VSYS: track 0.00 -> 84.1 mm, vias 0 -> 1
- net /SCL: track 0.00 -> 82.0 mm
- net /VBUS: track 0.00 -> 79.1 mm
- net /CSA: track 0.00 -> 53.2 mm, vias 0 -> 1
- net /5V: track 0.00 -> 49.2 mm, vias 0 -> 1
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
Commit message: 07/09/25 11:15 Arrakis.local
Routing:
- net GND: track 297.0 -> 0.00 mm, vias 2 -> 0
- net /3V3: track 206.2 -> 0.00 mm
- net /CSD: track 103.4 -> 0.00 mm, vias 1 -> 0
- net /RST: track 102.5 -> 0.00 mm
- net /CSC: track 100.3 -> 0.00 mm, vias 1 -> 0
- net /MISO: track 100.0 -> 0.00 mm
- net /MOSI: track 96.6 -> 0.00 mm
- net /SCK: track 93.5 -> 0.00 mm
- net /CSB: track 88.8 -> 0.00 mm, vias 1 -> 0
- net /SDA: track 85.4 -> 0.00 mm, vias 1 -> 0
- net /VSYS: track 84.1 -> 0.00 mm, vias 1 -> 0
- net /SCL: track 82.0 -> 0.00 mm
- net /VBUS: track 79.1 -> 0.00 mm
- net /CSA: track 53.2 -> 0.00 mm, vias 1 -> 0
- net /5V: track 49.2 -> 0.00 mm, vias 1 -> 0
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