File: PicoRfid/PicoRfd.kicad_sch (KiCad schematic)
At the start: 19 parts, among them J1 12v, J2 CBUS, J3 5V select, J5 Grove 2mm, Q1 DMG2305UX-7, SW2 SW_Push, U1 AMS1117-3.3, U2 AMS1117-5.0, U3 Pico_RaspberryPico, U5 CAT24C256

Commit message: 07/09/25 10:05 Arrakis.local
Parts:
- added J5: Grove 2mm, Seed Grove etc:HW4-2.0, symbol Connector:Screw_Terminal_01x04
- added J6: IDC_A, Connector_IDC:IDC-Header_2x04_P2.54mm_Vertical, symbol Connector_Generic:Conn_01x08
- added J7: IDC_B, Connector_IDC:IDC-Header_2x04_P2.54mm_Vertical, symbol Connector_Generic:Conn_01x08
- added J8: IDC_C, Connector_IDC:IDC-Header_2x04_P2.54mm_Vertical, symbol Connector_Generic:Conn_01x08
- added J9: IDC_D, Connector_IDC:IDC-Header_2x04_P2.54mm_Vertical, symbol Connector_Generic:Conn_01x08
- renumbered C3 to C2, C4 to C3, J5 to J4, SW2 to SW1, U5 to U3, U3 to U4
Connections:
- net 3V3: now also J5.3 (Pin_3), J6.8 (Pin_8), J7.8 (Pin_8), J8.8 (Pin_8), J9.8 (Pin_8)
- net GND: now also J5.4 (Pin_4), J6.6 (Pin_6), J7.6 (Pin_6), J8.6 (Pin_6), J9.6 (Pin_6)
- net SCL: now also J5.1 (Pin_1)
- net SDA: now also J5.2 (Pin_2)
- net CSB: now reaches U4.11 (GPIO8)
- net CSB: now also J7.1 (Pin_1)
- net CSC: now reaches U4.12 (GPIO9)
- net CSC: now also J8.1 (Pin_1)
- net CSD: now reaches U4.14 (GPIO10)
- net CSD: now also J9.1 (Pin_1)
- net RST: now reaches U4.20 (GPIO15)
- net RST: now also J6.7 (Pin_7), J7.7 (Pin_7), J8.7 (Pin_7), J9.7 (Pin_7)
- net MOSI: now reaches U4.21 (GPIO16)
- net MOSI: now also J6.3 (Pin_3), J7.3 (Pin_3), J8.3 (Pin_3), J9.3 (Pin_3)
- net SCK: now reaches U4.22 (GPIO17)
- net SCK: now also J6.2 (Pin_2), J7.2 (Pin_2), J8.2 (Pin_2), J9.2 (Pin_2)
- net CSA: now reaches U4.24 (GPIO18)
- net CSA: now also J6.1 (Pin_1)
- net MISO: now reaches U4.25 (GPIO19)
- net MISO: now also J6.4 (Pin_4), J7.4 (Pin_4), J8.4 (Pin_4), J9.4 (Pin_4)
- new net IRQ: J6.5 (Pin_5), J7.5 (Pin_5), J8.5 (Pin_5), J9.5 (Pin_5)
- no-connect marks 39 -> 32

Commit message: 07/09/25 10:39 Titan.local
Parts:
- removed U3: CAT24C256, Package_DIP:DIP-8_W7.62mm_LongPads, symbol Memory_EEPROM:CAT24C256
Connections:
- net RST: now also U4.26 (GPIO20); no longer U4.20 (GPIO15)
- no-connect marks 32 -> 28
Other:
- moved on the sheet: U4

Commit message: 07/09/25 11:15 Arrakis.local
Other:
- moved on the sheet: D1, J4, U4
