File: PcbBare/PcbBare.kicad_pcb (KiCad board)
At the start: 2 copper layers, 76.2 x 50.8 mm, 4 parts

Commit message: 07/09/25 21:50 Titan.local
Parts:
- removed REF** (x4): MountingHole_2.1mm, MountingHole:MountingHole_2.1mm
- added H1: MountingHole_3.2mm_M3, MountingHole:MountingHole_3.2mm_M3, F.Cu at (78.7, 123.2)
- added h2: MountingHole_3.2mm_M3, MountingHole:MountingHole_3.2mm_M3, F.Cu at (55.9, 107.3)
- added h3: MountingHole_3.2mm_M3, MountingHole:MountingHole_3.2mm_M3, F.Cu at (55.2, 146.7)
- added h4: MountingHole_3.2mm_M3, MountingHole:MountingHole_3.2mm_M3, F.Cu at (122.6, 146.7)
- added h5: MountingHole_3.2mm_M3, MountingHole:MountingHole_3.2mm_M3, F.Cu at (121.9, 106.0)
Other:
- board text added: "Add holes as fottprint change grid to position and delete names etc Chage Ref ** to a name before trying to route or it won't work"
- board text removed: "Add holes as fottprint change grid to position and delete names etc"
Changed lines of the file:
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@@
   )
   (net 0 "")
-  (footprint "MountingHole:MountingHole_2.1mm" (layer "F.Cu")
-    (at 54.61 105.41)
-    (descr "Mounting Hole 2.1mm, no annular")
-    (tags "mounting hole 2.1mm no annular")
+  (footprint "MountingHole:MountingHole_3.2mm_M3" (layer "F.Cu")
+    (at 55.245 146.685)
+    (descr "Mounting Hole 3.2mm, no annular, M3")
+    (tags "mounting hole 3.2mm no annular m3")
     (attr exclude_from_pos_files exclude_from_bom)
-    (fp_text reference "REF**" (at 0 -3.2) (layer "F.SilkS") hide
+    (fp_text reference "h3" (at 0 -4.2) (layer "F.SilkS")
         (effects (font (size 1 1) (thickness 0.15)))
     )
-    (fp_text value "MountingHole_2.1mm" (at 0 3.2) (layer "F.Fab") hide
+    (fp_text value "MountingHole_3.2mm_M3" (at 0 4.2) (layer "F.Fab") hide
         (effects (font (size 1 1) (thickness 0.15)))
     )
@@
         (effects (font (size 1 1) (thickness 0.15)))
     )
-    (fp_circle (center 0 0) (end 2.1 0)
+    (fp_circle (center 0 0) (end 3.2 0)
       (stroke (width 0.15) (type solid)) (fill none) (layer "Cmts.User"))
-    (fp_circle (center 0 0) (end 2.35 0)
+    (fp_circle (center 0 0) (end 3.45 0)
       (stroke (width 0.05) (type solid)) (fill none) (layer "F.CrtYd"))
-    (pad "" np_thru_hole circle (at 0 0) (size 2.1 2.1) (drill 2.1) (layers "*.Cu" "*.Mask"))
+    (pad "" np_thru_hole circle (at 0 0) (size 3.2 3.2) (drill 3.2) (layers "*.Cu" "*.Mask"))
   )
-  (footprint "MountingHole:MountingHole_2.1mm" (layer "F.Cu")
-    (at 123.19 147.955)
-    (descr "Mounting Hole 2.1mm, no annular")
-    (tags "mounting hole 2.1mm no annular")
+  (footprint "MountingHole:MountingHole_3.2mm_M3" (layer "F.Cu")
+    (at 121.92 106.045)
+    (descr "Mounting Hole 3.2mm, no annular, M3")
+    (tags "mounting hole 3.2mm no annular m3")
     (attr exclude_from_pos_files exclude_from_bom)
-    (fp_text reference "REF**" (at 0 -3.2) (layer "F.SilkS") hide
+    (fp_text reference "h5" (at 0 -4.2) (layer "F.SilkS")
         (effects (font (size 1 1) (thickness 0.15)))
     )
-    (fp_text value "MountingHole_2.1mm" (at 0 3.2) (layer "F.Fab") hide
+    (fp_text value "MountingHole_3.2mm_M3" (at 0 4.2) (layer "F.Fab") hide
         (effects (font (size 1 1) (thickness 0.15)))
     )
@@
         (effects (font (size 1 1) (thickness 0.15)))
     )
-    (fp_circle (center 0 0) (end 2.1 0)
+    (fp_circle (center 0 0) (end 3.2 0)
       (stroke (width 0.15) (type solid)) (fill none) (layer "Cmts.User"))
-    (fp_circle (center 0 0) (end 2.35 0)
+    (fp_circle (center 0 0) (end 3.45 0)
       (stroke (width 0.05) (type solid)) (fill none) (layer "F.CrtYd"))
-    (pad "" np_thru_hole circle (at 0 0) (size 2.1 2.1) (drill 2.1) (layers "*.Cu" "*.Mask"))
+    (pad "" np_thru_hole circle (at 0 0) (size 3.2 3.2) (drill 3.2) (layers "*.Cu" "*.Mask"))
   )
-  (footprint "MountingHole:MountingHole_2.1mm" (layer "F.Cu")
-    (at 54.61 147.955)
-    (descr "Mounting Hole 2.1mm, no annular")
-    (tags "mounting hole 2.1mm no annular")
+  (footprint "MountingHole:MountingHole_3.2mm_M3" (layer "F.Cu")
+    (at 55.88 107.315)
+    (descr "Mounting Hole 3.2mm, no annular, M3")
+    (tags "mounting hole 3.2mm no annular m3")
     (attr exclude_from_pos_files exclude_from_bom)
-    (fp_text reference "REF**" (at 0 -3.2) (layer "F.SilkS") hide
+    (fp_text reference "h2" (at 0 -4.2) (layer "F.SilkS")
         (effects (font (size 1 1) (thickness 0.15)))
     )
-    (fp_text value "MountingHole_2.1mm" (at 0 3.2) (layer "F.Fab") hide
+    (fp_text value "MountingHole_3.2mm_M3" (at 0 4.2) (layer "F.Fab") hide
         (effects (font (size 1 1) (thickness 0.15)))
     )
@@
         (effects (font (size 1 1) (thickness 0.15)))
     )
-    (fp_circle (center 0 0) (end 2.1 0)
+    (fp_circle (center 0 0) (end 3.2 0)
       (stroke (width 0.15) (type solid)) (fill none) (layer "Cmts.User"))
-    (fp_circle (center 0 0) (end 2.35 0)
+    (fp_circle (center 0 0) (end 3.45 0)
       (stroke (width 0.05) (type solid)) (fill none) (layer "F.CrtYd"))
-    (pad "" np_thru_hole circle (at 0 0) (size 2.1 2.1) (drill 2.1) (layers "*.Cu" "*.Mask"))
+    (pad "" np_thru_hole circle (at 0 0) (size 3.2 3.2) (drill 3.2) (layers "*.Cu" "*.Mask"))
   )
-  (footprint "MountingHole:MountingHole_2.1mm" (layer "F.Cu")
-    (at 123.19 105.41)
-    (descr "Mounting Hole 2.1mm, no annular")
-    (tags "mounting hole 2.1mm no annular")
+  (footprint "MountingHole:MountingHole_3.2mm_M3" (layer "F.Cu")
+    (at 122.555 146.685)
+    (descr "Mounting Hole 3.2mm, no annular, M3")
+    (tags "mounting hole 3.2mm no annular m3")
     (attr exclude_from_pos_files exclude_from_bom)
-    (fp_text reference "REF**" (at 0 -3.2) (layer "F.SilkS") hide
+    (fp_text reference "h4" (at 0 -4.2) (layer "F.SilkS")
         (effects (font (size 1 1) (thickness 0.15)))
     )
-    (fp_text value "MountingHole_2.1mm" (at 0 3.2) (layer "F.Fab") hide
+    (fp_text value "MountingHole_3.2mm_M3" (at 0 4.2) (layer "F.Fab") hide
         (effects (font (size 1 1) (thickness 0.15)))
     )
@@
         (effects (font (size 1 1) (thickness 0.15)))
     )
-    (fp_circle (center 0 0) (end 2.1 0)
+    (fp_circle (center 0 0) (end 3.2 0)
       (stroke (width 0.15) (type solid)) (fill none) (layer "Cmts.User"))
-    (fp_circle (center 0 0) (end 2.35 0)
+    (fp_circle (center 0 0) (end 3.45 0)
       (stroke (width 0.05) (type solid)) (fill none) (layer "F.CrtYd"))
-    (pad "" np_thru_hole circle (at 0 0) (size 2.1 2.1) (drill 2.1) (layers "*.Cu" "*.Mask"))
+    (pad "" np_thru_hole circle (at 0 0) (size 3.2 3.2) (drill 3.2) (layers "*.Cu" "*.Mask"))
+  )
+  (footprint "MountingHole:MountingHole_3.2mm_M3" (layer "F.Cu")
+    (at 78.74 123.19)
+    (descr "Mounting Hole 3.2mm, no annular, M3")
+    (tags "mounting hole 3.2mm no annular m3")
+    (attr exclude_from_pos_files exclude_from_bom)
+    (fp_text reference "H1" (at 0 -4.2) (layer "F.SilkS")
+        (effects (font (size 1 1) (thickness 0.15)))
+    )
+    (fp_text value "MountingHole_3.2mm_M3" (at 0 4.2) (layer "F.Fab")
+        (effects (font (size 1 1) (thickness 0.15)))
+    )
+    (fp_text user "${REFERENCE}" (at 0 0) (layer "F.Fab")
+        (effects (font (size 1 1) (thickness 0.15)))
+    )
+    (fp_circle (center 0 0) (end 3.2 0)
+      (stroke (width 0.15) (type solid)) (fill none) (layer "Cmts.User"))
+    (fp_circle (center 0 0) (end 3.45 0)
+      (stroke (width 0.05) (type solid)) (fill none) (layer "F.CrtYd"))
+    (pad "" np_thru_hole circle (at 0 0) (size 3.2 3.2) (drill 3.2) (layers "*.Cu" "*.Mask"))
   )
   (gr_line (start 127 106.68) (end 127 147.32)
@@
   (gr_arc (start 127 147.32) (mid 125.512102 150.912102) (end 121.92 152.4)
     (stroke (width 0.1) (type default)) (layer "Edge.Cuts"))
-  (gr_text "ground plane is a zone on B Cu" (at 68.58 114.3) (layer "F.SilkS")
+  (gr_text "ground plane is a zone on B Cu" (at 68.58 116.84) (layer "F.SilkS")
     (effects (font (size 1 1) (thickness 0.15)) (justify left bottom))
   )
@@
     (effects (font (size 1 1) (thickness 0.15)) (justify left bottom))
   )
-  (gr_text "Add holes as fottprint change grid to position and delete names etc\n" (at 68.58 111.76) (layer "F.SilkS")
+  (gr_text "Add holes as fottprint change grid to position and delete names etc\nChage Ref ** to a name before trying to route or it won't work\n\n" (at 67.945 114.935) (layer "F.SilkS")
     (effects (font (size 1 1) (thickness 0.15)) (justify left bottom))
   )

Commit message: 07/09/25 22:02 Titan.local
Routing:
- added copper zone on F.Cu, net (none)
- removed copper zone on B.Cu, net (none)
Other:
- board text added: "ground plane is a zone on B Cu create from rect and filet lines, the right click and create zone"
- board text removed: "ground plane is a zone on B Cu"
Changed lines of the file:
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@@
   (gr_arc (start 127 147.32) (mid 125.512102 150.912102) (end 121.92 152.4)
     (stroke (width 0.1) (type default)) (layer "Edge.Cuts"))
-  (gr_text "ground plane is a zone on B Cu" (at 68.58 116.84) (layer "F.SilkS")
+  (gr_text "ground plane is a zone on B Cu create from rect and \nfilet lines, the right click and create zone" (at 68.58 116.84) (layer "F.SilkS")
     (effects (font (size 1 1) (thickness 0.15)) (justify left bottom))
   )
@@
     (effects (font (size 1 1) (thickness 0.15)) (justify left bottom))
   )
-  (zone (net 0) (net_name "") (layer "B.Cu") (hatch edge 0.5)
+  (zone (net 0) (net_name "") (layer "F.Cu") (hatch edge 0.5)
+    (connect_pads (clearance 0.5))
+    (min_thickness 0.25) (filled_areas_thickness no)
+    (fill (thermal_gap 0.5) (thermal_bridge_width 0.5) (island_removal_mode 1) (island_area_min 9.999999))
+    (polygon
+      (pts
+        (arc (start 125.095 116.205) (mid 121.375256 107.224744) (end 112.395 103.505))
+        (arc (start 66.04 103.505) (mid 57.059744 107.224744) (end 53.34 116.205))
+        (arc (start 53.34 137.16) (mid 57.059744 146.140256) (end 66.04 149.86))
+        (arc (start 112.395 149.86) (mid 121.375256 146.140256) (end 125.095 137.16))
+      )
+    )
+  )
+  (zone (net 0) (net_name "") (layer "F.Cu") (hatch edge 0.5)
     (connect_pads (clearance 0.5))
     (min_thickness 0.25) (filled_areas_thickness no)
@@
     (polygon
       (pts
-        (xy 53.34 110.49)
-        (xy 59.055 104.775)
-        (xy 119.38 104.775)
-        (xy 124.46 109.855)
-        (xy 124.46 144.145)
-        (xy 118.11 149.225)
-        (xy 59.055 149.225)
-        (xy 52.705 142.24)
-        (xy 52.705 110.49)
+        (arc (start 100.33 123.19) (mid 99.431974 123.561974) (end 99.06 124.46))
+        (arc (start 99.06 127.635) (mid 99.431974 128.533026) (end 100.33 128.905))
+        (arc (start 110.49 128.905) (mid 111.388026 128.533026) (end 111.76 127.635))
+        (arc (start 111.76 124.46) (mid 111.388026 123.561974) (end 110.49 123.19))
       )
     )
