File: PicoRfc522/PicoRfc522_pro.kicad_sch (KiCad schematic)
At the start: 19 parts, among them J1 5V sel, J2 Grove 2mm, J3 Screw_Terminal_01x04, J4 Screw_Terminal_01x02, J5 IDC1, J6 IDC1, J7 IDC1, J8 IDC1, Q1 DMG2305UX-7, SW1 SW_Push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

Commit message: 07/09/25 22:20 Titan.local
Parts:
- removed H1, H2, H3, H4: MountingHole, MountingHole:MountingHole_3.2mm_M3_DIN965, symbol Mechanical:MountingHole
Changed lines of the file:
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@@
     (effects (font (size 1.27 1.27)) (justify right bottom))
-  )
-  (symbol (lib_id "Mechanical:MountingHole") (at 120.65 102.87 0) (unit 1)
-    (in_bom yes) (on_board yes) (dnp no) (fields_autoplaced)
-    (property "Reference" "H3" (at 123.19 102.235 0)
-      (effects (font (size 1.27 1.27)) (justify left) hide)
-    )
-    (property "Value" "MountingHole" (at 123.19 104.775 0)
-      (effects (font (size 1.27 1.27)) (justify left) hide)
-    )
-    (property "Footprint" "MountingHole:MountingHole_3.2mm_M3_DIN965" (at 120.65 102.87 0)
-      (effects (font (size 1.27 1.27)) hide)
-    )
-    (property "Datasheet" "~" (at 120.65 102.87 0)
-      (effects (font (size 1.27 1.27)) hide)
-    )
-    (instances
-      (project "PicoRfc522_pro"
-        (path "/9472a9f5-95f0-4abd-b6a1-4228d4355bea"
-          (reference "H3") (unit 1)
-        )
-      )
-    )
   )
   (symbol (lib_id "Connector:Conn_01x03_Pin") (at 30.48 64.77 0) (unit 1)
@@
         (path "/9472a9f5-95f0-4abd-b6a1-4228d4355bea"
           (reference "Q1") (unit 1)
-        )
-      )
-    )
-  )
-  (symbol (lib_id "Mechanical:MountingHole") (at 104.775 102.235 0) (unit 1)
-    (in_bom yes) (on_board yes) (dnp no) (fields_autoplaced)
-    (property "Reference" "H2" (at 107.315 101.6 0)
-      (effects (font (size 1.27 1.27)) (justify left) hide)
-    )
-    (property "Value" "MountingHole" (at 107.315 104.14 0)
-      (effects (font (size 1.27 1.27)) (justify left) hide)
-    )
-    (property "Footprint" "MountingHole:MountingHole_3.2mm_M3_DIN965" (at 104.775 102.235 0)
-      (effects (font (size 1.27 1.27)) hide)
-    )
-    (property "Datasheet" "~" (at 104.775 102.235 0)
-      (effects (font (size 1.27 1.27)) hide)
-    )
-    (instances
-      (project "PicoRfc522_pro"
-        (path "/9472a9f5-95f0-4abd-b6a1-4228d4355bea"
-          (reference "H2") (unit 1)
-        )
-      )
-    )
-  )
-  (symbol (lib_id "Mechanical:MountingHole") (at 141.605 102.235 0) (unit 1)
-    (in_bom yes) (on_board yes) (dnp no) (fields_autoplaced)
-    (property "Reference" "H4" (at 144.145 101.6 0)
-      (effects (font (size 1.27 1.27)) (justify left) hide)
-    )
-    (property "Value" "MountingHole" (at 144.145 104.14 0)
-      (effects (font (size 1.27 1.27)) (justify left) hide)
-    )
-    (property "Footprint" "MountingHole:MountingHole_3.2mm_M3_DIN965" (at 141.605 102.235 0)
-      (effects (font (size 1.27 1.27)) hide)
-    )
-    (property "Datasheet" "~" (at 141.605 102.235 0)
-      (effects (font (size 1.27 1.27)) hide)
-    )
-    (instances
-      (project "PicoRfc522_pro"
-        (path "/9472a9f5-95f0-4abd-b6a1-4228d4355bea"
-          (reference "H4") (unit 1)
         )
       )
@@
         )
       )
-    )
-  )
-  (symbol (lib_id "Mechanical:MountingHole") (at 74.93 102.235 0) (unit 1)
-    (in_bom yes) (on_board yes) (dnp no) (fields_autoplaced)
-    (property "Reference" "H1" (at 77.47 101.6 0)
-      (effects (font (size 1.27 1.27)) (justify left) hide)
-    )
-    (property "Value" "MountingHole" (at 77.47 104.14 0)
-      (effects (font (size 1.27 1.27)) (justify left) hide)
-    )
-    (property "Footprint" "MountingHole:MountingHole_3.2mm_M3_DIN965" (at 74.93 102.235 0)
-      (effects (font (size 1.27 1.27)) hide)
-    )
-    (property "Datasheet" "~" (at 74.93 102.235 0)
-      (effects (font (size 1.27 1.27)) hide)
-    )
-    (instances
-      (project "PicoRfc522_pro"
-        (path "/9472a9f5-95f0-4abd-b6a1-4228d4355bea"
-          (reference "H1") (unit 1)
-        )
-      )
