File: PicoRfc522/PicoRfc522.kicad_pcb (KiCad board)
At the start: 2 copper layers, 100 x 90 mm, 19 parts, among them J1 5V sel, J2 Grove 2mm, J3 Screw_Terminal_01x04, J4 Screw_Terminal_01x02, J5 IDC1, J6 IDC1, J7 IDC1, J8 IDC1, Q1 DMG2305UX-7, SW1 SW_Push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

Commit message: 08/09/25 08:45 Titan.local
Parts:
- turned J2 to 180 degrees
Routing:
- net /3V3: track 184.0 -> 149.1 mm
- net /CS3: track 87.5 -> 98.4 mm, vias 1 -> 2
- net /GND: track 235.7 -> 245.4 mm
- net /5V: track 67.0 -> 76.7 mm
- net /VSYS: track 80.5 -> 71.6 mm
- net /RST: track 93.4 -> 101.1 mm, vias 1 -> 0
- net /SCL: track 82.4 -> 75.3 mm, vias 1 -> 0
- net /CS4: track 102.1 -> 95.9 mm
- net /VBUS: track 70.9 -> 73.6 mm
- net /12V: track 18.8 -> 16.8 mm
- net /CS2: track 88.8 -> 87.0 mm, vias 1 -> 2
- net /SDA: track 75.8 -> 77.6 mm, vias 0 -> 1
- net /MISO: track 92.4 -> 91.0 mm, vias 1 -> 0
- net /MOSI: track 93.9 -> 94.8 mm
Other:
- board text added: "3V3"
- board text added: "GND"
- board text added: "SCL"
- board text added: "SDA"

Commit message: 08/09/25 21:54 Titan.local
Parts:
- U3: value Pico_RaspberryPico -> Pico; footprint PicoNoSwd:RaspberryPico_TH_NoSWD -> Kicad-RP-Pico:RPi_Pico_SMD_TH
- moved U3 25.6 mm to (174.0, 89.5)
- moved J1 15.1 mm to (196.2, 76.2)
Connections:
- U3 pad 13: unconnected-(U3-GND-Pad13) -> /GND
- U3 pad 21: /MOSI -> /MISO
- U3 pad 22: /SCK -> /CS1
- U3 pad 24: /CS1 -> /SCK
- U3 pad 25: /MISO -> /MOSI
- U3 pad 3: /GND -> unconnected-(U3-GND-Pad3)
Routing:
- net /SCL: track 75.3 -> 90.8 mm
- net /5Vopt: track 54.4 -> 65.2 mm
- net /5V: track 76.7 -> 85.5 mm, vias 1 -> 2
- net /GND: track 245.4 -> 236.9 mm
- net /IRQ: track 51.1 -> 43.6 mm
- net /SCK: track 87.5 -> 94.3 mm
- net /3V3: track 149.1 -> 144.2 mm, vias 0 -> 2
- net /MISO: track 91.0 -> 86.8 mm, vias 0 -> 1
- net /RST: track 101.1 -> 97.0 mm, vias 0 -> 1
- net /CS3: track 98.4 -> 94.5 mm, vias 2 -> 1
- net /SDA: track 77.6 -> 73.7 mm, vias 1 -> 0
- net Net-(U3-RUN): track 38.6 -> 35.1 mm
- net /VBUS: track 73.6 -> 70.7 mm
- net /CS2: track 87.0 -> 84.5 mm, vias 2 -> 1
- net /12V: track 16.8 -> 19.0 mm
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
Commit message: 09/09/25 09:18 Arrakis.local
Parts:
- removed H1, H2, H3, H4: MountingHole_3.2mm_M3, MountingHole:MountingHole_3.2mm_M3
Routing:
- net /SCL: track 90.8 -> 76.8 mm
- net /CS4: track 94.8 -> 107.6 mm
- net /GND: track 236.9 -> 248.4 mm, vias 1 -> 0
- net /CS1: track 56.7 -> 67.4 mm
- net /RST: track 97.0 -> 92.0 mm, vias 1 -> 2
- net /SDA: track 73.7 -> 78.0 mm
- net /CS2: track 84.5 -> 81.0 mm
- net /5V: track 85.5 -> 82.6 mm
- net /VBUS: track 70.7 -> 68.5 mm
- net /3V3: track 144.2 -> 145.9 mm, vias 2 -> 1
- net /CS3: track 94.5 -> 95.5 mm
- net /MOSI: track 96.1 -> 95.4 mm
- net /SCK: track 94.3 -> 93.9 mm, vias 0 -> 1
- net /IRQ: track 43.6 -> 43.8 mm, vias 0 -> 1
- net /MISO: vias 1 -> 0

Commit message: 09/09/25 12:23 Arrakis.local
Routing:
- net /SCL: track 76.8 -> 90.8 mm
- net /CS4: track 107.6 -> 95.0 mm
- net /CS1: track 67.4 -> 56.8 mm
- net /RST: track 92.0 -> 99.2 mm, vias 2 -> 0
- net /CS2: track 81.0 -> 88.2 mm
- net /GND: track 248.4 -> 253.9 mm, vias 0 -> 2
- net /3V3: track 145.9 -> 151.1 mm, vias 1 -> 0
- net /SDA: track 78.0 -> 73.5 mm
- net /CS3: track 95.5 -> 98.8 mm, vias 1 -> 2
- net /12V: track 18.7 -> 15.9 mm, vias 1 -> 0
- net /5V: track 82.6 -> 85.0 mm, vias 2 -> 1
- net /MISO: track 86.8 -> 84.9 mm, vias 0 -> 1
- net /Pin: track 40.9 -> 42.7 mm
- net /IRQ: track 43.8 -> 42.6 mm, vias 1 -> 0
- net /VSYS: track 73.1 -> 72.2 mm
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
Commit message: 10/09/25 13:02 Titan.local
Parts:
- J2: footprint Seed Grove etc:HW4-2.0 -> OPL_Kicad_Library:HW4-2.0
Changed lines of the file:
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@@
     )
   )
-  (footprint "Seed Grove etc:HW4-2.0" (layer "F.Cu")
+  (footprint "OPL_Kicad_Library:HW4-2.0" (layer "F.Cu")
     (at 205.0018 68 180)
     (property "Sheetfile" "PicoRfc522.kicad_sch")
@@
     (property "ki_keywords" "screw terminal")
     (attr exclude_from_pos_files)
-    (fp_text reference "J2" (at -0.025 1.96) (layer "F.SilkS")
-        (effects (font (size 1 1) (thickness 0.15)))
-    )
-    (fp_text value "Grove 2mm" (at -0.025 5.3) (layer "F.Fab") hide
+    (fp_text reference "J2" (at -0.025 -3.375 180) (layer "F.SilkS") hide
+        (effects (font (size 1 1) (thickness 0.15)))
+    )
+    (fp_text value "Grove 2mm" (at -0.025 5.3 180) (layer "F.Fab")
+        (effects (font (size 1 1) (thickness 0.15)))
+    )
+    (fp_text user "${REFERENCE}" (at -0.1032 3.865 180) (layer "F.Fab")
         (effects (font (size 1 1) (thickness 0.15)))
     )
@@
         (effects (font (size 0.8 0.8) (thickness 0.15)))
     )
-    (fp_text user "Copper Keepouts shown on Dwgs layer" (at 0.1 -30.2) (layer "Cmts.User")
-        (effects (font (size 1 1) (thickness 0.15)))
-    )
     (fp_text user "${REFERENCE}" (at 0 0 180) (layer "F.Fab")

Commit message: 10/09/25 15:44 Titan.local
Routing:
- net /SCL: track 90.8 -> 72.6 mm
- net /CS1: track 56.8 -> 72.3 mm
- net /GND: track 253.9 -> 238.7 mm, vias 2 -> 1
- net /CS4: track 95.0 -> 108.2 mm
- net /3V3: track 151.1 -> 159.4 mm
- net /SDA: track 73.5 -> 80.6 mm
- net /SCK: track 93.5 -> 87.7 mm
- net /VSYS: track 72.2 -> 68.1 mm
- net /12V: track 15.9 -> 19.0 mm, vias 0 -> 1
- net /5V: track 85.0 -> 87.7 mm, vias 1 -> 2
- net /IRQ: track 42.6 -> 44.7 mm
- net /Pin: track 42.7 -> 41.0 mm
- net /MISO: track 84.9 -> 86.6 mm, vias 1 -> 0
- net /RST: track 99.2 -> 100.7 mm, vias 0 -> 1
- net /MOSI: track 95.9 -> 97.3 mm, vias 1 -> 0
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