File: PicoRfc522/PicoRfc522.kicad_sch (KiCad schematic)
At the start: 15 parts, among them J1 5V sel, J2 Grove 2mm, J3 Screw_Terminal_01x04, J4 Screw_Terminal_01x02, J5 IDC1, J6 IDC1, J7 IDC1, J8 IDC1, Q1 DMG2305UX-7, SW1 SW_Push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

Commit message: 08/09/25 21:54 Titan.local
Parts:
- removed U3: Pico_RaspberryPico, PicoNoSwd:RaspberryPico_TH_NoSWD, symbol PicoNoSwd:RaspberryPico-Pico
- added U3: Pico, Kicad-RP-Pico:RPi_Pico_SMD_TH, symbol Kicad-RP-Pico:Pico
Connections:
- net CS1: now also U3.22 (GPIO17)
- net CS2: now also U3.11 (GPIO8)
- net CS3: now also U3.12 (GPIO9)
- net CS4: now also U3.14 (GPIO10)
- net GND: now also U3.13 (GND)
- net MISO: now also U3.21 (GPIO16)
- net MOSI: now also U3.25 (GPIO19)
- net RST: now also U3.26 (GPIO20)
- net SCK: now also U3.24 (GPIO18)
- net SCL: now also U3.7 (GPIO5)
- net SDA: now also U3.6 (GPIO4)
- net VBUS: now also U3.40 (VBUS)
- net VSYS: now also U3.39 (VSYS)
- net at SW1.2: now also U3.30 (RUN)
- no-connect marks 28 -> 31
Other:
- moved on the sheet: J2, J6, J7, J8, SW1

Commit message: 10/09/25 13:02 Titan.local
Parts:
- J2: footprint Seed Grove etc:HW4-2.0 -> OPL_Kicad_Library:HW4-2.0
Changed lines of the file:
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@@
       (effects (font (size 1.27 1.27)))
     )
-    (property "Footprint" "Seed Grove etc:HW4-2.0" (at 30.48 115.57 0)
+    (property "Footprint" "OPL_Kicad_Library:HW4-2.0" (at 30.48 115.57 0)
       (effects (font (size 1.27 1.27)) hide)
     )

Commit message: 10/09/25 15:44 Titan.local
Parts:
- J2: footprint OPL_Kicad_Library:HW4-2.0 -> OPL_Connector:HW4-2.0
Changed lines of the file:
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@@
       (effects (font (size 1.27 1.27)))
     )
-    (property "Footprint" "OPL_Kicad_Library:HW4-2.0" (at 30.48 115.57 0)
+    (property "Footprint" "OPL_Connector:HW4-2.0" (at 30.48 115.57 0)
       (effects (font (size 1.27 1.27)) hide)
     )
