File: Untitled/Untitled.kicad_pcb (KiCad board)
At the start: 2 copper layers, 114 x 78 mm, 3 parts, among them J1 Screw_Terminal_01x04, J2 Screw_Terminal_01x04, U1 Pico

Commit message: 08/09/25 20:07 Titan.local
Parts:
- moved J2 83.9 mm to (149.2, 75.1)
- moved U1 46.3 mm to (116.8, 88.3)
- moved J1 15.1 mm to (190.2, 74.9)
Routing:
- net Net-(J1-Pin_2): track 48.8 -> 41.1 mm
- net Net-(J1-Pin_1): track 48.8 -> 41.1 mm
- net Net-(J1-Pin_4): track 48.8 -> 41.1 mm
- net Net-(J1-Pin_3): track 48.8 -> 41.1 mm
Other:
- board size 114 x 78 mm -> 122.6 x 82.6 mm

Commit message: 09/09/25 14:27 Titan.local
Parts:
- U1: footprint Kicad-RP-Pico:RPi_Pico_SMD_TH -> RP-Pico-Libraries:RP2040Pico

Commit message: 09/09/25 14:42 Arrakis.local
Parts:
- U1: footprint RP-Pico-Libraries:RP2040Pico -> RP-Pico Libraries:RP2040Pico

Commit message: 10/09/25 07:25 Titan.local
Parts:
- added Brd1: SSD1306, SSD1306:128x64OLED, F.Cu at (168.6, 96.4)
- added U2: Pico_RaspberryPico, Kicad-RP-Pico:RPi_Pico_SMD_TH, F.Cu at (74.9, 83.8)
- U1: footprint RP-Pico Libraries:RP2040Pico -> Kicad-RP-Pico:RPi_Pico_SMD_TH
Other:
- board size 122.6 x 82.6 mm -> 152.4 x 74.9 mm

Commit message: 10/09/25 12:32 Titan.local
Parts:
- added Brd2: SSD1306, SSD1306:128x64OLED, F.Cu at (171.8, 61.5)
- added J3: GROVE-CONNECTOR-DIP_4P-2.0_, OPL_Connector:HW4-2.0, F.Cu at (144.3, 87.6)
Changed lines of the file:
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@@
   (net 90 "unconnected-(U2-VSYS-Pad39)")
   (net 91 "unconnected-(U2-VBUS-Pad40)")
+  (net 92 "unconnected-(J3-Pad1)")
+  (net 93 "unconnected-(J3-Pad2)")
+  (net 94 "unconnected-(J3-Pad3)")
+  (net 95 "unconnected-(J3-Pad4)")
+  (net 96 "unconnected-(Brd2-GND-Pad1)")
+  (net 97 "unconnected-(Brd2-VCC-Pad2)")
+  (net 98 "unconnected-(Brd2-SCL-Pad3)")
+  (net 99 "unconnected-(Brd2-SDA-Pad4)")
   (footprint "TerminalBlock_Phoenix:TerminalBlock_Phoenix_PT-1,5-4-3.5-H_1x04_P3.50mm_Horizontal" (layer "F.Cu")
     (at 190.16 74.93 90)
@@
       (rotate (xyz 0 0 0))
     )
+  )
+  (footprint "OPL_Connector:HW4-2.0" (layer "F.Cu")
+    (at 144.32026 87.63)
+    (property "SKU" "320110033")
+    (property "Sheetfile" "Untitled.kicad_sch")
+    (property "Sheetname" "")
+    (attr exclude_from_pos_files)
+    (fp_text reference "J3" (at -0.025 -3.375) (layer "F.SilkS")
+        (effects (font (size 1 1) (thickness 0.15)))
+    )
+    (fp_text value "GROVE-CONNECTOR-DIP_4P-2.0_" (at -0.025 5.3) (layer "F.Fab")
+        (effects (font (size 1 1) (thickness 0.15)))
+    )
+    (fp_text user "${REFERENCE}" (at -0.025 -3.375) (layer "F.Fab")
+        (effects (font (size 1 1) (thickness 0.15)))
+    )
+    (fp_line (start -5.00086 2.95) (end -3.2 2.95)
+      (stroke (width 0.127) (type solid)) (layer "F.SilkS"))
+    (fp_line (start -4.99872 -2.19964) (end -4.99872 2.95)
+      (stroke (width 0.127) (type solid)) (layer "F.SilkS"))
+    (fp_line (start -4.99872 -2.19964) (end 4.99872 -2.19964)
+      (stroke (width 0.127) (type solid)) (layer "F.SilkS"))
+    (fp_line (start -4.99872 -0.99822) (end -4.99872 0.99822)
+      (stroke (width 0.127) (type solid)) (layer "F.SilkS"))
+    (fp_line (start -3.175 2.159) (end -1.778 2.159)
+      (stroke (width 0.127) (type solid)) (layer "F.SilkS"))
+    (fp_line (start -3.175 2.95) (end -3.175 2.159)
+      (stroke (width 0.127) (type solid)) (layer "F.SilkS"))
+    (fp_line (start -1.781 2.95) (end 1.775 2.95)
+      (stroke (width 0.127) (type solid)) (layer "F.SilkS"))
+    (fp_line (start -1.778 2.159) (end -1.778 2.95)
+      (stroke (width 0.127) (type solid)) (layer "F.SilkS"))
+    (fp_line (start 1.775 2.95) (end 1.775 2.159)
+      (stroke (width 0.127) (type solid)) (layer "F.SilkS"))
+    (fp_line (start 1.778 2.159) (end 3.175 2.159)
+      (stroke (width 0.127) (type solid)) (layer "F.SilkS"))
+    (fp_line (start 3.175 2.159) (end 3.175 2.95)
+      (stroke (width 0.127) (type solid)) (layer "F.SilkS"))
+    (fp_line (start 3.175 2.95) (end 5 2.95)
+      (stroke (width 0.127) (type solid)) (layer "F.SilkS"))
+    (fp_line (start 5 2.95) (end 5 -2.19964)
+      (stroke (width 0.127) (type solid)) (layer "F.SilkS"))
+    (fp_line (start -5.25 -2.4) (end 5.25 -2.4)
+      (stroke (width 0.05) (type solid)) (layer "F.CrtYd"))
+    (fp_line (start -5.25 3.2) (end -5.25 -2.4)
+      (stroke (width 0.05) (type solid)) (layer "F.CrtYd"))
+    (fp_line (start 5.25 -2.4) (end 5.25 3.2)
+      (stroke (width 0.05) (type solid)) (layer "F.CrtYd"))
+    (fp_line (start 5.25 3.2) (end -5.25 3.2)
+      (stroke (width 0.05) (type solid)) (layer "F.CrtYd"))
+    (fp_line (start -5 -2.15) (end 5 -2.15)
+      (stroke (width 0.1) (type solid)) (layer "F.Fab"))
+    (fp_line (start -5 2.95) (end -5 -2.15)
+      (stroke (width 0.1) (type solid)) (layer "F.Fab"))
+    (fp_line (start -4.99872 2.95) (end -3.19786 2.95)
+      (stroke (width 0.1) (type solid)) (layer "F.Fab"))
+    (fp_line (start -3.175 2.159) (end -1.778 2.159)
+      (stroke (width 0.1) (type solid)) (layer "F.Fab"))
+    (fp_line (start -3.175 2.95) (end -3.175 2.159)
+      (stroke (width 0.1) (type solid)) (layer "F.Fab"))
+    (fp_line (start -1.778 2.159) (end -1.778 2.95)
+      (stroke (width 0.1) (type solid)) (layer "F.Fab"))
+    (fp_line (start -1.778 2.95) (end 1.778 2.95)
+      (stroke (width 0.1) (type solid)) (layer "F.Fab"))
+    (fp_line (start 1.778 2.159) (end 3.175 2.159)
+      (stroke (width 0.1) (type solid)) (layer "F.Fab"))
+    (fp_line (start 1.778 2.95) (end 1.778 2.159)
+      (stroke (width 0.1) (type solid)) (layer "F.Fab"))
+    (fp_line (start 3.175 2.159) (end 3.175 2.95)
+      (stroke (width 0.1) (type solid)) (layer "F.Fab"))
+    (fp_line (start 3.175 2.95) (end 5 2.95)
+      (stroke (width 0.1) (type solid)) (layer "F.Fab"))
+    (fp_line (start 5 2.95) (end 5 -2.15)
+      (stroke (width 0.1) (type solid)) (layer "F.Fab"))
+    (pad "1" thru_hole rect (at -2.99974 0) (size 1.27 1.27) (drill 0.79756) (layers "*.Cu" "*.Mask")
+      (net 92 "unconnected-(J3-Pad1)") (pinfunction "1") (pintype "bidirectional"))
+    (pad "2" thru_hole circle (at -0.99822 0) (size 1.27 1.27) (drill 0.79756) (layers "*.Cu" "*.Mask")
+      (net 93 "unconnected-(J3-Pad2)") (pinfunction "2") (pintype "bidirectional"))
+    (pad "3" thru_hole circle (at 0.99822 0) (size 1.27 1.27) (drill 0.79756) (layers "*.Cu" "*.Mask")
+      (net 94 "unconnected-(J3-Pad3)") (pinfunction "3") (pintype "bidirectional"))
+    (pad "4" thru_hole circle (at 2.99974 0) (size 1.27 1.27) (drill 0.79756) (layers "*.Cu" "*.Mask")
+      (net 95 "unconnected-(J3-Pad4)") (pinfunction "4") (pintype "bidirectional"))
   )
   (footprint "SSD1306:128x64OLED" (layer "F.Cu")
@@
       (offset (xyz 0 0 0))
       (scale (xyz 1 1 1))
+      (rotate (xyz 0 0 0))
+    )
+  )
+  (footprint "SSD1306:128x64OLED" (layer "F.Cu")
+    (at 171.785 61.515)
+    (property "Sheetfile" "Untitled.kicad_sch")
+    (property "Sheetname" "")
+    (property "ki_description" "SSD1306 OLED")
+    (property "ki_keywords" "SSD1306")
+    (attr through_hole)
+    (fp_text reference "Brd2" (at 0 0.254) (layer "F.SilkS")
+        (effects (font (size 1 1) (thickness 0.15)))
+    )
+    (fp_text value "SSD1306" (at -7.747 -7.62) (layer "F.Fab")
+        (effects (font (size 1 1) (thickness 0.15)))
+    )
+    (fp_line (start -13.4 -12.3) (end 14 -12.3)
+      (stroke (width 0.12) (type solid)) (layer "F.SilkS"))
+    (fp_line (start -13.4 15) (end -13.4 -12.3)
+      (stroke (width 0.12) (type solid)) (layer "F.SilkS"))
+    (fp_line (start -12.978 -9.005) (end 10.122 -9.005)
+      (stroke (width 0.12) (type solid)) (layer "F.SilkS"))
+    (fp_line (start -12.978 7.595) (end -12.978 -9.005)
+      (stroke (width 0.12) (type solid)) (layer "F.SilkS"))
+    (fp_line (start -4.699 -11.811) (end -4.699 -9.398)
+      (stroke (width 0.12) (type solid)) (layer "F.SilkS"))
+    (fp_line (start -4.699 -11.811) (end 5.08 -11.811)
+      (stroke (width 0.12) (type solid)) (layer "F.SilkS"))
+    (fp_line (start 5.08 -11.811) (end 5.08 -9.398)
+      (stroke (width 0.12) (type solid)) (layer "F.SilkS"))
+    (fp_line (start 5.08 -9.398) (end -4.699 -9.398)
+      (stroke (width 0.12) (type solid)) (layer "F.SilkS"))
+    (fp_line (start 10.122 -9.005) (end 13.208 -9.005)
+      (stroke (width 0.12) (type solid)) (layer "F.SilkS"))
+    (fp_line (start 10.122 7.595) (end -12.978 7.595)
+      (stroke (width 0.12) (type solid)) (layer "F.SilkS"))
+    (fp_line (start 10.122 7.595) (end 13.462 7.62)
+      (stroke (width 0.12) (type solid)) (layer "F.SilkS"))
+    (fp_line (start 13.462 -9.017) (end 13.208 -9.005)
+      (stroke (width 0.12) (type solid)) (layer "F.SilkS"))
+    (fp_line (start 13.462 7.62) (end 13.462 -9.017)
+      (stroke (width 0.12) (type solid)) (layer "F.SilkS"))
+    (fp_line (start 14 -12.3) (end 14 15)
+      (stroke (width 0.12) (type solid)) (layer "F.SilkS"))
+    (fp_line (start 14 15) (end -13.4 15)
+      (stroke (width 0.12) (type solid)) (layer "F.SilkS"))
+    (pad "1" thru_hole oval (at -3.62 -10.6 90) (size 2 1.6) (drill 1) (layers "*.Cu" "*.Mask")
+      (net 96 "unconnected-(Brd2-GND-Pad1)") (pinfunction "GND") (pintype "input"))
+    (pad "2" thru_hole oval (at -1.08 -10.6 90) (size 2 1.6) (drill 1) (layers "*.Cu" "*.Mask")
+      (net 97 "unconnected-(Brd2-VCC-Pad2)") (pinfunction "VCC") (pintype "input"))
+    (pad "3" thru_hole oval (at 1.46 -10.6 90) (size 2 1.6) (drill 1) (layers "*.Cu" "*.Mask")
+      (net 98 "unconnected-(Brd2-SCL-Pad3)") (pinfunction "SCL") (pintype "input"))
+    (pad "4" thru_hole oval (at 4 -10.6 90) (size 2 1.6) (drill 1) (layers "*.Cu" "*.Mask")
+      (net 99 "unconnected-(Brd2-SDA-Pad4)") (pinfunction "SDA") (pintype "input"))
+    (model "/Users/colinc/Documents/Kicad/KiCadLibs/KiCad-SSD1306-128x64-master/images/ssd1306_3d.jpg"
+      (offset (xyz 0 0 0))
+      (scale (xyz 1 1 1))
