File: Untitled/Untitled.kicad_sch (KiCad schematic)
At the start: 3 parts, among them J1 Screw_Terminal_01x04, J2 Screw_Terminal_01x04, U1 Pico

Commit message: 08/09/25 20:07 Titan.local
Changed lines of the file:
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@@
 (kicad_sch (version 20230121) (generator eeschema)
   (paper "A4")
-  (wire (pts (xy 128.905 66.675) (xy 178.435 66.675))
+  (wire (pts (xy 114.3 76.2) (xy 124.46 76.2))
     (stroke (width 0) (type default))
   )
-  (wire (pts (xy 128.905 64.135) (xy 178.435 64.135))
+  (wire (pts (xy 114.3 81.28) (xy 124.46 81.28))
     (stroke (width 0) (type default))
   )
-  (wire (pts (xy 128.905 61.595) (xy 178.435 61.595))
+  (wire (pts (xy 114.3 83.82) (xy 124.46 83.82))
     (stroke (width 0) (type default))
   )
-  (wire (pts (xy 128.905 69.215) (xy 178.435 69.215))
+  (wire (pts (xy 114.3 78.74) (xy 124.46 78.74))
     (stroke (width 0) (type default))
   )
-  (symbol (lib_id "Connector:Screw_Terminal_01x04") (at 183.515 64.135 0) (unit 1)
+  (symbol (lib_id "Connector:Screw_Terminal_01x04") (at 129.54 78.74 0) (unit 1)
     (in_bom yes) (on_board yes) (dnp no) (fields_autoplaced)
-    (property "Reference" "J1" (at 186.69 64.77 0)
+    (property "Reference" "J1" (at 132.08 78.74 0)
       (effects (font (size 1.27 1.27)) (justify left))
     )
-    (property "Value" "Screw_Terminal_01x04" (at 186.69 67.31 0)
+    (property "Value" "Screw_Terminal_01x04" (at 132.08 81.28 0)
       (effects (font (size 1.27 1.27)) (justify left))
     )
-    (property "Footprint" "TerminalBlock_Phoenix:TerminalBlock_Phoenix_PT-1,5-4-3.5-H_1x04_P3.50mm_Horizontal" (at 183.515 64.135 0)
+    (property "Footprint" "TerminalBlock_Phoenix:TerminalBlock_Phoenix_PT-1,5-4-3.5-H_1x04_P3.50mm_Horizontal" (at 129.54 78.74 0)
       (effects (font (size 1.27 1.27)) hide)
     )
-    (property "Datasheet" "~" (at 183.515 64.135 0)
+    (property "Datasheet" "~" (at 129.54 78.74 0)
       (effects (font (size 1.27 1.27)) hide)
     )
@@
     (instances
       (project "Untitled"
-        (path "/0c7b1023-00a5-46d3-9a5b-6b9e17609b4b"
+        (path "/774ca873-b611-4971-865b-08f86387ffba"
           (reference "J1") (unit 1)
         )
@@
     )
   )
-  (symbol (lib_id "Kicad-RP-Pico:Pico") (at 154.94 113.665 0) (unit 1)
+  (symbol (lib_id "Connector:Screw_Terminal_01x04") (at 109.22 78.74 0) (mirror y) (unit 1)
     (in_bom yes) (on_board yes) (dnp no) (fields_autoplaced)
-    (property "Reference" "U1" (at 154.94 83.82 0)
+    (property "Reference" "J2" (at 109.22 69.85 0)
       (effects (font (size 1.27 1.27)))
     )
-    (property "Value" "Pico" (at 154.94 86.36 0)
+    (property "Value" "Screw_Terminal_01x04" (at 109.22 72.39 0)
       (effects (font (size 1.27 1.27)))
     )
-    (property "Footprint" "Kicad-RP-Pico:RPi_Pico_SMD_TH" (at 154.94 113.665 90)
+    (property "Footprint" "TerminalBlock_Phoenix:TerminalBlock_Phoenix_PT-1,5-4-3.5-H_1x04_P3.50mm_Horizontal" (at 109.22 78.74 0)
       (effects (font (size 1.27 1.27)) hide)
     )
-    (property "Datasheet" "" (at 154.94 113.665 0)
+    (property "Datasheet" "~" (at 109.22 78.74 0)
+      (effects (font (size 1.27 1.27)) hide)
+    )
+    (pin "1")
+    (pin "2")
+    (pin "3")
+    (pin "4")
+    (instances
+      (project "Untitled"
+        (path "/774ca873-b611-4971-865b-08f86387ffba"
+          (reference "J2") (unit 1)
+        )
+      )
+    )
+  )
+  (symbol (lib_id "Kicad-RP-Pico:Pico") (at 154.94 99.06 0) (unit 1)
+    (in_bom yes) (on_board yes) (dnp no) (fields_autoplaced)
+    (property "Reference" "U1" (at 154.94 67.31 0)
+      (effects (font (size 1.27 1.27)))
+    )
+    (property "Value" "Pico" (at 154.94 69.85 0)
+      (effects (font (size 1.27 1.27)))
+    )
+    (property "Footprint" "Kicad-RP-Pico:RPi_Pico_SMD_TH" (at 154.94 99.06 90)
+      (effects (font (size 1.27 1.27)) hide)
+    )
+    (property "Datasheet" "" (at 154.94 99.06 0)
       (effects (font (size 1.27 1.27)) hide)
     )
@@
     (instances
       (project "Untitled"
-        (path "/0c7b1023-00a5-46d3-9a5b-6b9e17609b4b"
+        (path "/774ca873-b611-4971-865b-08f86387ffba"
           (reference "U1") (unit 1)
         )
       )
-    )
-  )
-  (symbol (lib_id "Connector:Screw_Terminal_01x04") (at 123.825 64.135 0) (mirror y) (unit 1)
-    (in_bom yes) (on_board yes) (dnp no)
-    (property "Reference" "J2" (at 123.825 74.295 0)
-      (effects (font (size 1.27 1.27)))
-    )
-    (property "Value" "Screw_Terminal_01x04" (at 123.825 71.755 0)
-      (effects (font (size 1.27 1.27)))
-    )
-    (property "Footprint" "TerminalBlock_Phoenix:TerminalBlock_Phoenix_PT-1,5-4-3.5-H_1x04_P3.50mm_Horizontal" (at 123.825 64.135 0)
-      (effects (font (size 1.27 1.27)) hide)
-    )
-    (property "Datasheet" "~" (at 123.825 64.135 0)
-      (effects (font (size 1.27 1.27)) hide)
-    )
-    (pin "1")
-    (pin "2")
-    (pin "3")
-    (pin "4")
-    (instances
-      (project "Untitled"
-        (path "/0c7b1023-00a5-46d3-9a5b-6b9e17609b4b"
-          (reference "J2") (unit 1)
-        )
-      )

Commit message: 09/09/25 14:27 Titan.local
Parts:
- U1: footprint Kicad-RP-Pico:RPi_Pico_SMD_TH -> RPi_Pico:RPi_Pico_SMD_TH
Changed lines of the file:
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@@
       (effects (font (size 1.27 1.27)))
     )
-    (property "Footprint" "Kicad-RP-Pico:RPi_Pico_SMD_TH" (at 154.94 99.06 90)
+    (property "Footprint" "RPi_Pico:RPi_Pico_SMD_TH" (at 154.94 99.06 90)
       (effects (font (size 1.27 1.27)) hide)
     )

Commit message: 09/09/25 14:42 Arrakis.local
Parts:
- U1: footprint RPi_Pico:RPi_Pico_SMD_TH -> RP-Pico Libraries:RP2040Pico
Changed lines of the file:
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@@
       (effects (font (size 1.27 1.27)))
     )
-    (property "Footprint" "RPi_Pico:RPi_Pico_SMD_TH" (at 154.94 99.06 90)
+    (property "Footprint" "RP-Pico Libraries:RP2040Pico" (at 154.94 99.06 90)
       (effects (font (size 1.27 1.27)) hide)
     )

Commit message: 10/09/25 07:25 Titan.local
Parts:
- added Brd1: SSD1306, SSD1306:128x64OLED, symbol SSD1306:SSD1306
- added U2: Pico_RaspberryPico, Kicad-RP-Pico:RPi_Pico_SMD_TH, symbol PicoNoSwd:RaspberryPico-Pico
- U1: footprint RP-Pico Libraries:RP2040Pico -> Kicad-RP-Pico:RPi_Pico_SMD_TH
Changed lines of the file:
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@@
+    )
+  )
+  (symbol (lib_id "PicoNoSwd:RaspberryPico-Pico") (at 266.192 56.388 0) (unit 1)
+    (in_bom yes) (on_board yes) (dnp no) (fields_autoplaced)
+    (property "Reference" "U2" (at 254.762 49.53 0)
+      (effects (font (size 1.27 1.27)))
+    )
+    (property "Value" "Pico_RaspberryPico" (at 254.762 52.07 0)
+      (effects (font (size 1.27 1.27)))
+    )
+    (property "Footprint" "Kicad-RP-Pico:RPi_Pico_SMD_TH" (at 266.192 56.388 0)
+      (effects (font (size 1.27 1.27)) hide)
+    )
+    (property "Datasheet" "" (at 266.192 56.388 0)
+      (effects (font (size 1.27 1.27)) hide)
+    )
+    (pin "1")
+    (pin "10")
+    (pin "11")
+    (pin "12")
+    (pin "13")
+    (pin "14")
+    (pin "15")
+    (pin "16")
+    (pin "17")
+    (pin "18")
+    (pin "19")
+    (pin "2")
+    (pin "20")
+    (pin "21")
+    (pin "22")
+    (pin "23")
+    (pin "24")
+    (pin "25")
+    (pin "26")
+    (pin "27")
+    (pin "28")
+    (pin "29")
+    (pin "3")
+    (pin "30")
+    (pin "31")
+    (pin "32")
+    (pin "33")
+    (pin "34")
+    (pin "35")
+    (pin "36")
+    (pin "37")
+    (pin "38")
+    (pin "39")
+    (pin "4")
+    (pin "40")
+    (pin "5")
+    (pin "6")
+    (pin "7")
+    (pin "8")
+    (pin "9")
+    (instances
+      (project "Untitled"
+        (path "/774ca873-b611-4971-865b-08f86387ffba"
+          (reference "U2") (unit 1)
+        )
+      )
+    )
+  )
+  (symbol (lib_id "SSD1306:SSD1306") (at 215.138 82.804 0) (unit 1)
+    (in_bom yes) (on_board yes) (dnp no) (fields_autoplaced)
+    (property "Reference" "Brd1" (at 222.25 81.534 0)
+      (effects (font (size 1.27 1.27)) (justify left))
+    )
+    (property "Value" "SSD1306" (at 222.25 84.074 0)
+      (effects (font (size 1.27 1.27)) (justify left))
+    )
+    (property "Footprint" "SSD1306:128x64OLED" (at 215.138 76.454 0)
+      (effects (font (size 1.27 1.27)) hide)
+    )
+    (property "Datasheet" "" (at 215.138 76.454 0)
+      (effects (font (size 1.27 1.27)) hide)
+    )
+    (pin "1")
+    (pin "2")
+    (pin "3")
+    (pin "4")
+    (instances
+      (project "Untitled"
+        (path "/774ca873-b611-4971-865b-08f86387ffba"
+          (reference "Brd1") (unit 1)
+        )
+      )
     )
   )
@@
       (effects (font (size 1.27 1.27)))
     )
-    (property "Footprint" "RP-Pico Libraries:RP2040Pico" (at 154.94 99.06 90)
+    (property "Footprint" "Kicad-RP-Pico:RPi_Pico_SMD_TH" (at 154.94 99.06 90)
       (effects (font (size 1.27 1.27)) hide)
     )

Commit message: 10/09/25 12:32 Titan.local
Parts:
- added Brd2: SSD1306, SSD1306:128x64OLED, symbol SSD1306-128x64_OLED:SSD1306
- added J3: GROVE-CONNECTOR-DIP_4P-2.0_, OPL_Connector:HW4-2.0, symbol OPL_Connector:GROVE-CONNECTOR-DIP_4P-2.0_
Changed lines of the file:
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@@
     (stroke (width 0) (type default))
+  )
+  (symbol (lib_id "OPL_Connector:GROVE-CONNECTOR-DIP_4P-2.0_") (at 69.85 116.078 0) (unit 1)
+    (in_bom yes) (on_board yes) (dnp no) (fields_autoplaced)
+    (property "Reference" "J3" (at 74.93 114.808 0)
+      (effects (font (size 1.143 1.143)) (justify left))
+    )
+    (property "Value" "GROVE-CONNECTOR-DIP_4P-2.0_" (at 74.93 117.348 0)
+      (effects (font (size 1.143 1.143)) (justify left))
+    )
+    (property "Footprint" "OPL_Connector:HW4-2.0" (at 69.85 116.078 0)
+      (effects (font (size 1.27 1.27)) hide)
+    )
+    (property "Datasheet" "" (at 69.85 116.078 0)
+      (effects (font (size 1.27 1.27)) hide)
+    )
+    (property "SKU" "320110033" (at 70.612 112.268 0)
+      (effects (font (size 0.508 0.508)) hide)
+    )
+    (pin "1")
+    (pin "2")
+    (pin "3")
+    (pin "4")
+    (instances
+      (project "Untitled"
+        (path "/774ca873-b611-4971-865b-08f86387ffba"
+          (reference "J3") (unit 1)
+        )
+      )
+    )
   )
   (symbol (lib_id "Connector:Screw_Terminal_01x04") (at 129.54 78.74 0) (unit 1)
@@
         )
       )
+    )
+  )
+  (symbol (lib_id "SSD1306-128x64_OLED:SSD1306") (at 92.964 102.362 0) (unit 1)
+    (in_bom yes) (on_board yes) (dnp no) (fields_autoplaced)
+    (property "Reference" "Brd2" (at 100.33 101.092 0)
+      (effects (font (size 1.27 1.27)) (justify left))
+    )
+    (property "Value" "SSD1306" (at 100.33 103.632 0)
+      (effects (font (size 1.27 1.27)) (justify left))
+    )
+    (property "Footprint" "SSD1306:128x64OLED" (at 92.964 96.012 0)
+      (effects (font (size 1.27 1.27)) hide)
+    )
+    (property "Datasheet" "" (at 92.964 96.012 0)
+      (effects (font (size 1.27 1.27)) hide)
+    )
+    (pin "1")
+    (pin "2")
+    (pin "3")
+    (pin "4")
+    (instances
+      (project "Untitled"
+        (path "/774ca873-b611-4971-865b-08f86387ffba"
+          (reference "Brd2") (unit 1)
+        )
+      )
