File: EspRfid522/EspRfid522.kicad_pcb (KiCad board)
At the start: 2 copper layers, 100 x 34 mm, 15 parts, among them J1 Screw_Terminal_01x02, J2 IDC1, J3 IDC2, J4 IDC3, J5 IDC4, U1 AP7384-50Y, U2 AMS1117-3.3, U3 ESP32-DEVKITC-32D

Commit message: 13/09/25 20:26 Titan.local
Parts:
- added J6: DIP-BLACK-MALE-HEADER-VERT_2P-2.54_, Connector_PinHeader_2.54mm:PinHeader_2x01_P2.54mm_Vertical, F.Cu at (128.9, 74.9)
- added J7: DIP-BLACK-FEMALE-HEADER_2X4P-2.54_, Connector_PinHeader_2.54mm:PinHeader_2x04_P2.54mm_Vertical, F.Cu at (113.7, 78.1)
- moved J1 6.44 mm to (115.0, 55.4)
- moved D2 4.97 mm to (125.7, 56.7)
- moved D1 4.97 mm to (125.7, 52.1)
- moved D3 4.97 mm to (125.7, 61.2)
- moved D4 4.97 mm to (125.7, 65.8)
- moved C3 4.84 mm to (139.7, 71.1)
Connections:
- J2 pad 5: /IRQ -> /IRQ1
- J3 pad 5: /IRQ -> /IRQ2
- J4 pad 5: /IRQ -> /IRQ3
- J5 pad 5: /IRQ -> /IRQ4
- U3 pad J2-19: /5V -> /EXT_5V
- U3 pad J2-5: unconnected-(U3-IO34-PadJ2-5) -> /IO34
- U3 pad J2-6: unconnected-(U3-IO35-PadJ2-6) -> /IO35
- U3 pad J2-7: unconnected-(U3-IO32-PadJ2-7) -> /IO32
- U3 pad J2-8: unconnected-(U3-IO33-PadJ2-8) -> /IO33
Routing:
- net /IRQ4: track 0.00 -> 86.0 mm, vias 0 -> 1
- net /IO34: track 0.00 -> 75.2 mm
- net /IO35: track 0.00 -> 74.0 mm
- net /IO32: track 0.00 -> 72.0 mm
- net /IO33: track 0.00 -> 70.1 mm
- net /IRQ2: track 0.00 -> 69.3 mm, vias 0 -> 1
- net /IRQ3: track 0.00 -> 67.9 mm, vias 0 -> 1
- net /IRQ1: track 0.00 -> 40.0 mm
- net /IRQ: track 38.9 -> 0.00 mm
- net /EXT_5V: track 0.00 -> 25.0 mm
- net /GND: track 144.9 -> 124.6 mm
- net /+V: track 45.3 -> 65.1 mm
- net /3V3: track 81.2 -> 97.2 mm
- net /5V: track 36.1 -> 40.1 mm
- net /RST: track 47.0 -> 49.9 mm, vias 0 -> 1
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Other:
- board text added: "4 3 2 1"
- board text added: "5v sel"
- board text added: "IRQ"

Commit message: 14/09/25 14:58 Arrakis.local
Parts:
- added H1: MountingHole, MountingHole:MountingHole_3.2mm_M3_ISO14580, F.Cu at (206.0, 52.0)
- added H2: MountingHole, MountingHole:MountingHole_3.2mm_M3_ISO14580, F.Cu at (206.0, 80.0)
- added H3: MountingHole, MountingHole:MountingHole_3.2mm_M3_ISO14580, F.Cu at (112.0, 52.0)
- added H4: MountingHole, MountingHole:MountingHole_3.2mm_M3_ISO14580, F.Cu at (112.0, 80.0)
- added J10: IDC4, Connector_IDC:IDC-Header_2x04_P2.54mm_Vertical, F.Cu at (189.5, 62.5)
- added J8: IDC2, Connector_IDC:IDC-Header_2x04_P2.54mm_Vertical, F.Cu at (163.2, 62.2)
- added J9: IDC3, Connector_IDC:IDC-Header_2x04_P2.54mm_Vertical, F.Cu at (174.2, 62.2)
- J2: value IDC1 -> Conn_01x02; footprint Connector_IDC:IDC-Header_2x04_P2.54mm_Vertical -> Connector_PinHeader_2.54mm:PinHeader_1x02_P2.54mm_Vertical
- J3: value IDC2 -> Conn_01x02; footprint Connector_IDC:IDC-Header_2x04_P2.54mm_Vertical -> Connector_PinHeader_2.54mm:PinHeader_1x02_P2.54mm_Vertical
- J4: value IDC3 -> Conn_01x02; footprint Connector_IDC:IDC-Header_2x04_P2.54mm_Vertical -> Connector_PinHeader_2.54mm:PinHeader_1x02_P2.54mm_Vertical
- J5: value IDC4 -> Conn_01x02; footprint Connector_IDC:IDC-Header_2x04_P2.54mm_Vertical -> Connector_PinHeader_2.54mm:PinHeader_1x02_P2.54mm_Vertical
- J6: value DIP-BLACK-MALE-HEADER-VERT_2P-2.54_ -> Conn_01x02; footprint Connector_PinHeader_2.54mm:PinHeader_2x01_P2.54mm_Vertical -> Connector_PinHeader_2.54mm:PinHeader_1x02_P2.54mm_Vertical
- J7: value DIP-BLACK-FEMALE-HEADER_2X4P-2.54_ -> IDC1; footprint Connector_PinHeader_2.54mm:PinHeader_2x04_P2.54mm_Vertical -> Connector_IDC:IDC-Header_2x04_P2.54mm_Vertical
- U1: value AP7384-50Y -> AMS1117-3.3; footprint Package_TO_SOT_SMD:SOT-89-3 -> Package_TO_SOT_SMD:SOT-223-3_TabPin2
- U2: value AMS1117-3.3 -> AMS1117-5.0
- moved J6 54.5 mm to (183.0, 68.5)
- moved J4 41.5 mm to (141.0, 72.5)
- moved J7 38.1 mm to (148.2, 62.0), turned to 0 degrees
- moved C2 22.0 mm to (125.0, 77.0), turned to 180 degrees
- moved C3 14.7 mm to (125.0, 72.0), turned to 180 degrees
- moved J3 13.7 mm to (157.0, 68.0)
- moved C1 10.9 mm to (134.6, 73.0)
- moved J5 10.2 mm to (183.0, 59.5)
- moved U1 9.06 mm to (137.0, 65.0)
- moved J1 8.60 mm to (115.0, 64.0)
- moved U2 8.06 mm to (137.0, 56.0)
- moved U3 3.12 mm to (175.0, 65.3)
- moved J2 1.46 mm to (157.0, 60.0)
Connections:
- J2 pad 1: /CS1 -> /IO32
- J2 pad 2: /SCK -> /IRQ1
- J3 pad 1: /CS2 -> /IO33
- J3 pad 2: /SCK -> /IRQ2
- J4 pad 1: /CS3 -> /EXT_5V
- J4 pad 2: /SCK -> /5V
- J5 pad 1: /CS4 -> /IO34
- J5 pad 2: /SCK -> /IRQ3
- J6 pad 1: /EXT_5V -> /IO35
- J6 pad 2: /5V -> /IRQ4
- J7 pad 1: /IO32 -> /CS1
- J7 pad 2: /IO33 -> /SCK
- J7 pad 3: /IO34 -> /MOSI
- J7 pad 4: /IO35 -> /MISO
- J7 pad 5: /IRQ4 -> /IRQ1
- J7 pad 6: /IRQ3 -> /GND
- J7 pad 7: /IRQ2 -> /RST
- J7 pad 8: /IRQ1 -> /3V3
- U1 pad 1: /5V -> /GND
- U1 pad 2: /GND -> /3V3
- U1 pad 3: /+V -> /5V
- U2 pad 2: /3V3 -> /5V
- U2 pad 3: /5V -> /+V
Routing:
- net /GND: track 124.6 -> 0.00 mm
- net /3V3: track 97.2 -> 0.00 mm, vias 1 -> 0
- net /IRQ4: track 86.0 -> 0.00 mm, vias 1 -> 0
- net /IO34: track 75.2 -> 0.00 mm
- net /IO35: track 74.0 -> 0.00 mm
- net /IO32: track 72.0 -> 0.00 mm
- net /IO33: track 70.1 -> 0.00 mm
- net /IRQ2: track 69.3 -> 0.00 mm, vias 1 -> 0
- net /IRQ3: track 67.9 -> 0.00 mm, vias 1 -> 0
- net /+V: track 65.1 -> 0.00 mm
- net /MOSI: track 50.9 -> 0.00 mm
- net /RST: track 49.9 -> 0.00 mm, vias 1 -> 0
- net /SCK: track 49.5 -> 0.00 mm
- net /MISO: track 49.3 -> 0.00 mm
- net /5V: track 40.1 -> 0.00 mm, vias 1 -> 0
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Other:
- board text removed: "4 3 2 1"
- board text removed: "IRQ"

Commit message: 14/09/25 15:04 Titan.local
Routing:
- net /GND: track 0.00 -> 143.9 mm
- net /3V3: track 0.00 -> 79.5 mm, vias 0 -> 1
- net /MISO: track 0.00 -> 60.7 mm
- net /RST: track 0.00 -> 59.3 mm
- net /MOSI: track 0.00 -> 57.9 mm
- net /SCK: track 0.00 -> 55.0 mm
- net /5V: track 0.00 -> 51.3 mm, vias 0 -> 1
- net /+V: track 0.00 -> 48.8 mm, vias 0 -> 2
- net /IO32: track 0.00 -> 30.7 mm
- net /CS4: track 0.00 -> 29.3 mm
- net /CS1: track 0.00 -> 29.2 mm
- net /IO33: track 0.00 -> 26.5 mm
- net /DCC1: track 0.00 -> 20.8 mm, vias 0 -> 1
- net /IO34: track 0.00 -> 19.4 mm
- net /DCC2: track 0.00 -> 18.5 mm
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
Commit message: 14/09/25 16:21 Arrakis.local
Parts:
- removed H1, H2, H3, H4: MountingHole, MountingHole:MountingHole_3.2mm_M3_ISO14580
- moved J10 5.02 mm to (194.5, 62.0)
- moved J7 4.21 mm to (152.5, 62.0)
- moved J8 4.21 mm to (167.5, 62.2)
- moved J2 4.12 mm to (161.0, 59.0)
- moved J3 4.00 mm to (161.0, 68.0)
- moved J5 4.00 mm to (187.0, 59.5)
- moved J6 4.00 mm to (187.0, 68.5)
- moved J9 4.00 mm to (178.2, 62.2)
Routing:
- net /+V: track 48.8 -> 69.7 mm
- net /CS4: track 29.3 -> 37.4 mm, vias 0 -> 1
- net /SCK: track 55.0 -> 62.6 mm
- net /MISO: track 60.7 -> 56.8 mm
- net /RST: track 59.3 -> 55.7 mm
- net /CS2: track 12.1 -> 15.2 mm
- net /DCC1: track 20.8 -> 23.8 mm, vias 1 -> 2
- net /3V3: track 79.5 -> 81.8 mm, vias 1 -> 0
- net /CS1: track 29.2 -> 27.1 mm
- net /5V: track 51.3 -> 53.4 mm
- net /IO32: track 30.7 -> 28.8 mm
- net /IO35: track 10.3 -> 11.8 mm
- net /IO34: track 19.4 -> 20.7 mm
- net /GND: track 143.9 -> 142.6 mm, vias 0 -> 1
- net /IRQ4: track 7.89 -> 9.08 mm
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Other:
- outline, holes or cut-outs redrawn
