File: EspRfid522/EspRfid522.kicad_sch (KiCad schematic)
At the start: 15 parts, among them J1 Screw_Terminal_01x02, J2 IDC1, J3 IDC2, J4 IDC3, J5 IDC4, U1 AP7384-50Y, U2 AMS1117-3.3, U3 ESP32-DEVKITC-32D

Commit message: 13/09/25 20:26 Titan.local
Parts:
- added J6: DIP-BLACK-MALE-HEADER-VERT_2P-2.54_, Connector_PinHeader_2.54mm:PinHeader_2x01_P2.54mm_Vertical, symbol OPL_Connector:DIP-BLACK-MALE-HEADER-VERT_2P-2.54_
- added J7: DIP-BLACK-FEMALE-HEADER_2X4P-2.54_, Connector_PinHeader_2.54mm:PinHeader_2x04_P2.54mm_Vertical, symbol OPL_Connector:DIP-BLACK-FEMALE-HEADER_2X4P-2.54_
Connections:
- net 5V: now also J6.2; no longer U3.J2-19 (EXT_5V)
- net IO34: now reaches U3.J2-5 (IO34)
- net IO34: now also J7.3
- net IO35: now reaches U3.J2-6 (IO35)
- net IO35: now also J7.4
- net IO32: now reaches U3.J2-7 (IO32)
- net IO32: now also J7.1
- net IO33: now reaches U3.J2-8 (IO33)
- net IO33: now also J7.2
- removed net IRQ: J2.5 (Pin_5), J3.5 (Pin_5), J4.5 (Pin_5), J5.5 (Pin_5)
- new net EXT_5V: J6.1, U3.J2-19 (EXT_5V)
- new net IRQ1: J2.5 (Pin_5), J7.8
- new net IRQ2: J3.5 (Pin_5), J7.7
- new net IRQ3: J4.5 (Pin_5), J7.6
- new net IRQ4: J5.5 (Pin_5), J7.5
Changed lines of the file:
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@@
   (junction (at 86.36 35.56) (diameter 0) (color 0 0 0 0)
   )
+  (junction (at 45.72 79.248) (diameter 0) (color 0 0 0 0)
+  )
   (junction (at 92.71 35.56) (diameter 0) (color 0 0 0 0)
   )
@@
     (stroke (width 0) (type default))
   )
+  (wire (pts (xy 45.72 79.248) (xy 45.72 95.25))
+    (stroke (width 0) (type default))
+  )
   (wire (pts (xy 86.36 35.56) (xy 92.71 35.56))
     (stroke (width 0) (type default))
@@
     (stroke (width 0) (type default))
   )
+  (wire (pts (xy 101.854 78.74) (xy 158.115 78.74))
+    (stroke (width 0) (type default))
+  )
   (wire (pts (xy 26.67 27.94) (xy 38.1 27.94))
     (stroke (width 0) (type default))
@@
     (stroke (width 0) (type default))
   )
+  (wire (pts (xy 101.854 78.74) (xy 101.854 79.248))
+    (stroke (width 0) (type default))
+  )
   (wire (pts (xy 111.76 48.26) (xy 111.76 52.07))
     (stroke (width 0) (type default))
@@
     (stroke (width 0) (type default))
   )
-  (wire (pts (xy 45.72 35.56) (xy 45.72 95.25))
+  (wire (pts (xy 45.72 35.56) (xy 45.72 79.248))
     (stroke (width 0) (type default))
   )
@@
     (stroke (width 0) (type default))
   )
+  (wire (pts (xy 45.72 79.248) (xy 96.774 79.248))
+    (stroke (width 0) (type default))
+  )
   (wire (pts (xy 123.19 52.07) (xy 120.65 52.07))
     (stroke (width 0) (type default))
@@
     (stroke (width 0) (type default))
   )
-  (wire (pts (xy 151.13 78.74) (xy 158.115 78.74))
-    (stroke (width 0) (type default))
-  )
   (wire (pts (xy 123.19 60.96) (xy 121.92 60.96))
     (stroke (width 0) (type default))
@@
     (effects (font (size 1.27 1.27)) (justify right bottom))
   )
+  (label "IO34" (at 149.86 101.854 180) (fields_autoplaced)
+    (effects (font (size 1.27 1.27)) (justify right bottom))
+  )
   (label "SCK" (at 249.555 100.33 180) (fields_autoplaced)
     (effects (font (size 1.27 1.27)) (justify right bottom))
@@
     (effects (font (size 1.27 1.27)) (justify left bottom))
   )
-  (label "IRQ" (at 249.555 36.83 180) (fields_autoplaced)
+  (label "IRQ1" (at 249.555 36.83 180) (fields_autoplaced)
     (effects (font (size 1.27 1.27)) (justify right bottom))
   )
@@
     (effects (font (size 1.27 1.27)) (justify right bottom))
   )
-  (label "IRQ" (at 249.555 60.325 180) (fields_autoplaced)
-    (effects (font (size 1.27 1.27)) (justify right bottom))
+  (label "IRQ2" (at 249.555 60.325 180) (fields_autoplaced)
+    (effects (font (size 1.27 1.27)) (justify right bottom))
+  )
+  (label "IRQ1" (at 167.64 96.774 0) (fields_autoplaced)
+    (effects (font (size 1.27 1.27)) (justify left bottom))
   )
   (label "MISO" (at 249.555 81.915 180) (fields_autoplaced)
     (effects (font (size 1.27 1.27)) (justify right bottom))
   )
+  (label "IRQ2" (at 167.64 99.314 0) (fields_autoplaced)
+    (effects (font (size 1.27 1.27)) (justify left bottom))
+  )
   (label "CS4" (at 198.755 63.5 0) (fields_autoplaced)
     (effects (font (size 1.27 1.27)) (justify left bottom))
@@
     (effects (font (size 1.27 1.27)) (justify right bottom))
   )
+  (label "IO33" (at 158.115 50.8 180) (fields_autoplaced)
+    (effects (font (size 1.27 1.27)) (justify right bottom))
+  )
   (label "CS4" (at 249.555 97.79 180) (fields_autoplaced)
     (effects (font (size 1.27 1.27)) (justify right bottom))
@@
     (effects (font (size 1.27 1.27)) (justify right bottom))
   )
+  (label "IO32" (at 158.115 48.26 180) (fields_autoplaced)
+    (effects (font (size 1.27 1.27)) (justify right bottom))
+  )
   (label "CS2" (at 198.755 58.42 0) (fields_autoplaced)
     (effects (font (size 1.27 1.27)) (justify left bottom))
@@
     (effects (font (size 1.27 1.27)) (justify right bottom))
   )
-  (label "IRQ" (at 249.555 107.95 180) (fields_autoplaced)
+  (label "IRQ4" (at 249.555 107.95 180) (fields_autoplaced)
+    (effects (font (size 1.27 1.27)) (justify right bottom))
+  )
+  (label "IO32" (at 149.86 96.774 180) (fields_autoplaced)
     (effects (font (size 1.27 1.27)) (justify right bottom))
   )
@@
     (effects (font (size 1.27 1.27)) (justify right bottom))
   )
-  (label "IRQ" (at 249.555 84.455 180) (fields_autoplaced)
+  (label "IRQ3" (at 249.555 84.455 180) (fields_autoplaced)
+    (effects (font (size 1.27 1.27)) (justify right bottom))
+  )
+  (label "IO35" (at 149.86 104.394 180) (fields_autoplaced)
     (effects (font (size 1.27 1.27)) (justify right bottom))
   )
@@
     (effects (font (size 1.27 1.27)) (justify left bottom))
   )
+  (label "IO34" (at 158.115 43.18 180) (fields_autoplaced)
+    (effects (font (size 1.27 1.27)) (justify right bottom))
+  )
   (label "SCK" (at 249.555 52.705 180) (fields_autoplaced)
     (effects (font (size 1.27 1.27)) (justify right bottom))
@@
     (effects (font (size 1.27 1.27)) (justify left bottom))
   )
-  (label "5V" (at 151.13 78.74 0) (fields_autoplaced)
+  (label "EXT_5V" (at 151.13 78.74 0) (fields_autoplaced)
     (effects (font (size 1.27 1.27)) (justify left bottom))
   )
@@
     (effects (font (size 1.27 1.27)) (justify right bottom))
   )
+  (label "IRQ4" (at 167.64 104.394 0) (fields_autoplaced)
+    (effects (font (size 1.27 1.27)) (justify left bottom))
+  )
   (label "MISO" (at 249.555 105.41 180) (fields_autoplaced)
     (effects (font (size 1.27 1.27)) (justify right bottom))
@@
     (effects (font (size 1.27 1.27)) (justify left bottom))
   )
+  (label "IO35" (at 158.115 45.72 180) (fields_autoplaced)
+    (effects (font (size 1.27 1.27)) (justify right bottom))
+  )
   (label "MOSI" (at 198.755 35.56 0) (fields_autoplaced)
     (effects (font (size 1.27 1.27)) (justify left bottom))
   )
+  (label "IRQ3" (at 167.64 101.854 0) (fields_autoplaced)
+    (effects (font (size 1.27 1.27)) (justify left bottom))
+  )
   (label "RST" (at 249.555 65.405 180) (fields_autoplaced)
+    (effects (font (size 1.27 1.27)) (justify right bottom))
+  )
+  (label "IO33" (at 149.86 99.314 180) (fields_autoplaced)
     (effects (font (size 1.27 1.27)) (justify right bottom))
   )
@@
         (path "/5704e254-5676-4e5e-88a0-6bc38578f992"
           (reference "U2") (unit 1)
+        )
+      )
+    )
+  )
+  (symbol (lib_id "OPL_Connector:DIP-BLACK-MALE-HEADER-VERT_2P-2.54_") (at 99.314 86.868 270) (unit 1)
+    (in_bom yes) (on_board yes) (dnp no) (fields_autoplaced)
+    (property "Reference" "J6" (at 105.41 85.598 90)
+      (effects (font (size 1.143 1.143)) (justify left))
+    )
+    (property "Value" "DIP-BLACK-MALE-HEADER-VERT_2P-2.54_" (at 105.41 88.138 90)
+      (effects (font (size 1.143 1.143)) (justify left))
+    )
+    (property "Footprint" "Connector_PinHeader_2.54mm:PinHeader_2x01_P2.54mm_Vertical" (at 99.314 86.868 0)
+      (effects (font (size 1.27 1.27)) hide)
+    )
+    (property "Datasheet" "" (at 99.314 86.868 0)
+      (effects (font (size 1.27 1.27)) hide)
+    )
+    (property "MPN" "P125-1102A0BS116A1" (at 103.124 87.63 0)
+      (effects (font (size 0.508 0.508)) hide)
+    )
+    (property "SKU" "320020016" (at 103.124 87.63 0)
+      (effects (font (size 0.508 0.508)) hide)
+    )
+    (pin "1")
+    (pin "2")
+    (instances
+      (project "EspRfid522"
+        (path "/5704e254-5676-4e5e-88a0-6bc38578f992"
+          (reference "J6") (unit 1)
         )
       )
@@
         )
       )
+    )
+  )
+  (symbol (lib_id "OPL_Connector:DIP-BLACK-FEMALE-HEADER_2X4P-2.54_") (at 158.75 100.584 0) (unit 1)
+    (in_bom yes) (on_board yes) (dnp no) (fields_autoplaced)
+    (property "Reference" "J7" (at 158.75 90.17 0)
+      (effects (font (size 1.143 1.143)))
+    )
+    (property "Value" "DIP-BLACK-FEMALE-HEADER_2X4P-2.54_" (at 158.75 92.71 0)
+      (effects (font (size 1.143 1.143)))
+    )
+    (property "Footprint" "Connector_PinHeader_2.54mm:PinHeader_2x04_P2.54mm_Vertical" (at 158.75 100.584 0)
+      (effects (font (size 1.27 1.27)) hide)
+    )
+    (property "Datasheet" "" (at 158.75 100.584 0)
+      (effects (font (size 1.27 1.27)) hide)
+    )
+    (property "SKU" "320030087" (at 159.512 96.774 0)
+      (effects (font (size 0.508 0.508)) hide)
+    )
+    (pin "1")
+    (pin "2")
+    (pin "3")
+    (pin "4")
+    (pin "5")
+    (pin "6")
+    (pin "7")
+    (pin "8")
+    (instances
+      (project "EspRfid522"
+        (path "/5704e254-5676-4e5e-88a0-6bc38578f992"
+          (reference "J7") (unit 1)
+        )
+      )

Commit message: 14/09/25 14:58 Arrakis.local
Parts:
- removed J6: DIP-BLACK-MALE-HEADER-VERT_2P-2.54_, Connector_PinHeader_2.54mm:PinHeader_2x01_P2.54mm_Vertical, symbol OPL_Connector:DIP-BLACK-MALE-HEADER-VERT_2P-2.54_
- removed J7: DIP-BLACK-FEMALE-HEADER_2X4P-2.54_, Connector_PinHeader_2.54mm:PinHeader_2x04_P2.54mm_Vertical, symbol OPL_Connector:DIP-BLACK-FEMALE-HEADER_2X4P-2.54_
- removed U1: AP7384-50Y, Package_TO_SOT_SMD:SOT-89-3, symbol Regulator_Linear:AP7384-50Y
- added H1, H2, H3, H4: MountingHole, MountingHole:MountingHole_3.2mm_M3_ISO14580, symbol Mechanical:MountingHole
- added J2, J3, J4, J5, J6: Conn_01x02, Connector_PinHeader_2.54mm:PinHeader_1x02_P2.54mm_Vertical, symbol Connector_Generic:Conn_01x02
- added U2: AMS1117-5.0, Package_TO_SOT_SMD:SOT-223-3_TabPin2, symbol Regulator_Linear:AMS1117-5.0
- renumbered J5 to J10, J2 to J7, J3 to J8, J4 to J9, U2 to U1
Connections:
- net +V: now also U2.3 (VI)
- net 5V: now also J4.2 (Pin_2), U2.2 (VO)
- net EXT_5V: now also J4.1 (Pin_1)
- net GND: now also U2.1 (GND)
- net IO32: now also J2.1 (Pin_1)
- net IO33: now also J3.1 (Pin_1)
- net IO34: now also J5.1 (Pin_1)
- net IO35: now also J6.1 (Pin_1)
- net IRQ1: now also J2.2 (Pin_2)
- net IRQ2: now also J3.2 (Pin_2)
- net IRQ3: now also J5.2 (Pin_2)
- net IRQ4: now also J6.2 (Pin_2)
- no-connect marks 0 -> 23
Other:
- note added: "AP7384 or AP7387Q alternate"
- note added: "Cap 25v Size 2412 Vishay 593D106X9025C2TE3"
- note added: "Other possible diodes B340LA-13-F"
- note added: "SCL"
- note added: "SDA"
- note removed: "Size 2412 Vishay 593D106X9025C2TE3"

Commit message: 14/09/25 16:21 Arrakis.local
Parts:
- removed H1, H2, H3, H4: MountingHole, MountingHole:MountingHole_3.2mm_M3_ISO14580, symbol Mechanical:MountingHole
Changed lines of the file:
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@@
-    )
-  )
-  (symbol (lib_id "Mechanical:MountingHole") (at 88.9 137.795 0) (unit 1)
-    (in_bom yes) (on_board yes) (dnp no) (fields_autoplaced)
-    (property "Reference" "H4" (at 91.44 137.16 0)
-      (effects (font (size 1.27 1.27)) (justify left))
-    )
-    (property "Value" "MountingHole" (at 91.44 139.7 0)
-      (effects (font (size 1.27 1.27)) (justify left))
-    )
-    (property "Footprint" "MountingHole:MountingHole_3.2mm_M3_ISO14580" (at 88.9 137.795 0)
-      (effects (font (size 1.27 1.27)) hide)
-    )
-    (property "Datasheet" "~" (at 88.9 137.795 0)
-      (effects (font (size 1.27 1.27)) hide)
-    )
-    (instances
-      (project "EspRfid522"
-        (path "/5704e254-5676-4e5e-88a0-6bc38578f992"
-          (reference "H4") (unit 1)
-        )
-      )
     )
   )
@@
         (path "/5704e254-5676-4e5e-88a0-6bc38578f992"
           (reference "J4") (unit 1)
-        )
-      )
-    )
-  )
-  (symbol (lib_id "Mechanical:MountingHole") (at 60.96 137.16 0) (unit 1)
-    (in_bom yes) (on_board yes) (dnp no) (fields_autoplaced)
-    (property "Reference" "H2" (at 63.5 136.525 0)
-      (effects (font (size 1.27 1.27)) (justify left))
-    )
-    (property "Value" "MountingHole" (at 63.5 139.065 0)
-      (effects (font (size 1.27 1.27)) (justify left))
-    )
-    (property "Footprint" "MountingHole:MountingHole_3.2mm_M3_ISO14580" (at 60.96 137.16 0)
-      (effects (font (size 1.27 1.27)) hide)
-    )
-    (property "Datasheet" "~" (at 60.96 137.16 0)
-      (effects (font (size 1.27 1.27)) hide)
-    )
-    (instances
-      (project "EspRfid522"
-        (path "/5704e254-5676-4e5e-88a0-6bc38578f992"
-          (reference "H2") (unit 1)
-        )
-      )
-    )
-  )
-  (symbol (lib_id "Mechanical:MountingHole") (at 45.085 137.16 0) (unit 1)
-    (in_bom yes) (on_board yes) (dnp no) (fields_autoplaced)
-    (property "Reference" "H1" (at 48.26 136.525 0)
-      (effects (font (size 1.27 1.27)) (justify left))
-    )
-    (property "Value" "MountingHole" (at 48.26 139.065 0)
-      (effects (font (size 1.27 1.27)) (justify left))
-    )
-    (property "Footprint" "MountingHole:MountingHole_3.2mm_M3_ISO14580" (at 45.085 137.16 0)
-      (effects (font (size 1.27 1.27)) hide)
-    )
-    (property "Datasheet" "~" (at 45.085 137.16 0)
-      (effects (font (size 1.27 1.27)) hide)
-    )
-    (instances
-      (project "EspRfid522"
-        (path "/5704e254-5676-4e5e-88a0-6bc38578f992"
-          (reference "H1") (unit 1)
         )
       )
@@
         )
       )
-    )
-  )
-  (symbol (lib_id "Mechanical:MountingHole") (at 74.295 137.795 0) (unit 1)
-    (in_bom yes) (on_board yes) (dnp no) (fields_autoplaced)
-    (property "Reference" "H3" (at 77.47 137.16 0)
-      (effects (font (size 1.27 1.27)) (justify left))
-    )
-    (property "Value" "MountingHole" (at 77.47 139.7 0)
-      (effects (font (size 1.27 1.27)) (justify left))
-    )
-    (property "Footprint" "MountingHole:MountingHole_3.2mm_M3_ISO14580" (at 74.295 137.795 0)
-      (effects (font (size 1.27 1.27)) hide)
-    )
-    (property "Datasheet" "~" (at 74.295 137.795 0)
-      (effects (font (size 1.27 1.27)) hide)
-    )
-    (instances
-      (project "EspRfid522"
-        (path "/5704e254-5676-4e5e-88a0-6bc38578f992"
-          (reference "H3") (unit 1)
-        )
-      )
